File: MOD_Foot_Prototype1/MOD_Foot_Prototype1.kicad_pcb (KiCad board)
At the start: 2 copper layers, 248.9 x 74.2 mm, 91 parts, among them CN1 CONN_PANNEL_2X2, CN2 CONN_PANNEL_2X2, J1 RJ45_CHAIN, J2 RJ45_CHAIN, P1 HEADER_5X1, P2 HEADER_5X2, Q1 MMBT3904, Q2 MMBT3904, Q3 MMBT3904, U1 LPC111X_LQFP48, U2 MC7805, U3 NCP1117DT33G, U4 SN75176BDR, U5 74HC245, U6 74HC245, X1 10MHz

Commit message: fix issue #14: Broken component/footprint map file This commit makes the mod-arduino-shield a dependency. We must still move the footprint library to a single repository and declare it properly as a git submodule.
Parts:
- C1, C3: value 10uF -> 100uF; footprint CAP_RAD_5MM -> MODArduinoLib:CAP_RAD_5MM
- C10, C11, C12, C13, C14, C15, C17, C2, C4, C5, C7, C8, C9, R1, R10, R14, R15, R16, R17, R18, R19, R2, R20, R21, R22, R23, R24, R25, R27, R28, R29, R30, R31, R32, R33, R36, R40, R41, R7, R8, R9: footprint SM0603 -> MODArduinoLib:SM0603
- C16, C6: footprint CAP_RAD_5MM -> MODArduinoLib:CAP_RAD_5MM
- CN1, CN2: footprint CONN_PANNEL -> MODArduinoLib:CONN_PANNEL
- D1: footprint DO-214AC(SMA) -> MODArduinoLib:DO-214AC(SMA)
- D2, D3: footprint SOD123 -> MODArduinoLib:SOD123
- D4: footprint SOD323 -> MODArduinoLib:SOD323
- FOOT1, FOOT2, FOOT3, FOOT4: footprint PIN_ARRAY_2X1 -> MODArduinoLib:PIN_ARRAY_2X1
- J1, J2: footprint RJ45-RJHSE5084 -> MODArduinoLib:RJ45-RJHSE5084
- LCD1: footprint LCD-AGM-2004A-204 -> MODArduinoLib:LCD-AGM-2004A-204
- LED1, LED2, LED3, LED4: footprint LED_CLRTB_GFSF_1 -> MODArduinoLib:LED_CLRTB_GFSF_1
- P1: footprint PIN_ARRAY_5x1 -> MODArduinoLib:PIN_ARRAY_5x1
- P2: footprint PIN_ARRAY_5x2 -> MODArduinoLib:PIN_ARRAY_5x2
- Q1, Q2, Q3: footprint SOT23 -> MODArduinoLib:SOT23
- R11, R12, R13, R26, R3, R34, R35, R37, R38, R39, R4, R5, R6: footprint SM0805 -> MODArduinoLib:SM0805
- RT1: footprint SM2920 -> MODArduinoLib:SM2920
- TP1, TP2, TP3: footprint SIL-1 -> MODArduinoLib:SIL-1
- U1: footprint LQFP48 -> MODArduinoLib:LQFP48
- U2, U3: footprint DPAK(369C) -> MODArduinoLib:DPAK(369C)
- U4: footprint SO8E -> MODArduinoLib:SO8E
- U5, U6: footprint TSSOP20 -> MODArduinoLib:TSSOP20
- X1: footprint HC_49US -> MODArduinoLib:HC_49US
Connections:
- net LED1 renamed LED5
- net LED2 renamed TX_CHAIN
- CN1 pad 1: (no net) -> Net-(CN1-Pad1)
- CN2 pad 1: (no net) -> Net-(CN2-Pad1)
- P2 pad 6: (no net) -> Net-(P2-Pad6)
- P2 pad 8: (no net) -> Net-(P2-Pad8)
- U1 pad 10: (no net) -> Net-(U1-Pad10)
- U1 pad 18: (no net) -> Net-(U1-Pad18)
- U1 pad 21: (no net) -> Net-(U1-Pad21)
- U1 pad 22: (no net) -> Net-(U1-Pad22)
- U1 pad 9: (no net) -> Net-(U1-Pad9)
- U6 pad 14: (no net) -> Net-(U6-Pad14)
- U6 pad 15: (no net) -> Net-(U6-Pad15)
- U6 pad 16: (no net) -> Net-(U6-Pad16)
- U6 pad 17: (no net) -> Net-(U6-Pad17)
- U6 pad 18: (no net) -> Net-(U6-Pad18)
- U6 pad 2: (no net) -> Net-(U6-Pad2)
- U6 pad 3: (no net) -> Net-(U6-Pad3)
- U6 pad 4: (no net) -> Net-(U6-Pad4)
- U6 pad 5: (no net) -> Net-(U6-Pad5)
- U6 pad 6: (no net) -> Net-(U6-Pad6)
Routing:
- added copper zone on B.Cu, net N-0000012
- added copper zone on F.Cu, net N-0000012
- removed copper zone on B.Cu, net Net-(C6-Pad1)
- removed copper zone on F.Cu, net Net-(C6-Pad1)

Commit message: update footprint lib references in the kicad_pcb file as well... (and a relative path in the netlist file)
Parts:
- C1, C16, C3, C6: footprint MODArduinoLib:CAP_RAD_5MM -> MOD_Footprints_Lib:CAP_RAD_5MM
- C10, C11, C12, C13, C14, C15, C17, C2, C4, C5, C7, C8, C9, R1, R10, R14, R15, R16, R17, R18, R19, R2, R20, R21, R22, R23, R24, R25, R27, R28, R29, R30, R31, R32, R33, R36, R40, R41, R7, R8, R9: footprint MODArduinoLib:SM0603 -> MOD_Footprints_Lib:SM0603
- CN1, CN2: footprint MODArduinoLib:CONN_PANNEL -> MOD_Footprints_Lib:CONN_PANNEL
- D1: footprint MODArduinoLib:DO-214AC(SMA) -> MOD_Footprints_Lib:DO-214AC(SMA)
- D2, D3: footprint MODArduinoLib:SOD123 -> MOD_Footprints_Lib:SOD123
- D4: footprint MODArduinoLib:SOD323 -> MOD_Footprints_Lib:SOD323
- FOOT1, FOOT2, FOOT3, FOOT4: footprint MODArduinoLib:PIN_ARRAY_2X1 -> MOD_Footprints_Lib:PIN_ARRAY_2X1
- J1, J2: footprint MODArduinoLib:RJ45-RJHSE5084 -> MOD_Footprints_Lib:RJ45-RJHSE5084
- LCD1: footprint MODArduinoLib:LCD-AGM-2004A-204 -> MOD_Footprints_Lib:LCD-AGM-2004A-204
- LED1, LED2, LED3, LED4: footprint MODArduinoLib:LED_CLRTB_GFSF_1 -> MOD_Footprints_Lib:LED_CLRTB_GFSF_1
- P1: footprint MODArduinoLib:PIN_ARRAY_5x1 -> MOD_Footprints_Lib:PIN_ARRAY_5x1
- P2: footprint MODArduinoLib:PIN_ARRAY_5x2 -> MOD_Footprints_Lib:PIN_ARRAY_5x2
- Q1, Q2, Q3: footprint MODArduinoLib:SOT23 -> MOD_Footprints_Lib:SOT23
- R11, R12, R13, R26, R3, R34, R35, R37, R38, R39, R4, R5, R6: footprint MODArduinoLib:SM0805 -> MOD_Footprints_Lib:SM0805
- RT1: footprint MODArduinoLib:SM2920 -> MOD_Footprints_Lib:SM2920
- TP1, TP2, TP3: footprint MODArduinoLib:SIL-1 -> MOD_Footprints_Lib:SIL-1
- U1: footprint MODArduinoLib:LQFP48 -> MOD_Footprints_Lib:LQFP48
- U2, U3: footprint MODArduinoLib:DPAK(369C) -> MOD_Footprints_Lib:DPAK(369C)
- U4: footprint MODArduinoLib:SO8E -> MOD_Footprints_Lib:SO8E
- U5, U6: footprint MODArduinoLib:TSSOP20 -> MOD_Footprints_Lib:TSSOP20
- X1: footprint MODArduinoLib:HC_49US -> MOD_Footprints_Lib:HC_49US

Commit message: grounding the mechanical connectors (and regenerating Gerber files)
Connections:
- CN1 pad 1: Net-(CN1-Pad1) -> DGND
- CN2 pad 1: Net-(CN2-Pad1) -> DGND
