File: MOD_Foot_Prototype1/MOD_Foot_Prototype1.kicad_pcb (KiCad board)
At the start: 2 copper layers, 248.9 x 74.2 mm, 91 parts, among them CN1 CONN_PANNEL_2X2, CN2 CONN_PANNEL_2X2, J1 RJ45_CHAIN, J2 RJ45_CHAIN, P1 HEADER_5X1, P2 HEADER_5X2, Q1 MMBT3904, Q2 MMBT3904, Q3 MMBT3904, U1 LPC111X_LQFP48, U2 MC7805, U3 NCP1117DT33G, U4 SN75176BDR, U5 74HC245, U6 74HC245, X1 10MHz

Commit message: rearrange R38 and C3 components (fix issue #7)
Parts:
- moved R38 6.04 mm to (349.3, 184.4), turned to 270 degrees
Routing:
- net +5V: track 162.5 -> 164.8 mm

Commit message: updating pcb traces (fixes issue #13: ADC availability)
Connections:
- U1 pad 18: Net-(U1-Pad18) -> LED1_R
- U1 pad 21: Net-(U1-Pad21) -> LED1_B
- U1 pad 40: LED1_B -> Net-(U1-Pad40)
- U1 pad 42: LED1_R -> Net-(U1-Pad42)
Routing:
- net LED1_B: track 42.7 -> 51.3 mm, vias 0 -> 2
- net LED1_R: track 45.7 -> 54.4 mm, vias 0 -> 2

Commit message: fix issue #11: protect the U4 IC when the board is being debugged Updated PCB traces and regenerated Gerbers.
Parts:
- added R42: 0R, MOD_Footprints_Lib:SM0805, F.Cu at (338.7, 202.4)
- added R43: 0R, MOD_Footprints_Lib:SM0805, F.Cu at (344.4, 207.1)
- P1: value HEADER_5X1 -> HEADER_5X2; footprint MOD_Footprints_Lib:PIN_ARRAY_5x1 -> MOD_Footprints_Lib:PIN_ARRAY_5x2
- moved P1 1.26 mm to (342.7, 199.3)
- moved R39 0.09 mm to (340.9, 234.5), turned to 270 degrees
Connections:
- P1 pad 2: +5V -> DGND
- P1 pad 3: RX_CHAIN -> +5V
- P1 pad 4: TX_CHAIN -> +5V
- P1 pad 5: EN_CHAIN -> RX_CHAIN
- R2 pad 1: TX_CHAIN -> LED6
- R31 pad 2: TX_CHAIN -> LED6
- R39 pad 1: +3.3V -> Net-(P2-Pad1)
- R39 pad 2: Net-(P2-Pad1) -> +3.3V
- U1 pad 46: RX_CHAIN -> Net-(P1-Pad6)
- U1 pad 47: TX_CHAIN -> Net-(P1-Pad8)
- U4 pad 4: TX_CHAIN -> LED6
Routing:
- net TX_CHAIN: track 43.2 -> 0.00 mm, vias 2 -> 0
- net LED6: track 0.00 -> 31.4 mm, vias 0 -> 2
- net Net-(P1-Pad6): track 0.00 -> 21.8 mm
- net Net-(P1-Pad8): track 0.00 -> 20.5 mm, vias 0 -> 2
- net RX_CHAIN: track 25.8 -> 12.7 mm
- net +5V: track 164.8 -> 167.3 mm
Other:
- board text added: "UART DEBUGGER"

Commit message: fixed issue #9 by adding an SM1210 footprint for a second fuse. It's up to us to decide which kind of fuse to solder in the board, but the PCB has got both footprints.
Parts:
- added RT2: PTC_FUSE_500mA, MOD_Footprints_Lib:SM2920, F.Cu at (355.2, 181.4)
- RT1: footprint MOD_Footprints_Lib:SM2920 -> MOD_Footprints_Lib:SM1210
Connections:
- net LED6 renamed TX_CHAIN
Routing:
- net +9V: track 16.6 -> 18.4 mm
- net Net-(D1-Pad2): track 4.32 -> 6.10 mm

Commit message: wip - retracing PCB to accomodate schematic changes from previous recent commits.
Parts:
- removed D4: 1N4148, MOD_Footprints_Lib:SOD323
- added C18: 100nF_X7R, MOD_Footprints_Lib:SM0603, F.Cu at (350.9, 202.3)
- added R44: 0R/NC, MOD_Footprints_Lib:SM0805, F.Cu at (348.1, 213.1)
- added R45: 0R, MOD_Footprints_Lib:SM0805, F.Cu at (343.7, 213.1)
- C5: value 100nF_X7R -> 100uF; footprint MOD_Footprints_Lib:SM0603 -> MOD_Footprints_Lib:CAP_RAD_5MM
- J1: value RJ45_CHAIN -> RJ45_CHAIN_MAIN
- J2: value RJ45_CHAIN -> RJ45_CHAIN_EXTENSION
- Q2: value MMBT3904 -> MMBT3906
- R11: value 120R -> 100R 0.5W; footprint MOD_Footprints_Lib:SM0805 -> MOD_Footprints_Lib:SM1210
- R12, R13: value 10R -> 10k; footprint MOD_Footprints_Lib:SM0805 -> MOD_Footprints_Lib:SM0603
- R2: value 1k -> 100R 0.5W; footprint MOD_Footprints_Lib:SM0603 -> MOD_Footprints_Lib:SM1210
- R28: value 1k -> 10k
- RT1: footprint MOD_Footprints_Lib:SM1210 -> MOD_Footprints_Lib:SM2920
- RT2: footprint MOD_Footprints_Lib:SM2920 -> MOD_Footprints_Lib:SM1210
- U4: value SN75176BDR -> MAX13450E; footprint MOD_Footprints_Lib:SO8E -> MOD_Footprints_Lib:TSSOP14
- moved R11 21.7 mm to (352.9, 217.7)
- moved R2 5.45 mm to (352.9, 213.7), turned to 180 degrees
- moved R27 5.29 mm to (360.7, 200.4)
- moved C8 3.91 mm to (355.9, 194.3), turned to 0 degrees
- moved R30 2.72 mm to (348.4, 193.9), turned to 0 degrees
- moved U4 2.34 mm to (351.5, 199.0)
- moved R28 2.34 mm to (353.7, 204.1)
- moved R43 0.60 mm to (343.8, 207.0)
- moved R31 0.13 mm to (349.9, 207.9)
- turned R42 to 270 degrees
Connections:
- C5 pad 1: VCC -> Net-(C5-Pad1)
- C8 pad 1: +5V -> Net-(C5-Pad1)
- D2 pad 2: Net-(D2-Pad2) -> RS485_RX+
- D3 pad 2: Net-(D3-Pad2) -> RS485_RX-
- J1 pad 1: VCC -> RS485_TX+
- J1 pad 11: Net-(J1-Pad11) -> DGND
- J1 pad 2: VCC -> RS485_TX-
- J1 pad 3: RS422_A -> RS485_RX+
- J1 pad 4: RS422_A -> VCC
- J1 pad 5: RS422_B -> VCC
- J1 pad 6: RS422_B -> RS485_RX-
- J1 pad 7: DGND -> Net-(J1-Pad7)
- J1 pad 8: DGND -> Net-(J1-Pad7)
- J2 pad 1: VCC -> RS485_RX+
- J2 pad 11: Net-(J1-Pad11) -> DGND
- J2 pad 2: VCC -> RS485_RX-
- J2 pad 3: RS422_A -> RS485_TX+
- J2 pad 4: RS422_A -> VCC
- J2 pad 5: RS422_B -> VCC
- J2 pad 6: RS422_B -> RS485_TX-
- J2 pad 7: DGND -> Net-(C5-Pad1)
- J2 pad 8: DGND -> Net-(J2-Pad8)
- P1 pad 10: EN_CHAIN -> UC_TX_CHAIN_EN
- P1 pad 6: Net-(P1-Pad6) -> UC_RX_CHAIN
- P1 pad 8: Net-(P1-Pad8) -> UC_TX_CHAIN
- P1 pad 9: EN_CHAIN -> TX_CHAIN_EN
- Q1 pad 1: DGND -> Net-(Q1-Pad1)
- Q1 pad 2: Net-(Q1-Pad2) -> DGND
- Q2 pad 1: DGND -> Net-(Q2-Pad1)
- Q2 pad 2: Net-(Q2-Pad2) -> +5V
- Q2 pad 3: Net-(J1-Pad11) -> RTERM_CHAIN
- Q3 pad 1: DGND -> Net-(Q3-Pad1)
- Q3 pad 2: Net-(Q3-Pad2) -> DGND
- R1 pad 2: Net-(Q1-Pad2) -> Net-(Q1-Pad1)
- R11 pad 1: RS422_B -> Net-(J2-Pad8)
- R11 pad 2: RS422_A -> DGND
- R12 pad 1: RS422_B -> Net-(C5-Pad1)
- R12 pad 2: Net-(D3-Pad2) -> Net-(R12-Pad2)
- R13 pad 1: RS422_A -> +5V
- R13 pad 2: Net-(D2-Pad2) -> Net-(R12-Pad2)
- R2 pad 1: TX_CHAIN -> Net-(J1-Pad7)
- R2 pad 2: Net-(Q2-Pad2) -> DGND
- R27 pad 1: DGND -> Net-(R12-Pad2)
- R27 pad 2: Net-(D3-Pad2) -> Net-(Q2-Pad1)
- R28 pad 1: Net-(D4-Pad1) -> RTERM_CHAIN
- R28 pad 2: +5V -> DGND
- R29 pad 2: EN_CHAIN -> RX_CHAIN
- R30 pad 2: RX_CHAIN -> Net-(R30-Pad2)
- R31 pad 1: +5V -> TX_CHAIN_EN
- R31 pad 2: TX_CHAIN -> DGND
- R36 pad 2: Net-(Q3-Pad2) -> Net-(Q3-Pad1)
- R39 pad 1: Net-(P2-Pad1) -> +3.3V
- R39 pad 2: +3.3V -> Net-(P2-Pad1)
- R42 pad 1: Net-(P1-Pad6) -> RX_CHAIN
- R42 pad 2: RX_CHAIN -> UC_RX_CHAIN
- R43 pad 1: Net-(P1-Pad8) -> TX_CHAIN
- R43 pad 2: TX_CHAIN -> UC_TX_CHAIN
- U1 pad 18: LED1_R -> Net-(U1-Pad18)
- U1 pad 21: LED1_B -> Net-(U1-Pad21)
- U1 pad 40: Net-(U1-Pad40) -> LED1_B
- U1 pad 42: Net-(U1-Pad42) -> LED1_R
- U1 pad 45: EN_CHAIN -> UC_TX_CHAIN_EN
- U1 pad 46: Net-(P1-Pad6) -> UC_RX_CHAIN
- U1 pad 47: Net-(P1-Pad8) -> UC_TX_CHAIN
- U4 pad 1: RX_CHAIN -> TX_CHAIN_EN
- U4 pad 2: EN_CHAIN -> DGND
- U4 pad 3: EN_CHAIN -> TX_CHAIN
- U4 pad 4: TX_CHAIN -> +5V
- U4 pad 5: DGND -> RTERM_CHAIN
- U4 pad 6: Net-(D2-Pad2) -> Net-(C18-Pad1)
- U4 pad 7: Net-(D3-Pad2) -> RX_CHAIN
- U4 pad 8: +5V -> RS485_RX+
Routing:
- net LED1_R: track 54.4 -> 0.00 mm, vias 2 -> 0
- net LED1_B: track 51.3 -> 0.42 mm, vias 2 -> 0
- net VCC: track 42.1 -> 2.40 mm
- net RS422_A: track 34.0 -> 0.00 mm, vias 1 -> 0
- net RS422_B: track 32.5 -> 0.00 mm, vias 2 -> 0
- net EN_CHAIN: track 29.4 -> 0.00 mm, vias 1 -> 0
- net Net-(J1-Pad11): track 25.5 -> 0.00 mm, vias 1 -> 0
- net UC_TX_CHAIN: track 0.00 -> 25.1 mm, vias 0 -> 2
- net UC_TX_CHAIN_EN: track 0.00 -> 24.8 mm, vias 0 -> 3
- net Net-(J1-Pad9): track 24.8 -> 0.34 mm, vias 1 -> 0
- net TX_CHAIN_EN: track 0.00 -> 22.1 mm, vias 0 -> 3
- net Net-(P1-Pad6): track 21.8 -> 0.00 mm
- net UC_RX_CHAIN: track 0.00 -> 21.4 mm
- net Net-(P1-Pad8): track 20.5 -> 0.00 mm, vias 2 -> 0
- net Net-(C5-Pad1): track 0.00 -> 20.2 mm
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
Commit message: fix issues #4 and #11 - traced all pcb signals and regenerated Gerber files.
Routing:
- net RS485_TX+: track 0.00 -> 58.3 mm, vias 0 -> 4
- net VCC: track 2.40 -> 51.0 mm, vias 0 -> 4
- net RS485_RX+: track 4.20 -> 51.3 mm, vias 0 -> 4
- net LED1_R: track 0.00 -> 45.8 mm
- net RS485_TX-: track 0.00 -> 44.9 mm, vias 0 -> 3
- net LED1_B: track 0.42 -> 42.9 mm
- net Net-(J1-Pad7): track 0.00 -> 33.5 mm, vias 0 -> 4
- net RS485_RX-: track 4.22 -> 34.4 mm, vias 0 -> 3
- net +5V: track 161.8 -> 191.9 mm, vias 6 -> 9
- net Net-(J1-Pad9): track 0.34 -> 25.7 mm, vias 0 -> 2
- net Net-(C5-Pad1): track 20.2 -> 43.8 mm, vias 0 -> 1
- net DGND: track 144.9 -> 166.9 mm, vias 56 -> 58
- net Net-(Q2-Pad1): track 0.00 -> 21.3 mm, vias 0 -> 4
- net Net-(R30-Pad2): track 6.79 -> 24.7 mm, vias 0 -> 2
- net RTERM_CHAIN: track 7.91 -> 25.0 mm, vias 0 -> 2
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
Commit message: changing the position of the C5 capacitor to make it fit (it was too tight to place it between the RJ45 connectors)
Parts:
- moved C5 22.2 mm to (368.5, 222.5)
Routing:
- net Net-(C5-Pad1): track 43.8 -> 49.0 mm, vias 1 -> 2
Changed lines of the file:
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@@
     (thickness 1.6)
     (drawings 30)
-    (tracks 1148)
+    (tracks 1152)
     (zones 0)
     (modules 96)
@@
   )
   (module MOD_Footprints_Lib:CAP_RAD_5MM (layer F.Cu)
-    (at 372.4529 200.6727)
+    (at 368.5 222.5)
     (attr smd)
     (fp_text reference C5 (at -3.6529 1.1273) (layer F.SilkS)
@@
   (segment (start 342.773 202.946) (end 342.773 206.9465) (width 0.381) (layer F.Cu) (net 96))
   (segment (start 342.773 206.9465) (end 342.8365 207.01) (width 0.381) (layer F.Cu) (net 96))
+  (via (at 369.4 216.7) (size 0.508) (drill 0.3048) (layers F.Cu B.Cu) (net 97))
+  (segment (start 368.5 221.5) (end 368.5 217.6) (width 0.381) (layer F.Cu) (net 97))
+  (segment (start 368.5 217.6) (end 369.4 216.7) (width 0.381) (layer F.Cu) (net 97))
   (segment (start 372.4529 199.6727) (end 372.4529 199.8471) (width 0.381) (layer F.Cu) (net 97))
   (segment (start 372.4529 199.8471) (end 368.5 203.8) (width 0.381) (layer F.Cu) (net 97))
   (segment (start 371.5131 215.4869) (end 371.5131 213.8553) (width 0.381) (layer B.Cu) (net 97))
   (segment (start 370.3 216.7) (end 371.5131 215.4869) (width 0.381) (layer B.Cu) (net 97))
-  (segment (start 368.9 216.7) (end 370.3 216.7) (width 0.381) (layer B.Cu) (net 97))
+  (segment (start 368.9 216.7) (end 369.4 216.7) (width 0.381) (layer B.Cu) (net 97))
+  (segment (start 369.4 216.7) (end 370.3 216.7) (width 0.381) (layer B.Cu) (net 97))
   (segment (start 368.4 216.2) (end 368.9 216.7) (width 0.381) (layer B.Cu) (net 97))
   (segment (start 368.4 213.6) (end 368.4 216.2) (width 0.381) (layer B.Cu) (net 97))

Commit message: tweaking the pcb layout to avoid islands without copper in the ground plane.
Routing:
- net Net-(C5-Pad1): track 49.0 -> 46.0 mm
- net RS485_RX+: track 51.3 -> 49.9 mm
- net Net-(Q2-Pad1): track 21.3 -> 22.1 mm
- net UC_TX_CHAIN: track 25.1 -> 25.7 mm
