File: MOD_Foot_Prototype1/MOD_Foot_Prototype1.kicad_pcb (KiCad board)
At the start: 2 copper layers, 248.9 x 74.2 mm, 96 parts, among them CN1 CONN_PANNEL_2X2, CN2 CONN_PANNEL_2X2, J1 RJ45_CHAIN_MAIN, J2 RJ45_CHAIN_EXTENSION, P1 HEADER_5X2, P2 HEADER_5X2, Q1 MMBT3904, Q2 MMBT3906, Q3 MMBT3904, U1 LPC111X_LQFP48, U2 MC7805, U3 NCP1117DT33G, U4 MAX13450E, U5 74HC245, U6 74HC245, X1 10MHz

Commit message: fix issue #1: Add "CC by-SA" license logo to the PCB silk layer
Parts:
- added G***: LOGO, MOD_Footprints_Lib:MOD_Logo, F.Cu at (275.3, 220.8)
Other:
- board text added: "(c) 2014 Musical Operating Devices Licensed under CC By-SA https://github.com/portalmod/mod-hw-footswitch/"
- board text removed: "MOD FOOT PROTOTYPE 1 - 2014/04/23"

Commit message: fix issue #10: updating the PCB layout with the added pull up resistors for LCD ENABLE and RW signals
Parts:
- added R46: 10k, MOD_Footprints_Lib:SM0603, F.Cu at (313.9, 214.4)
- added R47: 10k, MOD_Footprints_Lib:SM0603, F.Cu at (313.9, 212.4)
Routing:
- net +3.3V: track 460.4 -> 481.1 mm, vias 15 -> 16
- net UC_LCD_E: track 44.1 -> 51.4 mm, vias 2 -> 4
- net UC_LCD_RW: track 45.1 -> 52.3 mm, vias 2 -> 4

Commit message: updating pcb layout
Parts:
- R12: value 10k -> 100k
Connections:
- C18 pad 1: Net-(C18-Pad1) -> +3.3V
- Q2 pad 2: +5V -> +3.3V
- R13 pad 1: +5V -> +3.3V
- R29 pad 1: +5V -> +3.3V
- R30 pad 1: +5V -> +3.3V
- U4 pad 6: Net-(C18-Pad1) -> +3.3V
Routing:
- net +3.3V: track 481.1 -> 538.0 mm, vias 16 -> 22
- net +5V: track 191.9 -> 151.3 mm, vias 9 -> 5
- net Net-(C18-Pad1): track 3.18 -> 0.00 mm
