File: MOD_Foot_Prototype1/MOD_Foot_Prototype1.sch (KiCad schematic (older format))
At the start: 79 parts, among them CN1 CONN_PANNEL_2X2, CN2 CONN_PANNEL_2X2, J1 RJ45_CHAIN, J2 RJ45_CHAIN, P1 HEADER_5X1, P2 HEADER_5X2, Q1 MMBT3904, Q2 MMBT3904, U1 LPC111X_LQFP48, U2 MC7805, U3 NCP1117DT33G, U4 SN75176BDR, X1 10MHz

Commit message: BOM for ITEAD quotes.
Parts:
- C1, C3: value 10uF -> 100uF
Other:
- moved on the sheet: CN1, CN2, P1, P2, R39, R40, R41
Changed lines of the file:
@@
 LIBS:MOD_Foot_Prototype1
 LIBS:MOD_Foot_Prototype1-cache
-EELAYER 27 0
+EELAYER 24 0
 EELAYER END
 $Descr A4 11693 8268
@@
 P 2950 1550
 F 0 "C3" V 3050 1650 50  0000 L CNN
-F 1 "10uF" V 2800 1450 50  0000 L CNN
+F 1 "100uF" V 2800 1450 50  0000 L CNN
 F 2 "CAP_RAD_5MM" H 2950 1550 60  0001 C CNN
 F 3 "~" H 2950 1550 60  0000 C CNN
@@
 L CONN_5X2 P2
 U 1 1 5347E35E
-P 8750 5100
-F 0 "P2" H 8750 5400 60  0000 C CNN
-F 1 "HEADER_5X2" H 8750 4800 50  0000 C CNN
-F 2 "PIN_ARRAY_5x2" H 8750 5100 60  0001 C CNN
-F 3 "" H 8750 5100 60  0000 C CNN
-	1    8750 5100
-	1    0    0    -1
-$EndComp
-Text GLabel 9850 4900 2    50   BiDi ~ 0
+P 8350 4850
+F 0 "P2" H 8350 5150 60  0000 C CNN
+F 1 "HEADER_5X2" H 8350 4550 50  0000 C CNN
+F 2 "PIN_ARRAY_5x2" H 8350 4850 60  0001 C CNN
+F 3 "" H 8350 4850 60  0000 C CNN
+	1    8350 4850
+	1    0    0    -1
+$EndComp
+Text GLabel 9450 4650 2    50   BiDi ~ 0
 SWDIO
-Text GLabel 9850 5000 2    50   Output ~ 0
+Text GLabel 9450 4750 2    50   Output ~ 0
 SWDCLK
 Text GLabel 7150 3150 0    50   BiDi ~ 0
@@
 L DGND #PWR033
 U 1 1 5347F0C7
-P 8250 5400
-F 0 "#PWR033" H 8250 5400 40  0001 C CNN
-F 1 "DGND" H 8250 5330 40  0000 C CNN
-F 2 "" H 8250 5400 60  0000 C CNN
-F 3 "" H 8250 5400 60  0000 C CNN
-	1    8250 5400
+P 7850 5150
+F 0 "#PWR033" H 7850 5150 40  0001 C CNN
+F 1 "DGND" H 7850 5080 40  0000 C CNN
+F 2 "" H 7850 5150 60  0000 C CNN
+F 3 "" H 7850 5150 60  0000 C CNN
+	1    7850 5150
 	1    0    0    -1
 $EndComp
 Text GLabel 7000 1450 0    50   Input ~ 0
 RESET
-Text GLabel 9250 5300 2    50   Output ~ 0
+Text GLabel 8850 5050 2    50   Output ~ 0
 RESET
-NoConn ~ 9150 5100
-NoConn ~ 9150 5200
+NoConn ~ 8750 4850
+NoConn ~ 8750 4950
 Text GLabel 7150 3650 0    50   Output ~ 0
 TX_CHAIN
@@
 P 1800 1550
 F 0 "C1" V 1900 1650 50  0000 L CNN
-F 1 "10uF" V 1650 1450 50  0000 L CNN
+F 1 "100uF" V 1650 1450 50  0000 L CNN
 F 2 "CAP_RAD_5MM" H 1800 1550 60  0001 C CNN
 F 3 "~" H 1800 1550 60  0000 C CNN
@@
 	1    0    0    -1
 $EndComp
-Text GLabel 6750 5000 0    50   Output ~ 0
+Text GLabel 6300 4850 0    50   Output ~ 0
 RX_CHAIN
-Text GLabel 6750 5100 0    50   Input ~ 0
+Text GLabel 6300 4950 0    50   Input ~ 0
 TX_CHAIN
 $Comp
 L +5V #PWR043
 U 1 1 53483CA1
-P 6700 4900
-F 0 "#PWR043" H 6700 4990 20  0001 C CNN
-F 1 "+5V" H 6700 4990 30  0000 C CNN
-F 2 "" H 6700 4900 60  0000 C CNN
-F 3 "" H 6700 4900 60  0000 C CNN
-	1    6700 4900
+P 6250 4750
+F 0 "#PWR043" H 6250 4840 20  0001 C CNN
+F 1 "+5V" H 6250 4840 30  0000 C CNN
+F 2 "" H 6250 4750 60  0000 C CNN
+F 3 "" H 6250 4750 60  0000 C CNN
+	1    6250 4750
 	0    -1   -1   0
 $EndComp
@@
 L DGND #PWR044
 U 1 1 53484031
-P 6800 4800
-F 0 "#PWR044" H 6800 4800 40  0001 C CNN
-F 1 "DGND" H 6800 4725 40  0000 C CNN
-F 2 "" H 6800 4800 60  0000 C CNN
-F 3 "" H 6800 4800 60  0000 C CNN
-	1    6800 4800
+P 6350 4650
+F 0 "#PWR044" H 6350 4650 40  0001 C CNN
+F 1 "DGND" H 6350 4575 40  0000 C CNN
+F 2 "" H 6350 4650 60  0000 C CNN
+F 3 "" H 6350 4650 60  0000 C CNN
+	1    6350 4650
 	0    1    -1   0
 $EndComp
@@
 $EndComp
 $Sheet
-S 7550 5850 2250 1050
+S 7500 5400 2250 1050
 U 53485BBD
 F0 "Display" 50
@@
 	7150 3150 7350 3150
 Wire Wire Line
-	9150 4900 9250 4900
-Wire Wire Line
-	9250 5000 9150 5000
-Wire Wire Line
-	8250 5000 8250 5400
-Connection ~ 8250 5200
-Connection ~ 8250 5100
-Connection ~ 8250 5300
+	8750 4650 8850 4650
+Wire Wire Line
+	8850 4750 8750 4750
+Wire Wire Line
+	7850 4750 7850 5150
+Connection ~ 7850 4950
+Connection ~ 7850 4850
+Connection ~ 7850 5050
 Wire Wire Line
 	7150 1300 7250 1300
@@
 Connection ~ 7250 1450
 Wire Wire Line
-	9150 5300 9250 5300
+	8750 5050 8850 5050
 Wire Wire Line
 	7150 3550 7350 3550
@@
 	2450 1600 2450 1700
 Wire Wire Line
-	6750 5100 6900 5100
-Wire Wire Line
-	6750 5000 6900 5000
-Wire Wire Line
-	6700 4900 6900 4900
-Wire Wire Line
-	6800 4800 6900 4800
+	6300 4950 6450 4950
+Wire Wire Line
+	6300 4850 6450 4850
+Wire Wire Line
+	6250 4750 6450 4750
+Wire Wire Line
+	6350 4650 6450 4650
 Wire Wire Line
 	6300 1550 6350 1550
@@
 	6850 1550 7350 1550
 Wire Wire Line
-	8250 5300 8350 5300
-Wire Wire Line
-	8350 5200 8250 5200
-Wire Wire Line
-	8250 5100 8350 5100
-Wire Wire Line
-	8350 5000 8250 5000
+	7850 5050 7950 5050
+Wire Wire Line
+	7950 4950 7850 4950
+Wire Wire Line
+	7850 4850 7950 4850
+Wire Wire Line
+	7950 4750 7850 4750
 Wire Wire Line
 	2900 4650 2900 4750
@@
 	3200 1150 3200 1350
 Connection ~ 3200 1250
-NoConn ~ 11050 6100
-NoConn ~ 11050 6200
-NoConn ~ 10250 6100
-NoConn ~ 10250 6200
-NoConn ~ 11050 6550
-NoConn ~ 11050 6650
-NoConn ~ 10250 6550
-NoConn ~ 10250 6650
+NoConn ~ 11000 5750
+NoConn ~ 11000 5850
+NoConn ~ 10200 5750
+NoConn ~ 10200 5850
+NoConn ~ 11000 6200
+NoConn ~ 11000 6300
+NoConn ~ 10200 6200
+NoConn ~ 10200 6300
 $Comp
 L CONN_PANNEL_2X2 CN1
 U 1 1 534AEC1C
-P 10650 6150
-F 0 "CN1" H 10650 6300 50  0000 C CNN
-F 1 "CONN_PANNEL_2X2" H 10660 6020 40  0000 C CNN
-F 2 "CONN_PANNEL" H 10650 6150 60  0001 C CNN
-F 3 "" H 10650 6150 60  0000 C CNN
-	1    10650 6150
+P 10600 5800
+F 0 "CN1" H 10600 5950 50  0000 C CNN
+F 1 "CONN_PANNEL_2X2" H 10610 5670 40  0000 C CNN
+F 2 "CONN_PANNEL" H 10600 5800 60  0001 C CNN
+F 3 "" H 10600 5800 60  0000 C CNN
+	1    10600 5800
 	1    0    0    -1
 $EndComp
@@
 L CONN_PANNEL_2X2 CN2
 U 1 1 534AEC33
-P 10650 6600
-F 0 "CN2" H 10650 6750 50  0000 C CNN
-F 1 "CONN_PANNEL_2X2" H 10660 6470 40  0000 C CNN
-F 2 "CONN_PANNEL" H 10650 6600 60  0001 C CNN
-F 3 "" H 10650 6600 60  0000 C CNN
-	1    10650 6600
+P 10600 6250
+F 0 "CN2" H 10600 6400 50  0000 C CNN
+F 1 "CONN_PANNEL_2X2" H 10610 6120 40  0000 C CNN
+F 2 "CONN_PANNEL" H 10600 6250 60  0001 C CNN
+F 3 "" H 10600 6250 60  0000 C CNN
+	1    10600 6250
 	1    0    0    -1
 $EndComp
@@
 L R R41
 U 1 1 534AC71A
-P 9500 5000
-F 0 "R41" V 9600 5000 40  0000 C CNN
-F 1 "100R" V 9507 5001 40  0000 C CNN
-F 2 "SM0603" V 9430 5000 30  0001 C CNN
-F 3 "~" H 9500 5000 30  0000 C CNN
-	1    9500 5000
+P 9100 4750
+F 0 "R41" V 9200 4750 40  0000 C CNN
+F 1 "100R" V 9107 4751 40  0000 C CNN
+F 2 "SM0603" V 9030 4750 30  0001 C CNN
+F 3 "~" H 9100 4750 30  0000 C CNN
+	1    9100 4750
 	0    1    1    0
 $EndComp
@@
 L R R40
 U 1 1 534AC720
-P 9500 4900
-F 0 "R40" V 9400 4900 40  0000 C CNN
-F 1 "100R" V 9507 4901 40  0000 C CNN
-F 2 "SM0603" V 9430 4900 30  0001 C CNN
-F 3 "~" H 9500 4900 30  0000 C CNN
-	1    9500 4900
+P 9100 4650
+F 0 "R40" V 9000 4650 40  0000 C CNN
+F 1 "100R" V 9107 4651 40  0000 C CNN
+F 2 "SM0603" V 9030 4650 30  0001 C CNN
+F 3 "~" H 9100 4650 30  0000 C CNN
+	1    9100 4650
 	0    1    1    0
 $EndComp
 Wire Wire Line
-	9750 4900 9850 4900
-Wire Wire Line
-	9850 5000 9750 5000
+	9350 4650 9450 4650
+Wire Wire Line
+	9450 4750 9350 4750
 $Comp
 L R R39
 U 1 1 534ACBE2
-P 8050 4900
-F 0 "R39" V 8130 4900 40  0000 C CNN
-F 1 "0R" V 8057 4901 40  0000 C CNN
-F 2 "SM0805" V 7980 4900 30  0001 C CNN
-F 3 "~" H 8050 4900 30  0000 C CNN
-	1    8050 4900
-	0    -1   -1   0
-$EndComp
-Wire Wire Line
-	8350 4900 8300 4900
+P 7650 4650
+F 0 "R39" V 7730 4650 40  0000 C CNN
+F 1 "0R" V 7657 4651 40  0000 C CNN
+F 2 "SM0805" V 7580 4650 30  0001 C CNN
+F 3 "~" H 7650 4650 30  0000 C CNN
+	1    7650 4650
+	0    -1   -1   0
+$EndComp
+Wire Wire Line
+	7950 4650 7900 4650
 $Comp
 L +3.3V #PWR050
 U 1 1 534ACD23
-P 7750 4900
-F 0 "#PWR050" H 7750 4860 30  0001 C CNN
-F 1 "+3.3V" H 7750 5010 30  0000 C CNN
-F 2 "" H 7750 4900 60  0000 C CNN
-F 3 "" H 7750 4900 60  0000 C CNN
-	1    7750 4900
-	0    -1   -1   0
-$EndComp
-Wire Wire Line
-	7750 4900 7800 4900
+P 7350 4650
+F 0 "#PWR050" H 7350 4610 30  0001 C CNN
+F 1 "+3.3V" H 7350 4760 30  0000 C CNN
+F 2 "" H 7350 4650 60  0000 C CNN
+F 3 "" H 7350 4650 60  0000 C CNN
+	1    7350 4650
+	0    -1   -1   0
+$EndComp
+Wire Wire Line
+	7350 4650 7400 4650
 $Comp
 L CONN_5 P1
 U 1 1 534C5616
-P 7300 5000
-F 0 "P1" H 7300 5300 50  0000 C CNN
-F 1 "HEADER_5X1" H 7300 4700 50  0000 C CNN
-F 2 "PIN_ARRAY_5x1" H 7300 5000 60  0001 C CNN
-F 3 "" H 7300 5000 60  0000 C CNN
-	1    7300 5000
-	1    0    0    -1
-$EndComp
-Text GLabel 6750 5200 0    50   Input ~ 0
+P 6850 4850
+F 0 "P1" H 6850 5150 50  0000 C CNN
+F 1 "HEADER_5X1" H 6850 4550 50  0000 C CNN
+F 2 "PIN_ARRAY_5x1" H 6850 4850 60  0001 C CNN
+F 3 "" H 6850 4850 60  0000 C CNN
+	1    6850 4850
+	1    0    0    -1
+$EndComp
+Text GLabel 6300 5050 0    50   Input ~ 0
 EN_CHAIN
 Wire Wire Line
-	6750 5200 6900 5200
+	6300 5050 6450 5050
 Wire Wire Line
 	10150 3000 9950 3000

Commit message: Solved schematic diagram of rs422 protection zener diodes.
Parts:
- removed D2, D3: MMSZ5242B, SOD123, symbol ZENERSMALL
- added D2, D3: MMSZ5242B, SOD123, symbol ZENERsmall
Connections:
- net labels added: LED5, LED6
- net labels removed: LED1, LED2
Changed lines of the file:
@@
 $EndComp
 Text GLabel 750  6950 0    50   Input ~ 0
-LED1
+LED5
 Text GLabel 950  7450 0    50   Input ~ 0
-LED2
+LED6
 $Comp
 L DGND #PWR015
@@
 F 3 "~" H 4200 6250 30  0000 C CNN
 	1    4200 6250
-	0    -1   -1   0
-$EndComp
-$Comp
-L ZENERSMALL D3
-U 1 1 53479C92
-P 4750 6450
-F 0 "D3" H 4750 6500 40  0000 C CNN
-F 1 "MMSZ5242B" H 4775 6375 30  0000 C CNN
-F 2 "SOD123" H 4750 6450 60  0001 C CNN
-F 3 "~" H 4750 6450 60  0000 C CNN
-	1    4750 6450
-	0    -1   -1   0
-$EndComp
-$Comp
-L ZENERSMALL D2
-U 1 1 53479CBA
-P 4550 6450
-F 0 "D2" H 4550 6500 40  0000 C CNN
-F 1 "MMSZ5242B" H 4575 6375 30  0000 C CNN
-F 2 "SOD123" H 4550 6450 60  0001 C CNN
-F 3 "~" H 4550 6450 60  0000 C CNN
-	1    4550 6450
 	0    -1   -1   0
 $EndComp
@@
 FOOT_4
 Text GLabel 10150 3000 2    50   Output ~ 0
-LED1
+LED5
 $Comp
 L LINEAR_REGULATOR_DPAK_3P U2
@@
 $EndComp
 Text GLabel 6250 6450 3    50   Input ~ 0
-LED2
+LED6
 $Comp
 L +5V #PWR047
@@
 	2850 650  2950 650
 Connection ~ 2950 650
+$Comp
+L ZENERsmall D3
+U 1 1 538F9A06
+P 4750 6450
+F 0 "D3" H 4748 6512 40  0000 C CNN
+F 1 "MMSZ5242B" H 4746 6378 30  0000 C CNN
+F 2 "SOD123" H 4750 6450 60  0001 C CNN
+F 3 "" H 4750 6450 60  0000 C CNN
+	1    4750 6450
+	0    -1   -1   0
+$EndComp
+$Comp
+L ZENERsmall D2
+U 1 1 538F9A7D
+P 4550 6450
+F 0 "D2" H 4548 6512 40  0000 C CNN
+F 1 "MMSZ5242B" H 4548 6384 30  0000 C CNN
+F 2 "SOD123" H 4550 6450 60  0001 C CNN
+F 3 "" H 4550 6450 60  0000 C CNN
+	1    4550 6450
+	0    -1   -1   0
+$EndComp
 $EndSCHEMATC

Commit message: fix issue #14: Broken component/footprint map file This commit makes the mod-arduino-shield a dependency. We must still move the footprint library to a single repository and declare it properly as a git submodule.
Parts:
- C1, C3, C6: footprint CAP_RAD_5MM -> MODArduinoLib:CAP_RAD_5MM
- C10, C11, C12, C13, C2, C4, C5, C7, C8, C9, R1, R10, R14, R15, R16, R17, R18, R19, R2, R20, R21, R22, R23, R24, R25, R27, R28, R29, R30, R31, R32, R33, R40, R41, R7, R8, R9: footprint SM0603 -> MODArduinoLib:SM0603
- CN1, CN2: footprint CONN_PANNEL -> MODArduinoLib:CONN_PANNEL
- D1: footprint DO-214AC(SMA) -> MODArduinoLib:DO-214AC(SMA)
- D2, D3: footprint SOD123 -> MODArduinoLib:SOD123
- D4: footprint SOD323 -> MODArduinoLib:SOD323
- FOOT1, FOOT2, FOOT3, FOOT4: footprint PIN_ARRAY_2X1 -> MODArduinoLib:PIN_ARRAY_2X1
- J1, J2: footprint RJ45-RJHSE5084 -> MODArduinoLib:RJ45-RJHSE5084
- LED1, LED2, LED3, LED4: footprint LED_CLRTB_GFSF_1 -> MODArduinoLib:LED_CLRTB_GFSF_1
- P1: footprint PIN_ARRAY_5x1 -> MODArduinoLib:PIN_ARRAY_5x1
- P2: footprint PIN_ARRAY_5x2 -> MODArduinoLib:PIN_ARRAY_5x2
- Q1, Q2: footprint SOT23 -> MODArduinoLib:SOT23
- R11, R12, R13, R26, R3, R38, R39, R4, R5, R6: footprint SM0805 -> MODArduinoLib:SM0805
- RT1: footprint SM2920 -> MODArduinoLib:SM2920
- TP1, TP2, TP3: footprint SIL-1 -> MODArduinoLib:SIL-1
- U1: footprint LQFP48 -> MODArduinoLib:LQFP48
- U2, U3: footprint DPAK(369C) -> MODArduinoLib:DPAK(369C)
- U4: footprint SO8E -> MODArduinoLib:SO8E
- X1: footprint HC_49US -> MODArduinoLib:HC_49US

Commit message: removing local footprint library and adding a submodule to use the footprint library available at the https://github.com/portalmod/mod-kicad-footprints repository.
Parts:
- C1, C3, C6: footprint MODArduinoLib:CAP_RAD_5MM -> MOD_Footprints_Lib:CAP_RAD_5MM
- C10, C11, C12, C13, C2, C4, C5, C7, C8, C9, R1, R10, R14, R15, R16, R17, R18, R19, R2, R20, R21, R22, R23, R24, R25, R27, R28, R29, R30, R31, R32, R33, R40, R41, R7, R8, R9: footprint MODArduinoLib:SM0603 -> MOD_Footprints_Lib:SM0603
- CN1, CN2: footprint MODArduinoLib:CONN_PANNEL -> MOD_Footprints_Lib:CONN_PANNEL
- D1: footprint MODArduinoLib:DO-214AC(SMA) -> MOD_Footprints_Lib:DO-214AC(SMA)
- D2, D3: footprint MODArduinoLib:SOD123 -> MOD_Footprints_Lib:SOD123
- D4: footprint MODArduinoLib:SOD323 -> MOD_Footprints_Lib:SOD323
- FOOT1, FOOT2, FOOT3, FOOT4: footprint MODArduinoLib:PIN_ARRAY_2X1 -> MOD_Footprints_Lib:PIN_ARRAY_2X1
- J1, J2: footprint MODArduinoLib:RJ45-RJHSE5084 -> MOD_Footprints_Lib:RJ45-RJHSE5084
- LED1, LED2, LED3, LED4: footprint MODArduinoLib:LED_CLRTB_GFSF_1 -> MOD_Footprints_Lib:LED_CLRTB_GFSF_1
- P1: footprint MODArduinoLib:PIN_ARRAY_5x1 -> MOD_Footprints_Lib:PIN_ARRAY_5x1
- P2: footprint MODArduinoLib:PIN_ARRAY_5x2 -> MOD_Footprints_Lib:PIN_ARRAY_5x2
- Q1, Q2: footprint MODArduinoLib:SOT23 -> MOD_Footprints_Lib:SOT23
- R11, R12, R13, R26, R3, R38, R39, R4, R5, R6: footprint MODArduinoLib:SM0805 -> MOD_Footprints_Lib:SM0805
- RT1: footprint MODArduinoLib:SM2920 -> MOD_Footprints_Lib:SM2920
- TP1, TP2, TP3: footprint MODArduinoLib:SIL-1 -> MOD_Footprints_Lib:SIL-1
- U1: footprint MODArduinoLib:LQFP48 -> MOD_Footprints_Lib:LQFP48
- U2, U3: footprint MODArduinoLib:DPAK(369C) -> MOD_Footprints_Lib:DPAK(369C)
- U4: footprint MODArduinoLib:SO8E -> MOD_Footprints_Lib:SO8E
- X1: footprint MODArduinoLib:HC_49US -> MOD_Footprints_Lib:HC_49US

Commit message: grounding the mechanical connectors (and regenerating Gerber files)
Connections:
- net DGND: now also CN1.1, CN2.1
- no-connect marks 15 -> 7
Changed lines of the file:
@@
 	3200 1150 3200 1350
 Connection ~ 3200 1250
-NoConn ~ 11000 5750
-NoConn ~ 11000 5850
-NoConn ~ 10200 5750
-NoConn ~ 10200 5850
-NoConn ~ 11000 6200
-NoConn ~ 11000 6300
-NoConn ~ 10200 6200
-NoConn ~ 10200 6300
 $Comp
 L CONN_PANNEL_2X2 CN1
@@
 	0    -1   -1   0
 $EndComp
+$Comp
+L DGND #PWR?
+U 1 1 5482017F
+P 10100 6400
+F 0 "#PWR?" H 10100 6400 40  0001 C CNN
+F 1 "DGND" H 10100 6330 40  0000 C CNN
+F 2 "" H 10100 6400 60  0000 C CNN
+F 3 "" H 10100 6400 60  0000 C CNN
+	1    10100 6400
+	1    0    0    -1
+$EndComp
+$Comp
+L DGND #PWR?
+U 1 1 548204A6
+P 11100 6400
+F 0 "#PWR?" H 11100 6400 40  0001 C CNN
+F 1 "DGND" H 11100 6330 40  0000 C CNN
+F 2 "" H 11100 6400 60  0000 C CNN
+F 3 "" H 11100 6400 60  0000 C CNN
+	1    11100 6400
+	1    0    0    -1
+$EndComp
+Wire Wire Line
+	11000 5750 11100 5750
+Wire Wire Line
+	11100 5750 11100 6400
+Wire Wire Line
+	11000 6300 11100 6300
+Connection ~ 11100 6300
+Wire Wire Line
+	11000 6200 11100 6200
+Connection ~ 11100 6200
+Wire Wire Line
+	11000 5850 11100 5850
+Connection ~ 11100 5850
+Wire Wire Line
+	10200 5750 10100 5750
+Wire Wire Line
+	10100 5750 10100 6400
+Wire Wire Line
+	10200 6300 10100 6300
+Connection ~ 10100 6300
+Wire Wire Line
+	10200 6200 10100 6200
+Connection ~ 10100 6200
+Wire Wire Line
+	10200 5850 10100 5850
+Connection ~ 10100 5850
 $EndSCHEMATC
