File: MOD_Foot_Prototype1/MOD_Foot_Prototype1.sch (KiCad schematic (older format))
At the start: 79 parts, among them CN1 CONN_PANNEL_2X2, CN2 CONN_PANNEL_2X2, J1 RJ45_CHAIN, J2 RJ45_CHAIN, P1 HEADER_5X1, P2 HEADER_5X2, Q1 MMBT3904, Q2 MMBT3904, U1 LPC111X_LQFP48, U2 MC7805, U3 NCP1117DT33G, U4 SN75176BDR, X1 10MHz

Commit message: wip issue #11: protect the U4 IC when the board is being debugged - made the changes in the schematics
Parts:
- removed P1: HEADER_5X1, MOD_Footprints_Lib:PIN_ARRAY_5x1, symbol CONN_5
- added P1: HEADER_5X2, MOD_Footprints_Lib:PIN_ARRAY_5x2, symbol CONN_5X2
- added R? (x2): 0R, MOD_Footprints_Lib:SM0805, symbol R
Connections:
- net +3.3V: now also R39.2; no longer R39.1
- net +5V: now also P1.3, P1.4
- net DGND: now also P1.1, P1.2
- net EN_CHAIN: now also P1.10, P1.9
- net LED6: now also P1.7, R?.2; no longer U1.47 (PIO1_7/TXD/CT32B0_MAT1)
- net RX_CHAIN: now also P1.5, R?.2; no longer U1.46 (PIO1_6/RXD/CT32B0_MAT0)
- net at P2.1: now also R39.1; no longer R39.2
- new net: P1.6, R?.1, U1.46 (PIO1_6/RXD/CT32B0_MAT0)
- new net: P1.8, R?.1, U1.47 (PIO1_7/TXD/CT32B0_MAT1)
Other:
- moved on the sheet: LED1, LED2, LED3, LED4, P2, R14, R15, R16, R17, R18, R19, R20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

Commit message: fix issue #11: protect the U4 IC when the board is being debugged Updated PCB traces and regenerated Gerbers.
Parts:
- gave numbers to parts that had none: 2

Commit message: fixed issue #9 by adding an SM1210 footprint for a second fuse. It's up to us to decide which kind of fuse to solder in the board, but the PCB has got both footprints.
Parts:
- added RT2: PTC_FUSE_500mA, MOD_Footprints_Lib:SM2920, symbol FUSE
- RT1: footprint MOD_Footprints_Lib:SM2920 -> MOD_Footprints_Lib:SM1210
Connections:
- net +9V: now also RT2.2
- net at D1.2 (K), RT1.1: now also RT2.1
Other:
- moved on the sheet: D1, RT1

Commit message: sch: created one sheet for each part of the circuit
Parts:
- removed C1, C3, C6: 100uF, MOD_Footprints_Lib:CAP_RAD_5MM, symbol CP1
- removed C10, C11: 18pF_NP0, MOD_Footprints_Lib:SM0603, symbol C
- removed C12, C13, C2, C4, C5, C7, C8, C9: 100nF_X7R, MOD_Footprints_Lib:SM0603, symbol C
- removed CN1, CN2: CONN_PANNEL_2X2, MOD_Footprints_Lib:CONN_PANNEL, symbol CONN_PANNEL_2X2
- removed D1: CGRA4007-G, MOD_Footprints_Lib:DO-214AC(SMA), symbol DIODE
- removed D2, D3: MMSZ5242B, MOD_Footprints_Lib:SOD123, symbol ZENERsmall
- removed D4: 1N4148, MOD_Footprints_Lib:SOD323, symbol DIODE
- removed FOOT1, FOOT2, FOOT3, FOOT4: HEADER_2X1_180, MOD_Footprints_Lib:PIN_ARRAY_2X1, symbol CONN_2
- removed J1, J2: RJ45_CHAIN, MOD_Footprints_Lib:RJ45-RJHSE5084, symbol RJ45_CHAIN
- removed LED1, LED2, LED3, LED4: LED_RGB, MOD_Footprints_Lib:LED_CLRTB_GFSF_1, symbol LED_RGB
- removed P1, P2: HEADER_5X2, MOD_Footprints_Lib:PIN_ARRAY_5x2, symbol CONN_5X2
- removed Q1, Q2: MMBT3904, MOD_Footprints_Lib:SOT23, symbol NPN
- removed R1, R14, R15, R16, R17, R18, R19, R2, R20, R21, R22, R23, R24, R25, R27, R28: 1k, MOD_Footprints_Lib:SM0603, symbol R
- removed R10, R29, R30, R31, R32, R33, R7, R8, R9: 10k, MOD_Footprints_Lib:SM0603, symbol R
- removed R11: 120R, MOD_Footprints_Lib:SM0805, symbol R
- removed R12, R13: 10R, MOD_Footprints_Lib:SM0805, symbol R
- removed R26, R38, R39, R42, R43: 0R, MOD_Footprints_Lib:SM0805, symbol R
- removed R3, R4, R5, R6: 470R, MOD_Footprints_Lib:SM0805, symbol R
- removed R40, R41: 100R, MOD_Footprints_Lib:SM0603, symbol R
- removed RT1: PTC_FUSE_500mA, MOD_Footprints_Lib:SM1210, symbol FUSE
- removed RT2: PTC_FUSE_500mA, MOD_Footprints_Lib:SM2920, symbol FUSE
- removed TP1, TP2, TP3: CONN_1, MOD_Footprints_Lib:SIL-1, symbol CONN_1
- removed U1: LPC111X_LQFP48, MOD_Footprints_Lib:LQFP48, symbol LPC111X_LQFP48
- removed U2: MC7805, MOD_Footprints_Lib:DPAK(369C), symbol LINEAR_REGULATOR_DPAK_3P
- removed U3: NCP1117DT33G, MOD_Footprints_Lib:DPAK(369C), symbol NCP1117DT33G
- removed U4: SN75176BDR, MOD_Footprints_Lib:SO8E, symbol SN75176BDR
- removed X1: 10MHz, MOD_Footprints_Lib:HC_49US, symbol CRYSTAL
Connections:
- no-connect marks 7 -> 0
