File: MOD_Foot_Prototype1/control-chain.sch (KiCad schematic (older format))
At the start: 25 parts, among them J1 RJ45_CHAIN_MAIN, J2 RJ45_CHAIN_EXTENSION, Q1 MMBT3904, Q2 MMBT3906, U4 MAX13450E

Commit message: Modifying the control chain RTERM_CHAIN circuit to generate a 3.3V logic signal. (instead of 5 volts)
Parts:
- R12: value 10k -> 100k
Connections:
- net +3.3V: now also Q2.2 (E), R13.1
- net +5V: no longer Q2.2 (E), R13.1
Changed lines of the file:
@@
 P 4600 4550
 F 0 "R12" V 4500 4550 40  0000 C CNN
-F 1 "10k" V 4607 4551 40  0000 C CNN
+F 1 "100k" V 4607 4551 40  0000 C CNN
 F 2 "MOD_Footprints_Lib:SM0603" V 4530 4550 30  0001 C CNN
 F 3 "~" H 4600 4550 30  0000 C CNN
@@
 Text GLabel 6300 4850 2    50   Input ~ 0
 RTERM_CHAIN
-$Comp
-L +5V #PWR019
-U 1 1 5488151E
-P 5000 3750
-F 0 "#PWR019" H 5000 3840 20  0001 C CNN
-F 1 "+5V" H 5000 3840 30  0000 C CNN
-F 2 "" H 5000 3750 60  0000 C CNN
-F 3 "" H 5000 3750 60  0000 C CNN
-	1    5000 3750
-	1    0    0    -1
-$EndComp
-Wire Wire Line
-	3600 2200 3850 2200
-Wire Wire Line
-	3850 2200 4400 2200
-Wire Wire Line
-	3600 4350 3700 4350
-Wire Wire Line
-	3700 4350 4100 4350
+Wire Wire Line
+	3600 2200 4400 2200
+Wire Wire Line
+	3600 4350 4100 4350
 Wire Wire Line
 	8900 2600 9150 2600
@@
 	3600 2900 3700 2900
 Wire Wire Line
-	3700 2800 3700 2900
-Wire Wire Line
-	3700 2900 3700 3050
+	3700 2800 3700 3050
 Wire Wire Line
 	3600 2800 3700 2800
 Wire Wire Line
-	3600 2700 4300 2700
-Wire Wire Line
-	4300 2700 4400 2700
-Wire Wire Line
-	4100 2550 4200 2550
-Wire Wire Line
-	4200 2550 4400 2550
+	3600 2700 4400 2700
+Wire Wire Line
+	4100 2550 4400 2550
 Wire Wire Line
 	4100 2400 4100 2550
@@
 	4100 2300 4100 2350
 Wire Wire Line
-	3600 2300 3950 2300
-Wire Wire Line
-	3950 2300 4100 2300
+	3600 2300 4100 2300
 Connection ~ 3950 2300
 Wire Wire Line
@@
 Connection ~ 2300 1600
 Wire Wire Line
-	2300 1700 2300 1600
+	2300 1600 2300 1700
 Connection ~ 2150 1600
 Wire Wire Line
@@
 Connection ~ 2000 1600
 Wire Wire Line
-	2000 1600 2150 1600
-Wire Wire Line
-	2150 1600 2300 1600
-Wire Wire Line
-	2300 1600 2450 1600
+	2000 1600 2450 1600
 Wire Wire Line
 	2450 1600 2450 1700
 Wire Wire Line
-	2000 1500 2000 1600
-Wire Wire Line
-	2000 1600 2000 1700
+	2000 1500 2000 1700
 Wire Wire Line
 	2450 2350 2450 2500
@@
 	2450 2200 2450 2250
 Wire Wire Line
-	7050 2250 7450 2250
-Wire Wire Line
-	7450 2250 7700 2250
-Wire Wire Line
-	7050 2050 7250 2050
-Wire Wire Line
-	7250 2050 7700 2050
+	7050 2250 7700 2250
+Wire Wire Line
+	7050 2050 7700 2050
 Wire Wire Line
 	7050 3050 7700 3050
@@
 	9500 2450 9500 2000
 Wire Wire Line
-	8900 2450 9500 2450
-Wire Wire Line
-	9500 2450 9650 2450
-Wire Wire Line
-	9500 1300 9500 1400
-Wire Wire Line
-	9500 1400 9500 1500
+	8900 2450 9650 2450
+Wire Wire Line
+	9500 1300 9500 1500
 Wire Wire Line
 	9000 2300 9000 2350
@@
 	9250 2000 9250 2150
 Wire Wire Line
-	8900 2150 9250 2150
-Wire Wire Line
-	9250 2150 9750 2150
+	8900 2150 9750 2150
 Connection ~ 9600 2750
 Wire Wire Line
 	9600 3350 9600 3450
 Wire Wire Line
-	8900 2750 9600 2750
-Wire Wire Line
-	9600 2750 9850 2750
+	8900 2750 9850 2750
 Wire Wire Line
 	8900 2950 9050 2950
@@
 	9000 2000 8900 2000
 Wire Wire Line
-	8050 3550 8050 3650
-Wire Wire Line
-	8050 3650 8050 3800
+	8050 3550 8050 3800
 Wire Wire Line
 	8050 4200 8050 4300
@@
 	7350 2650 7350 2700
 Wire Wire Line
-	7250 2650 7350 2650
-Wire Wire Line
-	7350 2650 7450 2650
+	7250 2650 7450 2650
 Wire Wire Line
 	7250 2550 7250 2650
@@
 Connection ~ 2300 4600
 Wire Wire Line
-	2300 2850 2300 4600
-Wire Wire Line
-	2300 4600 2300 4900
+	2300 2850 2300 4900
 Wire Wire Line
 	4100 4350 4100 4200
@@
 	3700 2600 3600 2600
 Wire Wire Line
-	3700 1900 3700 2500
-Wire Wire Line
-	3700 2500 3700 2600
+	3700 1900 3700 2600
 Wire Wire Line
 	3600 2500 3700 2500
@@
 	3700 4650 3700 4800
 Wire Wire Line
-	3600 4550 4000 4550
-Wire Wire Line
-	4000 4550 4250 4550
-Wire Wire Line
-	4250 4550 4350 4550
-Wire Wire Line
-	4850 4550 5000 4550
-Wire Wire Line
-	5000 4550 5150 4550
+	3600 4550 4350 4550
+Wire Wire Line
+	4850 4550 5150 4550
 Wire Wire Line
 	5000 4450 5000 4550
 Connection ~ 5000 4550
 Wire Wire Line
-	5000 3750 5000 3850
-Wire Wire Line
-	5000 3850 5000 3950
+	5000 3750 5000 3950
 Wire Wire Line
 	6050 3850 6050 4350
@@
 Connection ~ 5000 3850
 Wire Wire Line
-	6050 4750 6050 4850
-Wire Wire Line
-	6050 4850 6050 4950
+	6050 4750 6050 4950
 Wire Wire Line
 	6050 5450 6050 5550
@@
 	7850 3650 8050 3650
 Connection ~ 8050 3650
+$Comp
+L +3.3V #PWR?
+U 1 1 5491D651
+P 5000 3750
+F 0 "#PWR?" H 5000 3710 30  0001 C CNN
+F 1 "+3.3V" H 5000 3860 30  0000 C CNN
+F 2 "" H 5000 3750 60  0000 C CNN
+F 3 "" H 5000 3750 60  0000 C CNN
+	1    5000 3750
+	1    0    0    -1
+$EndComp
 $EndSCHEMATC
