File: MOD_Foot_Prototype1/Display.sch (KiCad schematic (older format))
At the start: 12 parts, among them Q3 MMBT3904, U5 74HC245, U6 74HC245

Commit message: fix issue #14: Broken component/footprint map file This commit makes the mod-arduino-shield a dependency. We must still move the footprint library to a single repository and declare it properly as a git submodule.
Parts:
- C14, C15, C17, R36: footprint SM0603 -> MODArduinoLib:SM0603
- C16: footprint CAP_RAD_5MM -> MODArduinoLib:CAP_RAD_5MM
- LCD1: footprint LCD-AGM-2004A-204 -> MODArduinoLib:LCD-AGM-2004A-204
- Q3: footprint SOT23 -> MODArduinoLib:SOT23
- R34, R35, R37: footprint SM0805 -> MODArduinoLib:SM0805
- U5, U6: footprint TSSOP20 -> MODArduinoLib:TSSOP20
Changed lines of the file:
@@
 LIBS:MOD_Foot_Prototype1
 LIBS:MOD_Foot_Prototype1-cache
-EELAYER 24 0
+EELAYER 25 0
 EELAYER END
 $Descr A4 11693 8268
@@
 F 0 "U5" H 4350 3700 60  0000 L BNN
 F 1 "74HC245" H 4250 2600 60  0000 L TNN
-F 2 "TSSOP20" H 4400 3150 60  0001 C CNN
+F 2 "MODArduinoLib:TSSOP20" H 4400 3150 60  0001 C CNN
 F 3 "~" H 4400 3150 60  0000 C CNN
 	1    4400 3150
@@
 F 0 "U6" H 4350 5450 60  0000 L BNN
 F 1 "74HC245" H 4250 4350 60  0000 L TNN
-F 2 "TSSOP20" H 4400 4900 60  0001 C CNN
+F 2 "MODArduinoLib:TSSOP20" H 4400 4900 60  0001 C CNN
 F 3 "~" H 4400 4900 60  0000 C CNN
 	1    4400 4900
@@
 F 0 "C14" V 4450 2350 40  0000 L CNN
 F 1 "100nF_X7R" V 4750 2250 40  0000 L CNN
-F 2 "SM0603" H 4638 2250 30  0001 C CNN
+F 2 "MODArduinoLib:SM0603" H 4638 2250 30  0001 C CNN
 F 3 "~" H 4600 2400 60  0000 C CNN
 	1    4600 2400
@@
 F 0 "C17" V 8600 2750 40  0000 L CNN
 F 1 "100nF_X7R" V 8800 2500 40  0000 L CNN
-F 2 "SM0603" H 8688 2500 30  0001 C CNN
+F 2 "MODArduinoLib:SM0603" H 8688 2500 30  0001 C CNN
 F 3 "~" H 8650 2650 60  0000 C CNN
 	1    8650 2650
@@
 F 0 "C15" V 4450 4000 40  0000 L CNN
 F 1 "100nF_X7R" V 4750 3900 40  0000 L CNN
-F 2 "SM0603" H 4638 3900 30  0001 C CNN
+F 2 "MODArduinoLib:SM0603" H 4638 3900 30  0001 C CNN
 F 3 "~" H 4600 4050 60  0000 C CNN
 	1    4600 4050
@@
 F 0 "C16" V 8700 2950 50  0000 L CNN
 F 1 "100uF" V 8500 2750 50  0000 L CNN
-F 2 "CAP_RAD_5MM" H 8650 2850 60  0001 C CNN
+F 2 "MODArduinoLib:CAP_RAD_5MM" H 8650 2850 60  0001 C CNN
 F 3 "~" H 8650 2850 60  0000 C CNN
 	1    8650 2850
@@
 F 0 "Q3" H 8400 5400 50  0000 R CNN
 F 1 "MMBT3904" V 8650 5750 50  0000 R CNN
-F 2 "SOT23" H 8400 5550 60  0001 C CNN
+F 2 "MODArduinoLib:SOT23" H 8400 5550 60  0001 C CNN
 F 3 "~" H 8400 5550 60  0000 C CNN
 	1    8400 5550
@@
 F 0 "R36" V 7930 5550 40  0000 C CNN
 F 1 "1k" V 7857 5551 40  0000 C CNN
-F 2 "SM0603" V 7780 5550 30  0001 C CNN
+F 2 "MODArduinoLib:SM0603" V 7780 5550 30  0001 C CNN
 F 3 "~" H 7850 5550 30  0000 C CNN
 	1    7850 5550
@@
 F 0 "R35" V 7830 3700 40  0000 C CNN
 F 1 "330R" V 7757 3701 40  0000 C CNN
-F 2 "SM0805" V 7680 3700 30  0001 C CNN
+F 2 "MODArduinoLib:SM0805" V 7680 3700 30  0001 C CNN
 F 3 "~" H 7750 3700 30  0000 C CNN
 	1    7750 3700
@@
 F 0 "R34" V 7830 3000 40  0000 C CNN
 F 1 "3k" V 7757 3001 40  0000 C CNN
-F 2 "SM0805" V 7680 3000 30  0001 C CNN
+F 2 "MODArduinoLib:SM0805" V 7680 3000 30  0001 C CNN
 F 3 "~" H 7750 3000 30  0000 C CNN
 	1    7750 3000
@@
 F 0 "LCD1" H 8950 4800 60  0000 C CNN
 F 1 "AGM-2004A-204" V 9600 3950 60  0000 C CNN
-F 2 "LCD-AGM-2004A-204" H 8950 3900 60  0001 C CNN
+F 2 "MODArduinoLib:LCD-AGM-2004A-204" H 8950 3900 60  0001 C CNN
 F 3 "" H 8950 3900 60  0000 C CNN
 	1    8950 3900
@@
 F 0 "R37" V 8580 5000 40  0000 C CNN
 F 1 "0R" V 8507 5001 40  0000 C CNN
-F 2 "SM0805" V 8430 5000 30  0001 C CNN
+F 2 "MODArduinoLib:SM0805" V 8430 5000 30  0001 C CNN
 F 3 "~" H 8500 5000 30  0000 C CNN
 	1    8500 5000

Commit message: removing local footprint library and adding a submodule to use the footprint library available at the https://github.com/portalmod/mod-kicad-footprints repository.
Parts:
- C14, C15, C17, R36: footprint MODArduinoLib:SM0603 -> MOD_Footprints_Lib:SM0603
- C16: footprint MODArduinoLib:CAP_RAD_5MM -> MOD_Footprints_Lib:CAP_RAD_5MM
- LCD1: footprint MODArduinoLib:LCD-AGM-2004A-204 -> MOD_Footprints_Lib:LCD-AGM-2004A-204
- Q3: footprint MODArduinoLib:SOT23 -> MOD_Footprints_Lib:SOT23
- R34, R35, R37: footprint MODArduinoLib:SM0805 -> MOD_Footprints_Lib:SM0805
- U5, U6: footprint MODArduinoLib:TSSOP20 -> MOD_Footprints_Lib:TSSOP20
Changed lines of the file:
@@
 F 0 "U5" H 4350 3700 60  0000 L BNN
 F 1 "74HC245" H 4250 2600 60  0000 L TNN
-F 2 "MODArduinoLib:TSSOP20" H 4400 3150 60  0001 C CNN
+F 2 "MOD_Footprints_Lib:TSSOP20" H 4400 3150 60  0001 C CNN
 F 3 "~" H 4400 3150 60  0000 C CNN
 	1    4400 3150
@@
 F 0 "U6" H 4350 5450 60  0000 L BNN
 F 1 "74HC245" H 4250 4350 60  0000 L TNN
-F 2 "MODArduinoLib:TSSOP20" H 4400 4900 60  0001 C CNN
+F 2 "MOD_Footprints_Lib:TSSOP20" H 4400 4900 60  0001 C CNN
 F 3 "~" H 4400 4900 60  0000 C CNN
 	1    4400 4900
@@
 F 0 "C14" V 4450 2350 40  0000 L CNN
 F 1 "100nF_X7R" V 4750 2250 40  0000 L CNN
-F 2 "MODArduinoLib:SM0603" H 4638 2250 30  0001 C CNN
+F 2 "MOD_Footprints_Lib:SM0603" H 4638 2250 30  0001 C CNN
 F 3 "~" H 4600 2400 60  0000 C CNN
 	1    4600 2400
@@
 F 0 "C17" V 8600 2750 40  0000 L CNN
 F 1 "100nF_X7R" V 8800 2500 40  0000 L CNN
-F 2 "MODArduinoLib:SM0603" H 8688 2500 30  0001 C CNN
+F 2 "MOD_Footprints_Lib:SM0603" H 8688 2500 30  0001 C CNN
 F 3 "~" H 8650 2650 60  0000 C CNN
 	1    8650 2650
@@
 F 0 "C15" V 4450 4000 40  0000 L CNN
 F 1 "100nF_X7R" V 4750 3900 40  0000 L CNN
-F 2 "MODArduinoLib:SM0603" H 4638 3900 30  0001 C CNN
+F 2 "MOD_Footprints_Lib:SM0603" H 4638 3900 30  0001 C CNN
 F 3 "~" H 4600 4050 60  0000 C CNN
 	1    4600 4050
@@
 F 0 "C16" V 8700 2950 50  0000 L CNN
 F 1 "100uF" V 8500 2750 50  0000 L CNN
-F 2 "MODArduinoLib:CAP_RAD_5MM" H 8650 2850 60  0001 C CNN
+F 2 "MOD_Footprints_Lib:CAP_RAD_5MM" H 8650 2850 60  0001 C CNN
 F 3 "~" H 8650 2850 60  0000 C CNN
 	1    8650 2850
@@
 F 0 "Q3" H 8400 5400 50  0000 R CNN
 F 1 "MMBT3904" V 8650 5750 50  0000 R CNN
-F 2 "MODArduinoLib:SOT23" H 8400 5550 60  0001 C CNN
+F 2 "MOD_Footprints_Lib:SOT23" H 8400 5550 60  0001 C CNN
 F 3 "~" H 8400 5550 60  0000 C CNN
 	1    8400 5550
@@
 F 0 "R36" V 7930 5550 40  0000 C CNN
 F 1 "1k" V 7857 5551 40  0000 C CNN
-F 2 "MODArduinoLib:SM0603" V 7780 5550 30  0001 C CNN
+F 2 "MOD_Footprints_Lib:SM0603" V 7780 5550 30  0001 C CNN
 F 3 "~" H 7850 5550 30  0000 C CNN
 	1    7850 5550
@@
 F 0 "R35" V 7830 3700 40  0000 C CNN
 F 1 "330R" V 7757 3701 40  0000 C CNN
-F 2 "MODArduinoLib:SM0805" V 7680 3700 30  0001 C CNN
+F 2 "MOD_Footprints_Lib:SM0805" V 7680 3700 30  0001 C CNN
 F 3 "~" H 7750 3700 30  0000 C CNN
 	1    7750 3700
@@
 F 0 "R34" V 7830 3000 40  0000 C CNN
 F 1 "3k" V 7757 3001 40  0000 C CNN
-F 2 "MODArduinoLib:SM0805" V 7680 3000 30  0001 C CNN
+F 2 "MOD_Footprints_Lib:SM0805" V 7680 3000 30  0001 C CNN
 F 3 "~" H 7750 3000 30  0000 C CNN
 	1    7750 3000
@@
 F 0 "LCD1" H 8950 4800 60  0000 C CNN
 F 1 "AGM-2004A-204" V 9600 3950 60  0000 C CNN
-F 2 "MODArduinoLib:LCD-AGM-2004A-204" H 8950 3900 60  0001 C CNN
+F 2 "MOD_Footprints_Lib:LCD-AGM-2004A-204" H 8950 3900 60  0001 C CNN
 F 3 "" H 8950 3900 60  0000 C CNN
 	1    8950 3900
@@
 F 0 "R37" V 8580 5000 40  0000 C CNN
 F 1 "0R" V 8507 5001 40  0000 C CNN
-F 2 "MODArduinoLib:SM0805" V 8430 5000 30  0001 C CNN
+F 2 "MOD_Footprints_Lib:SM0805" V 8430 5000 30  0001 C CNN
 F 3 "~" H 8500 5000 30  0000 C CNN
 	1    8500 5000
