File: MOD_Foot_Prototype1/io.sch (KiCad schematic (older format))
At the start: 24 parts

Commit message: Fixing schematics references numbering. Also regenerated .net and .cmp files.
Parts:
- renumbered R23 to R10, R24 to R14, R25 to R15, R26 to R16, R27 to R17, R28 to R18, R29 to R19, R30 to R20, R31 to R21, R32 to R22, R33 to R23, R38 to R24, R39 to R25, R20 to R7, R21 to R8, R22 to R9
Changed lines of the file:
@@
 FOOT_4
 $Comp
-L R R23
+L R R10
 U 1 1 548337D0
 P 2900 1900
-F 0 "R23" V 3000 1900 40  0000 C CNN
+F 0 "R10" V 3000 1900 40  0000 C CNN
 F 1 "10k" V 2907 1901 40  0000 C CNN
 F 2 "MOD_Footprints_Lib:SM0603" V 2830 1900 30  0001 C CNN
@@
 $EndComp
 $Comp
-L R R22
+L R R9
 U 1 1 548337D7
 P 2800 1900
-F 0 "R22" V 2850 2125 40  0000 C CNN
+F 0 "R9" V 2850 2125 40  0000 C CNN
 F 1 "10k" V 2807 1901 40  0000 C CNN
 F 2 "MOD_Footprints_Lib:SM0603" V 2730 1900 30  0001 C CNN
@@
 $EndComp
 $Comp
-L R R21
+L R R8
 U 1 1 548337DE
 P 2700 1900
-F 0 "R21" V 2750 2125 40  0000 C CNN
+F 0 "R8" V 2750 2125 40  0000 C CNN
 F 1 "10k" V 2707 1901 40  0000 C CNN
 F 2 "MOD_Footprints_Lib:SM0603" V 2630 1900 30  0001 C CNN
@@
 $EndComp
 $Comp
-L R R20
+L R R7
 U 1 1 548337E5
 P 2600 1900
-F 0 "R20" V 2500 1900 40  0000 C CNN
+F 0 "R7" V 2500 1900 40  0000 C CNN
 F 1 "10k" V 2607 1901 40  0000 C CNN
 F 2 "MOD_Footprints_Lib:SM0603" V 2530 1900 30  0001 C CNN
@@
 $EndComp
 $Comp
-L R R24
+L R R14
 U 1 1 548337F9
 P 4550 1600
-F 0 "R24" V 4475 1600 40  0000 C CNN
+F 0 "R14" V 4475 1600 40  0000 C CNN
 F 1 "1k" V 4557 1601 40  0000 C CNN
 F 2 "MOD_Footprints_Lib:SM0603" V 4480 1600 30  0001 C CNN
@@
 $EndComp
 $Comp
-L R R25
+L R R15
 U 1 1 54833800
 P 4550 1750
-F 0 "R25" V 4475 1750 40  0000 C CNN
+F 0 "R15" V 4475 1750 40  0000 C CNN
 F 1 "1k" V 4557 1751 40  0000 C CNN
 F 2 "MOD_Footprints_Lib:SM0603" V 4480 1750 30  0001 C CNN
@@
 $EndComp
 $Comp
-L R R26
+L R R16
 U 1 1 54833807
 P 4550 1900
-F 0 "R26" V 4475 1900 40  0000 C CNN
+F 0 "R16" V 4475 1900 40  0000 C CNN
 F 1 "1k" V 4557 1901 40  0000 C CNN
 F 2 "MOD_Footprints_Lib:SM0603" V 4480 1900 30  0001 C CNN
@@
 $EndComp
 $Comp
-L R R27
+L R R17
 U 1 1 5483381E
 P 4550 2300
-F 0 "R27" V 4475 2300 40  0000 C CNN
+F 0 "R17" V 4475 2300 40  0000 C CNN
 F 1 "1k" V 4557 2301 40  0000 C CNN
 F 2 "MOD_Footprints_Lib:SM0603" V 4480 2300 30  0001 C CNN
@@
 $EndComp
 $Comp
-L R R28
+L R R18
 U 1 1 54833825
 P 4550 2450
-F 0 "R28" V 4475 2450 40  0000 C CNN
+F 0 "R18" V 4475 2450 40  0000 C CNN
 F 1 "1k" V 4557 2451 40  0000 C CNN
 F 2 "MOD_Footprints_Lib:SM0603" V 4480 2450 30  0001 C CNN
@@
 $EndComp
 $Comp
-L R R29
+L R R19
 U 1 1 5483382C
 P 4550 2600
-F 0 "R29" V 4475 2600 40  0000 C CNN
+F 0 "R19" V 4475 2600 40  0000 C CNN
 F 1 "1k" V 4557 2601 40  0000 C CNN
 F 2 "MOD_Footprints_Lib:SM0603" V 4480 2600 30  0001 C CNN
@@
 $EndComp
 $Comp
-L R R30
+L R R20
 U 1 1 54833843
 P 4550 3000
-F 0 "R30" V 4475 3000 40  0000 C CNN
+F 0 "R20" V 4475 3000 40  0000 C CNN
 F 1 "1k" V 4557 3001 40  0000 C CNN
 F 2 "MOD_Footprints_Lib:SM0603" V 4480 3000 30  0001 C CNN
@@
 $EndComp
 $Comp
-L R R31
+L R R21
 U 1 1 5483384A
 P 4550 3150
-F 0 "R31" V 4475 3150 40  0000 C CNN
+F 0 "R21" V 4475 3150 40  0000 C CNN
 F 1 "1k" V 4557 3151 40  0000 C CNN
 F 2 "MOD_Footprints_Lib:SM0603" V 4480 3150 30  0001 C CNN
@@
 $EndComp
 $Comp
-L R R32
+L R R22
 U 1 1 54833851
 P 4550 3300
-F 0 "R32" V 4475 3300 40  0000 C CNN
+F 0 "R22" V 4475 3300 40  0000 C CNN
 F 1 "1k" V 4557 3301 40  0000 C CNN
 F 2 "MOD_Footprints_Lib:SM0603" V 4480 3300 30  0001 C CNN
@@
 $EndComp
 $Comp
-L R R33
+L R R23
 U 1 1 54833868
 P 4550 3700
-F 0 "R33" V 4475 3700 40  0000 C CNN
+F 0 "R23" V 4475 3700 40  0000 C CNN
 F 1 "1k" V 4557 3701 40  0000 C CNN
 F 2 "MOD_Footprints_Lib:SM0603" V 4480 3700 30  0001 C CNN
@@
 $EndComp
 $Comp
-L R R38
+L R R24
 U 1 1 5483386F
 P 4550 3850
-F 0 "R38" V 4475 3850 40  0000 C CNN
+F 0 "R24" V 4475 3850 40  0000 C CNN
 F 1 "1k" V 4557 3851 40  0000 C CNN
 F 2 "MOD_Footprints_Lib:SM0603" V 4480 3850 30  0001 C CNN
@@
 $EndComp
 $Comp
-L R R39
+L R R25
 U 1 1 54833876
 P 4550 4000
-F 0 "R39" V 4475 4000 40  0000 C CNN
+F 0 "R25" V 4475 4000 40  0000 C CNN
 F 1 "1k" V 4557 4001 40  0000 C CNN
 F 2 "MOD_Footprints_Lib:SM0603" V 4480 4000 30  0001 C CNN
