File: MOD_Foot_Prototype1/power.sch (KiCad schematic (older format))
At the start: 16 parts, among them U3 MC7805, U4 NCP1117DT33G

Commit message: sch: ERC passing
Changed lines of the file:
@@
 $EndComp
 $Comp
-L DGND #PWR46
+L DGND #PWR044
 U 1 1 54831906
 P 5600 2950
-F 0 "#PWR46" H 5600 2950 40  0001 C CNN
+F 0 "#PWR044" H 5600 2950 40  0001 C CNN
 F 1 "DGND" H 5600 2880 40  0000 C CNN
 F 2 "" H 5600 2950 60  0000 C CNN
@@
 $EndComp
 $Comp
-L DGND #PWR43
+L DGND #PWR045
 U 1 1 5483190C
 P 4550 2950
-F 0 "#PWR43" H 4550 2950 40  0001 C CNN
+F 0 "#PWR045" H 4550 2950 40  0001 C CNN
 F 1 "DGND" H 4550 2880 40  0000 C CNN
 F 2 "" H 4550 2950 60  0000 C CNN
@@
 $EndComp
 $Comp
-L DGND #PWR45
+L DGND #PWR046
 U 1 1 54831919
 P 5200 2800
-F 0 "#PWR45" H 5200 2800 40  0001 C CNN
+F 0 "#PWR046" H 5200 2800 40  0001 C CNN
 F 1 "DGND" H 5200 2730 40  0000 C CNN
 F 2 "" H 5200 2800 60  0000 C CNN
@@
 $EndComp
 $Comp
-L +3.3V #PWR48
+L +3.3V #PWR047
 U 1 1 5483191F
 P 6550 2200
-F 0 "#PWR48" H 6550 2160 30  0001 C CNN
+F 0 "#PWR047" H 6550 2160 30  0001 C CNN
 F 1 "+3.3V" H 6550 2310 30  0000 C CNN
 F 2 "" H 6550 2200 60  0000 C CNN
@@
 $EndComp
 $Comp
-L DGND #PWR47
+L DGND #PWR048
 U 1 1 5483192C
 P 5850 2950
-F 0 "#PWR47" H 5850 2950 40  0001 C CNN
+F 0 "#PWR048" H 5850 2950 40  0001 C CNN
 F 1 "DGND" H 5850 2880 40  0000 C CNN
 F 2 "" H 5850 2950 60  0000 C CNN
@@
 $EndComp
 $Comp
-L PWR_FLAG #FLG5
+L PWR_FLAG #FLG049
 U 1 1 54831939
 P 6750 2250
-F 0 "#FLG5" H 6750 2345 30  0001 C CNN
+F 0 "#FLG049" H 6750 2345 30  0001 C CNN
 F 1 "PWR_FLAG" H 6750 2430 30  0000 C CNN
 F 2 "" H 6750 2250 60  0000 C CNN
@@
 $EndComp
 $Comp
-L DGND #PWR44
+L DGND #PWR050
 U 1 1 54831946
 P 4800 2950
-F 0 "#PWR44" H 4800 2950 40  0001 C CNN
+F 0 "#PWR050" H 4800 2950 40  0001 C CNN
 F 1 "DGND" H 4800 2880 40  0000 C CNN
 F 2 "" H 4800 2950 60  0000 C CNN
@@
 $EndComp
 $Comp
-L DGND #PWR39
+L DGND #PWR051
 U 1 1 54831960
-P 3400 2950
-F 0 "#PWR39" H 3400 2950 40  0001 C CNN
-F 1 "DGND" H 3400 2880 40  0000 C CNN
-F 2 "" H 3400 2950 60  0000 C CNN
-F 3 "" H 3400 2950 60  0000 C CNN
-	1    3400 2950
+P 3400 3200
+F 0 "#PWR051" H 3400 3200 40  0001 C CNN
+F 1 "DGND" H 3400 3130 40  0000 C CNN
+F 2 "" H 3400 3200 60  0000 C CNN
+F 3 "" H 3400 3200 60  0000 C CNN
+	1    3400 3200
 	-1   0    0    -1
 $EndComp
@@
 $EndComp
 $Comp
-L +9V #PWR38
+L +9V #PWR052
 U 1 1 5483196D
 P 3400 2200
-F 0 "#PWR38" H 3400 2170 20  0001 C CNN
+F 0 "#PWR052" H 3400 2170 20  0001 C CNN
 F 1 "+9V" H 3400 2310 30  0000 C CNN
 F 2 "" H 3400 2200 60  0000 C CNN
@@
 $EndComp
 $Comp
-L VCC #PWR37
+L VCC #PWR053
 U 1 1 54831973
 P 1900 2250
-F 0 "#PWR37" H 1900 2350 30  0001 C CNN
+F 0 "#PWR053" H 1900 2350 30  0001 C CNN
 F 1 "VCC" H 1900 2350 30  0000 C CNN
 F 2 "" H 1900 2250 60  0000 C CNN
@@
 $EndComp
 $Comp
-L DGND #PWR40
+L DGND #PWR054
 U 1 1 5483198E
 P 3650 2950
-F 0 "#PWR40" H 3650 2950 40  0001 C CNN
+F 0 "#PWR054" H 3650 2950 40  0001 C CNN
 F 1 "DGND" H 3650 2880 40  0000 C CNN
 F 2 "" H 3650 2950 60  0000 C CNN
@@
 $EndComp
 $Comp
-L PWR_FLAG #FLG3
+L PWR_FLAG #FLG055
 U 1 1 54831994
 P 3650 2250
-F 0 "#FLG3" H 3650 2345 30  0001 C CNN
+F 0 "#FLG055" H 3650 2345 30  0001 C CNN
 F 1 "PWR_FLAG" H 3650 2430 30  0000 C CNN
 F 2 "" H 3650 2250 60  0000 C CNN
@@
 $EndComp
 $Comp
-L +5V #PWR42
+L +5V #PWR056
 U 1 1 5483199A
 P 4550 1700
-F 0 "#PWR42" H 4550 1790 20  0001 C CNN
+F 0 "#PWR056" H 4550 1790 20  0001 C CNN
 F 1 "+5V" H 4550 1790 30  0000 C CNN
 F 2 "" H 4550 1700 60  0000 C CNN
@@
 $EndComp
 $Comp
-L DGND #PWR41
+L DGND #PWR057
 U 1 1 548319A0
 P 4050 2800
-F 0 "#PWR41" H 4050 2800 40  0001 C CNN
+F 0 "#PWR057" H 4050 2800 40  0001 C CNN
 F 1 "DGND" H 4050 2730 40  0000 C CNN
 F 2 "" H 4050 2800 60  0000 C CNN
@@
 	4800 2850 4800 2950
 Wire Wire Line
-	3400 2850 3400 2950
+	3400 2850 3400 3200
 Wire Wire Line
 	3100 2350 3700 2350
@@
 	1900 2250 1900 2350
 Wire Wire Line
-	1900 2350 1950 2350
+	1650 2350 1950 2350
 Wire Wire Line
 	4050 2700 4050 2800
@@
 Connection ~ 3400 2900
 $Comp
-L PWR_FLAG #FLG4
+L PWR_FLAG #FLG058
 U 1 1 548319DC
 P 4450 1750
-F 0 "#FLG4" H 4450 1845 30  0001 C CNN
+F 0 "#FLG058" H 4450 1845 30  0001 C CNN
 F 1 "PWR_FLAG" H 4450 1930 30  0000 C CNN
 F 2 "" H 4450 1750 60  0000 C CNN
@@
 	3200 2050 3200 2350
 Connection ~ 3200 2350
+$Comp
+L PWR_FLAG #FLG059
+U 1 1 54879B32
+P 1650 2300
+F 0 "#FLG059" H 1650 2395 30  0001 C CNN
+F 1 "PWR_FLAG" H 1650 2480 30  0000 C CNN
+F 2 "" H 1650 2300 60  0000 C CNN
+F 3 "" H 1650 2300 60  0000 C CNN
+	1    1650 2300
+	1    0    0    -1
+$EndComp
+Wire Wire Line
+	1650 2300 1650 2350
+Connection ~ 1900 2350
+$Comp
+L PWR_FLAG #FLG060
+U 1 1 54879C64
+P 3300 3100
+F 0 "#FLG060" H 3300 3195 30  0001 C CNN
+F 1 "PWR_FLAG" H 3300 3280 30  0000 C CNN
+F 2 "" H 3300 3100 60  0000 C CNN
+F 3 "" H 3300 3100 60  0000 C CNN
+	1    3300 3100
+	0    -1   1    0
+$EndComp
+Wire Wire Line
+	3300 3100 3400 3100
+Connection ~ 3400 3100
 $EndSCHEMATC

Commit message: Fixing schematics references numbering. Also regenerated .net and .cmp files.
Parts:
- renumbered C8 to C1, C9 to C2, C10 to C3, C11 to C4, C12 to C6, C13 to C7, D4 to D1, R41 to R26, R40 to R38, TP3 to TP1, TP1 to TP3, U3 to U2, U4 to U3
Changed lines of the file:
@@
 $EndDescr
 $Comp
-L NCP1117DT33G U4
+L NCP1117DT33G U3
 U 1 1 548318F8
 P 5200 2400
-F 0 "U4" H 5200 2600 60  0000 C CNN
+F 0 "U3" H 5200 2600 60  0000 C CNN
 F 1 "NCP1117DT33G" H 5300 2700 60  0000 C CNN
 F 2 "MOD_Footprints_Lib:DPAK(369C)" H 5200 2450 60  0001 C CNN
@@
 $EndComp
 $Comp
-L CP1 C12
+L CP1 C6
 U 1 1 548318FF
 P 5600 2650
-F 0 "C12" V 5700 2750 50  0000 L CNN
+F 0 "C6" V 5700 2750 50  0000 L CNN
 F 1 "100uF" V 5450 2550 50  0000 L CNN
 F 2 "MOD_Footprints_Lib:CAP_RAD_5MM" H 5600 2650 60  0001 C CNN
@@
 $EndComp
 $Comp
-L CP1 C10
+L CP1 C3
 U 1 1 54831912
 P 4550 2650
-F 0 "C10" V 4650 2750 50  0000 L CNN
+F 0 "C3" V 4650 2750 50  0000 L CNN
 F 1 "100uF" V 4400 2550 50  0000 L CNN
 F 2 "MOD_Footprints_Lib:CAP_RAD_5MM" H 4550 2650 60  0001 C CNN
@@
 $EndComp
 $Comp
-L C C13
+L C C7
 U 1 1 54831925
 P 5850 2650
-F 0 "C13" V 5800 2750 40  0000 L CNN
+F 0 "C7" V 5800 2750 40  0000 L CNN
 F 1 "100nF_X7R" V 6000 2500 40  0000 L CNN
 F 2 "MOD_Footprints_Lib:SM0603" H 5888 2500 30  0001 C CNN
@@
 $EndComp
 $Comp
-L R R41
+L R R26
 U 1 1 54831932
 P 6200 2350
-F 0 "R41" V 6280 2350 40  0000 C CNN
+F 0 "R26" V 6280 2350 40  0000 C CNN
 F 1 "0R" V 6207 2351 40  0000 C CNN
 F 2 "MOD_Footprints_Lib:SM0805" V 6130 2350 30  0001 C CNN
@@
 $EndComp
 $Comp
-L C C11
+L C C4
 U 1 1 5483193F
 P 4800 2650
-F 0 "C11" V 4750 2750 40  0000 L CNN
+F 0 "C4" V 4750 2750 40  0000 L CNN
 F 1 "100nF_X7R" V 4950 2500 40  0000 L CNN
 F 2 "MOD_Footprints_Lib:SM0603" H 4838 2500 30  0001 C CNN
@@
 $EndComp
 $Comp
-L CONN_1 TP3
+L CONN_1 TP1
 U 1 1 5483194C
 P 5850 2100
-F 0 "TP3" V 5950 2050 40  0000 L CNN
+F 0 "TP1" V 5950 2050 40  0000 L CNN
 F 1 "CONN_1" H 5850 2155 30  0001 C CNN
 F 2 "MOD_Footprints_Lib:SIL-1" H 5850 2100 60  0001 C CNN
@@
 $EndComp
 $Comp
-L LINEAR_REGULATOR_DPAK_3P U3
+L LINEAR_REGULATOR_DPAK_3P U2
 U 1 1 54831959
 P 4050 2400
-F 0 "U3" H 4050 2600 60  0000 C CNN
+F 0 "U2" H 4050 2600 60  0000 C CNN
 F 1 "MC7805" H 4050 2700 60  0000 C CNN
 F 2 "MOD_Footprints_Lib:DPAK(369C)" H 4050 2450 60  0001 C CNN
@@
 $EndComp
 $Comp
-L CP1 C8
+L CP1 C1
 U 1 1 54831966
 P 3400 2650
-F 0 "C8" V 3500 2750 50  0000 L CNN
+F 0 "C1" V 3500 2750 50  0000 L CNN
 F 1 "100uF" V 3250 2550 50  0000 L CNN
 F 2 "MOD_Footprints_Lib:CAP_RAD_5MM" H 3400 2650 60  0001 C CNN
@@
 $EndComp
 $Comp
-L DIODE D4
+L DIODE D1
 U 1 1 54831979
 P 2150 2350
-F 0 "D4" H 2150 2450 40  0000 C CNN
+F 0 "D1" H 2150 2450 40  0000 C CNN
 F 1 "CGRA4007-G" H 2150 2250 40  0000 C CNN
 F 2 "MOD_Footprints_Lib:DO-214AC(SMA)" H 2150 2350 60  0001 C CNN
@@
 $EndComp
 $Comp
-L C C9
+L C C2
 U 1 1 54831987
 P 3650 2650
-F 0 "C9" V 3600 2750 40  0000 L CNN
+F 0 "C2" V 3600 2750 40  0000 L CNN
 F 1 "100nF_X7R" V 3800 2500 40  0000 L CNN
 F 2 "MOD_Footprints_Lib:SM0603" H 3688 2500 30  0001 C CNN
@@
 Connection ~ 4800 2350
 $Comp
-L R R40
+L R R38
 U 1 1 548319C3
 P 4550 2050
-F 0 "R40" V 4630 2050 40  0000 C CNN
+F 0 "R38" V 4630 2050 40  0000 C CNN
 F 1 "0R" V 4557 2051 40  0000 C CNN
 F 2 "MOD_Footprints_Lib:SM0805" V 4480 2050 30  0001 C CNN
@@
 $EndComp
 $Comp
-L CONN_1 TP1
+L CONN_1 TP3
 U 1 1 548319D3
 P 3200 2900
-F 0 "TP1" V 3300 2850 40  0000 L CNN
+F 0 "TP3" V 3300 2850 40  0000 L CNN
 F 1 "CONN_1" H 3200 2955 30  0001 C CNN
 F 2 "MOD_Footprints_Lib:SIL-1" H 3200 2900 60  0001 C CNN
