File: hw-design/control-chain.sch (KiCad schematic (older format))
At the start: 25 parts, among them J1 RJ45_CHAIN_MAIN, J2 RJ45_CHAIN_EXTENSION, Q1 MMBT3904, Q2 MMBT3906, U4 MAX13450E

Commit message: updating MAX13450E symbol
Parts:
- U4: footprint MOD_Footprints_Lib:TSSOP14 -> TSSOP-14EP
Connections:
- wire segments 102 -> 105
Other:
- moved on the sheet: C18, D2, D3, R29, R30, R31, R44

Commit message: fixing name of the standard RS-485 -> RS-422
Connections:
- net RS485_RX+ renamed RS422_RX+
- net RS485_RX- renamed RS422_RX-
- net RS485_TX+ renamed RS422_TX+
- net RS485_TX- renamed RS422_TX-
Changed lines of the file:
@@
 LED5
 Text GLabel 7000 1850 0    60   Input ~ 0
-RS485_RX+
+RS422_RX+
 Text GLabel 7000 2050 0    60   Input ~ 0
-RS485_RX-
+RS422_RX-
 $Comp
 L DGND #PWR04
@@
 $EndComp
 Text GLabel 7100 2750 0    60   Output ~ 0
-RS485_TX+
+RS422_TX+
 Text GLabel 7100 2950 0    60   Output ~ 0
-RS485_TX-
+RS422_TX-
 $Comp
 L DGND #PWR011
@@
 $EndComp
 Text GLabel 4400 2200 2    60   Output ~ 0
-RS485_TX+
+RS422_TX+
 Text GLabel 4400 2350 2    60   Output ~ 0
-RS485_TX-
+RS422_TX-
 Text GLabel 4400 2550 2    60   Input ~ 0
-RS485_RX+
+RS422_RX+
 Text GLabel 4400 2700 2    60   Input ~ 0
-RS485_RX-
+RS422_RX-
 $Comp
 L VCC #PWR013

Commit message: using RJ45 leds to indicate cable connection status instead of power status
Parts:
- added C19: 100uF, MOD_Footprints_Lib:CAP_RAD_5MM, symbol CP1
- added C20: 100nF_X7R, MOD_Footprints_Lib:SM0603, symbol C
- added Q4, Q5, Q6: MMBT3904, MOD_Footprints_Lib:SOT23, symbol NPN
- added R48, R49, R52: 100k, MOD_Footprints_Lib:SM0603, symbol R
- added R50, R51, R54: 10k, MOD_Footprints_Lib:SM0603, symbol R
- added R53: 1k, MOD_Footprints_Lib:SM0603, symbol R
- R1: value 1k -> 10k
- R12: renamed from R13; value 10k -> 100k
- R13: renamed from R12; value 100k -> 10k
- R27: value 1k -> 100k
- R3, R4, R5, R6: value 470R -> 1K2
Connections:
- net +3.3V: now also R13.1, Q4.3 (C); no longer R12.1, R3.1, R4.1, R5.1, R6.1
- net DGND: now also R27.2, C19.2, C20.2, R49.2, R52.2; no longer J2.11 (LED2A)
- net TX_CHAIN_EN: now also R51.1; no longer R31.1, U4.1 (DE)
- net VCC: now also J2.12 (LED2C), Q6.3 (C), R48.1; no longer J1.5
- net at J1.12 (LED2C): now also R6.1; no longer R6.2
- net at J1.9 (LED1A), Q1.3 (C): no longer J2.9 (LED1A)
- net at J2.10 (LED1C): now also Q6.2 (E); no longer R3.2
- net GND_FB: now reaches R4.2
- net GND_FB: now also C5.1, C8.1, J2.7, R12.2, R3.2, R48.2; no longer J2.12 (LED2C)
- net at Q2.1 (B): now also R53.1; no longer R27.2
- net LED5 renamed LED_STATUS
- net LED_STATUS: now also R54.1
- new net: J2.11 (LED2A), R4.1
- new net: J2.9 (LED1A), R3.1
- new net: Q5.2 (E), R31.1, U4.1 (DE)
- new net: R12.1, R13.2, R53.2
- new net: Q4.1 (B), R27.1, R50.2
- new net: Q4.2 (E), Q5.3 (C)
- new net: Q5.1 (B), R49.1, R51.2
- new net: Q6.1 (B), R54.2
- new net VCC_FB: C19.1, C20.1, J1.5, R5.1, R50.1, R52.1, R6.2
Other:
- moved on the sheet: C18, C5, C8, D2, D3, J1, J2, Q1, Q2, R1, R11, R12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

Commit message: wip: breaking pcbs apart
Parts:
- added CN1, CN2: CONN_PANNEL_2X2, MOD_Footprints_Lib:CONN_PANNEL, symbol CONN_PANNEL_2X2
- added P3, P4: CONN_8X2, MOD_Footprints_Lib:pin_array_8x2, symbol CONN_8X2
- U4: footprint TSSOP-14EP -> MOD_Footprints_Lib:TSSOP14
Connections:
- net DGND: now also P4.15; no longer J1.11 (LED2A)
- net GND_FB: now also P4.11; no longer J2.7
- net RS422_RX+: now also P4.5; no longer J1.3, J2.1
- net RS422_RX-: now also P4.7; no longer J1.6, J2.2
- net RS422_TX+: now also P4.1; no longer J1.1, J2.3
- net RS422_TX-: now also P4.3; no longer J1.2, J2.6
- net VCC: now also P4.2; no longer J1.4, J2.12 (LED2C), J2.4, J2.5
- net VCC_FB: now also P4.9; no longer J1.5
- net MAIN_LED1C: now reaches R5.2
- net MAIN_LED1C: now also P4.6; no longer J1.10 (LED1C)
- net MAIN_LED2C: now reaches R6.1
- net MAIN_LED2C: now also P4.4; no longer J1.12 (LED2C)
- net P3_MAIN_LOAD: now reaches J1.7, J1.8
- net P3_MAIN_LOAD: now also P3.13; no longer R2.1
- net MAIN_LED1A: now reaches Q1.3 (C)
- net MAIN_LED1A: now also P4.8; no longer J1.9 (LED1A)
- net EXT_LED1C: now reaches Q6.2 (E)
- net EXT_LED1C: now also P4.12; no longer J2.10 (LED1C)
- net EXT_LED2A: now reaches R4.1
- net EXT_LED2A: now also P4.10; no longer J2.11 (LED2A)
- net EXT_LOAD: now reaches R11.1
- net EXT_LOAD: now also P4.16; no longer J2.8
- net EXT_LED1A: now reaches R3.1
- net EXT_LED1A: now also P4.14; no longer J2.9 (LED1A)
- new net MAIN_LOAD: P4.13, R2.1
- new net P3_DGND: CN1.1, CN2.1, J1.11 (LED2A), P3.15
- new net P3_EXT_LED1A: J2.9 (LED1A), P3.14
- new net P3_EXT_LED1C: J2.10 (LED1C), P3.12
- new net P3_EXT_LED2A: J2.11 (LED2A), P3.10
- new net P3_EXT_LOAD: J2.8, P3.16
- new net P3_GND_FB: J2.7, P3.11
- new net P3_MAIN_LED1A: J1.9 (LED1A), P3.8
- new net P3_MAIN_LED1C: J1.10 (LED1C), P3.6
- new net P3_MAIN_LED2C: J1.12 (LED2C), P3.4
- new net P3_RS422_RX+: J1.3, J2.1, P3.5
- new net P3_RS422_RX-: J1.6, J2.2, P3.7
- new net P3_RS422_TX+: J1.1, J2.3, P3.1
- new net P3_RS422_TX-: J1.2, J2.6, P3.3
- new net P3_VCC: J1.4, J2.12 (LED2C), J2.4, J2.5, P3.2
- new net P3_VCC_FB: J1.5, P3.9
Other:
- moved on the sheet: C19, C20, C5, C8, J1, J2, Q1, Q2, Q4, Q6, R1, R11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
