File: hw-design/cpu.sch (KiCad schematic (older format))
At the start: 21 parts, among them CN1 CONN_PANNEL_2X2, CN2 CONN_PANNEL_2X2, P1 HEADER_5X2, P2 HEADER_5X2, U1 LPC111X_LQFP48, X1 10MHz

Commit message: using RJ45 leds to indicate cable connection status instead of power status
Connections:
- net LED5 renamed LED_STATUS
Changed lines of the file:
@@
 $EndComp
 $Comp
-L DGND #PWR023
+L DGND #PWR030
 U 1 1 54834712
 P 5550 4000
-F 0 "#PWR023" H 5550 4000 40  0001 C CNN
+F 0 "#PWR030" H 5550 4000 40  0001 C CNN
 F 1 "DGND" H 5550 3930 40  0000 C CNN
 F 2 "" H 5550 4000 60  0000 C CNN
@@
 $EndComp
 $Comp
-L DGND #PWR024
+L DGND #PWR031
 U 1 1 5483471F
 P 6550 3600
-F 0 "#PWR024" H 6550 3600 40  0001 C CNN
+F 0 "#PWR031" H 6550 3600 40  0001 C CNN
 F 1 "DGND" H 6550 3530 40  0000 C CNN
 F 2 "" H 6550 3600 60  0000 C CNN
@@
 $EndComp
 $Comp
-L DGND #PWR025
+L DGND #PWR032
 U 1 1 54834725
 P 6550 3400
-F 0 "#PWR025" H 6550 3400 40  0001 C CNN
+F 0 "#PWR032" H 6550 3400 40  0001 C CNN
 F 1 "DGND" H 6550 3330 40  0000 C CNN
 F 2 "" H 6550 3400 60  0000 C CNN
@@
 $EndComp
 $Comp
-L +3.3V #PWR026
+L +3.3V #PWR033
 U 1 1 5483472B
 P 5950 3350
-F 0 "#PWR026" H 5950 3310 30  0001 C CNN
+F 0 "#PWR033" H 5950 3310 30  0001 C CNN
 F 1 "+3.3V" H 5950 3460 30  0000 C CNN
 F 2 "" H 5950 3350 60  0000 C CNN
@@
 $EndComp
 $Comp
-L DGND #PWR027
+L DGND #PWR034
 U 1 1 5483473F
 P 6350 4900
-F 0 "#PWR027" H 6350 4900 40  0001 C CNN
+F 0 "#PWR034" H 6350 4900 40  0001 C CNN
 F 1 "DGND" H 6350 4830 40  0000 C CNN
 F 2 "" H 6350 4900 60  0000 C CNN
@@
 $EndComp
 $Comp
-L DGND #PWR028
+L DGND #PWR035
 U 1 1 54834745
 P 6350 4100
-F 0 "#PWR028" H 6350 4100 40  0001 C CNN
+F 0 "#PWR035" H 6350 4100 40  0001 C CNN
 F 1 "DGND" H 6350 4030 40  0000 C CNN
 F 2 "" H 6350 4100 60  0000 C CNN
@@
 $EndComp
 $Comp
-L DGND #PWR029
+L DGND #PWR036
 U 1 1 54834760
 P 2150 1400
-F 0 "#PWR029" H 2150 1400 40  0001 C CNN
+F 0 "#PWR036" H 2150 1400 40  0001 C CNN
 F 1 "DGND" H 2150 1330 40  0000 C CNN
 F 2 "" H 2150 1400 60  0000 C CNN
@@
 $EndComp
 $Comp
-L +3.3V #PWR030
+L +3.3V #PWR037
 U 1 1 54834766
 P 2750 800
-F 0 "#PWR030" H 2750 760 30  0001 C CNN
+F 0 "#PWR037" H 2750 760 30  0001 C CNN
 F 1 "+3.3V" H 2750 910 30  0000 C CNN
 F 2 "" H 2750 800 60  0000 C CNN
@@
 SWDCLK
 $Comp
-L DGND #PWR031
+L DGND #PWR038
 U 1 1 54834777
 P 4250 6450
-F 0 "#PWR031" H 4250 6450 40  0001 C CNN
+F 0 "#PWR038" H 4250 6450 40  0001 C CNN
 F 1 "DGND" H 4250 6380 40  0000 C CNN
 F 2 "" H 4250 6450 60  0000 C CNN
@@
 FOOT_4
 Text GLabel 5650 3100 2    50   Output ~ 0
-LED5
-Text GLabel 1250 6500 0    50   Output ~ 0
-RX_CHAIN
-Text GLabel 1250 6600 0    50   Input ~ 0
-TX_CHAIN
-$Comp
-L +5V #PWR032
+LED_STATUS
+$Comp
+L +5V #PWR039
 U 1 1 5483479B
 P 1100 6400
-F 0 "#PWR032" H 1100 6490 20  0001 C CNN
+F 0 "#PWR039" H 1100 6490 20  0001 C CNN
 F 1 "+5V" H 1100 6490 30  0000 C CNN
 F 2 "" H 1100 6400 60  0000 C CNN
@@
 $EndComp
 $Comp
-L DGND #PWR033
+L DGND #PWR040
 U 1 1 548347A1
 P 1200 6300
-F 0 "#PWR033" H 1200 6300 40  0001 C CNN
+F 0 "#PWR040" H 1200 6300 40  0001 C CNN
 F 1 "DGND" H 1200 6225 40  0000 C CNN
 F 2 "" H 1200 6300 60  0000 C CNN
@@
 $EndComp
 $Comp
-L +3.3V #PWR034
+L +3.3V #PWR041
 U 1 1 548347AE
 P 1800 1650
-F 0 "#PWR034" H 1800 1610 30  0001 C CNN
+F 0 "#PWR041" H 1800 1610 30  0001 C CNN
 F 1 "+3.3V" H 1800 1760 30  0000 C CNN
 F 2 "" H 1800 1650 60  0000 C CNN
@@
 $EndComp
 $Comp
-L +3.3V #PWR035
+L +3.3V #PWR042
 U 1 1 54834827
 P 3750 5950
-F 0 "#PWR035" H 3750 5910 30  0001 C CNN
+F 0 "#PWR042" H 3750 5910 30  0001 C CNN
 F 1 "+3.3V" H 3750 6060 30  0000 C CNN
 F 2 "" H 3750 5950 60  0000 C CNN
@@
 	0    -1   -1   0
 $EndComp
-Text GLabel 1250 6700 0    50   Input ~ 0
-TX_CHAIN_EN
 NoConn ~ 2850 2150
 NoConn ~ 2850 1750
@@
 NoConn ~ 5450 3300
 $Comp
-L DGND #PWR036
+L DGND #PWR043
 U 1 1 5483484A
 P 7350 5950
-F 0 "#PWR036" H 7350 5950 40  0001 C CNN
+F 0 "#PWR043" H 7350 5950 40  0001 C CNN
 F 1 "DGND" H 7350 5880 40  0000 C CNN
 F 2 "" H 7350 5950 60  0000 C CNN
@@
 $EndComp
 $Comp
-L DGND #PWR037
+L DGND #PWR044
 U 1 1 54834850
 P 8350 5950
-F 0 "#PWR037" H 8350 5950 40  0001 C CNN
+F 0 "#PWR044" H 8350 5950 40  0001 C CNN
 F 1 "DGND" H 8350 5880 40  0000 C CNN
 F 2 "" H 8350 5950 60  0000 C CNN
@@
 $EndComp
 $Comp
-L +5V #PWR038
+L +5V #PWR045
 U 1 1 548788DF
 P 2800 6400
-F 0 "#PWR038" H 2800 6490 20  0001 C CNN
+F 0 "#PWR045" H 2800 6490 20  0001 C CNN
 F 1 "+5V" H 2800 6490 30  0000 C CNN
 F 2 "" H 2800 6400 60  0000 C CNN
@@
 $EndComp
 $Comp
-L DGND #PWR039
+L DGND #PWR046
 U 1 1 548788E5
 P 2700 6300
-F 0 "#PWR039" H 2700 6300 40  0001 C CNN
+F 0 "#PWR046" H 2700 6300 40  0001 C CNN
 F 1 "DGND" H 2700 6225 40  0000 C CNN
 F 2 "" H 2700 6300 60  0000 C CNN
@@
 Connection ~ 1400 1950
 $Comp
-L +3.3V #PWR040
+L +3.3V #PWR047
 U 1 1 54908FE8
 P 1400 1100
-F 0 "#PWR040" H 1400 1060 30  0001 C CNN
+F 0 "#PWR047" H 1400 1060 30  0001 C CNN
 F 1 "+3.3V" H 1400 1210 30  0000 C CNN
 F 2 "" H 1400 1100 60  0000 C CNN
@@
 $EndComp
 Connection ~ 1400 1250
+Text GLabel 1250 6500 0    50   Input ~ 0
+RX_CHAIN
+Text GLabel 1250 6600 0    50   Output ~ 0
+TX_CHAIN
+Text GLabel 1250 6700 0    50   Output ~ 0
+TX_CHAIN_EN
 $EndSCHEMATC

Commit message: wip: breaking pcbs apart
Parts:
- removed CN1, CN2: CONN_PANNEL_2X2, MOD_Footprints_Lib:CONN_PANNEL, symbol CONN_PANNEL_2X2
Changed lines of the file:
@@
 EESchema Schematic File Version 2
 LIBS:footswitch
+LIBS:conn
 LIBS:footswitch-cache
 EELAYER 25 0
@@
 $EndComp
 $Comp
-L DGND #PWR030
+L DGND #PWR028
 U 1 1 54834712
 P 5550 4000
-F 0 "#PWR030" H 5550 4000 40  0001 C CNN
+F 0 "#PWR028" H 5550 4000 40  0001 C CNN
 F 1 "DGND" H 5550 3930 40  0000 C CNN
 F 2 "" H 5550 4000 60  0000 C CNN
@@
 $EndComp
 $Comp
-L DGND #PWR031
+L DGND #PWR029
 U 1 1 5483471F
 P 6550 3600
-F 0 "#PWR031" H 6550 3600 40  0001 C CNN
+F 0 "#PWR029" H 6550 3600 40  0001 C CNN
 F 1 "DGND" H 6550 3530 40  0000 C CNN
 F 2 "" H 6550 3600 60  0000 C CNN
@@
 $EndComp
 $Comp
-L DGND #PWR032
+L DGND #PWR030
 U 1 1 54834725
 P 6550 3400
-F 0 "#PWR032" H 6550 3400 40  0001 C CNN
+F 0 "#PWR030" H 6550 3400 40  0001 C CNN
 F 1 "DGND" H 6550 3330 40  0000 C CNN
 F 2 "" H 6550 3400 60  0000 C CNN
@@
 $EndComp
 $Comp
-L +3.3V #PWR033
+L +3.3V #PWR031
 U 1 1 5483472B
 P 5950 3350
-F 0 "#PWR033" H 5950 3310 30  0001 C CNN
+F 0 "#PWR031" H 5950 3310 30  0001 C CNN
 F 1 "+3.3V" H 5950 3460 30  0000 C CNN
 F 2 "" H 5950 3350 60  0000 C CNN
@@
 $EndComp
 $Comp
-L DGND #PWR034
+L DGND #PWR032
 U 1 1 5483473F
 P 6350 4900
-F 0 "#PWR034" H 6350 4900 40  0001 C CNN
+F 0 "#PWR032" H 6350 4900 40  0001 C CNN
 F 1 "DGND" H 6350 4830 40  0000 C CNN
 F 2 "" H 6350 4900 60  0000 C CNN
@@
 $EndComp
 $Comp
-L DGND #PWR035
+L DGND #PWR033
 U 1 1 54834745
 P 6350 4100
-F 0 "#PWR035" H 6350 4100 40  0001 C CNN
+F 0 "#PWR033" H 6350 4100 40  0001 C CNN
 F 1 "DGND" H 6350 4030 40  0000 C CNN
 F 2 "" H 6350 4100 60  0000 C CNN
@@
 $EndComp
 $Comp
-L DGND #PWR036
+L DGND #PWR034
 U 1 1 54834760
 P 2150 1400
-F 0 "#PWR036" H 2150 1400 40  0001 C CNN
+F 0 "#PWR034" H 2150 1400 40  0001 C CNN
 F 1 "DGND" H 2150 1330 40  0000 C CNN
 F 2 "" H 2150 1400 60  0000 C CNN
@@
 $EndComp
 $Comp
-L +3.3V #PWR037
+L +3.3V #PWR035
 U 1 1 54834766
 P 2750 800
-F 0 "#PWR037" H 2750 760 30  0001 C CNN
+F 0 "#PWR035" H 2750 760 30  0001 C CNN
 F 1 "+3.3V" H 2750 910 30  0000 C CNN
 F 2 "" H 2750 800 60  0000 C CNN
@@
 SWDCLK
 $Comp
-L DGND #PWR038
+L DGND #PWR036
 U 1 1 54834777
 P 4250 6450
-F 0 "#PWR038" H 4250 6450 40  0001 C CNN
+F 0 "#PWR036" H 4250 6450 40  0001 C CNN
 F 1 "DGND" H 4250 6380 40  0000 C CNN
 F 2 "" H 4250 6450 60  0000 C CNN
@@
 LED_STATUS
 $Comp
-L +5V #PWR039
+L +5V #PWR037
 U 1 1 5483479B
 P 1100 6400
-F 0 "#PWR039" H 1100 6490 20  0001 C CNN
+F 0 "#PWR037" H 1100 6490 20  0001 C CNN
 F 1 "+5V" H 1100 6490 30  0000 C CNN
 F 2 "" H 1100 6400 60  0000 C CNN
@@
 $EndComp
 $Comp
-L DGND #PWR040
+L DGND #PWR038
 U 1 1 548347A1
 P 1200 6300
-F 0 "#PWR040" H 1200 6300 40  0001 C CNN
+F 0 "#PWR038" H 1200 6300 40  0001 C CNN
 F 1 "DGND" H 1200 6225 40  0000 C CNN
 F 2 "" H 1200 6300 60  0000 C CNN
@@
 $EndComp
 $Comp
-L +3.3V #PWR041
+L +3.3V #PWR039
 U 1 1 548347AE
 P 1800 1650
-F 0 "#PWR041" H 1800 1610 30  0001 C CNN
+F 0 "#PWR039" H 1800 1610 30  0001 C CNN
 F 1 "+3.3V" H 1800 1760 30  0000 C CNN
 F 2 "" H 1800 1650 60  0000 C CNN
@@
 UC_LCD_DIR
 $Comp
-L CONN_PANNEL_2X2 CN1
-U 1 1 54834801
-P 7850 5350
-F 0 "CN1" H 7850 5500 50  0000 C CNN
-F 1 "CONN_PANNEL_2X2" H 7860 5220 40  0000 C CNN
-F 2 "MOD_Footprints_Lib:CONN_PANNEL" H 7850 5350 60  0001 C CNN
-F 3 "" H 7850 5350 60  0000 C CNN
-	1    7850 5350
-	1    0    0    -1
-$EndComp
-$Comp
-L CONN_PANNEL_2X2 CN2
-U 1 1 54834808
-P 7850 5800
-F 0 "CN2" H 7850 5950 50  0000 C CNN
-F 1 "CONN_PANNEL_2X2" H 7860 5670 40  0000 C CNN
-F 2 "MOD_Footprints_Lib:CONN_PANNEL" H 7850 5800 60  0001 C CNN
-F 3 "" H 7850 5800 60  0000 C CNN
-	1    7850 5800
-	1    0    0    -1
-$EndComp
-$Comp
 L R R41
 U 1 1 5483480F
@@
 $EndComp
 $Comp
-L +3.3V #PWR042
+L +3.3V #PWR040
 U 1 1 54834827
 P 3750 5950
-F 0 "#PWR042" H 3750 5910 30  0001 C CNN
+F 0 "#PWR040" H 3750 5910 30  0001 C CNN
 F 1 "+3.3V" H 3750 6060 30  0000 C CNN
 F 2 "" H 3750 5950 60  0000 C CNN
@@
 NoConn ~ 5450 3200
 NoConn ~ 5450 3300
-$Comp
-L DGND #PWR043
-U 1 1 5483484A
-P 7350 5950
-F 0 "#PWR043" H 7350 5950 40  0001 C CNN
-F 1 "DGND" H 7350 5880 40  0000 C CNN
-F 2 "" H 7350 5950 60  0000 C CNN
-F 3 "" H 7350 5950 60  0000 C CNN
-	1    7350 5950
-	1    0    0    -1
-$EndComp
-$Comp
-L DGND #PWR044
-U 1 1 54834850
-P 8350 5950
-F 0 "#PWR044" H 8350 5950 40  0001 C CNN
-F 1 "DGND" H 8350 5880 40  0000 C CNN
-F 2 "" H 8350 5950 60  0000 C CNN
-F 3 "" H 8350 5950 60  0000 C CNN
-	1    8350 5950
-	1    0    0    -1
-$EndComp
 $Comp
 L CONN_5X2 P1
@@
 $EndComp
 $Comp
-L +5V #PWR045
+L +5V #PWR041
 U 1 1 548788DF
 P 2800 6400
-F 0 "#PWR045" H 2800 6490 20  0001 C CNN
+F 0 "#PWR041" H 2800 6490 20  0001 C CNN
 F 1 "+5V" H 2800 6490 30  0000 C CNN
 F 2 "" H 2800 6400 60  0000 C CNN
@@
 $EndComp
 $Comp
-L DGND #PWR046
+L DGND #PWR042
 U 1 1 548788E5
 P 2700 6300
-F 0 "#PWR046" H 2700 6300 40  0001 C CNN
+F 0 "#PWR042" H 2700 6300 40  0001 C CNN
 F 1 "DGND" H 2700 6225 40  0000 C CNN
 F 2 "" H 2700 6300 60  0000 C CNN
@@
 	2850 2250 2650 2250
 Wire Wire Line
-	8250 5300 8350 5300
-Wire Wire Line
-	8350 5300 8350 5950
-Wire Wire Line
-	8250 5850 8350 5850
-Connection ~ 8350 5850
-Wire Wire Line
-	8250 5750 8350 5750
-Connection ~ 8350 5750
-Wire Wire Line
-	8250 5400 8350 5400
-Connection ~ 8350 5400
-Wire Wire Line
-	7450 5300 7350 5300
-Wire Wire Line
-	7350 5300 7350 5950
-Wire Wire Line
-	7450 5850 7350 5850
-Connection ~ 7350 5850
-Wire Wire Line
-	7450 5750 7350 5750
-Connection ~ 7350 5750
-Wire Wire Line
-	7450 5400 7350 5400
-Connection ~ 7350 5400
-Wire Wire Line
 	1250 6500 1550 6500
 Wire Wire Line
@@
 Connection ~ 1400 1950
 $Comp
-L +3.3V #PWR047
+L +3.3V #PWR043
 U 1 1 54908FE8
 P 1400 1100
-F 0 "#PWR047" H 1400 1060 30  0001 C CNN
+F 0 "#PWR043" H 1400 1060 30  0001 C CNN
 F 1 "+3.3V" H 1400 1210 30  0000 C CNN
 F 2 "" H 1400 1100 60  0000 C CNN
