File: hw-design/footswitch.kicad_pcb (KiCad board)
At the start: 2 copper layers, 248.9 x 74.2 mm, 99 parts, among them CN1 CONN_PANNEL_2X2, CN2 CONN_PANNEL_2X2, J1 RJ45_CHAIN_MAIN, J2 RJ45_CHAIN_EXTENSION, P1 HEADER_5X2, P2 HEADER_5X2, Q1 MMBT3904, Q2 MMBT3906, Q3 MMBT3904, U1 LPC111X_LQFP48, U2 MC7805, U3 NCP1117DT33G, U4 MAX13450E, U5 74HC245, U6 74HC245, X1 10MHz

Commit message: fixing name of the standard RS-485 -> RS-422
Connections:
- net RS485_RX+ renamed RS422_RX+
- net RS485_RX- renamed RS422_RX-
- net RS485_TX+ renamed RS422_TX+
- net RS485_TX- renamed RS422_TX-

Commit message: wip: breaking pcbs apart
Parts:
- added P3: CONN_8X2, MOD_Footprints_Lib:pin_array_8x2, F.Cu at (223.5, 187.5)
- added P4: CONN_8X2, MOD_Footprints_Lib:pin_array_8x2, F.Cu at (296.2, 211.3)
- R1: value 1k -> 10k
- R27: value 1k -> 100k
- R3, R4, R5, R6: value 470R -> 1K2
- moved CN2 184.6 mm to (196.1, 176.8), turned to 180 degrees
- moved J1 159.3 mm to (212.9, 176.3), turned to 180 degrees
- moved J2 141.7 mm to (234.2, 176.3), turned to 180 degrees
- moved CN1 120.4 mm to (251.0, 176.8), turned to 180 degrees
Connections:
- net LED5 renamed LED_STATUS
- C5 pad 1: Net-(C5-Pad1) -> GND_FB
- C8 pad 1: Net-(C5-Pad1) -> GND_FB
- CN1 pad 1: DGND -> P3_DGND
- CN2 pad 1: DGND -> P3_DGND
- J1 pad 1: RS422_TX+ -> P3_RS422_TX+
- J1 pad 10: Net-(J1-Pad10) -> P3_MAIN_LED1C
- J1 pad 11: DGND -> P3_DGND
- J1 pad 12: Net-(J1-Pad12) -> P3_MAIN_LED2C
- J1 pad 2: RS422_TX- -> P3_RS422_TX-
- J1 pad 3: RS422_RX+ -> P3_RS422_RX+
- J1 pad 4: VCC -> P3_VCC
- J1 pad 5: VCC -> P3_VCC_FB
- J1 pad 6: RS422_RX- -> P3_RS422_RX-
- J1 pad 7: Net-(J1-Pad7) -> P3_MAIN_LOAD
- J1 pad 8: Net-(J1-Pad7) -> P3_MAIN_LOAD
- J1 pad 9: Net-(J1-Pad9) -> P3_MAIN_LED1A
- J2 pad 1: RS422_RX+ -> P3_RS422_RX+
- J2 pad 10: Net-(J2-Pad10) -> P3_EXT_LED1C
- J2 pad 11: DGND -> P3_EXT_LED2A
- J2 pad 12: Net-(J2-Pad12) -> P3_VCC
- J2 pad 2: RS422_RX- -> P3_RS422_RX-
- J2 pad 3: RS422_TX+ -> P3_RS422_TX+
- J2 pad 4: VCC -> P3_VCC
- J2 pad 5: VCC -> P3_VCC
- J2 pad 6: RS422_TX- -> P3_RS422_TX-
- J2 pad 7: Net-(C5-Pad1) -> P3_GND_FB
- J2 pad 8: Net-(J2-Pad8) -> P3_EXT_LOAD
- J2 pad 9: Net-(J1-Pad9) -> P3_EXT_LED1A
- Q1 pad 3: Net-(J1-Pad9) -> MAIN_LED1A
- R11 pad 1: Net-(J2-Pad8) -> EXT_LOAD
- R12 pad 1: Net-(C5-Pad1) -> Net-(R12-Pad1)
- R12 pad 2: Net-(R12-Pad2) -> GND_FB
- R13 pad 2: Net-(R12-Pad2) -> Net-(R12-Pad1)
- R2 pad 1: Net-(J1-Pad7) -> MAIN_LOAD
- R27 pad 1: Net-(R12-Pad2) -> Net-(Q4-Pad1)
- R27 pad 2: Net-(Q2-Pad1) -> DGND
- R3 pad 1: +3.3V -> EXT_LED1A
- R3 pad 2: Net-(J2-Pad10) -> GND_FB
- R31 pad 1: TX_CHAIN_EN -> Net-(Q5-Pad2)
- R4 pad 1: +3.3V -> EXT_LED2A
- R4 pad 2: Net-(J2-Pad12) -> GND_FB
- R5 pad 1: +3.3V -> VCC_FB
- R5 pad 2: Net-(J1-Pad10) -> MAIN_LED1C
- R6 pad 1: +3.3V -> MAIN_LED2C
- R6 pad 2: Net-(J1-Pad12) -> VCC_FB
- U4 pad 1: TX_CHAIN_EN -> Net-(Q5-Pad2)
Routing:
- net P3_DGND: track 0.00 -> 101.3 mm
- net P3_VCC: track 0.00 -> 53.9 mm
- net GND_FB: track 0.00 -> 46.1 mm, vias 0 -> 2
- net Net-(C5-Pad1): track 46.0 -> 0.00 mm, vias 2 -> 0
- net (no net): track 0.00 -> 34.1 mm, vias 0 -> 5
- net Net-(J1-Pad7): track 33.5 -> 0.00 mm, vias 4 -> 0
- net MAIN_LOAD: track 0.00 -> 33.5 mm, vias 0 -> 4
- net P3_RS422_RX-: track 0.00 -> 33.1 mm
- net P3_RS422_RX+: track 0.00 -> 32.8 mm
- net VCC: track 51.0 -> 22.5 mm, vias 4 -> 0
- net Net-(J1-Pad9): track 25.7 -> 0.00 mm, vias 2 -> 0
- net MAIN_LED1A: track 0.00 -> 25.7 mm, vias 0 -> 2
- net P3_RS422_TX-: track 0.00 -> 24.5 mm, vias 0 -> 1
- net P3_VCC_FB: track 0.00 -> 21.7 mm, vias 0 -> 3
- net Net-(Q2-Pad1): track 22.1 -> 3.66 mm, vias 4 -> 2
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
Commit message: wip: tracing signals and adding a ground plane to the mini-pcb with connectors
Parts:
- moved CN1 0.80 mm to (251.2, 176.0)
- moved CN2 0.76 mm to (196.1, 176.0)
Routing:
- net P3_RS422_TX-: track 24.5 -> 60.9 mm, vias 1 -> 4
- net P3_DGND: track 101.3 -> 130.3 mm, vias 0 -> 2
- net P3_GND_FB: track 0.00 -> 27.0 mm, vias 0 -> 2
- net P3_RS422_TX+: track 17.7 -> 43.6 mm
- net P3_MAIN_LED1A: track 0.00 -> 23.9 mm, vias 0 -> 3
- net P3_MAIN_LOAD: track 2.20 -> 23.4 mm, vias 0 -> 4
- net Net-(R12-Pad1): track 7.57 -> 23.6 mm, vias 0 -> 1
- net GND_FB: track 46.1 -> 30.1 mm, vias 2 -> 1
- net P3_VCC: track 53.9 -> 40.3 mm, vias 0 -> 2
- net P3_EXT_LOAD: track 0.00 -> 12.0 mm, vias 0 -> 1
- net DGND: track 179.8 -> 170.0 mm, vias 59 -> 58
- net Net-(Q2-Pad1): track 3.66 -> 13.4 mm, vias 2 -> 3
- net P3_EXT_LED1C: track 0.00 -> 6.56 mm, vias 0 -> 1
- net P3_RS422_RX+: track 32.8 -> 37.5 mm
- net P3_EXT_LED1A: track 0.00 -> 4.35 mm
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Other:
- outline, holes or cut-outs redrawn

Commit message: adding another ground plane
Routing:
- net P3_DGND: track 130.3 -> 0.00 mm, vias 2 -> 0
- net +3.3V: track 521.2 -> 433.2 mm, vias 22 -> 18
- net EXT_LED1A: track 2.43 -> 67.5 mm, vias 0 -> 3
- net EXT_LED2A: track 3.01 -> 25.6 mm, vias 0 -> 1
- net TX_CHAIN_EN: track 31.3 -> 18.9 mm, vias 4 -> 2
- net Net-(Q5-Pad2): track 1.71 -> 14.2 mm, vias 0 -> 2
- net DGND: track 170.0 -> 181.4 mm, vias 58 -> 60
- net Net-(Q2-Pad1): track 13.4 -> 2.04 mm, vias 3 -> 1
- net Net-(R12-Pad1): track 23.6 -> 12.9 mm, vias 1 -> 0
- net GND_FB: track 30.1 -> 40.7 mm, vias 1 -> 2
- added copper zone on B.Cu, net P3_DGND
- added copper zone on F.Cu, net P3_DGND

Commit message: exporting mini-pcb to a VRML file
Parts:
- removed C1, C16, C3, C5, C6: 100uF, MOD_Footprints_Lib:CAP_RAD_5MM
- removed C10, C11: 18pF_NP0, MOD_Footprints_Lib:SM0603
- removed C12, C13, C14, C15, C17, C18, C2, C4, C7, C8, C9: 100nF_X7R, MOD_Footprints_Lib:SM0603
- removed D1: CGRA4007-G, MOD_Footprints_Lib:DO-214AC(SMA)
- removed D2, D3: MMSZ5242B, MOD_Footprints_Lib:SOD123
- removed FOOT1, FOOT2, FOOT3, FOOT4: HEADER_2X1_180, MOD_Footprints_Lib:PIN_ARRAY_2X1
- removed G***: LOGO, MOD_Footprints_Lib:MOD_Logo
- removed LCD1: AGM-2004A-204, MOD_Footprints_Lib:LCD-AGM-2004A-204
- removed LED1, LED2, LED3, LED4: LED_RGB, MOD_Footprints_Lib:LED_CLRTB_GFSF_1
- removed P1, P2: HEADER_5X2, MOD_Footprints_Lib:PIN_ARRAY_5x2
- removed P4: CONN_8X2, MOD_Footprints_Lib:pin_array_8x2
- removed Q1, Q3: MMBT3904, MOD_Footprints_Lib:SOT23
- removed Q2: MMBT3906, MOD_Footprints_Lib:SOT23
- removed R1, R10, R13, R28, R29, R30, R31, R32, R33, R46, R47, R7, R8, R9: 10k, MOD_Footprints_Lib:SM0603
- removed R11, R2: 100R 0.5W, MOD_Footprints_Lib:SM1210
- removed R12, R27: 100k, MOD_Footprints_Lib:SM0603
- removed R14, R15, R16, R17, R18, R19, R20, R21, R22, R23, R24, R25, R36: 1k, MOD_Footprints_Lib:SM0603
- removed R26, R37, R38, R39, R42, R43, R45: 0R, MOD_Footprints_Lib:SM0805
- removed R3, R4, R5, R6: 1K2, MOD_Footprints_Lib:SM0805
- removed R34: 3k, MOD_Footprints_Lib:SM0805
- removed R35: 330R, MOD_Footprints_Lib:SM0805
- removed R40, R41: 100R, MOD_Footprints_Lib:SM0603
- removed R44: 0R/NC, MOD_Footprints_Lib:SM0805
- removed RT1: PTC_FUSE_500mA, MOD_Footprints_Lib:SM2920
- removed RT2: PTC_FUSE_500mA, MOD_Footprints_Lib:SM1210
- removed TP1, TP2, TP3: CONN_1, MOD_Footprints_Lib:SIL-1
- removed U1: LPC111X_LQFP48, MOD_Footprints_Lib:LQFP48
- removed U2: MC7805, MOD_Footprints_Lib:DPAK(369C)
- removed U3: NCP1117DT33G, MOD_Footprints_Lib:DPAK(369C)
- removed U4: MAX13450E, MOD_Footprints_Lib:TSSOP14
- removed U5, U6: 74HC245, MOD_Footprints_Lib:TSSOP20
- removed X1: 10MHz, MOD_Footprints_Lib:HC_49US
- moved J1 39.1 mm to (199.1, 139.7)
- moved J2 39.1 mm to (220.5, 139.7)
- moved P3 39.1 mm to (209.8, 150.9)
- moved CN1 39.1 mm to (237.5, 139.4)
- moved CN2 39.1 mm to (182.4, 139.4)
Routing:
- net +3.3V: track 433.2 -> 0.00 mm, vias 18 -> 0
- net FOOT_4: track 203.3 -> 0.00 mm
- net LED4_B: track 199.0 -> 0.00 mm, vias 2 -> 0
- net LED4_R: track 198.7 -> 0.00 mm, vias 2 -> 0
- net LED4_G: track 196.4 -> 0.00 mm
- net DGND: track 181.4 -> 0.00 mm, vias 60 -> 0
- net +5V: track 151.3 -> 0.00 mm, vias 5 -> 0
- net FOOT_3: track 129.6 -> 0.00 mm
- net LED3_G: track 124.0 -> 0.00 mm
- net LED3_R: track 123.9 -> 0.00 mm
- net LED3_B: track 123.5 -> 0.00 mm
- net Net-(C6-Pad1): track 105.3 -> 0.00 mm, vias 33 -> 0
- net EXT_LED1A: track 67.5 -> 0.00 mm, vias 3 -> 0
- net LCD_RS: track 58.6 -> 0.00 mm
- net RS422_TX+: track 58.5 -> 0.00 mm, vias 4 -> 0
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- removed copper zone on B.Cu, net DGND
- removed copper zone on F.Cu, net DGND
- removed copper zone on B.Cu, net N-0000012
- removed copper zone on F.Cu, net N-0000012
Other:
- board size 248.9 x 74.2 mm -> 68.6 x 19.6 mm
- board text removed: "(c) 2014 Musical Operating Devices Licensed under CC By-SA https://github.com/portalmod/mod-hw-footswitch/"
- board text removed: "+3.3V"
- board text removed: "+5V"
- board text removed: "12"
- board text removed: "24"
- board text removed: "36"
- board text removed: "GND"
- board text removed: "UART DEBUGGER"
