File: hw-design/board/cpu.sch (KiCad schematic (older format))
At the start: 21 parts, among them CN1 CONN_PANNEL_2X2, CN2 CONN_PANNEL_2X2, P1 HEADER_5X2, P2 HEADER_5X2, U1 LPC111X_LQFP48, X1 10MHz

Commit message: importing common sheets from expression-pedal project
Parts:
- removed C9: 100nF_X7R, MOD_Footprints_Lib:SM0603, symbol C
- removed CN1, CN2: CONN_PANNEL_2X2, MOD_Footprints_Lib:CONN_PANNEL, symbol CONN_PANNEL_2X2
- removed P1, P2: HEADER_5X2, MOD_Footprints_Lib:PIN_ARRAY_5x2, symbol CONN_5X2
- removed R32, R33, R46, R47: 10k, MOD_Footprints_Lib:SM0603, symbol R
- removed R39, R42, R43, R45: 0R, MOD_Footprints_Lib:SM0805, symbol R
- removed R40, R41: 100R, MOD_Footprints_Lib:SM0603, symbol R
- removed U1: LPC111X_LQFP48, MOD_Footprints_Lib:LQFP48, symbol LPC111X_LQFP48
- removed X1: 10MHz, MOD_Footprints_Lib:HC_49US, symbol CRYSTAL
- added C14, C15, C16: 100nF X7R, Capacitors_SMD:C_0603, symbol C
- added P1: CHAIN, Pin_Headers:Pin_Header_Straight_1x04, symbol CONN_01X04
- added P2: USB_OTG, Connect:USB_Mini-B, symbol USB_OTG
- added P3: SWD, Pin_Headers:Pin_Header_Straight_2x05_Pitch1.27mm, symbol CONN_02X05
- added Q7: BC857, Housings_SOT-23_SOT-143_TSOT-6:SOT-23, symbol Q_PNP_BEC
- added R14: 3k, Resistors_SMD:R_0603, symbol R
- added R15: 24k, Resistors_SMD:R_0603, symbol R
- added R16: 1k5, Resistors_SMD:R_0603, symbol R
- added R17: 1M, Resistors_SMD:R_0603, symbol R
- added R18, R19: 33R, Resistors_SMD:R_0603, symbol R
- added R20: 100R, Resistors_SMD:R_0603, symbol R
- added R21: 10k, Resistors_SMD:R_0603, symbol R
- added SW1: SW_PUSH, Buttons_Switches_SMD:SW_SPST_FSMSM, symbol SW_PUSH
- added U4: LPC11U24FBD48/401, Housings_QFP:LQFP-80_12x12mm_Pitch0.5mm, symbol LPC11U24FBD48/401
- added Y1: 12MHz, Crystals:Crystal_HC49-SD_SMD, symbol Crystal_Small
- C10: value 18pF_NP0 -> 10nF 500V; footprint MOD_Footprints_Lib:SM0603 -> Capacitors_SMD:C_1206; MPN (none) -> 501R18W103KV4E
- C11: value 18pF_NP0 -> 18pF; footprint MOD_Footprints_Lib:SM0603 -> Capacitors_SMD:C_0603; MPN (none) -> C1608C0G1H180J080AA
- C12: value 100nF_X7R -> 18pF; footprint MOD_Footprints_Lib:SM0603 -> Capacitors_SMD:C_0603; MPN (none) -> C1608C0G1H180J080AA
- C13: value 100nF_X7R -> 10nF; footprint MOD_Footprints_Lib:SM0603 -> Capacitors_SMD:C_0603; MPN (none) -> C1608X7R1E103K080AA
Connections:
- net labels added: CH1, CH2, CH3, CHAIN_DE, CHAIN_RX, CHAIN_TX, FS1, FS1_LED_B, FS1_LED_G, FS1_LED_R, GNDD, POT, RX_LED, SWCLK, SWO, TX_LED, USB_CONNECT, USB_DM, USB_DP, USB_VBUS, VCC
- net labels removed: +5V, DGND, FOOT_1, FOOT_2, FOOT_3, FOOT_4, LED1_B, LED1_G, LED1_R, LED2_B, LED2_G, LED2_R, LED3_B, LED3_G, LED3_R, LED4_B, LED4_G, LED4_R, LED_STATUS, RX_CHAIN, SWDCLK, TX_CHAIN, TX_CHAIN_EN, UC_LCD0, UC_LCD1, UC_LCD2, UC_LCD3, UC_LCD4, UC_LCD5, UC_LCD6, UC_LCD7, UC_LCD_BACK, UC_LCD_DIR, UC_LCD_E, UC_LCD_RS, UC_LCD_RW, UC_RX_CHAIN, UC_TX_CHAIN, UC_TX_CHAIN_EN
- wire segments 108 -> 90
- no-connect marks 7 -> 25
Other:
- note added: "RESET"
- note added: "SWD"
- note added: "USB DEVICE"

Commit message: sch: schematic updated (missing displays circuit)
Connections:
- net FS3: now reaches U4.1 (PIO1_25/CT32B0_MAT1)
- net FS4: now reaches U4.11 (PIO1_26/CT32B0_MAT2/RXD)
- net LEDS_SCL: now reaches U4.15 (PIO0_4/SCL)
- net LEDS_SDA: now reaches U4.16 (PIO0_5/SDA)
- net FS2: now reaches U4.21 (PIO1_24/CT32B0_MAT0)
- net LEDS_OE: now reaches U4.23 (PIO0_7/~CTS~)
- net FS1_LED_B: no longer names the net of U4.25 (PIO1_31)
- net FS1_LED_G: no longer names the net of U4.31 (PIO1_29/SCK0/CT32B0_CAP1)
- net FS1_LED_R: no longer names the net of U4.24 (PIO1_28/CT32B0_CAP0/SCLK)
- net POT: no longer names the net of U4.32 (TDI/PIO0_11/AD0/CT32B0_MAT3)
- no-connect marks 25 -> 23
Other:
- moved on the sheet: P3
Changed lines of the file:
@@
 LIBS:transistors
 LIBS:nxp_armmcu
+LIBS:philips
 LIBS:footswitch-cache
 EELAYER 25 0
@@
 L GNDD #PWR045
 U 1 1 54E5DFA7
-P 9200 3950
-F 0 "#PWR045" H 9200 3700 60  0001 C CNN
-F 1 "GNDD" H 9200 3800 60  0000 C CNN
-F 2 "" H 9200 3950 60  0000 C CNN
-F 3 "" H 9200 3950 60  0000 C CNN
-	1    9200 3950
+P 9200 4250
+F 0 "#PWR045" H 9200 4000 60  0001 C CNN
+F 1 "GNDD" H 9200 4100 60  0000 C CNN
+F 2 "" H 9200 4250 60  0000 C CNN
+F 3 "" H 9200 4250 60  0000 C CNN
+	1    9200 4250
 	1    0    0    -1
 $EndComp
@@
 L CONN_02X05 P3
 U 1 1 54F2A3AF
-P 9650 3650
-F 0 "P3" H 9650 3950 50  0000 C CNN
-F 1 "SWD" H 9650 3350 50  0000 C CNN
-F 2 "Pin_Headers:Pin_Header_Straight_2x05_Pitch1.27mm" H 9650 2450 60  0001 C CNN
-F 3 "" H 9650 2450 60  0000 C CNN
-F 4 "-" H 0   0   50  0001 C CNN "MPN"
-	1    9650 3650
+P 9650 3950
+F 0 "P3" H 9650 4250 50  0000 C CNN
+F 1 "SWD" H 9650 3650 50  0000 C CNN
+F 2 "Pin_Headers:Pin_Header_Straight_2x05_Pitch1.27mm" H 9650 2750 60  0001 C CNN
+F 3 "" H 9650 2750 60  0000 C CNN
+F 4 "-" H 0   300 50  0001 C CNN "MPN"
+	1    9650 3950
 	1    0    0    -1
 $EndComp
@@
 	-1   0    0    -1
 $EndComp
-Text GLabel 10100 3850 2    50   Input ~ 0
+Text GLabel 10100 4150 2    50   Input ~ 0
 RESET
-Text Notes 9500 3250 0    100  ~ 0
+Text Notes 9500 3550 0    100  ~ 0
 SWD
 Text GLabel 7850 2200 2    50   Input ~ 0
@@
 Text GLabel 1800 1100 2    50   Input ~ 0
 CHAIN_DE
-Text GLabel 10100 3650 2    50   Output ~ 0
+Text GLabel 10100 3950 2    50   Output ~ 0
 SWO
-Text GLabel 10100 3550 2    50   Input ~ 0
+Text GLabel 10100 3850 2    50   Input ~ 0
 SWCLK
-Text GLabel 10100 3450 2    50   BiDi ~ 0
+Text GLabel 10100 3750 2    50   BiDi ~ 0
 SWDIO
 Text GLabel 7850 1900 2    50   Input ~ 0
@@
 Text GLabel 7850 2800 2    50   Output ~ 0
 SWO
-Text GLabel 7850 3000 2    50   Input ~ 0
-POT
 Text GLabel 3900 2800 0    50   Input ~ 0
 FS1
@@
 Text GLabel 7850 3800 2    50   Output ~ 0
 TX_LED
-Text GLabel 3900 3300 0    50   Output ~ 0
-FS1_LED_R
-Text GLabel 3900 3400 0    50   Output ~ 0
-FS1_LED_G
-Text GLabel 3900 3500 0    50   Output ~ 0
-FS1_LED_B
-Wire Wire Line
-	9200 3550 9200 3950
+Text GLabel 7850 2400 2    50   Output ~ 0
+LEDS_SDA
+Text GLabel 7850 2300 2    50   Output ~ 0
+LEDS_SCL
+Text GLabel 7850 2600 2    50   Output ~ 0
+LEDS_OE
+Wire Wire Line
+	9200 3850 9200 4250
+Wire Wire Line
+	9900 4150 10100 4150
+Wire Wire Line
+	9200 4150 9400 4150
+Wire Wire Line
+	9200 3950 9400 3950
+Wire Wire Line
+	9200 3850 9400 3850
+Wire Wire Line
+	4100 4100 4050 4100
+Wire Wire Line
+	4050 4100 4050 4200
+Wire Wire Line
+	4050 4200 3550 4200
+Wire Wire Line
+	3550 4200 3550 4250
+Wire Wire Line
+	3300 4250 3300 3900
+Wire Wire Line
+	3300 3900 4050 3900
+Wire Wire Line
+	4050 3900 4050 4000
+Wire Wire Line
+	4050 4000 4100 4000
+Wire Wire Line
+	3850 3950 3850 3900
+Wire Wire Line
+	3850 4150 3850 4200
+Wire Wire Line
+	3300 4550 3300 4600
+Wire Wire Line
+	3550 4550 3550 4600
+Wire Wire Line
+	7850 2200 7700 2200
+Wire Wire Line
+	5800 1600 5800 900
+Wire Wire Line
+	5600 900  6200 900
+Wire Wire Line
+	6000 900  6000 1600
+Wire Wire Line
+	5900 850  5900 900
+Wire Wire Line
+	7700 2500 7850 2500
+Wire Wire Line
+	5600 1050 5600 900
+Wire Wire Line
+	6200 900  6200 1050
+Wire Wire Line
+	5600 1450 5600 1350
+Wire Wire Line
+	6200 1450 6200 1350
+Wire Wire Line
+	5800 4600 5800 4700
+Wire Wire Line
+	5800 4700 6000 4700
+Wire Wire Line
+	6000 4700 6000 4600
+Wire Wire Line
+	5900 4750 5900 4700
+Wire Wire Line
+	4300 7350 4150 7350
+Wire Wire Line
+	3350 6400 3350 7350
+Wire Wire Line
+	4300 7200 4150 7200
+Wire Wire Line
+	3850 7200 3450 7200
+Wire Wire Line
+	3450 7200 3450 6400
+Wire Wire Line
+	4200 6450 4350 6450
+Wire Wire Line
+	3550 6450 3900 6450
+Wire Wire Line
+	3550 6450 3550 6400
+Wire Wire Line
+	3750 6300 3750 6550
+Wire Wire Line
+	2850 6100 2850 6000
+Wire Wire Line
+	2650 6000 2950 6000
+Wire Wire Line
+	2650 6000 2650 6100
+Wire Wire Line
+	2650 6400 2650 6500
+Wire Wire Line
+	2650 6500 3150 6500
+Wire Wire Line
+	3150 6500 3150 6400
+Wire Wire Line
+	2850 6400 2850 6600
+Wire Wire Line
+	3900 3700 4100 3700
+Wire Wire Line
+	4100 3800 3900 3800
+Wire Wire Line
+	1950 7100 2150 7100
+Wire Wire Line
+	2050 7000 2050 7100
+Wire Wire Line
+	1650 7100 1500 7100
+Wire Wire Line
+	2050 6500 2050 6700
+Wire Wire Line
+	2450 6900 2450 6600
+Wire Wire Line
+	2450 6600 2050 6600
+Wire Wire Line
+	2450 7300 2450 7350
+Wire Wire Line
+	2450 7350 2600 7350
+Wire Wire Line
+	2900 7350 3850 7350
+Wire Wire Line
+	3750 6900 3750 6850
+Wire Wire Line
+	3900 2000 4100 2000
+Wire Wire Line
+	3900 2100 4100 2100
+Wire Wire Line
+	4100 2200 3900 2200
+Wire Wire Line
+	1650 1300 1800 1300
+Wire Wire Line
+	1800 1200 1650 1200
+Wire Wire Line
+	1650 1100 1800 1100
+Wire Wire Line
+	1650 1400 1700 1400
+Wire Wire Line
+	1700 1400 1700 1450
+Wire Wire Line
+	9900 3950 10100 3950
 Wire Wire Line
 	9900 3850 10100 3850
 Wire Wire Line
-	9200 3850 9400 3850
-Wire Wire Line
-	9200 3650 9400 3650
-Wire Wire Line
-	9200 3550 9400 3550
-Wire Wire Line
-	4100 4100 4050 4100
-Wire Wire Line
-	4050 4100 4050 4200
-Wire Wire Line
-	4050 4200 3550 4200
-Wire Wire Line
-	3550 4200 3550 4250
-Wire Wire Line
-	3300 4250 3300 3900
-Wire Wire Line
-	3300 3900 4050 3900
-Wire Wire Line
-	4050 3900 4050 4000
-Wire Wire Line
-	4050 4000 4100 4000
-Wire Wire Line
-	3850 3950 3850 3900
-Wire Wire Line
-	3850 4150 3850 4200
-Wire Wire Line
-	3300 4550 3300 4600
-Wire Wire Line
-	3550 4550 3550 4600
-Wire Wire Line
-	7850 2200 7700 2200
-Wire Wire Line
-	5800 1600 5800 900
-Wire Wire Line
-	5600 900  6200 900
-Wire Wire Line
-	6000 900  6000 1600
-Wire Wire Line
-	5900 850  5900 900
-Wire Wire Line
-	7700 2500 7850 2500
-Wire Wire Line
-	5600 1050 5600 900
-Wire Wire Line
-	6200 900  6200 1050
-Wire Wire Line
-	5600 1450 5600 1350
-Wire Wire Line
-	6200 1450 6200 1350
-Wire Wire Line
-	5800 4600 5800 4700
-Wire Wire Line
-	5800 4700 6000 4700
-Wire Wire Line
-	6000 4700 6000 4600
-Wire Wire Line
-	5900 4750 5900 4700
-Wire Wire Line
-	4300 7350 4150 7350
-Wire Wire Line
-	3350 6400 3350 7350
-Wire Wire Line
-	4300 7200 4150 7200
-Wire Wire Line
-	3850 7200 3450 7200
-Wire Wire Line
-	3450 7200 3450 6400
-Wire Wire Line
-	4200 6450 4350 6450
-Wire Wire Line
-	3550 6450 3900 6450
-Wire Wire Line
-	3550 6450 3550 6400
-Wire Wire Line
-	3750 6300 3750 6550
-Wire Wire Line
-	2850 6100 2850 6000
-Wire Wire Line
-	2650 6000 2950 6000
-Wire Wire Line
-	2650 6000 2650 6100
-Wire Wire Line
-	2650 6400 2650 6500
-Wire Wire Line
-	2650 6500 3150 6500
-Wire Wire Line
-	3150 6500 3150 6400
-Wire Wire Line
-	2850 6400 2850 6600
-Wire Wire Line
-	3900 3700 4100 3700
-Wire Wire Line
-	4100 3800 3900 3800
-Wire Wire Line
-	1950 7100 2150 7100
-Wire Wire Line
-	2050 7000 2050 7100
-Wire Wire Line
-	1650 7100 1500 7100
-Wire Wire Line
-	2050 6500 2050 6700
-Wire Wire Line
-	2450 6900 2450 6600
-Wire Wire Line
-	2450 6600 2050 6600
-Wire Wire Line
-	2450 7300 2450 7350
-Wire Wire Line
-	2450 7350 2600 7350
-Wire Wire Line
-	2900 7350 3850 7350
-Wire Wire Line
-	3750 6900 3750 6850
-Wire Wire Line
-	3900 2000 4100 2000
-Wire Wire Line
-	3900 2100 4100 2100
-Wire Wire Line
-	4100 2200 3900 2200
-Wire Wire Line
-	1650 1300 1800 1300
-Wire Wire Line
-	1800 1200 1650 1200
-Wire Wire Line
-	1650 1100 1800 1100
-Wire Wire Line
-	1650 1400 1700 1400
-Wire Wire Line
-	1700 1400 1700 1450
-Wire Wire Line
-	9900 3650 10100 3650
-Wire Wire Line
-	9900 3550 10100 3550
-Wire Wire Line
-	9900 3450 10100 3450
+	9900 3750 10100 3750
 Wire Wire Line
 	7850 2900 7700 2900
@@
 	7850 2800 7700 2800
 Wire Wire Line
-	7850 3000 7700 3000
-Wire Wire Line
 	3900 2400 4100 2400
 Wire Wire Line
@@
 Wire Wire Line
 	7850 3800 7700 3800
-Wire Wire Line
-	4100 3300 3900 3300
-Wire Wire Line
-	3900 3400 4100 3400
-Wire Wire Line
-	4100 3500 3900 3500
-Connection ~ 9200 3650
-Connection ~ 9200 3850
+Connection ~ 9200 3950
+Connection ~ 9200 4150
 Connection ~ 3850 3900
 Connection ~ 3850 4200
@@
 Connection ~ 9600 1750
 NoConn ~ 3250 6400
+NoConn ~ 9400 4050
 NoConn ~ 9400 3750
-NoConn ~ 9400 3450
-NoConn ~ 9900 3750
+NoConn ~ 9900 4050
 NoConn ~ 4100 2700
-NoConn ~ 4100 2900
-NoConn ~ 4100 3000
-NoConn ~ 4100 3100
 NoConn ~ 4100 3200
 NoConn ~ 7700 2000
 NoConn ~ 7700 2100
-NoConn ~ 7700 2300
-NoConn ~ 7700 2400
-NoConn ~ 7700 2600
 NoConn ~ 7700 2700
 NoConn ~ 7700 3100
@@
 NoConn ~ 7700 4200
 NoConn ~ 4100 2300
+Wire Wire Line
+	7700 2300 7850 2300
+Wire Wire Line
+	7850 2400 7700 2400
+Wire Wire Line
+	7850 2600 7700 2600
+Text GLabel 3900 2900 0    50   Input ~ 0
+FS2
+Wire Wire Line
+	4100 2900 3900 2900
+Text GLabel 3900 3000 0    50   Input ~ 0
+FS3
+Wire Wire Line
+	4100 3000 3900 3000
+Text GLabel 3900 3100 0    50   Input ~ 0
+FS4
+Wire Wire Line
+	4100 3100 3900 3100
+NoConn ~ 4100 3300
+NoConn ~ 4100 3400
+NoConn ~ 4100 3500
+NoConn ~ 7700 3000
 $EndSCHEMATC

Commit message: sch: display circuit done
Connections:
- net LCD_RW: now reaches U4.17 (PIO0_21/CT16B1_MAT0/MOSI1)
- net LCD_CONTRAST: now reaches U4.27 (PIO0_8/MISO0/CT16B0_MAT0)
- net LCD1_EN: now reaches U4.30 (PIO0_22/AD6/CT16B1_MAT1/MISO1)
- net LCD_D7: now reaches U4.32 (TDI/PIO0_11/AD0/CT32B0_MAT3)
- net LCD_D6: now reaches U4.33 (TMS/PIO0_12/AD1/CT32B1_CAP0)
- net LCD_D5: now reaches U4.34 (TDO/PIO0_13/AD2/CT32B1_MAT0)
- net LCD_D4: now reaches U4.35 (~TRST~/PIO0_14/AD3/CT32B1_MAT1)
- net LCD1_BL: now reaches U4.40 (PIO0_16/AD5/CT32B1_MAT3/WAKEUP)
- net LCD2_EN: now reaches U4.42 (PIO0_23/AD7)
- net LCD2_BL: now reaches U4.45 (PIO0_17/~RTS~/CT32B0_CAP0/SCLK)
- net LCD_RS: now reaches U4.9 (PIO0_20/CT16B1_CAP0)
- no-connect marks 23 -> 12
Changed lines of the file:
@@
 LIBS:regul
 LIBS:transistors
+LIBS:display
 LIBS:nxp_armmcu
 LIBS:philips
@@
 NoConn ~ 7700 2000
 NoConn ~ 7700 2100
-NoConn ~ 7700 2700
-NoConn ~ 7700 3100
-NoConn ~ 7700 3200
-NoConn ~ 7700 3300
-NoConn ~ 7700 3500
-NoConn ~ 7700 3600
-NoConn ~ 7700 3900
-NoConn ~ 7700 4000
-NoConn ~ 7700 4100
-NoConn ~ 7700 4200
 NoConn ~ 4100 2300
 Wire Wire Line
@@
 NoConn ~ 4100 3400
 NoConn ~ 4100 3500
-NoConn ~ 7700 3000
+Text GLabel 7850 3000 2    50   BiDi ~ 0
+LCD_D7
+Text GLabel 7850 3100 2    50   BiDi ~ 0
+LCD_D6
+Text GLabel 7850 3200 2    50   BiDi ~ 0
+LCD_D5
+Text GLabel 7850 3300 2    50   BiDi ~ 0
+LCD_D4
+Text GLabel 7850 3900 2    50   Output ~ 0
+LCD_RS
+Text GLabel 7850 4000 2    50   Output ~ 0
+LCD_RW
+Text GLabel 7850 4100 2    50   Output ~ 0
+LCD1_EN
+Text GLabel 7850 4200 2    50   Output ~ 0
+LCD2_EN
+Text GLabel 7850 3500 2    50   Output ~ 0
+LCD1_BL
+Text GLabel 7850 3600 2    50   Output ~ 0
+LCD2_BL
+Text GLabel 7850 2700 2    50   Output ~ 0
+LCD_CONTRAST
+Wire Wire Line
+	7850 3000 7700 3000
+Wire Wire Line
+	7700 3100 7850 3100
+Wire Wire Line
+	7850 3200 7700 3200
+Wire Wire Line
+	7700 3300 7850 3300
+Wire Wire Line
+	7700 3900 7850 3900
+Wire Wire Line
+	7850 4000 7700 4000
+Wire Wire Line
+	7700 4100 7850 4100
+Wire Wire Line
+	7850 4200 7700 4200
+Wire Wire Line
+	7700 2700 7850 2700
+Wire Wire Line
+	7850 3500 7700 3500
+Wire Wire Line
+	7700 3600 7850 3600
 $EndSCHEMATC

Commit message: sch: fixing VBUS signal and FS1 I/O
Parts:
- added R21: 3K3, Resistors_SMD:R_0603, symbol R
- R20: value 100R -> 2K; MPN RMCF0603JT100R -> RMCF0603JT2K00
- renumbered R21 to R22
Connections:
- net FS1: now also U4.4 (PIO0_1/CLKOUT/CT32B0_MAT2/USB_FTOGGLE); no longer U4.18 (PIO1_23/CT16B1_MAT1/SSEL1)
- net GNDD: now also R21.1
- net USB_VBUS: now also R21.2

Commit message: sch: DRC checked
Changed lines of the file:
@@
 $EndDescr
 $Comp
-L GNDD #PWR52
+L GNDD #PWR045
 U 1 1 54E5DFA7
 P 9200 4250
-F 0 "#PWR52" H 9200 4000 60  0001 C CNN
+F 0 "#PWR045" H 9200 4000 60  0001 C CNN
 F 1 "GNDD" H 9200 4100 60  0000 C CNN
 F 2 "" H 9200 4250 60  0000 C CNN
@@
 $EndComp
 $Comp
-L GNDD #PWR43
+L GNDD #PWR046
 U 1 1 556F6417
 P 3300 4600
-F 0 "#PWR43" H 3300 4350 50  0001 C CNN
+F 0 "#PWR046" H 3300 4350 50  0001 C CNN
 F 1 "GNDD" H 3300 4450 50  0000 C CNN
 F 2 "" H 3300 4600 60  0000 C CNN
@@
 $EndComp
 $Comp
-L GNDD #PWR44
+L GNDD #PWR047
 U 1 1 556F65EC
 P 3550 4600
-F 0 "#PWR44" H 3550 4350 50  0001 C CNN
+F 0 "#PWR047" H 3550 4350 50  0001 C CNN
 F 1 "GNDD" H 3550 4450 50  0000 C CNN
 F 2 "" H 3550 4600 60  0000 C CNN
@@
 $EndComp
 $Comp
-L +3.3V #PWR49
+L +3.3V #PWR048
 U 1 1 55705A80
 P 5900 850
-F 0 "#PWR49" H 5900 700 50  0001 C CNN
+F 0 "#PWR048" H 5900 700 50  0001 C CNN
 F 1 "+3.3V" H 5900 990 50  0000 C CNN
 F 2 "" H 5900 850 60  0000 C CNN
@@
 $EndComp
 $Comp
-L GNDD #PWR48
+L GNDD #PWR049
 U 1 1 557DC875
 P 5600 1450
-F 0 "#PWR48" H 5600 1200 50  0001 C CNN
+F 0 "#PWR049" H 5600 1200 50  0001 C CNN
 F 1 "GNDD" H 5600 1300 50  0000 C CNN
 F 2 "" H 5600 1450 60  0000 C CNN
@@
 $EndComp
 $Comp
-L GNDD #PWR51
+L GNDD #PWR050
 U 1 1 557DCAD9
 P 6200 1450
-F 0 "#PWR51" H 6200 1200 50  0001 C CNN
+F 0 "#PWR050" H 6200 1200 50  0001 C CNN
 F 1 "GNDD" H 6200 1300 50  0000 C CNN
 F 2 "" H 6200 1450 60  0000 C CNN
@@
 $EndComp
 $Comp
-L GNDD #PWR50
+L GNDD #PWR051
 U 1 1 557DD01E
 P 5900 4750
-F 0 "#PWR50" H 5900 4500 50  0001 C CNN
+F 0 "#PWR051" H 5900 4500 50  0001 C CNN
 F 1 "GNDD" H 5900 4600 50  0000 C CNN
 F 2 "" H 5900 4750 60  0000 C CNN
@@
 $EndComp
 $Comp
-L GNDD #PWR42
+L GNDD #PWR052
 U 1 1 557DE7E3
 P 2850 6600
-F 0 "#PWR42" H 2850 6350 50  0001 C CNN
+F 0 "#PWR052" H 2850 6350 50  0001 C CNN
 F 1 "GNDD" H 2850 6450 50  0000 C CNN
 F 2 "" H 2850 6600 60  0000 C CNN
@@
 $EndComp
 $Comp
-L VCC #PWR45
+L VCC #PWR053
 U 1 1 557DE7F0
 P 3750 6300
-F 0 "#PWR45" H 3750 6150 50  0001 C CNN
+F 0 "#PWR053" H 3750 6150 50  0001 C CNN
 F 1 "VCC" H 3750 6450 50  0000 C CNN
 F 2 "" H 3750 6300 60  0000 C CNN
@@
 $EndComp
 $Comp
-L +3.3V #PWR41
+L +3.3V #PWR054
 U 1 1 557E22DB
 P 2050 6500
-F 0 "#PWR41" H 2050 6350 50  0001 C CNN
+F 0 "#PWR054" H 2050 6350 50  0001 C CNN
 F 1 "+3.3V" H 2050 6640 50  0000 C CNN
 F 2 "" H 2050 6500 60  0000 C CNN
@@
 $EndComp
 $Comp
-L GNDD #PWR46
+L GNDD #PWR055
 U 1 1 557EA320
 P 3750 6900
-F 0 "#PWR46" H 3750 6650 50  0001 C CNN
+F 0 "#PWR055" H 3750 6650 50  0001 C CNN
 F 1 "GNDD" H 3750 6750 50  0000 C CNN
 F 2 "" H 3750 6900 60  0000 C CNN
@@
 $EndComp
 $Comp
-L GNDD #PWR40
+L GNDD #PWR056
 U 1 1 557F3440
 P 1700 1450
-F 0 "#PWR40" H 1700 1200 50  0001 C CNN
+F 0 "#PWR056" H 1700 1200 50  0001 C CNN
 F 1 "GNDD" H 1700 1300 50  0000 C CNN
 F 2 "" H 1700 1450 60  0000 C CNN
@@
 $EndComp
 $Comp
-L +3.3V #PWR54
+L +3.3V #PWR057
 U 1 1 55802FA1
 P 10000 1250
-F 0 "#PWR54" H 10000 1100 50  0001 C CNN
+F 0 "#PWR057" H 10000 1100 50  0001 C CNN
 F 1 "+3.3V" H 10000 1390 50  0000 C CNN
 F 2 "" H 10000 1250 60  0000 C CNN
@@
 $EndComp
 $Comp
-L GNDD #PWR55
+L GNDD #PWR058
 U 1 1 55803C49
 P 10000 2250
-F 0 "#PWR55" H 10000 2000 50  0001 C CNN
+F 0 "#PWR058" H 10000 2000 50  0001 C CNN
 F 1 "GNDD" H 10000 2100 50  0000 C CNN
 F 2 "" H 10000 2250 60  0000 C CNN
@@
 $EndComp
 $Comp
-L GNDD #PWR53
+L GNDD #PWR059
 U 1 1 55806665
 P 9600 2550
-F 0 "#PWR53" H 9600 2300 50  0001 C CNN
+F 0 "#PWR059" H 9600 2300 50  0001 C CNN
 F 1 "GNDD" H 9600 2400 50  0000 C CNN
 F 2 "" H 9600 2550 60  0000 C CNN
@@
 LCD_CONTRAST
 Wire Wire Line
-	9200 3850 9200 3950
-Wire Wire Line
-	9200 3950 9200 4150
-Wire Wire Line
-	9200 4150 9200 4250
+	9200 3850 9200 4250
 Wire Wire Line
 	9900 4150 10100 4150
@@
 	4050 4100 4050 4200
 Wire Wire Line
-	4050 4200 3850 4200
-Wire Wire Line
-	3850 4200 3550 4200
+	4050 4200 3550 4200
 Wire Wire Line
 	3550 4200 3550 4250
@@
 	3300 4250 3300 3900
 Wire Wire Line
-	3300 3900 3850 3900
-Wire Wire Line
-	3850 3900 4050 3900
+	3300 3900 4050 3900
 Wire Wire Line
 	4050 3900 4050 4000
@@
 	5800 1600 5800 900
 Wire Wire Line
-	5600 900  5800 900
-Wire Wire Line
-	5800 900  5900 900
-Wire Wire Line
-	5900 900  6000 900
-Wire Wire Line
-	6000 900  6200 900
+	5600 900  6200 900
 Wire Wire Line
 	6000 900  6000 1600
@@
 	5800 4600 5800 4700
 Wire Wire Line
-	5800 4700 5900 4700
-Wire Wire Line
-	5900 4700 6000 4700
+	5800 4700 6000 4700
 Wire Wire Line
 	6000 4700 6000 4600
@@
 	3450 7200 3450 6400
 Wire Wire Line
-	4200 6450 4350 6450
-Wire Wire Line
-	4350 6450 4500 6450
-Wire Wire Line
-	3550 6450 3750 6450
-Wire Wire Line
-	3750 6450 3900 6450
+	4200 6450 4500 6450
+Wire Wire Line
+	3550 6450 3900 6450
 Wire Wire Line
 	3550 6450 3550 6400
 Wire Wire Line
-	3750 6300 3750 6450
-Wire Wire Line
-	3750 6450 3750 6550
+	3750 6300 3750 6550
 Wire Wire Line
 	2850 6100 2850 6000
 Wire Wire Line
-	2650 6000 2850 6000
-Wire Wire Line
-	2850 6000 2950 6000
+	2650 6000 2950 6000
 Wire Wire Line
 	2650 6000 2650 6100
@@
 	2650 6400 2650 6500
 Wire Wire Line
-	2650 6500 2850 6500
-Wire Wire Line
-	2850 6500 3150 6500
+	2650 6500 3150 6500
 Wire Wire Line
 	3150 6500 3150 6400
 Wire Wire Line
-	2850 6400 2850 6500
-Wire Wire Line
-	2850 6500 2850 6600
+	2850 6400 2850 6600
 Wire Wire Line
 	3950 3700 4100 3700
@@
 	4100 3800 3950 3800
 Wire Wire Line
-	1950 7100 2050 7100
-Wire Wire Line
-	2050 7100 2150 7100
+	1950 7100 2150 7100
 Wire Wire Line
 	2050 7000 2050 7100
@@
 	1650 7100 1500 7100
 Wire Wire Line
-	2050 6500 2050 6600
-Wire Wire Line
-	2050 6600 2050 6700
+	2050 6500 2050 6700
 Wire Wire Line
 	2450 6900 2450 6600
@@
 	2450 7350 2600 7350
 Wire Wire Line
-	2900 7350 3350 7350
-Wire Wire Line
-	3350 7350 3850 7350
+	2900 7350 3850 7350
 Wire Wire Line
 	3750 6900 3750 6850
@@
 	10000 1350 10000 1250
 Wire Wire Line
-	10000 1650 10000 1750
-Wire Wire Line
-	10000 1750 10000 1850
+	10000 1650 10000 1850
 Wire Wire Line
 	10000 2150 10000 2250
 Wire Wire Line
-	9350 1750 9600 1750
-Wire Wire Line
-	9600 1750 10000 1750
+	9350 1750 10000 1750
 Wire Wire Line
 	9600 1850 9600 1750
@@
 Connection ~ 4350 6450
 $Comp
-L GNDD #PWR47
+L GNDD #PWR060
 U 1 1 558C35D8
 P 4350 6900
-F 0 "#PWR47" H 4350 6650 50  0001 C CNN
+F 0 "#PWR060" H 4350 6650 50  0001 C CNN
 F 1 "GNDD" H 4350 6750 50  0000 C CNN
 F 2 "" H 4350 6900 60  0000 C CNN

Commit message: sch: fixing some footprints and MPN
Parts:
- U4: footprint Housings_QFP:LQFP-80_12x12mm_Pitch0.5mm -> Housings_QFP:LQFP-48_7x7mm_Pitch0.5mm
Changed lines of the file:
@@
 F 0 "U4" H 4400 4500 50  0000 C CNN
 F 1 "LPC11U24FBD48/401" H 7100 4500 50  0000 C CNN
-F 2 "Housings_QFP:LQFP-80_12x12mm_Pitch0.5mm" H 5900 2000 50  0000 C CNN
+F 2 "Housings_QFP:LQFP-48_7x7mm_Pitch0.5mm" H 5900 2000 50  0000 C CNN
 F 3 "" H 5850 3050 60  0000 C CNN
 F 4 "LPC11U24FBD48/401" H 0   0   50  0001 C CNN "MPN"
