File: hw-design/board/cpu.sch (KiCad schematic (older format))
At the start: 23 parts, among them P1 CHAIN, P2 USB_OTG, P3 SWD, Q7 BC857, SW1 SW_PUSH, U4 LPC11U24FBD48/401, Y1 12MHz

Commit message: sch: channel selector switch is no longer used
Connections:
- net CH1: no longer names the net of U4.2 (PIO1_19/~DTR~/SSEL1)
- net CH2: no longer names the net of U4.13 (PIO1_20/~DSR~/SCK1)
- net CH3: no longer names the net of U4.26 (PIO1_21/~DCD~/MISO1)
- no-connect marks 12 -> 15
Changed lines of the file:
@@
 Text GLabel 7850 2000 2    50   Input ~ 0
 FS1
-Text GLabel 3950 2400 0    50   Input ~ 0
-CH1
-Text GLabel 3950 2500 0    50   Input ~ 0
-CH2
-Text GLabel 3950 2600 0    50   Input ~ 0
-CH3
 Text GLabel 7850 3700 2    50   Output ~ 0
 RX_LED
@@
 Wire Wire Line
 	7850 2800 7700 2800
-Wire Wire Line
-	3950 2400 4100 2400
-Wire Wire Line
-	4100 2500 3950 2500
-Wire Wire Line
-	3950 2600 4100 2600
 Wire Wire Line
 	7700 2000 7850 2000
@@
 Wire Wire Line
 	4350 6900 4350 6850
+NoConn ~ 4100 2400
+NoConn ~ 4100 2500
+NoConn ~ 4100 2600
 $EndSCHEMATC

Commit message: sch: schematic files reorganized, new sheets for usb and rear board
Parts:
- removed C10: 10nF 500V, Capacitors_SMD:C_1206, symbol C
- removed C13: 10nF, Capacitors_SMD:C_0603, symbol C
- removed P2: USB_OTG, Connect:USB_Mini-B, symbol USB_OTG
- removed Q7: BC857, Housings_SOT-23_SOT-143_TSOT-6:SOT-23, symbol Q_PNP_BEC
- removed R14: 3k, Resistors_SMD:R_0603, symbol R
- removed R15: 24k, Resistors_SMD:R_0603, symbol R
- removed R16: 1k5, Resistors_SMD:R_0603, symbol R
- removed R17: 1M, Resistors_SMD:R_0603, symbol R
- removed R18, R19: 33R, Resistors_SMD:R_0603, symbol R
- removed R20: 2K, Resistors_SMD:R_0603, symbol R
- removed R21: 3K3, Resistors_SMD:R_0603, symbol R
- renumbered C12 to C10, C14 to C11, C15 to C12, C16 to C13, C11 to C9, P3 to P2, R22 to R6
Connections:
- net RX_LED renamed RX_LED_CPU
- net TX_LED renamed TX_LED_CPU
- net USB_DM renamed USB_DM_CPU
- net USB_DP renamed USB_DP_CPU
- no-connect marks 15 -> 14
Other:
- note removed: "USB DEVICE"
- moved on the sheet: C10, C11, C12, C13, C9, P1, P2, R6, SW1, U4, Y1

Commit message: connecting foot leds directly to cpu
Parts:
- P1: footprint Pin_Headers:Pin_Header_Straight_1x04 -> Pin_Headers:Pin_Header_Straight_1x03; symbol CONN_01X04 -> CONN_01X03
Connections:
- net LEDS_SCL is gone; now on net FS3: U4.15 (PIO0_4/SCL)
- net LEDS_SDA is gone; now on net FS4: U4.16 (PIO0_5/SDA)
- net CHAIN_DE: no longer P1.4 (P4)
- net FS2: now also U4.10 (PIO0_2/SSEL0/CT16B0_CAP0); no longer U4.21 (PIO1_24/CT32B0_MAT0)
- net FS3: no longer U4.1 (PIO1_25/CT32B0_MAT1)
- net FS4: no longer U4.11 (PIO1_26/CT32B0_MAT2/RXD)
- net LED_B4: now reaches U4.12 (PIO1_27/CT32B0_MAT3/TXD)
- net LED_G1: now reaches U4.13 (PIO1_20/~DSR~/SCK1)
- net LED_G2: now reaches U4.18 (PIO1_23/CT16B1_MAT1/SSEL1)
- net LED_R1: now reaches U4.2 (PIO1_19/~DTR~/SSEL1)
- net LED_R4: now reaches U4.24 (PIO1_28/CT32B0_CAP0/SCLK)
- net LED_B2: now reaches U4.26 (PIO1_21/~DCD~/MISO1)
- net LED_G4: now reaches U4.31 (PIO1_29/SCK0/CT32B0_CAP1)
- net LED_R2: now reaches U4.38 (PIO1_22/~RI~/MOSI1)
- net LED_B1: now reaches U4.48 (PIO1_16/~RI~/CT16B0_CAP0)
- net LEDS_OE: no longer names the net of U4.23 (PIO0_7/~CTS~)
- net RX_LED_CPU: no longer names the net of U4.46 (PIO0_18/RXD/CT32B0_MAT0)
- net TX_LED_CPU: no longer names the net of U4.47 (PIO0_19/TXD/CT32B0_MAT1)
- new net LED_B3: U4.21 (PIO1_24/CT32B0_MAT0)
- new net LED_G3: U4.11 (PIO1_26/CT32B0_MAT2/RXD)
- new net LED_R3: U4.1 (PIO1_25/CT32B0_MAT1)
- no-connect marks 14 -> 7
Changed lines of the file:
@@
-$EndComp
-$Comp
-L LPC11U24FBD48/401 U4
-U 1 1 556F3A3A
-P 5550 3750
-F 0 "U4" H 4050 5150 50  0000 C CNN
-F 1 "LPC11U24FBD48/401" H 6750 5150 50  0000 C CNN
-F 2 "Housings_QFP:LQFP-48_7x7mm_Pitch0.5mm" H 5550 2650 50  0000 C CNN
-F 3 "" H 5500 3700 60  0000 C CNN
-F 4 "LPC11U24FBD48/401" H -350 650 50  0001 C CNN "MPN"
-	1    5550 3750
-	1    0    0    -1
 $EndComp
 $Comp
@@
 F 0 "C10" H 3225 5150 50  0000 L CNN
 F 1 "18pF" H 3225 4950 50  0000 L CNN
-F 2 "Capacitors_SMD:C_0603" H 3238 4900 30  0000 C CNN
+F 2 "Capacitors_SMD:C_0603" H 3238 4900 30  0001 C CNN
 F 3 "" H 3200 5050 60  0000 C CNN
 F 4 "C1608C0G1H180J080AA" H -350 650 50  0001 C CNN "MPN"
@@
 F 0 "C9" H 2975 5150 50  0000 L CNN
 F 1 "18pF" H 2975 4950 50  0000 L CNN
-F 2 "Capacitors_SMD:C_0603" H 2988 4900 30  0000 C CNN
+F 2 "Capacitors_SMD:C_0603" H 2988 4900 30  0001 C CNN
 F 3 "" H 2950 5050 60  0000 C CNN
 F 4 "C1608C0G1H180J080AA" H -350 650 50  0001 C CNN "MPN"
@@
 $EndComp
 $Comp
-L CONN_01X04 P1
+L CONN_01X03 P1
 U 1 1 557F309A
-P 1800 2800
-F 0 "P1" H 1800 3050 50  0000 C CNN
-F 1 "CHAIN" V 1900 2800 50  0000 C CNN
-F 2 "Pin_Headers:Pin_Header_Straight_1x04" H 1800 2800 60  0001 C CNN
-F 3 "" H 1800 2800 60  0000 C CNN
-F 4 "-" H 350 1550 50  0001 C CNN "MPN"
-	1    1800 2800
+P 1800 2850
+F 0 "P1" H 1800 3100 50  0000 C CNN
+F 1 "CHAIN" V 1900 2850 50  0000 C CNN
+F 2 "Pin_Headers:Pin_Header_Straight_1x03" H 1800 2850 60  0001 C CNN
+F 3 "" H 1800 2850 60  0000 C CNN
+F 4 "-" H 350 1600 50  0001 C CNN "MPN"
+	1    1800 2850
 	-1   0    0    1
 $EndComp
@@
 F 0 "R6" V 9750 2150 50  0000 C CNN
 F 1 "10k" V 9650 2150 50  0000 C CNN
-F 2 "Resistors_SMD:R_0603" V 9580 2150 30  0000 C CNN
+F 2 "Resistors_SMD:R_0603" V 9580 2150 30  0001 C CNN
 F 3 "" H 9650 2150 30  0000 C CNN
 F 4 "RMCF0603JT10K0" H -350 650 50  0001 C CNN "MPN"
@@
 F 0 "SW1" H 9400 2910 50  0000 C CNN
 F 1 "SW_PUSH" H 9250 2720 50  0000 C CNN
-F 2 "Buttons_Switches_SMD:SW_SPST_FSMSM" H 9250 2800 60  0000 C CNN
+F 2 "Buttons_Switches_SMD:SW_SPST_FSMSM" H 9250 2800 60  0001 C CNN
 F 3 "" H 9250 2800 60  0000 C CNN
 F 4 "FSMSM" H -350 650 50  0001 C CNN "MPN"
@@
 Text GLabel 2150 2750 2    50   Output ~ 0
 CHAIN_RX
-Text GLabel 2150 2650 2    50   Input ~ 0
-CHAIN_DE
 Text GLabel 9750 4600 2    50   Output ~ 0
 SWO
@@
 Text GLabel 7500 2650 2    50   Input ~ 0
 FS1
-Text GLabel 7500 4350 2    50   Output ~ 0
-RX_LED_CPU
-Text GLabel 7500 4450 2    50   Output ~ 0
-TX_LED_CPU
-Text GLabel 7500 3050 2    50   Output ~ 0
-LEDS_SDA
-Text GLabel 7500 2950 2    50   Output ~ 0
-LEDS_SCL
-Text GLabel 7500 3250 2    50   Output ~ 0
-LEDS_OE
-Text GLabel 3600 3550 0    50   Input ~ 0
+Text GLabel 7500 2750 2    50   Input ~ 0
 FS2
-Text GLabel 3600 3650 0    50   Input ~ 0
+Text GLabel 7500 2950 2    50   Input ~ 0
 FS3
-Text GLabel 3600 3750 0    50   Input ~ 0
+Text GLabel 7500 3050 2    50   Input ~ 0
 FS4
 Text GLabel 7500 3650 2    50   BiDi ~ 0
@@
 	2150 2750 2000 2750
 Wire Wire Line
-	2000 2650 2150 2650
-Wire Wire Line
 	2000 2950 2050 2950
 Wire Wire Line
@@
 	7350 2650 7500 2650
 Wire Wire Line
-	7500 4350 7350 4350
-Wire Wire Line
-	7500 4450 7350 4450
-Wire Wire Line
-	7350 2950 7500 2950
+	7500 2750 7350 2750
+Wire Wire Line
+	7500 2950 7350 2950
 Wire Wire Line
 	7500 3050 7350 3050
-Wire Wire Line
-	7500 3250 7350 3250
-Wire Wire Line
-	3750 3550 3600 3550
-Wire Wire Line
-	3750 3650 3600 3650
-Wire Wire Line
-	3750 3750 3600 3750
 Wire Wire Line
 	7500 3650 7350 3650
@@
 NoConn ~ 9050 4400
 NoConn ~ 9550 4700
-NoConn ~ 3750 3350
-NoConn ~ 3750 3850
-NoConn ~ 7350 2750
-NoConn ~ 3750 2950
-NoConn ~ 3750 3950
-NoConn ~ 3750 4050
 NoConn ~ 3750 4150
-NoConn ~ 3750 3450
-NoConn ~ 3750 3050
-NoConn ~ 3750 3150
-NoConn ~ 3750 3250
+Text GLabel 3600 3050 0    50   Output ~ 0
+LED_R1
+Text GLabel 3600 3150 0    50   Output ~ 0
+LED_G1
+Text GLabel 3600 2950 0    50   Output ~ 0
+LED_B1
+Text GLabel 3600 3350 0    50   Output ~ 0
+LED_R2
+Text GLabel 3600 3450 0    50   Output ~ 0
+LED_G2
+Text GLabel 3600 3250 0    50   Output ~ 0
+LED_B2
+Text GLabel 3600 3650 0    50   Output ~ 0
+LED_R3
+Text GLabel 3600 3750 0    50   Output ~ 0
+LED_G3
+Text GLabel 3600 3550 0    50   Output ~ 0
+LED_B3
+Text GLabel 3600 3950 0    50   Output ~ 0
+LED_R4
+Text GLabel 3600 4050 0    50   Output ~ 0
+LED_G4
+Text GLabel 3600 3850 0    50   Output ~ 0
+LED_B4
+$Comp
+L LPC11U24FBD48/401 U4
+U 1 1 556F3A3A
+P 5550 3750
+F 0 "U4" H 4050 5150 50  0000 C CNN
+F 1 "LPC11U24FBD48/401" H 6750 5150 50  0000 C CNN
+F 2 "Housings_QFP:LQFP-48_7x7mm_Pitch0.5mm" H 5550 2650 50  0000 C CNN
+F 3 "" H 5500 3700 60  0000 C CNN
+F 4 "LPC11U24FBD48/401" H -350 650 50  0001 C CNN "MPN"
+	1    5550 3750
+	1    0    0    -1
+$EndComp
+Wire Wire Line
+	3600 2950 3750 2950
+Wire Wire Line
+	3600 3050 3750 3050
+Wire Wire Line
+	3750 3150 3600 3150
+Wire Wire Line
+	3600 3250 3750 3250
+Wire Wire Line
+	3600 3350 3750 3350
+Wire Wire Line
+	3750 3450 3600 3450
+Wire Wire Line
+	3600 3550 3750 3550
+Wire Wire Line
+	3750 3650 3600 3650
+Wire Wire Line
+	3600 3750 3750 3750
+Wire Wire Line
+	3750 3850 3600 3850
+Wire Wire Line
+	3600 3950 3750 3950
+Wire Wire Line
+	3750 4050 3600 4050
+NoConn ~ 7350 4350
+NoConn ~ 7350 4450
+NoConn ~ 7350 3250
 $EndSCHEMATC

Commit message: annotation and ERC
Parts:
- renumbered C11 to C12, C12 to C13, C13 to C21, C9 to C4, C10 to C6, P1 to P3, P2 to P9, R6 to R36, U4 to U3
Changed lines of the file:
@@
 $EndDescr
 $Comp
-L GNDD #PWR033
+L GNDD #PWR74
 U 1 1 54E5DFA7
 P 8850 4900
-F 0 "#PWR033" H 8850 4650 60  0001 C CNN
+F 0 "#PWR74" H 8850 4650 60  0001 C CNN
 F 1 "GNDD" H 8850 4750 60  0000 C CNN
 F 2 "" H 8850 4900 60  0000 C CNN
@@
 $EndComp
 $Comp
-L CONN_02X05 P2
+L CONN_02X05 P9
 U 1 1 54F2A3AF
 P 9300 4600
-F 0 "P2" H 9300 4900 50  0000 C CNN
+F 0 "P9" H 9300 4900 50  0000 C CNN
 F 1 "SWD" H 9300 4300 50  0000 C CNN
 F 2 "Pin_Headers:Pin_Header_Straight_2x05_Pitch1.27mm" H 9300 3400 60  0001 C CNN
@@
 $EndComp
 $Comp
-L C C10
+L C C6
 U 1 1 556F5E37
 P 3200 5050
-F 0 "C10" H 3225 5150 50  0000 L CNN
+F 0 "C6" H 3225 5150 50  0000 L CNN
 F 1 "18pF" H 3225 4950 50  0000 L CNN
 F 2 "Capacitors_SMD:C_0603" H 3238 4900 30  0001 C CNN
@@
 $EndComp
 $Comp
-L C C9
+L C C4
 U 1 1 556F5E74
 P 2950 5050
-F 0 "C9" H 2975 5150 50  0000 L CNN
+F 0 "C4" H 2975 5150 50  0000 L CNN
 F 1 "18pF" H 2975 4950 50  0000 L CNN
 F 2 "Capacitors_SMD:C_0603" H 2988 4900 30  0001 C CNN
@@
 $EndComp
 $Comp
-L GNDD #PWR034
+L GNDD #PWR24
 U 1 1 556F6417
 P 2950 5250
-F 0 "#PWR034" H 2950 5000 50  0001 C CNN
+F 0 "#PWR24" H 2950 5000 50  0001 C CNN
 F 1 "GNDD" H 2950 5100 50  0000 C CNN
 F 2 "" H 2950 5250 60  0000 C CNN
@@
 $EndComp
 $Comp
-L GNDD #PWR035
+L GNDD #PWR28
 U 1 1 556F65EC
 P 3200 5250
-F 0 "#PWR035" H 3200 5000 50  0001 C CNN
+F 0 "#PWR28" H 3200 5000 50  0001 C CNN
 F 1 "GNDD" H 3200 5100 50  0000 C CNN
 F 2 "" H 3200 5250 60  0000 C CNN
@@
 $EndComp
 $Comp
-L +3.3V #PWR036
+L +3.3V #PWR47
 U 1 1 55705A80
 P 5550 1500
-F 0 "#PWR036" H 5550 1350 50  0001 C CNN
+F 0 "#PWR47" H 5550 1350 50  0001 C CNN
 F 1 "+3.3V" H 5550 1640 50  0000 C CNN
 F 2 "" H 5550 1500 60  0000 C CNN
@@
 $EndComp
 $Comp
-L C C11
+L C C12
 U 1 1 557DBC57
 P 5250 1850
-F 0 "C11" V 5300 1650 40  0000 L CNN
+F 0 "C12" V 5300 1650 40  0000 L CNN
 F 1 "100nF X7R" V 5100 1700 40  0000 L CNN
 F 2 "Capacitors_SMD:C_0603" H 5288 1700 30  0001 C CNN
@@
 $EndComp
 $Comp
-L C C12
+L C C13
 U 1 1 557DBEEF
 P 5850 1850
-F 0 "C12" V 5900 1650 40  0000 L CNN
+F 0 "C13" V 5900 1650 40  0000 L CNN
 F 1 "100nF X7R" V 6000 1700 40  0000 L CNN
 F 2 "Capacitors_SMD:C_0603" H 5888 1700 30  0001 C CNN
@@
 $EndComp
 $Comp
-L GNDD #PWR037
+L GNDD #PWR46
 U 1 1 557DC875
 P 5250 2100
-F 0 "#PWR037" H 5250 1850 50  0001 C CNN
+F 0 "#PWR46" H 5250 1850 50  0001 C CNN
 F 1 "GNDD" H 5250 1950 50  0000 C CNN
 F 2 "" H 5250 2100 60  0000 C CNN
@@
 $EndComp
 $Comp
-L GNDD #PWR038
+L GNDD #PWR49
 U 1 1 557DCAD9
 P 5850 2100
-F 0 "#PWR038" H 5850 1850 50  0001 C CNN
+F 0 "#PWR49" H 5850 1850 50  0001 C CNN
 F 1 "GNDD" H 5850 1950 50  0000 C CNN
 F 2 "" H 5850 2100 60  0000 C CNN
@@
 $EndComp
 $Comp
-L GNDD #PWR039
+L GNDD #PWR48
 U 1 1 557DD01E
 P 5550 5400
-F 0 "#PWR039" H 5550 5150 50  0001 C CNN
+F 0 "#PWR48" H 5550 5150 50  0001 C CNN
 F 1 "GNDD" H 5550 5250 50  0000 C CNN
 F 2 "" H 5550 5400 60  0000 C CNN
@@
 $EndComp
 $Comp
-L CONN_01X03 P1
+L CONN_01X03 P3
 U 1 1 557F309A
 P 1800 2850
-F 0 "P1" H 1800 3100 50  0000 C CNN
+F 0 "P3" H 1800 3100 50  0000 C CNN
 F 1 "CHAIN" V 1900 2850 50  0000 C CNN
 F 2 "Pin_Headers:Pin_Header_Straight_1x03" H 1800 2850 60  0001 C CNN
@@
 $EndComp
 $Comp
-L GNDD #PWR040
+L GNDD #PWR6
 U 1 1 557F3440
 P 2050 3000
-F 0 "#PWR040" H 2050 2750 50  0001 C CNN
+F 0 "#PWR6" H 2050 2750 50  0001 C CNN
 F 1 "GNDD" H 2050 2850 50  0000 C CNN
 F 2 "" H 2050 3000 60  0000 C CNN
@@
 $EndComp
 $Comp
-L R R6
+L R R36
 U 1 1 558018EB
 P 9650 2150
-F 0 "R6" V 9750 2150 50  0000 C CNN
+F 0 "R36" V 9750 2150 50  0000 C CNN
 F 1 "10k" V 9650 2150 50  0000 C CNN
 F 2 "Resistors_SMD:R_0603" V 9580 2150 30  0001 C CNN
@@
 $EndComp
 $Comp
-L +3.3V #PWR041
+L +3.3V #PWR80
 U 1 1 55802FA1
 P 9650 1900
-F 0 "#PWR041" H 9650 1750 50  0001 C CNN
+F 0 "#PWR80" H 9650 1750 50  0001 C CNN
 F 1 "+3.3V" H 9650 2040 50  0000 C CNN
 F 2 "" H 9650 1900 60  0000 C CNN
@@
 $EndComp
 $Comp
-L GNDD #PWR042
+L GNDD #PWR81
 U 1 1 55803C49
 P 9650 2900
-F 0 "#PWR042" H 9650 2650 50  0001 C CNN
+F 0 "#PWR81" H 9650 2650 50  0001 C CNN
 F 1 "GNDD" H 9650 2750 50  0000 C CNN
 F 2 "" H 9650 2900 60  0000 C CNN
@@
 $EndComp
 $Comp
-L C C13
+L C C21
 U 1 1 55804D28
 P 9650 2650
-F 0 "C13" V 9700 2500 40  0000 L CNN
+F 0 "C21" V 9700 2500 40  0000 L CNN
 F 1 "100nF X7R" V 9500 2500 40  0000 L CNN
 F 2 "Capacitors_SMD:C_0603" H 9688 2500 30  0001 C CNN
@@
 $EndComp
 $Comp
-L GNDD #PWR043
+L GNDD #PWR76
 U 1 1 55806665
 P 9250 3200
-F 0 "#PWR043" H 9250 2950 50  0001 C CNN
+F 0 "#PWR76" H 9250 2950 50  0001 C CNN
 F 1 "GNDD" H 9250 3050 50  0000 C CNN
 F 2 "" H 9250 3200 60  0000 C CNN
@@
 LED_B4
 $Comp
-L LPC11U24FBD48/401 U4
+L LPC11U24FBD48/401 U3
 U 1 1 556F3A3A
 P 5550 3750
-F 0 "U4" H 4050 5150 50  0000 C CNN
+F 0 "U3" H 4050 5150 50  0000 C CNN
 F 1 "LPC11U24FBD48/401" H 6750 5150 50  0000 C CNN
 F 2 "Housings_QFP:LQFP-48_7x7mm_Pitch0.5mm" H 5550 2650 50  0000 C CNN

Commit message: replace reset button by pin header
Parts:
- removed SW1: SW_PUSH, Buttons_Switches_SMD:SW_SPST_FSMSM, symbol SW_PUSH
- added P10: CPU_RESET, Pin_Headers:Pin_Header_Straight_1x02, symbol CONN_01X02
Connections:
- net GNDD: now also P10.2 (P2)
- net RESET: now also P10.1 (P1)
Other:
- moved on the sheet: C21, R36

Commit message: fix usb resistors
Connections:
- net CHAIN_DE: now also U3.40 (PIO0_16/AD5/CT32B1_MAT3/WAKEUP); no longer U3.43 (PIO1_15/~DCD~/CT16B0_MAT2/SCK1)
- net LCD1_BL: now also U3.43 (PIO1_15/~DCD~/CT16B0_MAT2/SCK1); no longer U3.40 (PIO0_16/AD5/CT32B1_MAT3/WAKEUP)
Changed lines of the file:
@@
 Text GLabel 3600 2750 0    50   Input ~ 0
 CHAIN_RX
-Text GLabel 3600 2850 0    50   Output ~ 0
+Text GLabel 7500 4150 2    50   Output ~ 0
 CHAIN_DE
 Text GLabel 2150 2850 2    50   Input ~ 0
@@
 Text GLabel 7500 4850 2    50   Output ~ 0
 LCD2_EN
-Text GLabel 7500 4150 2    50   Output ~ 0
+Text GLabel 3600 2850 0    50   Output ~ 0
 LCD1_BL
 Text GLabel 7500 4250 2    50   Output ~ 0
@@
 	3600 2750 3750 2750
 Wire Wire Line
-	3750 2850 3600 2850
+	7350 4150 7500 4150
 Wire Wire Line
 	2000 2850 2150 2850
@@
 	7350 3350 7500 3350
 Wire Wire Line
-	7500 4150 7350 4150
+	3600 2850 3750 2850
 Wire Wire Line
 	7350 4250 7500 4250
