File: hw-design/board/cpu.sch (KiCad schematic (older format))
At the start: 11 parts, among them P10 CPU_RESET, P3 CHAIN, P9 SWD, U3 LPC11U24FBD48/401, Y1 12MHz

Commit message: use fixed contrast to displays
Parts:
- renumbered C12 to C13, C13 to C14, R36 to R37
Connections:
- net labels removed: LCD_CONTRAST
- wire segments 80 -> 79
- no-connect marks 7 -> 8
Changed lines of the file:
@@
 $EndDescr
 $Comp
-L GNDD #PWR74
+L GNDD #PWR70
 U 1 1 54E5DFA7
 P 8850 4900
-F 0 "#PWR74" H 8850 4650 60  0001 C CNN
+F 0 "#PWR70" H 8850 4650 60  0001 C CNN
 F 1 "GNDD" H 8850 4750 60  0000 C CNN
 F 2 "" H 8850 4900 60  0000 C CNN
@@
 $EndComp
 $Comp
-L GNDD #PWR24
+L GNDD #PWR22
 U 1 1 556F6417
 P 2950 5250
-F 0 "#PWR24" H 2950 5000 50  0001 C CNN
+F 0 "#PWR22" H 2950 5000 50  0001 C CNN
 F 1 "GNDD" H 2950 5100 50  0000 C CNN
 F 2 "" H 2950 5250 60  0000 C CNN
@@
 $EndComp
 $Comp
-L GNDD #PWR28
+L GNDD #PWR27
 U 1 1 556F65EC
 P 3200 5250
-F 0 "#PWR28" H 3200 5000 50  0001 C CNN
+F 0 "#PWR27" H 3200 5000 50  0001 C CNN
 F 1 "GNDD" H 3200 5100 50  0000 C CNN
 F 2 "" H 3200 5250 60  0000 C CNN
@@
 $EndComp
 $Comp
-L +3.3V #PWR47
+L +3.3V #PWR45
 U 1 1 55705A80
 P 5550 1500
-F 0 "#PWR47" H 5550 1350 50  0001 C CNN
+F 0 "#PWR45" H 5550 1350 50  0001 C CNN
 F 1 "+3.3V" H 5550 1640 50  0000 C CNN
 F 2 "" H 5550 1500 60  0000 C CNN
@@
 $EndComp
 $Comp
-L C C12
+L C C13
 U 1 1 557DBC57
 P 5250 1850
-F 0 "C12" V 5300 1650 40  0000 L CNN
+F 0 "C13" V 5300 1650 40  0000 L CNN
 F 1 "100nF" V 5100 1700 40  0000 L CNN
 F 2 "Capacitors_SMD:C_0603" H 5288 1700 30  0001 C CNN
@@
 $EndComp
 $Comp
-L C C13
+L C C14
 U 1 1 557DBEEF
 P 5850 1850
-F 0 "C13" V 5900 1650 40  0000 L CNN
+F 0 "C14" V 5900 1650 40  0000 L CNN
 F 1 "100nF" V 6000 1700 40  0000 L CNN
 F 2 "Capacitors_SMD:C_0603" H 5888 1700 30  0001 C CNN
@@
 $EndComp
 $Comp
-L GNDD #PWR46
+L GNDD #PWR44
 U 1 1 557DC875
 P 5250 2100
-F 0 "#PWR46" H 5250 1850 50  0001 C CNN
+F 0 "#PWR44" H 5250 1850 50  0001 C CNN
 F 1 "GNDD" H 5250 1950 50  0000 C CNN
 F 2 "" H 5250 2100 60  0000 C CNN
@@
 $EndComp
 $Comp
-L GNDD #PWR49
+L GNDD #PWR47
 U 1 1 557DCAD9
 P 5850 2100
-F 0 "#PWR49" H 5850 1850 50  0001 C CNN
+F 0 "#PWR47" H 5850 1850 50  0001 C CNN
 F 1 "GNDD" H 5850 1950 50  0000 C CNN
 F 2 "" H 5850 2100 60  0000 C CNN
@@
 $EndComp
 $Comp
-L GNDD #PWR48
+L GNDD #PWR46
 U 1 1 557DD01E
 P 5550 5400
-F 0 "#PWR48" H 5550 5150 50  0001 C CNN
+F 0 "#PWR46" H 5550 5150 50  0001 C CNN
 F 1 "GNDD" H 5550 5250 50  0000 C CNN
 F 2 "" H 5550 5400 60  0000 C CNN
@@
 $EndComp
 $Comp
-L R R36
+L R R37
 U 1 1 558018EB
 P 9300 2150
-F 0 "R36" V 9400 2150 50  0000 C CNN
+F 0 "R37" V 9400 2150 50  0000 C CNN
 F 1 "10K" V 9300 2150 50  0000 C CNN
 F 2 "Resistors_SMD:R_0603" V 9230 2150 30  0001 C CNN
@@
 $EndComp
 $Comp
-L +3.3V #PWR79
+L +3.3V #PWR72
 U 1 1 55802FA1
 P 9300 1900
-F 0 "#PWR79" H 9300 1750 50  0001 C CNN
+F 0 "#PWR72" H 9300 1750 50  0001 C CNN
 F 1 "+3.3V" H 9300 2040 50  0000 C CNN
 F 2 "" H 9300 1900 60  0000 C CNN
@@
 $EndComp
 $Comp
-L GNDD #PWR80
+L GNDD #PWR73
 U 1 1 55803C49
 P 9300 2900
-F 0 "#PWR80" H 9300 2650 50  0001 C CNN
+F 0 "#PWR73" H 9300 2650 50  0001 C CNN
 F 1 "GNDD" H 9300 2750 50  0000 C CNN
 F 2 "" H 9300 2900 60  0000 C CNN
@@
 $EndComp
 $Comp
-L GNDD #PWR82
+L GNDD #PWR77
 U 1 1 55806665
 P 9650 2650
-F 0 "#PWR82" H 9650 2400 50  0001 C CNN
+F 0 "#PWR77" H 9650 2400 50  0001 C CNN
 F 1 "GNDD" H 9650 2500 50  0000 C CNN
 F 2 "" H 9650 2650 60  0000 C CNN
@@
 Text GLabel 7500 4350 2    50   Output ~ 0
 LCD2_BL
-Text GLabel 7500 4850 2    50   Output ~ 0
-LCD_CONTRAST
 NoConn ~ 9050 4700
 NoConn ~ 9050 4400
@@
 	7500 4450 7350 4450
 Wire Wire Line
-	7350 4850 7500 4850
-Wire Wire Line
 	3600 3550 3750 3550
 Wire Wire Line
@@
 $EndComp
 NoConn ~ 3750 3050
+NoConn ~ 7350 4850
 $EndSCHEMATC

Commit message: only trigger isp when usb is connected
Connections:
- net labels added: ISP_TRIGGER
- wire segments 79 -> 80
- no-connect marks 8 -> 7
Changed lines of the file:
@@
 Text GLabel 7500 3450 2    50   Output ~ 0
 SWO
-Text GLabel 7500 2650 2    50   Input ~ 0
+Text GLabel 7500 3250 2    50   Input ~ 0
 FS1
 Text GLabel 3600 3950 0    50   Input ~ 0
@@
 LED_B4
 NoConn ~ 3750 3350
-NoConn ~ 7350 3250
 NoConn ~ 3750 3650
 $Comp
@@
 	7500 3450 7350 3450
 Wire Wire Line
-	7350 2650 7500 2650
+	7350 3250 7500 3250
 Wire Wire Line
 	3600 3950 3750 3950
@@
 NoConn ~ 3750 3050
 NoConn ~ 7350 4850
+Text GLabel 7500 2650 2    50   Input ~ 0
+ISP_TRIGGER
+Wire Wire Line
+	7350 2650 7500 2650
 $EndSCHEMATC

Commit message: update netlist
Parts:
- renumbered R37 to R39
Changed lines of the file:
@@
 $EndDescr
 $Comp
-L GNDD #PWR70
+L GNDD #PWR72
 U 1 1 54E5DFA7
 P 8850 4900
-F 0 "#PWR70" H 8850 4650 60  0001 C CNN
+F 0 "#PWR72" H 8850 4650 60  0001 C CNN
 F 1 "GNDD" H 8850 4750 60  0000 C CNN
 F 2 "" H 8850 4900 60  0000 C CNN
@@
 $EndComp
 $Comp
-L GNDD #PWR22
+L GNDD #PWR24
 U 1 1 556F6417
 P 2950 5250
-F 0 "#PWR22" H 2950 5000 50  0001 C CNN
+F 0 "#PWR24" H 2950 5000 50  0001 C CNN
 F 1 "GNDD" H 2950 5100 50  0000 C CNN
 F 2 "" H 2950 5250 60  0000 C CNN
@@
 $EndComp
 $Comp
-L GNDD #PWR27
+L GNDD #PWR29
 U 1 1 556F65EC
 P 3200 5250
-F 0 "#PWR27" H 3200 5000 50  0001 C CNN
+F 0 "#PWR29" H 3200 5000 50  0001 C CNN
 F 1 "GNDD" H 3200 5100 50  0000 C CNN
 F 2 "" H 3200 5250 60  0000 C CNN
@@
 $EndComp
 $Comp
-L +3.3V #PWR45
+L +3.3V #PWR47
 U 1 1 55705A80
 P 5550 1500
-F 0 "#PWR45" H 5550 1350 50  0001 C CNN
+F 0 "#PWR47" H 5550 1350 50  0001 C CNN
 F 1 "+3.3V" H 5550 1640 50  0000 C CNN
 F 2 "" H 5550 1500 60  0000 C CNN
@@
 $EndComp
 $Comp
-L GNDD #PWR44
+L GNDD #PWR46
 U 1 1 557DC875
 P 5250 2100
-F 0 "#PWR44" H 5250 1850 50  0001 C CNN
+F 0 "#PWR46" H 5250 1850 50  0001 C CNN
 F 1 "GNDD" H 5250 1950 50  0000 C CNN
 F 2 "" H 5250 2100 60  0000 C CNN
@@
 $EndComp
 $Comp
-L GNDD #PWR47
+L GNDD #PWR49
 U 1 1 557DCAD9
 P 5850 2100
-F 0 "#PWR47" H 5850 1850 50  0001 C CNN
+F 0 "#PWR49" H 5850 1850 50  0001 C CNN
 F 1 "GNDD" H 5850 1950 50  0000 C CNN
 F 2 "" H 5850 2100 60  0000 C CNN
@@
 $EndComp
 $Comp
-L GNDD #PWR46
+L GNDD #PWR48
 U 1 1 557DD01E
 P 5550 5400
-F 0 "#PWR46" H 5550 5150 50  0001 C CNN
+F 0 "#PWR48" H 5550 5150 50  0001 C CNN
 F 1 "GNDD" H 5550 5250 50  0000 C CNN
 F 2 "" H 5550 5400 60  0000 C CNN
@@
 $EndComp
 $Comp
-L R R37
+L R R39
 U 1 1 558018EB
 P 9300 2150
-F 0 "R37" V 9400 2150 50  0000 C CNN
+F 0 "R39" V 9400 2150 50  0000 C CNN
 F 1 "10K" V 9300 2150 50  0000 C CNN
 F 2 "Resistors_SMD:R_0603" V 9230 2150 30  0001 C CNN
@@
 $EndComp
 $Comp
-L +3.3V #PWR72
+L +3.3V #PWR74
 U 1 1 55802FA1
 P 9300 1900
-F 0 "#PWR72" H 9300 1750 50  0001 C CNN
+F 0 "#PWR74" H 9300 1750 50  0001 C CNN
 F 1 "+3.3V" H 9300 2040 50  0000 C CNN
 F 2 "" H 9300 1900 60  0000 C CNN
@@
 $EndComp
 $Comp
-L GNDD #PWR73
+L GNDD #PWR75
 U 1 1 55803C49
 P 9300 2900
-F 0 "#PWR73" H 9300 2650 50  0001 C CNN
+F 0 "#PWR75" H 9300 2650 50  0001 C CNN
 F 1 "GNDD" H 9300 2750 50  0000 C CNN
 F 2 "" H 9300 2900 60  0000 C CNN
@@
 $EndComp
 $Comp
-L GNDD #PWR77
+L GNDD #PWR79
 U 1 1 55806665
 P 9650 2650
-F 0 "#PWR77" H 9650 2400 50  0001 C CNN
+F 0 "#PWR79" H 9650 2400 50  0001 C CNN
 F 1 "GNDD" H 9650 2500 50  0000 C CNN
 F 2 "" H 9650 2650 60  0000 C CNN
