File: hw-design/board/io.sch (KiCad schematic (older format))
At the start: 24 parts

Commit message: importing common sheets from expression-pedal project
Parts:
- removed FOOT1, FOOT2, FOOT3, FOOT4: HEADER_2X1_180, MOD_Footprints_Lib:PIN_ARRAY_2X1, symbol CONN_2
- removed LED1, LED2, LED3, LED4: LED_RGB, MOD_Footprints_Lib:LED_CLRTB_GFSF_1, symbol LED_RGB
- removed R10, R7, R8, R9: 10k, MOD_Footprints_Lib:SM0603, symbol R
- removed R14, R15, R16, R17, R18, R19, R20, R21: 1k, MOD_Footprints_Lib:SM0603, symbol R
- added C17, C18: 100nF X7R, Capacitors_SMD:C_0603, symbol C
- added D5: LED_RGB, LEDs:LED_RGB_PLLC-6, symbol LED_RGB
- added P4: FOOT, Pin_Headers:Pin_Header_Straight_1x02, symbol CONN_01X02
- added P5: 10K POT, Pin_Headers:Pin_Header_Straight_1x03, symbol CONN_01X03
- added R26, R27, R28: 100R, Resistors_SMD:R_0603, symbol R
- added R29, R30, R31: 10k, Resistors_SMD:R_0603, symbol R
- added SW2: SP3T, local-footprints:OS103011MA7QP1, symbol SP3T
- R22, R23, R24: value 1k -> 220R; footprint MOD_Footprints_Lib:SM0603 -> Resistors_SMD:R_0603; MPN (none) -> ESR03EZPJ221
- R25: value 1k -> 10k; footprint MOD_Footprints_Lib:SM0603 -> Resistors_SMD:R_0603; MPN (none) -> RMCF0603JT10K0
Connections:
- net labels added: CH1, CH2, CH3, FS1, FS1_LED_B, FS1_LED_G, FS1_LED_R, GNDD, POT
- net labels removed: DGND, FOOT_1, FOOT_2, FOOT_3, FOOT_4, LED1_B, LED1_G, LED1_R, LED2_B, LED2_G, LED2_R, LED3_B, LED3_G, LED3_R, LED4_B, LED4_G, LED4_R
- wire segments 59 -> 44
Other:
- note added: "CHANNEL SELECTOR"
- note added: "FOOT"
- note added: "LED"
- note added: "PEDAL"

Commit message: sch: schematic updated (missing displays circuit)
Parts:
- removed P5: 10K POT, Pin_Headers:Pin_Header_Straight_1x03, symbol CONN_01X03
- removed R26: 100R, Resistors_SMD:R_0603, symbol R
- added C19, C20: 100nF X7R, Capacitors_SMD:C_0603, symbol C
- added D6, D7, D8: LED_RGB, LEDs:LED_RGB_PLLC-6, symbol LED_RGB
- added P5, P6, P7: FOOT, Pin_Headers:Pin_Header_Straight_1x02, symbol CONN_01X02
- added R23: 10k, Resistors_SMD:R_0603, symbol R
- added R32, R33, R34, R35, R36, R37, R38, R39, R40: 220R, Resistors_SMD:R_0603, symbol R
- added U5: PCA9685, TSSOP28, symbol PCA9685
- R27, R28: value 100R -> 10k; MPN RMCF0603JT100R -> RMCF0603JT10K0
- renumbered R25 to R22, R29 to R24, R30 to R25, R31 to R26, R22 to R29, R23 to R30, R24 to R31
Connections:
- net +3V3: now also R27.1, R28.1, C19.2, C20.2, D6.BA (BLUE_ANODE), D6.GA (GREEN_ANODE), D6.RA (RED_ANODE), D7.BA (BLUE_ANODE), D7.GA (GREEN_ANODE), D7.RA (RED_ANODE), D8.BA (BLUE_ANODE), D8.GA (GREEN_ANODE), D8.RA (RED_ANODE), R23.1, U5.1 (A0), U5.28 (VDD)
- net GNDD: now also C19.1, C20.1, P5.2 (P2), P6.2 (P2), P7.2 (P2), U5.14 (VSS), U5.2 (A1), U5.24 (A5), U5.25 (EXTCLK), U5.3 (A2), U5.4 (A3), U5.5 (A4); no longer R27.2
- net FS1_LED_B: no longer names the net of R31.1
- net FS1_LED_B: now also U5.8 (LED2)
- net FS1_LED_G: no longer names the net of R30.1
- net FS1_LED_G: now also U5.7 (LED1)
- net FS1_LED_R: no longer names the net of R29.1
- net FS1_LED_R: now also U5.6 (LED0)
- net POT renamed FS4
- net FS4: now also P7.1 (P1)
- new net: R32.1, U5.10 (LED4)
- new net: R33.1, U5.11 (LED5)
- new net: R34.1, U5.12 (LED6)
- new net: R35.1, U5.15 (LED8)
- new net: R36.1, U5.16 (LED9)
- new net: R37.1, U5.17 (LED10)
- new net: R38.1, U5.19 (LED12)
- new net: R39.1, U5.20 (LED13)
- new net: R40.1, U5.21 (LED14)
- new net: D6.RC (RED_CATHODE), R32.2
- new net: D6.BC (BLUE_CATHODE), R34.2
- new net: D6.GC (GREEN_CATHODE), R33.2
- new net: D7.RC (RED_CATHODE), R35.2
- new net: D7.BC (BLUE_CATHODE), R37.2
- new net: D7.GC (GREEN_CATHODE), R36.2
- new net: D8.RC (RED_CATHODE), R38.2
- new net: D8.BC (BLUE_CATHODE), R40.2
- new net: D8.GC (GREEN_CATHODE), R39.2
- new net FS2: P6.1 (P1), R27.2
- new net FS3: P5.1 (P1), R23.2
- new net LEDS_OE: U5.23 (~OE~)
- new net LEDS_SCL: U5.26 (SCL)
- new net LEDS_SDA: U5.27 (SDA)
- no-connect marks 0 -> 4
Other:
- note added: "FOOTSWITCHES"
- note added: "LEDs"
- note removed: "FOOT"
- note removed: "LED"
- note removed: "PEDAL"
- moved on the sheet: C17, D5, P4, R22, R24, R25, R26, R29, R30, R31, SW2

Commit message: sch: MPN added to all components
Parts:
- U5: footprint TSSOP28 -> Housings_SSOP:TSSOP-28_4.4x9.7mm_Pitch0.65mm; MPN (none) -> PCA9685PW,112

Commit message: sch: fixing VBUS signal and FS1 I/O
Parts:
- renumbered R22 to R23, R23 to R24, R24 to R25, R25 to R26, R26 to R27, R27 to R28, R28 to R29, R29 to R30, R30 to R31, R31 to R32, R32 to R33, R33 to R34, R34 to R35, R35 to R36, R36 to R37, R37 to R38, R38 to R39, R39 to R40, R40 to R41
Changed lines of the file:
@@
 $EndDescr
 $Comp
-L R R24
+L R R25
 U 1 1 54CBEC23
 P 2050 1700
-F 0 "R24" V 2100 1950 40  0000 C CNN
+F 0 "R25" V 2100 1950 40  0000 C CNN
 F 1 "10k" V 2057 1701 40  0000 C CNN
 F 2 "Resistors_SMD:R_0603" V 1980 1700 30  0001 C CNN
@@
 $EndComp
 $Comp
-L R R25
+L R R26
 U 1 1 54CBEC30
 P 2200 1700
-F 0 "R25" V 2250 1950 40  0000 C CNN
+F 0 "R26" V 2250 1950 40  0000 C CNN
 F 1 "10k" V 2207 1701 40  0000 C CNN
 F 2 "Resistors_SMD:R_0603" V 2130 1700 30  0001 C CNN
@@
 $EndComp
 $Comp
-L R R26
+L R R27
 U 1 1 54CBEC37
 P 2350 1700
-F 0 "R26" V 2400 1950 40  0000 C CNN
+F 0 "R27" V 2400 1950 40  0000 C CNN
 F 1 "10k" V 2357 1701 40  0000 C CNN
 F 2 "Resistors_SMD:R_0603" V 2280 1700 30  0001 C CNN
@@
 $EndComp
 $Comp
-L R R22
+L R R23
 U 1 1 54CBEC53
 P 1650 3950
-F 0 "R22" V 1730 3950 40  0000 C CNN
+F 0 "R23" V 1730 3950 40  0000 C CNN
 F 1 "10k" V 1657 3951 40  0000 C CNN
 F 2 "Resistors_SMD:R_0603" V 1580 3950 30  0001 C CNN
@@
 $EndComp
 $Comp
-L GNDD #PWR060
+L GNDD #PWR58
 U 1 1 54E65047
 P 1650 4450
-F 0 "#PWR060" H 1650 4200 60  0001 C CNN
+F 0 "#PWR58" H 1650 4200 60  0001 C CNN
 F 1 "GNDD" H 1650 4300 60  0000 C CNN
 F 2 "" H 1650 4450 60  0000 C CNN
@@
 $EndComp
 $Comp
-L GNDD #PWR061
+L GNDD #PWR56
 U 1 1 54E753B2
 P 1150 2150
-F 0 "#PWR061" H 1150 1900 60  0001 C CNN
+F 0 "#PWR56" H 1150 1900 60  0001 C CNN
 F 1 "GNDD" H 1150 2000 60  0000 C CNN
 F 2 "" H 1150 2150 60  0000 C CNN
@@
 $EndComp
 $Comp
-L +3.3V #PWR062
+L +3.3V #PWR57
 U 1 1 556F3C3C
 P 1650 3700
-F 0 "#PWR062" H 1650 3550 50  0001 C CNN
+F 0 "#PWR57" H 1650 3550 50  0001 C CNN
 F 1 "+3.3V" H 1650 3840 50  0000 C CNN
 F 2 "" H 1650 3700 60  0000 C CNN
@@
 $EndComp
 $Comp
-L +3.3V #PWR063
+L +3.3V #PWR61
 U 1 1 556F428C
 P 2200 1350
-F 0 "#PWR063" H 2200 1200 50  0001 C CNN
+F 0 "#PWR61" H 2200 1200 50  0001 C CNN
 F 1 "+3.3V" H 2200 1490 50  0000 C CNN
 F 2 "" H 2200 1350 60  0000 C CNN
@@
 $EndComp
 $Comp
-L +3.3V #PWR064
+L +3.3V #PWR71
 U 1 1 557A9EA8
 P 9900 1300
-F 0 "#PWR064" H 9900 1150 50  0001 C CNN
+F 0 "#PWR71" H 9900 1150 50  0001 C CNN
 F 1 "+3.3V" H 9900 1440 50  0000 C CNN
 F 2 "" H 9900 1300 60  0000 C CNN
@@
 $EndComp
 $Comp
-L GNDD #PWR065
+L GNDD #PWR75
 U 1 1 557AA05D
 P 10150 1800
-F 0 "#PWR065" H 10150 1550 50  0001 C CNN
+F 0 "#PWR75" H 10150 1550 50  0001 C CNN
 F 1 "GNDD" H 10150 1650 50  0000 C CNN
 F 2 "" H 10150 1800 60  0000 C CNN
@@
 $EndComp
 $Comp
-L R R29
+L R R30
 U 1 1 557AA39A
 P 8950 1400
-F 0 "R29" V 9030 1400 40  0000 C CNN
+F 0 "R30" V 9030 1400 40  0000 C CNN
 F 1 "220R" V 8957 1401 40  0000 C CNN
 F 2 "Resistors_SMD:R_0603" V 8880 1400 30  0001 C CNN
@@
 $EndComp
 $Comp
-L R R30
+L R R31
 U 1 1 557AADB8
 P 8950 1600
-F 0 "R30" V 9030 1600 40  0000 C CNN
+F 0 "R31" V 9030 1600 40  0000 C CNN
 F 1 "220R" V 8957 1601 40  0000 C CNN
 F 2 "Resistors_SMD:R_0603" V 8880 1600 30  0001 C CNN
@@
 $EndComp
 $Comp
-L R R31
+L R R32
 U 1 1 557AAE1B
 P 8950 1800
-F 0 "R31" V 9030 1800 40  0000 C CNN
+F 0 "R32" V 9030 1800 40  0000 C CNN
 F 1 "220R" V 8957 1801 40  0000 C CNN
 F 2 "Resistors_SMD:R_0603" V 8880 1800 30  0001 C CNN
@@
 $EndComp
 $Comp
-L +3.3V #PWR066
+L +3.3V #PWR72
 U 1 1 55899AA7
 P 9900 2300
-F 0 "#PWR066" H 9900 2150 50  0001 C CNN
+F 0 "#PWR72" H 9900 2150 50  0001 C CNN
 F 1 "+3.3V" H 9900 2440 50  0000 C CNN
 F 2 "" H 9900 2300 60  0000 C CNN
@@
 $EndComp
 $Comp
-L GNDD #PWR067
+L GNDD #PWR76
 U 1 1 55899AAD
 P 10150 2800
-F 0 "#PWR067" H 10150 2550 50  0001 C CNN
+F 0 "#PWR76" H 10150 2550 50  0001 C CNN
 F 1 "GNDD" H 10150 2650 50  0000 C CNN
 F 2 "" H 10150 2800 60  0000 C CNN
@@
 $EndComp
 $Comp
-L R R32
+L R R33
 U 1 1 55899AB4
 P 8950 2400
-F 0 "R32" V 9030 2400 40  0000 C CNN
+F 0 "R33" V 9030 2400 40  0000 C CNN
 F 1 "220R" V 8957 2401 40  0000 C CNN
 F 2 "Resistors_SMD:R_0603" V 8880 2400 30  0001 C CNN
@@
 $EndComp
 $Comp
-L R R33
+L R R34
 U 1 1 55899AC2
 P 8950 2600
-F 0 "R33" V 9030 2600 40  0000 C CNN
+F 0 "R34" V 9030 2600 40  0000 C CNN
 F 1 "220R" V 8957 2601 40  0000 C CNN
 F 2 "Resistors_SMD:R_0603" V 8880 2600 30  0001 C CNN
@@
 $EndComp
 $Comp
-L R R34
+L R R35
 U 1 1 55899AC9
 P 8950 2800
-F 0 "R34" V 9030 2800 40  0000 C CNN
+F 0 "R35" V 9030 2800 40  0000 C CNN
 F 1 "220R" V 8957 2801 40  0000 C CNN
 F 2 "Resistors_SMD:R_0603" V 8880 2800 30  0001 C CNN
@@
 $EndComp
 $Comp
-L +3.3V #PWR068
+L +3.3V #PWR73
 U 1 1 5589B19A
 P 9900 3300
-F 0 "#PWR068" H 9900 3150 50  0001 C CNN
+F 0 "#PWR73" H 9900 3150 50  0001 C CNN
 F 1 "+3.3V" H 9900 3440 50  0000 C CNN
 F 2 "" H 9900 3300 60  0000 C CNN
@@
 $EndComp
 $Comp
-L GNDD #PWR069
+L GNDD #PWR77
 U 1 1 5589B1A0
 P 10150 3800
-F 0 "#PWR069" H 10150 3550 50  0001 C CNN
+F 0 "#PWR77" H 10150 3550 50  0001 C CNN
 F 1 "GNDD" H 10150 3650 50  0000 C CNN
 F 2 "" H 10150 3800 60  0000 C CNN
@@
 $EndComp
 $Comp
-L R R35
+L R R36
 U 1 1 5589B1A7
 P 8950 3400
-F 0 "R35" V 9030 3400 40  0000 C CNN
+F 0 "R36" V 9030 3400 40  0000 C CNN
 F 1 "220R" V 8957 3401 40  0000 C CNN
 F 2 "Resistors_SMD:R_0603" V 8880 3400 30  0001 C CNN
@@
 $EndComp
 $Comp
-L R R36
+L R R37
 U 1 1 5589B1B5
 P 8950 3600
-F 0 "R36" V 9030 3600 40  0000 C CNN
+F 0 "R37" V 9030 3600 40  0000 C CNN
 F 1 "220R" V 8957 3601 40  0000 C CNN
 F 2 "Resistors_SMD:R_0603" V 8880 3600 30  0001 C CNN
@@
 $EndComp
 $Comp
-L R R37
+L R R38
 U 1 1 5589B1BC
 P 8950 3800
-F 0 "R37" V 9030 3800 40  0000 C CNN
+F 0 "R38" V 9030 3800 40  0000 C CNN
 F 1 "220R" V 8957 3801 40  0000 C CNN
 F 2 "Resistors_SMD:R_0603" V 8880 3800 30  0001 C CNN
@@
 $EndComp
 $Comp
-L +3.3V #PWR070
+L +3.3V #PWR74
 U 1 1 5589B1DB
 P 9900 4300
-F 0 "#PWR070" H 9900 4150 50  0001 C CNN
+F 0 "#PWR74" H 9900 4150 50  0001 C CNN
 F 1 "+3.3V" H 9900 4440 50  0000 C CNN
 F 2 "" H 9900 4300 60  0000 C CNN
@@
 $EndComp
 $Comp
-L GNDD #PWR071
+L GNDD #PWR78
 U 1 1 5589B1E1
 P 10150 4800
-F 0 "#PWR071" H 10150 4550 50  0001 C CNN
+F 0 "#PWR78" H 10150 4550 50  0001 C CNN
 F 1 "GNDD" H 10150 4650 50  0000 C CNN
 F 2 "" H 10150 4800 60  0000 C CNN
@@
 $EndComp
 $Comp
-L R R38
+L R R39
 U 1 1 5589B1E8
 P 8950 4400
-F 0 "R38" V 9030 4400 40  0000 C CNN
+F 0 "R39" V 9030 4400 40  0000 C CNN
 F 1 "220R" V 8957 4401 40  0000 C CNN
 F 2 "Resistors_SMD:R_0603" V 8880 4400 30  0001 C CNN
@@
 $EndComp
 $Comp
-L R R39
+L R R40
 U 1 1 5589B1F6
 P 8950 4600
-F 0 "R39" V 9030 4600 40  0000 C CNN
+F 0 "R40" V 9030 4600 40  0000 C CNN
 F 1 "220R" V 8957 4601 40  0000 C CNN
 F 2 "Resistors_SMD:R_0603" V 8880 4600 30  0001 C CNN
@@
 $EndComp
 $Comp
-L R R40
+L R R41
 U 1 1 5589B1FD
 P 8950 4800
-F 0 "R40" V 9030 4800 40  0000 C CNN
+F 0 "R41" V 9030 4800 40  0000 C CNN
 F 1 "220R" V 8957 4801 40  0000 C CNN
 F 2 "Resistors_SMD:R_0603" V 8880 4800 30  0001 C CNN
@@
 $EndComp
 $Comp
-L R R27
+L R R28
 U 1 1 5589C3DA
 P 2700 3900
-F 0 "R27" V 2780 3900 40  0000 C CNN
+F 0 "R28" V 2780 3900 40  0000 C CNN
 F 1 "10k" V 2707 3901 40  0000 C CNN
 F 2 "Resistors_SMD:R_0603" V 2630 3900 30  0001 C CNN
@@
 $EndComp
 $Comp
-L GNDD #PWR072
+L GNDD #PWR63
 U 1 1 5589C3E0
 P 2700 4400
-F 0 "#PWR072" H 2700 4150 60  0001 C CNN
+F 0 "#PWR63" H 2700 4150 60  0001 C CNN
 F 1 "GNDD" H 2700 4250 60  0000 C CNN
 F 2 "" H 2700 4400 60  0000 C CNN
@@
 $EndComp
 $Comp
-L +3.3V #PWR073
+L +3.3V #PWR62
 U 1 1 5589C3ED
 P 2700 3650
-F 0 "#PWR073" H 2700 3500 50  0001 C CNN
+F 0 "#PWR62" H 2700 3500 50  0001 C CNN
 F 1 "+3.3V" H 2700 3790 50  0000 C CNN
 F 2 "" H 2700 3650 60  0000 C CNN
@@
 $EndComp
 $Comp
-L R R23
+L R R24
 U 1 1 5589C484
 P 1650 5350
-F 0 "R23" V 1730 5350 40  0000 C CNN
+F 0 "R24" V 1730 5350 40  0000 C CNN
 F 1 "10k" V 1657 5351 40  0000 C CNN
 F 2 "Resistors_SMD:R_0603" V 1580 5350 30  0001 C CNN
@@
 $EndComp
 $Comp
-L GNDD #PWR074
+L GNDD #PWR60
 U 1 1 5589C48A
 P 1650 5850
-F 0 "#PWR074" H 1650 5600 60  0001 C CNN
+F 0 "#PWR60" H 1650 5600 60  0001 C CNN
 F 1 "GNDD" H 1650 5700 60  0000 C CNN
 F 2 "" H 1650 5850 60  0000 C CNN
@@
 $EndComp
 $Comp
-L +3.3V #PWR075
+L +3.3V #PWR59
 U 1 1 5589C497
 P 1650 5100
-F 0 "#PWR075" H 1650 4950 50  0001 C CNN
+F 0 "#PWR59" H 1650 4950 50  0001 C CNN
 F 1 "+3.3V" H 1650 5240 50  0000 C CNN
 F 2 "" H 1650 5100 60  0000 C CNN
@@
 $EndComp
 $Comp
-L R R28
+L R R29
 U 1 1 5589C571
 P 2700 5350
-F 0 "R28" V 2780 5350 40  0000 C CNN
+F 0 "R29" V 2780 5350 40  0000 C CNN
 F 1 "10k" V 2707 5351 40  0000 C CNN
 F 2 "Resistors_SMD:R_0603" V 2630 5350 30  0001 C CNN
@@
 $EndComp
 $Comp
-L GNDD #PWR076
+L GNDD #PWR65
 U 1 1 5589C577
 P 2700 5850
-F 0 "#PWR076" H 2700 5600 60  0001 C CNN
+F 0 "#PWR65" H 2700 5600 60  0001 C CNN
 F 1 "GNDD" H 2700 5700 60  0000 C CNN
 F 2 "" H 2700 5850 60  0000 C CNN
@@
 $EndComp
 $Comp
-L +3.3V #PWR077
+L +3.3V #PWR64
 U 1 1 5589C584
 P 2700 5100
-F 0 "#PWR077" H 2700 4950 50  0001 C CNN
+F 0 "#PWR64" H 2700 4950 50  0001 C CNN
 F 1 "+3.3V" H 2700 5240 50  0000 C CNN
 F 2 "" H 2700 5100 60  0000 C CNN
@@
 $EndComp
 $Comp
-L GNDD #PWR078
+L GNDD #PWR67
 U 1 1 5589ADE1
 P 6600 2950
-F 0 "#PWR078" H 6600 2700 60  0001 C CNN
+F 0 "#PWR67" H 6600 2700 60  0001 C CNN
 F 1 "GNDD" H 6600 2800 60  0000 C CNN
 F 2 "" H 6600 2950 60  0000 C CNN
@@
 $EndComp
 $Comp
-L +3.3V #PWR079
+L +3.3V #PWR66
 U 1 1 5589B303
 P 6600 2200
-F 0 "#PWR079" H 6600 2050 50  0001 C CNN
+F 0 "#PWR66" H 6600 2050 50  0001 C CNN
 F 1 "+3.3V" H 6600 2340 50  0000 C CNN
 F 2 "" H 6600 2200 60  0000 C CNN
@@
 $EndComp
 $Comp
-L +3.3V #PWR080
+L +3.3V #PWR69
 U 1 1 5589B4DD
 P 7200 1900
-F 0 "#PWR080" H 7200 1750 50  0001 C CNN
+F 0 "#PWR69" H 7200 1750 50  0001 C CNN
 F 1 "+3.3V" H 7200 2040 50  0000 C CNN
 F 2 "" H 7200 1900 60  0000 C CNN
@@
 $EndComp
 $Comp
-L GNDD #PWR081
+L GNDD #PWR70
 U 1 1 5589B7E5
 P 7200 4300
-F 0 "#PWR081" H 7200 4050 60  0001 C CNN
+F 0 "#PWR70" H 7200 4050 60  0001 C CNN
 F 1 "GNDD" H 7200 4150 60  0000 C CNN
 F 2 "" H 7200 4300 60  0000 C CNN
@@
 $EndComp
 $Comp
-L GNDD #PWR082
+L GNDD #PWR68
 U 1 1 5589BC9B
 P 6650 3700
-F 0 "#PWR082" H 6650 3450 60  0001 C CNN
+F 0 "#PWR68" H 6650 3450 60  0001 C CNN
 F 1 "GNDD" H 6650 3550 60  0000 C CNN
 F 2 "" H 6650 3700 60  0000 C CNN

Commit message: sch: fixing some footprints and MPN
Parts:
- P4, P5, P6, P7: footprint Pin_Headers:Pin_Header_Straight_1x02 -> Pin_Headers:Pin_Header_Angled_1x02; MPN M20-9990246 -> M20-9960245
Changed lines of the file:
@@
 F 0 "P4" H 1350 4400 50  0000 C CNN
 F 1 "FOOT" V 1450 4250 50  0000 C CNN
-F 2 "Pin_Headers:Pin_Header_Straight_1x02" H 1350 4250 60  0001 C CNN
+F 2 "Pin_Headers:Pin_Header_Angled_1x02" H 1350 4250 60  0001 C CNN
 F 3 "" H 1350 4250 60  0000 C CNN
-F 4 "M20-9990246" H -400 2300 50  0001 C CNN "MPN"
+F 4 "M20-9960245" H -400 2300 50  0001 C CNN "MPN"
 	1    1350 4250
 	-1   0    0    -1
@@
 F 0 "P6" H 2400 4350 50  0000 C CNN
 F 1 "FOOT" V 2500 4200 50  0000 C CNN
-F 2 "Pin_Headers:Pin_Header_Straight_1x02" H 2400 4200 60  0001 C CNN
+F 2 "Pin_Headers:Pin_Header_Angled_1x02" H 2400 4200 60  0001 C CNN
 F 3 "" H 2400 4200 60  0000 C CNN
-F 4 "M20-9990246" H 650 2250 50  0001 C CNN "MPN"
+F 4 "M20-9960245" H 650 2250 50  0001 C CNN "MPN"
 	1    2400 4200
 	-1   0    0    -1
@@
 F 0 "P5" H 1350 5800 50  0000 C CNN
 F 1 "FOOT" V 1450 5650 50  0000 C CNN
-F 2 "Pin_Headers:Pin_Header_Straight_1x02" H 1350 5650 60  0001 C CNN
+F 2 "Pin_Headers:Pin_Header_Angled_1x02" H 1350 5650 60  0001 C CNN
 F 3 "" H 1350 5650 60  0000 C CNN
-F 4 "M20-9990246" H -400 3700 50  0001 C CNN "MPN"
+F 4 "M20-9960245" H -400 3700 50  0001 C CNN "MPN"
 	1    1350 5650
 	-1   0    0    -1
@@
 F 0 "P7" H 2400 5800 50  0000 C CNN
 F 1 "FOOT" V 2500 5650 50  0000 C CNN
-F 2 "Pin_Headers:Pin_Header_Straight_1x02" H 2400 5650 60  0001 C CNN
+F 2 "Pin_Headers:Pin_Header_Angled_1x02" H 2400 5650 60  0001 C CNN
 F 3 "" H 2400 5650 60  0000 C CNN
-F 4 "M20-9990246" H 650 3700 50  0001 C CNN "MPN"
+F 4 "M20-9960245" H 650 3700 50  0001 C CNN "MPN"
 	1    2400 5650
 	-1   0    0    -1
