File: hw-design/board/io.sch (KiCad schematic (older format))
At the start: 24 parts, among them P3 FOOT, P4 FOOT, P5 FOOT, P6 FOOT

Commit message: annotation and ERC
Parts:
- renumbered D4 to D5, D5 to D6, D6 to D7, D7 to D8, P3 to P1, P4 to P2, P5 to P4, P6 to P5, R7 to R1, R9 to R10, R10 to R11, R8 to R2, R11 to R22, R12 to R23, R13 to R24, R14 to R25, R15 to R26, R16 to R27, R17 to R28, R18 to R29, R19 to R30, R20 to R31, R21 to R32, R22 to R33
Changed lines of the file:
@@
 $EndDescr
 $Comp
-L R R7
+L R R1
 U 1 1 54CBEC53
 P 1850 1850
-F 0 "R7" V 1930 1850 40  0000 C CNN
+F 0 "R1" V 1930 1850 40  0000 C CNN
 F 1 "10k" V 1857 1851 40  0000 C CNN
 F 2 "Resistors_SMD:R_0603" V 1780 1850 30  0001 C CNN
@@
 $EndComp
 $Comp
-L GNDD #PWR044
+L GNDD #PWR3
 U 1 1 54E65047
 P 1850 2350
-F 0 "#PWR044" H 1850 2100 60  0001 C CNN
+F 0 "#PWR3" H 1850 2100 60  0001 C CNN
 F 1 "GNDD" H 1850 2200 60  0000 C CNN
 F 2 "" H 1850 2350 60  0000 C CNN
@@
 $EndComp
 $Comp
-L CONN_01X02 P3
+L CONN_01X02 P1
 U 1 1 54E6B5CA
 P 1550 2150
-F 0 "P3" H 1550 2300 50  0000 C CNN
+F 0 "P1" H 1550 2300 50  0000 C CNN
 F 1 "FOOT" V 1650 2150 50  0000 C CNN
 F 2 "Pin_Headers:Pin_Header_Angled_1x02" H 1550 2150 60  0001 C CNN
@@
 $EndComp
 $Comp
-L +3.3V #PWR045
+L +3.3V #PWR2
 U 1 1 556F3C3C
 P 1850 1600
-F 0 "#PWR045" H 1850 1450 50  0001 C CNN
+F 0 "#PWR2" H 1850 1450 50  0001 C CNN
 F 1 "+3.3V" H 1850 1740 50  0000 C CNN
 F 2 "" H 1850 1600 60  0000 C CNN
@@
 $EndComp
 $Comp
-L +3.3V #PWR046
+L +3.3V #PWR68
 U 1 1 557A9EA8
 P 8750 1500
-F 0 "#PWR046" H 8750 1350 50  0001 C CNN
+F 0 "#PWR68" H 8750 1350 50  0001 C CNN
 F 1 "+3.3V" H 8750 1640 50  0000 C CNN
 F 2 "" H 8750 1500 60  0000 C CNN
@@
 $EndComp
 $Comp
-L R R11
+L R R22
 U 1 1 557AA39A
 P 8000 1600
-F 0 "R11" V 8080 1600 40  0000 C CNN
+F 0 "R22" V 8080 1600 40  0000 C CNN
 F 1 "220R" V 8007 1601 40  0000 C CNN
 F 2 "Resistors_SMD:R_0603" V 7930 1600 30  0001 C CNN
@@
 $EndComp
 $Comp
-L LED_RGB D4
+L LED_RGB D5
 U 1 1 557AAC2C
 P 8450 1800
-F 0 "D4" H 8450 2250 50  0000 C CNN
+F 0 "D5" H 8450 2250 50  0000 C CNN
 F 1 "LED_RGB" H 8450 2150 50  0000 C CNN
 F 2 "LEDs:LED-RGB_PLLC-6" H 8450 1750 60  0001 C CNN
@@
 $EndComp
 $Comp
-L R R12
+L R R23
 U 1 1 557AADB8
 P 8000 1800
-F 0 "R12" V 8080 1800 40  0000 C CNN
+F 0 "R23" V 8080 1800 40  0000 C CNN
 F 1 "220R" V 8007 1801 40  0000 C CNN
 F 2 "Resistors_SMD:R_0603" V 7930 1800 30  0001 C CNN
@@
 $EndComp
 $Comp
-L R R13
+L R R24
 U 1 1 557AAE1B
 P 8000 2000
-F 0 "R13" V 8080 2000 40  0000 C CNN
+F 0 "R24" V 8080 2000 40  0000 C CNN
 F 1 "220R" V 8007 2001 40  0000 C CNN
 F 2 "Resistors_SMD:R_0603" V 7930 2000 30  0001 C CNN
@@
 $EndComp
 $Comp
-L +3.3V #PWR048
+L +3.3V #PWR69
 U 1 1 55899AA7
 P 8750 2500
-F 0 "#PWR048" H 8750 2350 50  0001 C CNN
+F 0 "#PWR69" H 8750 2350 50  0001 C CNN
 F 1 "+3.3V" H 8750 2640 50  0000 C CNN
 F 2 "" H 8750 2500 60  0000 C CNN
@@
 $EndComp
 $Comp
-L R R14
+L R R25
 U 1 1 55899AB4
 P 8000 2600
-F 0 "R14" V 8080 2600 40  0000 C CNN
+F 0 "R25" V 8080 2600 40  0000 C CNN
 F 1 "220R" V 8007 2601 40  0000 C CNN
 F 2 "Resistors_SMD:R_0603" V 7930 2600 30  0001 C CNN
@@
 $EndComp
 $Comp
-L LED_RGB D5
+L LED_RGB D6
 U 1 1 55899ABB
 P 8450 2800
-F 0 "D5" H 8450 3250 50  0000 C CNN
+F 0 "D6" H 8450 3250 50  0000 C CNN
 F 1 "LED_RGB" H 8450 3150 50  0000 C CNN
 F 2 "LEDs:LED-RGB_PLLC-6" H 8450 2750 60  0001 C CNN
@@
 $EndComp
 $Comp
-L R R15
+L R R26
 U 1 1 55899AC2
 P 8000 2800
-F 0 "R15" V 8080 2800 40  0000 C CNN
+F 0 "R26" V 8080 2800 40  0000 C CNN
 F 1 "220R" V 8007 2801 40  0000 C CNN
 F 2 "Resistors_SMD:R_0603" V 7930 2800 30  0001 C CNN
@@
 $EndComp
 $Comp
-L R R16
+L R R27
 U 1 1 55899AC9
 P 8000 3000
-F 0 "R16" V 8080 3000 40  0000 C CNN
+F 0 "R27" V 8080 3000 40  0000 C CNN
 F 1 "220R" V 8007 3001 40  0000 C CNN
 F 2 "Resistors_SMD:R_0603" V 7930 3000 30  0001 C CNN
@@
 $EndComp
 $Comp
-L +3.3V #PWR050
+L +3.3V #PWR70
 U 1 1 5589B19A
 P 8750 3500
-F 0 "#PWR050" H 8750 3350 50  0001 C CNN
+F 0 "#PWR70" H 8750 3350 50  0001 C CNN
 F 1 "+3.3V" H 8750 3640 50  0000 C CNN
 F 2 "" H 8750 3500 60  0000 C CNN
@@
 $EndComp
 $Comp
-L R R17
+L R R28
 U 1 1 5589B1A7
 P 8000 3600
-F 0 "R17" V 8080 3600 40  0000 C CNN
+F 0 "R28" V 8080 3600 40  0000 C CNN
 F 1 "220R" V 8007 3601 40  0000 C CNN
 F 2 "Resistors_SMD:R_0603" V 7930 3600 30  0001 C CNN
@@
 $EndComp
 $Comp
-L LED_RGB D6
+L LED_RGB D7
 U 1 1 5589B1AE
 P 8450 3800
-F 0 "D6" H 8450 4250 50  0000 C CNN
+F 0 "D7" H 8450 4250 50  0000 C CNN
 F 1 "LED_RGB" H 8450 4150 50  0000 C CNN
 F 2 "LEDs:LED-RGB_PLLC-6" H 8450 3750 60  0001 C CNN
@@
 $EndComp
 $Comp
-L R R18
+L R R29
 U 1 1 5589B1B5
 P 8000 3800
-F 0 "R18" V 8080 3800 40  0000 C CNN
+F 0 "R29" V 8080 3800 40  0000 C CNN
 F 1 "220R" V 8007 3801 40  0000 C CNN
 F 2 "Resistors_SMD:R_0603" V 7930 3800 30  0001 C CNN
@@
 $EndComp
 $Comp
-L R R19
+L R R30
 U 1 1 5589B1BC
 P 8000 4000
-F 0 "R19" V 8080 4000 40  0000 C CNN
+F 0 "R30" V 8080 4000 40  0000 C CNN
 F 1 "220R" V 8007 4001 40  0000 C CNN
 F 2 "Resistors_SMD:R_0603" V 7930 4000 30  0001 C CNN
@@
 $EndComp
 $Comp
-L +3.3V #PWR052
+L +3.3V #PWR71
 U 1 1 5589B1DB
 P 8750 4500
-F 0 "#PWR052" H 8750 4350 50  0001 C CNN
+F 0 "#PWR71" H 8750 4350 50  0001 C CNN
 F 1 "+3.3V" H 8750 4640 50  0000 C CNN
 F 2 "" H 8750 4500 60  0000 C CNN
@@
 $EndComp
 $Comp
-L R R20
+L R R31
 U 1 1 5589B1E8
 P 8000 4600
-F 0 "R20" V 8080 4600 40  0000 C CNN
+F 0 "R31" V 8080 4600 40  0000 C CNN
 F 1 "220R" V 8007 4601 40  0000 C CNN
 F 2 "Resistors_SMD:R_0603" V 7930 4600 30  0001 C CNN
@@
 $EndComp
 $Comp
-L LED_RGB D7
+L LED_RGB D8
 U 1 1 5589B1EF
 P 8450 4800
-F 0 "D7" H 8450 5250 50  0000 C CNN
+F 0 "D8" H 8450 5250 50  0000 C CNN
 F 1 "LED_RGB" H 8450 5150 50  0000 C CNN
 F 2 "LEDs:LED-RGB_PLLC-6" H 8450 4750 60  0001 C CNN
@@
 $EndComp
 $Comp
-L R R21
+L R R32
 U 1 1 5589B1F6
 P 8000 4800
-F 0 "R21" V 8080 4800 40  0000 C CNN
+F 0 "R32" V 8080 4800 40  0000 C CNN
 F 1 "220R" V 8007 4801 40  0000 C CNN
 F 2 "Resistors_SMD:R_0603" V 7930 4800 30  0001 C CNN
@@
 $EndComp
 $Comp
-L R R22
+L R R33
 U 1 1 5589B1FD
 P 8000 5000
-F 0 "R22" V 8080 5000 40  0000 C CNN
+F 0 "R33" V 8080 5000 40  0000 C CNN
 F 1 "220R" V 8007 5001 40  0000 C CNN
 F 2 "Resistors_SMD:R_0603" V 7930 5000 30  0001 C CNN
@@
 $EndComp
 $Comp
-L R R9
+L R R10
 U 1 1 5589C3DA
 P 2900 1850
-F 0 "R9" V 2980 1850 40  0000 C CNN
+F 0 "R10" V 2980 1850 40  0000 C CNN
 F 1 "10k" V 2907 1851 40  0000 C CNN
 F 2 "Resistors_SMD:R_0603" V 2830 1850 30  0001 C CNN
@@
 $EndComp
 $Comp
-L GNDD #PWR054
+L GNDD #PWR18
 U 1 1 5589C3E0
 P 2900 2350
-F 0 "#PWR054" H 2900 2100 60  0001 C CNN
+F 0 "#PWR18" H 2900 2100 60  0001 C CNN
 F 1 "GNDD" H 2900 2200 60  0000 C CNN
 F 2 "" H 2900 2350 60  0000 C CNN
@@
 $EndComp
 $Comp
-L CONN_01X02 P5
+L CONN_01X02 P4
 U 1 1 5589C3E7
 P 2600 2150
-F 0 "P5" H 2600 2300 50  0000 C CNN
+F 0 "P4" H 2600 2300 50  0000 C CNN
 F 1 "FOOT" V 2700 2150 50  0000 C CNN
 F 2 "Pin_Headers:Pin_Header_Angled_1x02" H 2600 2150 60  0001 C CNN
@@
 $EndComp
 $Comp
-L +3.3V #PWR055
+L +3.3V #PWR17
 U 1 1 5589C3ED
 P 2900 1600
-F 0 "#PWR055" H 2900 1450 50  0001 C CNN
+F 0 "#PWR17" H 2900 1450 50  0001 C CNN
 F 1 "+3.3V" H 2900 1740 50  0000 C CNN
 F 2 "" H 2900 1600 60  0000 C CNN
@@
 $EndComp
 $Comp
-L R R8
+L R R2
 U 1 1 5589C484
 P 1850 3250
-F 0 "R8" V 1930 3250 40  0000 C CNN
+F 0 "R2" V 1930 3250 40  0000 C CNN
 F 1 "10k" V 1857 3251 40  0000 C CNN
 F 2 "Resistors_SMD:R_0603" V 1780 3250 30  0001 C CNN
@@
 $EndComp
 $Comp
-L GNDD #PWR056
+L GNDD #PWR5
 U 1 1 5589C48A
 P 1850 3750
-F 0 "#PWR056" H 1850 3500 60  0001 C CNN
+F 0 "#PWR5" H 1850 3500 60  0001 C CNN
 F 1 "GNDD" H 1850 3600 60  0000 C CNN
 F 2 "" H 1850 3750 60  0000 C CNN
@@
 $EndComp
 $Comp
-L CONN_01X02 P4
+L CONN_01X02 P2
 U 1 1 5589C491
 P 1550 3550
-F 0 "P4" H 1550 3700 50  0000 C CNN
+F 0 "P2" H 1550 3700 50  0000 C CNN
 F 1 "FOOT" V 1650 3550 50  0000 C CNN
 F 2 "Pin_Headers:Pin_Header_Angled_1x02" H 1550 3550 60  0001 C CNN
@@
 $EndComp
 $Comp
-L +3.3V #PWR057
+L +3.3V #PWR4
 U 1 1 5589C497
 P 1850 3000
-F 0 "#PWR057" H 1850 2850 50  0001 C CNN
+F 0 "#PWR4" H 1850 2850 50  0001 C CNN
 F 1 "+3.3V" H 1850 3140 50  0000 C CNN
 F 2 "" H 1850 3000 60  0000 C CNN
@@
 $EndComp
 $Comp
-L R R10
+L R R11
 U 1 1 5589C571
 P 2900 3250
-F 0 "R10" V 2980 3250 40  0000 C CNN
+F 0 "R11" V 2980 3250 40  0000 C CNN
 F 1 "10k" V 2907 3251 40  0000 C CNN
 F 2 "Resistors_SMD:R_0603" V 2830 3250 30  0001 C CNN
@@
 $EndComp
 $Comp
-L GNDD #PWR058
+L GNDD #PWR20
 U 1 1 5589C577
 P 2900 3750
-F 0 "#PWR058" H 2900 3500 60  0001 C CNN
+F 0 "#PWR20" H 2900 3500 60  0001 C CNN
 F 1 "GNDD" H 2900 3600 60  0000 C CNN
 F 2 "" H 2900 3750 60  0000 C CNN
@@
 $EndComp
 $Comp
-L CONN_01X02 P6
+L CONN_01X02 P5
 U 1 1 5589C57E
 P 2600 3550
-F 0 "P6" H 2600 3700 50  0000 C CNN
+F 0 "P5" H 2600 3700 50  0000 C CNN
 F 1 "FOOT" V 2700 3550 50  0000 C CNN
 F 2 "Pin_Headers:Pin_Header_Angled_1x02" H 2600 3550 60  0001 C CNN
@@
 $EndComp
 $Comp
-L +3.3V #PWR059
+L +3.3V #PWR19
 U 1 1 5589C584
 P 2900 3000
-F 0 "#PWR059" H 2900 2850 50  0001 C CNN
+F 0 "#PWR19" H 2900 2850 50  0001 C CNN
 F 1 "+3.3V" H 2900 3140 50  0000 C CNN
 F 2 "" H 2900 3000 60  0000 C CNN

Commit message: update MPN
Parts:
- R1, R10, R11, R2: value 10k -> 10K
- R22, R23, R24, R25, R26, R27, R28, R29, R30, R31, R32, R33: MPN ESR03EZPJ221 -> RMCF0603JT220R
Changed lines of the file:
@@
 P 1850 1850
 F 0 "R1" V 1930 1850 40  0000 C CNN
-F 1 "10k" V 1857 1851 40  0000 C CNN
+F 1 "10K" V 1857 1851 40  0000 C CNN
 F 2 "Resistors_SMD:R_0603" V 1780 1850 30  0001 C CNN
 F 3 "~" H 1850 1850 30  0000 C CNN
@@
 F 2 "Resistors_SMD:R_0603" V 7930 1600 30  0001 C CNN
 F 3 "~" H 8000 1600 30  0000 C CNN
-F 4 "ESR03EZPJ221" H 6050 -2800 50  0001 C CNN "MPN"
+F 4 "RMCF0603JT220R" H 6050 -2800 50  0001 C CNN "MPN"
 	1    8000 1600
 	0    -1   1    0
@@
 F 2 "Resistors_SMD:R_0603" V 7930 1800 30  0001 C CNN
 F 3 "~" H 8000 1800 30  0000 C CNN
-F 4 "ESR03EZPJ221" H 6050 -2800 50  0001 C CNN "MPN"
+F 4 "RMCF0603JT220R" H 6050 -2800 50  0001 C CNN "MPN"
 	1    8000 1800
 	0    -1   1    0
@@
 F 2 "Resistors_SMD:R_0603" V 7930 2000 30  0001 C CNN
 F 3 "~" H 8000 2000 30  0000 C CNN
-F 4 "ESR03EZPJ221" H 6050 -2800 50  0001 C CNN "MPN"
+F 4 "RMCF0603JT220R" H 6050 -2800 50  0001 C CNN "MPN"
 	1    8000 2000
 	0    -1   1    0
@@
 F 2 "Resistors_SMD:R_0603" V 7930 2600 30  0001 C CNN
 F 3 "~" H 8000 2600 30  0000 C CNN
-F 4 "ESR03EZPJ221" H 6050 -1800 50  0001 C CNN "MPN"
+F 4 "RMCF0603JT220R" H 6050 -1800 50  0001 C CNN "MPN"
 	1    8000 2600
 	0    -1   1    0
@@
 F 2 "Resistors_SMD:R_0603" V 7930 2800 30  0001 C CNN
 F 3 "~" H 8000 2800 30  0000 C CNN
-F 4 "ESR03EZPJ221" H 6050 -1800 50  0001 C CNN "MPN"
+F 4 "RMCF0603JT220R" H 6050 -1800 50  0001 C CNN "MPN"
 	1    8000 2800
 	0    -1   1    0
@@
 F 2 "Resistors_SMD:R_0603" V 7930 3000 30  0001 C CNN
 F 3 "~" H 8000 3000 30  0000 C CNN
-F 4 "ESR03EZPJ221" H 6050 -1800 50  0001 C CNN "MPN"
+F 4 "RMCF0603JT220R" H 6050 -1800 50  0001 C CNN "MPN"
 	1    8000 3000
 	0    -1   1    0
@@
 F 2 "Resistors_SMD:R_0603" V 7930 3600 30  0001 C CNN
 F 3 "~" H 8000 3600 30  0000 C CNN
-F 4 "ESR03EZPJ221" H 6050 -800 50  0001 C CNN "MPN"
+F 4 "RMCF0603JT220R" H 6050 -800 50  0001 C CNN "MPN"
 	1    8000 3600
 	0    -1   1    0
@@
 F 2 "Resistors_SMD:R_0603" V 7930 3800 30  0001 C CNN
 F 3 "~" H 8000 3800 30  0000 C CNN
-F 4 "ESR03EZPJ221" H 6050 -800 50  0001 C CNN "MPN"
+F 4 "RMCF0603JT220R" H 6050 -800 50  0001 C CNN "MPN"
 	1    8000 3800
 	0    -1   1    0
@@
 F 2 "Resistors_SMD:R_0603" V 7930 4000 30  0001 C CNN
 F 3 "~" H 8000 4000 30  0000 C CNN
-F 4 "ESR03EZPJ221" H 6050 -800 50  0001 C CNN "MPN"
+F 4 "RMCF0603JT220R" H 6050 -800 50  0001 C CNN "MPN"
 	1    8000 4000
 	0    -1   1    0
@@
 F 2 "Resistors_SMD:R_0603" V 7930 4600 30  0001 C CNN
 F 3 "~" H 8000 4600 30  0000 C CNN
-F 4 "ESR03EZPJ221" H 6050 200 50  0001 C CNN "MPN"
+F 4 "RMCF0603JT220R" H 6050 200 50  0001 C CNN "MPN"
 	1    8000 4600
 	0    -1   1    0
@@
 F 2 "Resistors_SMD:R_0603" V 7930 4800 30  0001 C CNN
 F 3 "~" H 8000 4800 30  0000 C CNN
-F 4 "ESR03EZPJ221" H 6050 200 50  0001 C CNN "MPN"
+F 4 "RMCF0603JT220R" H 6050 200 50  0001 C CNN "MPN"
 	1    8000 4800
 	0    -1   1    0
@@
 F 2 "Resistors_SMD:R_0603" V 7930 5000 30  0001 C CNN
 F 3 "~" H 8000 5000 30  0000 C CNN
-F 4 "ESR03EZPJ221" H 6050 200 50  0001 C CNN "MPN"
+F 4 "RMCF0603JT220R" H 6050 200 50  0001 C CNN "MPN"
 	1    8000 5000
 	0    -1   1    0
@@
 P 2900 1850
 F 0 "R10" V 2980 1850 40  0000 C CNN
-F 1 "10k" V 2907 1851 40  0000 C CNN
+F 1 "10K" V 2907 1851 40  0000 C CNN
 F 2 "Resistors_SMD:R_0603" V 2830 1850 30  0001 C CNN
 F 3 "~" H 2900 1850 30  0000 C CNN
@@
 P 1850 3250
 F 0 "R2" V 1930 3250 40  0000 C CNN
-F 1 "10k" V 1857 3251 40  0000 C CNN
+F 1 "10K" V 1857 3251 40  0000 C CNN
 F 2 "Resistors_SMD:R_0603" V 1780 3250 30  0001 C CNN
 F 3 "~" H 1850 3250 30  0000 C CNN
@@
 P 2900 3250
 F 0 "R11" V 2980 3250 40  0000 C CNN
-F 1 "10k" V 2907 3251 40  0000 C CNN
+F 1 "10K" V 2907 3251 40  0000 C CNN
 F 2 "Resistors_SMD:R_0603" V 2830 3250 30  0001 C CNN
 F 3 "~" H 2900 3250 30  0000 C CNN

Commit message: DRC done
Parts:
- renumbered R11 to R10, R22 to R21, R23 to R22, R24 to R23, R25 to R26, R26 to R27, R27 to R28, R28 to R29, R29 to R30, R30 to R31, R31 to R32, R32 to R33, R33 to R34, R10 to R9
Changed lines of the file:
@@
 $EndComp
 $Comp
-L +3.3V #PWR68
+L +3.3V #PWR64
 U 1 1 557A9EA8
 P 8750 1500
-F 0 "#PWR68" H 8750 1350 50  0001 C CNN
+F 0 "#PWR64" H 8750 1350 50  0001 C CNN
 F 1 "+3.3V" H 8750 1640 50  0000 C CNN
 F 2 "" H 8750 1500 60  0000 C CNN
@@
 $EndComp
 $Comp
-L R R22
+L R R21
 U 1 1 557AA39A
 P 8000 1600
-F 0 "R22" V 8080 1600 40  0000 C CNN
+F 0 "R21" V 8080 1600 40  0000 C CNN
 F 1 "220R" V 8007 1601 40  0000 C CNN
 F 2 "Resistors_SMD:R_0603" V 7930 1600 30  0001 C CNN
@@
 $EndComp
 $Comp
-L R R23
+L R R22
 U 1 1 557AADB8
 P 8000 1800
-F 0 "R23" V 8080 1800 40  0000 C CNN
+F 0 "R22" V 8080 1800 40  0000 C CNN
 F 1 "220R" V 8007 1801 40  0000 C CNN
 F 2 "Resistors_SMD:R_0603" V 7930 1800 30  0001 C CNN
@@
 $EndComp
 $Comp
-L R R24
+L R R23
 U 1 1 557AAE1B
 P 8000 2000
-F 0 "R24" V 8080 2000 40  0000 C CNN
+F 0 "R23" V 8080 2000 40  0000 C CNN
 F 1 "220R" V 8007 2001 40  0000 C CNN
 F 2 "Resistors_SMD:R_0603" V 7930 2000 30  0001 C CNN
@@
 $EndComp
 $Comp
-L +3.3V #PWR69
+L +3.3V #PWR65
 U 1 1 55899AA7
 P 8750 2500
-F 0 "#PWR69" H 8750 2350 50  0001 C CNN
+F 0 "#PWR65" H 8750 2350 50  0001 C CNN
 F 1 "+3.3V" H 8750 2640 50  0000 C CNN
 F 2 "" H 8750 2500 60  0000 C CNN
@@
 $EndComp
 $Comp
-L R R25
+L R R26
 U 1 1 55899AB4
 P 8000 2600
-F 0 "R25" V 8080 2600 40  0000 C CNN
+F 0 "R26" V 8080 2600 40  0000 C CNN
 F 1 "220R" V 8007 2601 40  0000 C CNN
 F 2 "Resistors_SMD:R_0603" V 7930 2600 30  0001 C CNN
@@
 $EndComp
 $Comp
-L R R26
+L R R27
 U 1 1 55899AC2
 P 8000 2800
-F 0 "R26" V 8080 2800 40  0000 C CNN
+F 0 "R27" V 8080 2800 40  0000 C CNN
 F 1 "220R" V 8007 2801 40  0000 C CNN
 F 2 "Resistors_SMD:R_0603" V 7930 2800 30  0001 C CNN
@@
 $EndComp
 $Comp
-L R R27
+L R R28
 U 1 1 55899AC9
 P 8000 3000
-F 0 "R27" V 8080 3000 40  0000 C CNN
+F 0 "R28" V 8080 3000 40  0000 C CNN
 F 1 "220R" V 8007 3001 40  0000 C CNN
 F 2 "Resistors_SMD:R_0603" V 7930 3000 30  0001 C CNN
@@
 $EndComp
 $Comp
-L +3.3V #PWR70
+L +3.3V #PWR66
 U 1 1 5589B19A
 P 8750 3500
-F 0 "#PWR70" H 8750 3350 50  0001 C CNN
+F 0 "#PWR66" H 8750 3350 50  0001 C CNN
 F 1 "+3.3V" H 8750 3640 50  0000 C CNN
 F 2 "" H 8750 3500 60  0000 C CNN
@@
 $EndComp
 $Comp
-L R R28
+L R R29
 U 1 1 5589B1A7
 P 8000 3600
-F 0 "R28" V 8080 3600 40  0000 C CNN
+F 0 "R29" V 8080 3600 40  0000 C CNN
 F 1 "220R" V 8007 3601 40  0000 C CNN
 F 2 "Resistors_SMD:R_0603" V 7930 3600 30  0001 C CNN
@@
 $EndComp
 $Comp
-L R R29
+L R R30
 U 1 1 5589B1B5
 P 8000 3800
-F 0 "R29" V 8080 3800 40  0000 C CNN
+F 0 "R30" V 8080 3800 40  0000 C CNN
 F 1 "220R" V 8007 3801 40  0000 C CNN
 F 2 "Resistors_SMD:R_0603" V 7930 3800 30  0001 C CNN
@@
 $EndComp
 $Comp
-L R R30
+L R R31
 U 1 1 5589B1BC
 P 8000 4000
-F 0 "R30" V 8080 4000 40  0000 C CNN
+F 0 "R31" V 8080 4000 40  0000 C CNN
 F 1 "220R" V 8007 4001 40  0000 C CNN
 F 2 "Resistors_SMD:R_0603" V 7930 4000 30  0001 C CNN
@@
 $EndComp
 $Comp
-L +3.3V #PWR71
+L +3.3V #PWR67
 U 1 1 5589B1DB
 P 8750 4500
-F 0 "#PWR71" H 8750 4350 50  0001 C CNN
+F 0 "#PWR67" H 8750 4350 50  0001 C CNN
 F 1 "+3.3V" H 8750 4640 50  0000 C CNN
 F 2 "" H 8750 4500 60  0000 C CNN
@@
 $EndComp
 $Comp
-L R R31
+L R R32
 U 1 1 5589B1E8
 P 8000 4600
-F 0 "R31" V 8080 4600 40  0000 C CNN
+F 0 "R32" V 8080 4600 40  0000 C CNN
 F 1 "220R" V 8007 4601 40  0000 C CNN
 F 2 "Resistors_SMD:R_0603" V 7930 4600 30  0001 C CNN
@@
 $EndComp
 $Comp
-L R R32
+L R R33
 U 1 1 5589B1F6
 P 8000 4800
-F 0 "R32" V 8080 4800 40  0000 C CNN
+F 0 "R33" V 8080 4800 40  0000 C CNN
 F 1 "220R" V 8007 4801 40  0000 C CNN
 F 2 "Resistors_SMD:R_0603" V 7930 4800 30  0001 C CNN
@@
 $EndComp
 $Comp
-L R R33
+L R R34
 U 1 1 5589B1FD
 P 8000 5000
-F 0 "R33" V 8080 5000 40  0000 C CNN
+F 0 "R34" V 8080 5000 40  0000 C CNN
 F 1 "220R" V 8007 5001 40  0000 C CNN
 F 2 "Resistors_SMD:R_0603" V 7930 5000 30  0001 C CNN
@@
 $EndComp
 $Comp
-L R R10
+L R R9
 U 1 1 5589C3DA
 P 2900 1850
-F 0 "R10" V 2980 1850 40  0000 C CNN
+F 0 "R9" V 2980 1850 40  0000 C CNN
 F 1 "10K" V 2907 1851 40  0000 C CNN
 F 2 "Resistors_SMD:R_0603" V 2830 1850 30  0001 C CNN
@@
 $EndComp
 $Comp
-L GNDD #PWR18
+L GNDD #PWR16
 U 1 1 5589C3E0
 P 2900 2350
-F 0 "#PWR18" H 2900 2100 60  0001 C CNN
+F 0 "#PWR16" H 2900 2100 60  0001 C CNN
 F 1 "GNDD" H 2900 2200 60  0000 C CNN
 F 2 "" H 2900 2350 60  0000 C CNN
@@
 $EndComp
 $Comp
-L +3.3V #PWR17
+L +3.3V #PWR15
 U 1 1 5589C3ED
 P 2900 1600
-F 0 "#PWR17" H 2900 1450 50  0001 C CNN
+F 0 "#PWR15" H 2900 1450 50  0001 C CNN
 F 1 "+3.3V" H 2900 1740 50  0000 C CNN
 F 2 "" H 2900 1600 60  0000 C CNN
@@
 $EndComp
 $Comp
-L R R11
+L R R10
 U 1 1 5589C571
 P 2900 3250
-F 0 "R11" V 2980 3250 40  0000 C CNN
+F 0 "R10" V 2980 3250 40  0000 C CNN
 F 1 "10K" V 2907 3251 40  0000 C CNN
 F 2 "Resistors_SMD:R_0603" V 2830 3250 30  0001 C CNN
@@
 $EndComp
 $Comp
-L GNDD #PWR20
+L GNDD #PWR18
 U 1 1 5589C577
 P 2900 3750
-F 0 "#PWR20" H 2900 3500 60  0001 C CNN
+F 0 "#PWR18" H 2900 3500 60  0001 C CNN
 F 1 "GNDD" H 2900 3600 60  0000 C CNN
 F 2 "" H 2900 3750 60  0000 C CNN
@@
 $EndComp
 $Comp
-L +3.3V #PWR19
+L +3.3V #PWR17
 U 1 1 5589C584
 P 2900 3000
-F 0 "#PWR19" H 2900 2850 50  0001 C CNN
+F 0 "#PWR17" H 2900 2850 50  0001 C CNN
 F 1 "+3.3V" H 2900 3140 50  0000 C CNN
 F 2 "" H 2900 3000 60  0000 C CNN
