File: hw-design/board/io.sch (KiCad schematic (older format))
At the start: 24 parts, among them P1 FOOT, P2 FOOT, P4 FOOT, P5 FOOT

Commit message: update netlist
Parts:
- renumbered R9 to R11, R10 to R12, R21 to R23, R22 to R24, R23 to R25, R26 to R28, R27 to R29, R28 to R30, R29 to R31, R30 to R32, R31 to R33, R32 to R34, R33 to R35, R34 to R36
Changed lines of the file:
@@
 $EndComp
 $Comp
-L +3.3V #PWR64
+L +3.3V #PWR66
 U 1 1 557A9EA8
 P 8750 1500
-F 0 "#PWR64" H 8750 1350 50  0001 C CNN
+F 0 "#PWR66" H 8750 1350 50  0001 C CNN
 F 1 "+3.3V" H 8750 1640 50  0000 C CNN
 F 2 "" H 8750 1500 60  0000 C CNN
@@
 $EndComp
 $Comp
-L R R21
+L R R23
 U 1 1 557AA39A
 P 8000 1600
-F 0 "R21" V 8080 1600 40  0000 C CNN
+F 0 "R23" V 8080 1600 40  0000 C CNN
 F 1 "220R" V 8007 1601 40  0000 C CNN
 F 2 "Resistors_SMD:R_0603" V 7930 1600 30  0001 C CNN
@@
 $EndComp
 $Comp
-L R R22
+L R R24
 U 1 1 557AADB8
 P 8000 1800
-F 0 "R22" V 8080 1800 40  0000 C CNN
+F 0 "R24" V 8080 1800 40  0000 C CNN
 F 1 "220R" V 8007 1801 40  0000 C CNN
 F 2 "Resistors_SMD:R_0603" V 7930 1800 30  0001 C CNN
@@
 $EndComp
 $Comp
-L R R23
+L R R25
 U 1 1 557AAE1B
 P 8000 2000
-F 0 "R23" V 8080 2000 40  0000 C CNN
+F 0 "R25" V 8080 2000 40  0000 C CNN
 F 1 "220R" V 8007 2001 40  0000 C CNN
 F 2 "Resistors_SMD:R_0603" V 7930 2000 30  0001 C CNN
@@
 $EndComp
 $Comp
-L +3.3V #PWR65
+L +3.3V #PWR67
 U 1 1 55899AA7
 P 8750 2500
-F 0 "#PWR65" H 8750 2350 50  0001 C CNN
+F 0 "#PWR67" H 8750 2350 50  0001 C CNN
 F 1 "+3.3V" H 8750 2640 50  0000 C CNN
 F 2 "" H 8750 2500 60  0000 C CNN
@@
 $EndComp
 $Comp
-L R R26
+L R R28
 U 1 1 55899AB4
 P 8000 2600
-F 0 "R26" V 8080 2600 40  0000 C CNN
+F 0 "R28" V 8080 2600 40  0000 C CNN
 F 1 "220R" V 8007 2601 40  0000 C CNN
 F 2 "Resistors_SMD:R_0603" V 7930 2600 30  0001 C CNN
@@
 $EndComp
 $Comp
-L R R27
+L R R29
 U 1 1 55899AC2
 P 8000 2800
-F 0 "R27" V 8080 2800 40  0000 C CNN
+F 0 "R29" V 8080 2800 40  0000 C CNN
 F 1 "220R" V 8007 2801 40  0000 C CNN
 F 2 "Resistors_SMD:R_0603" V 7930 2800 30  0001 C CNN
@@
 $EndComp
 $Comp
-L R R28
+L R R30
 U 1 1 55899AC9
 P 8000 3000
-F 0 "R28" V 8080 3000 40  0000 C CNN
+F 0 "R30" V 8080 3000 40  0000 C CNN
 F 1 "220R" V 8007 3001 40  0000 C CNN
 F 2 "Resistors_SMD:R_0603" V 7930 3000 30  0001 C CNN
@@
 $EndComp
 $Comp
-L +3.3V #PWR66
+L +3.3V #PWR68
 U 1 1 5589B19A
 P 8750 3500
-F 0 "#PWR66" H 8750 3350 50  0001 C CNN
+F 0 "#PWR68" H 8750 3350 50  0001 C CNN
 F 1 "+3.3V" H 8750 3640 50  0000 C CNN
 F 2 "" H 8750 3500 60  0000 C CNN
@@
 $EndComp
 $Comp
-L R R29
+L R R31
 U 1 1 5589B1A7
 P 8000 3600
-F 0 "R29" V 8080 3600 40  0000 C CNN
+F 0 "R31" V 8080 3600 40  0000 C CNN
 F 1 "220R" V 8007 3601 40  0000 C CNN
 F 2 "Resistors_SMD:R_0603" V 7930 3600 30  0001 C CNN
@@
 $EndComp
 $Comp
-L R R30
+L R R32
 U 1 1 5589B1B5
 P 8000 3800
-F 0 "R30" V 8080 3800 40  0000 C CNN
+F 0 "R32" V 8080 3800 40  0000 C CNN
 F 1 "220R" V 8007 3801 40  0000 C CNN
 F 2 "Resistors_SMD:R_0603" V 7930 3800 30  0001 C CNN
@@
 $EndComp
 $Comp
-L R R31
+L R R33
 U 1 1 5589B1BC
 P 8000 4000
-F 0 "R31" V 8080 4000 40  0000 C CNN
+F 0 "R33" V 8080 4000 40  0000 C CNN
 F 1 "220R" V 8007 4001 40  0000 C CNN
 F 2 "Resistors_SMD:R_0603" V 7930 4000 30  0001 C CNN
@@
 $EndComp
 $Comp
-L +3.3V #PWR67
+L +3.3V #PWR69
 U 1 1 5589B1DB
 P 8750 4500
-F 0 "#PWR67" H 8750 4350 50  0001 C CNN
+F 0 "#PWR69" H 8750 4350 50  0001 C CNN
 F 1 "+3.3V" H 8750 4640 50  0000 C CNN
 F 2 "" H 8750 4500 60  0000 C CNN
@@
 $EndComp
 $Comp
-L R R32
+L R R34
 U 1 1 5589B1E8
 P 8000 4600
-F 0 "R32" V 8080 4600 40  0000 C CNN
+F 0 "R34" V 8080 4600 40  0000 C CNN
 F 1 "220R" V 8007 4601 40  0000 C CNN
 F 2 "Resistors_SMD:R_0603" V 7930 4600 30  0001 C CNN
@@
 $EndComp
 $Comp
-L R R33
+L R R35
 U 1 1 5589B1F6
 P 8000 4800
-F 0 "R33" V 8080 4800 40  0000 C CNN
+F 0 "R35" V 8080 4800 40  0000 C CNN
 F 1 "220R" V 8007 4801 40  0000 C CNN
 F 2 "Resistors_SMD:R_0603" V 7930 4800 30  0001 C CNN
@@
 $EndComp
 $Comp
-L R R34
+L R R36
 U 1 1 5589B1FD
 P 8000 5000
-F 0 "R34" V 8080 5000 40  0000 C CNN
+F 0 "R36" V 8080 5000 40  0000 C CNN
 F 1 "220R" V 8007 5001 40  0000 C CNN
 F 2 "Resistors_SMD:R_0603" V 7930 5000 30  0001 C CNN
@@
 $EndComp
 $Comp
-L R R9
+L R R11
 U 1 1 5589C3DA
 P 2900 1850
-F 0 "R9" V 2980 1850 40  0000 C CNN
+F 0 "R11" V 2980 1850 40  0000 C CNN
 F 1 "10K" V 2907 1851 40  0000 C CNN
 F 2 "Resistors_SMD:R_0603" V 2830 1850 30  0001 C CNN
@@
 $EndComp
 $Comp
-L GNDD #PWR16
+L GNDD #PWR18
 U 1 1 5589C3E0
 P 2900 2350
-F 0 "#PWR16" H 2900 2100 60  0001 C CNN
+F 0 "#PWR18" H 2900 2100 60  0001 C CNN
 F 1 "GNDD" H 2900 2200 60  0000 C CNN
 F 2 "" H 2900 2350 60  0000 C CNN
@@
 $EndComp
 $Comp
-L +3.3V #PWR15
+L +3.3V #PWR17
 U 1 1 5589C3ED
 P 2900 1600
-F 0 "#PWR15" H 2900 1450 50  0001 C CNN
+F 0 "#PWR17" H 2900 1450 50  0001 C CNN
 F 1 "+3.3V" H 2900 1740 50  0000 C CNN
 F 2 "" H 2900 1600 60  0000 C CNN
@@
 $EndComp
 $Comp
-L R R10
+L R R12
 U 1 1 5589C571
 P 2900 3250
-F 0 "R10" V 2980 3250 40  0000 C CNN
+F 0 "R12" V 2980 3250 40  0000 C CNN
 F 1 "10K" V 2907 3251 40  0000 C CNN
 F 2 "Resistors_SMD:R_0603" V 2830 3250 30  0001 C CNN
@@
 $EndComp
 $Comp
-L GNDD #PWR18
+L GNDD #PWR20
 U 1 1 5589C577
 P 2900 3750
-F 0 "#PWR18" H 2900 3500 60  0001 C CNN
+F 0 "#PWR20" H 2900 3500 60  0001 C CNN
 F 1 "GNDD" H 2900 3600 60  0000 C CNN
 F 2 "" H 2900 3750 60  0000 C CNN
@@
 $EndComp
 $Comp
-L +3.3V #PWR17
+L +3.3V #PWR19
 U 1 1 5589C584
 P 2900 3000
-F 0 "#PWR17" H 2900 2850 50  0001 C CNN
+F 0 "#PWR19" H 2900 2850 50  0001 C CNN
 F 1 "+3.3V" H 2900 3140 50  0000 C CNN
 F 2 "" H 2900 3000 60  0000 C CNN
