File: hw-design/board/io.sch (KiCad schematic (older format))
At the start: 24 parts, among them P1 FOOT, P2 FOOT, P4 FOOT, P5 FOOT

Commit message: update files to KiCAD 5
Parts:
- D5, D6, D7, D8: symbol LED_RGB -> footswitch-rescue:LED_RGB
- P1, P2, P4, P5: symbol CONN_01X02 -> footswitch-rescue:CONN_01X02; Note (none) -> place on the back side
- R1, R11, R12, R2, R23, R24, R25, R28, R29, R30, R31, R32, R33, R34, R35, R36: symbol R -> footswitch-rescue:R
Changed lines of the file:
@@
-EESchema Schematic File Version 2
-LIBS:conn
-LIBS:device
-LIBS:interface
-LIBS:power
-LIBS:regul
-LIBS:transistors
-LIBS:display
-LIBS:nxp_armmcu
-LIBS:philips
-LIBS:graphic_symbols
+EESchema Schematic File Version 4
 LIBS:footswitch-cache
 EELAYER 26 0
@@
 $EndDescr
 $Comp
-L R R1
+L footswitch-rescue:R R1
 U 1 1 54CBEC53
 P 1850 1850
@@
 $EndComp
 $Comp
-L GNDD #PWR039
+L footswitch-rescue:GNDD #PWR039
 U 1 1 54E65047
 P 1850 2350
@@
 $EndComp
 $Comp
-L CONN_01X02 P1
+L footswitch-rescue:CONN_01X02 P1
 U 1 1 54E6B5CA
 P 1550 2150
@@
 F 3 "" H 1550 2150 60  0000 C CNN
 F 4 "M20-9960245" H -200 200 50  0001 C CNN "MPN"
+F 5 "place on the back side" H 1550 2150 50  0001 C CNN "Note"
 	1    1550 2150
 	-1   0    0    -1
 $EndComp
 $Comp
-L +3.3V #PWR040
+L footswitch-rescue:+3.3V #PWR040
 U 1 1 556F3C3C
 P 1850 1600
@@
 $EndComp
 $Comp
-L +3.3V #PWR041
+L footswitch-rescue:+3.3V #PWR041
 U 1 1 557A9EA8
 P 8750 1500
@@
 $EndComp
 $Comp
-L R R23
+L footswitch-rescue:R R23
 U 1 1 557AA39A
 P 8000 1600
@@
 $EndComp
 $Comp
-L LED_RGB D5
+L footswitch-rescue:LED_RGB D5
 U 1 1 557AAC2C
 P 8450 1800
@@
 $EndComp
 $Comp
-L R R24
+L footswitch-rescue:R R24
 U 1 1 557AADB8
 P 8000 1800
@@
 $EndComp
 $Comp
-L R R25
+L footswitch-rescue:R R25
 U 1 1 557AAE1B
 P 8000 2000
@@
 $EndComp
 $Comp
-L +3.3V #PWR042
+L footswitch-rescue:+3.3V #PWR042
 U 1 1 55899AA7
 P 8750 2500
@@
 $EndComp
 $Comp
-L R R28
+L footswitch-rescue:R R28
 U 1 1 55899AB4
 P 8000 2600
@@
 $EndComp
 $Comp
-L LED_RGB D6
+L footswitch-rescue:LED_RGB D6
 U 1 1 55899ABB
 P 8450 2800
@@
 $EndComp
 $Comp
-L R R29
+L footswitch-rescue:R R29
 U 1 1 55899AC2
 P 8000 2800
@@
 $EndComp
 $Comp
-L R R30
+L footswitch-rescue:R R30
 U 1 1 55899AC9
 P 8000 3000
@@
 $EndComp
 $Comp
-L +3.3V #PWR043
+L footswitch-rescue:+3.3V #PWR043
 U 1 1 5589B19A
 P 8750 3500
@@
 $EndComp
 $Comp
-L R R31
+L footswitch-rescue:R R31
 U 1 1 5589B1A7
 P 8000 3600
@@
 $EndComp
 $Comp
-L LED_RGB D7
+L footswitch-rescue:LED_RGB D7
 U 1 1 5589B1AE
 P 8450 3800
@@
 $EndComp
 $Comp
-L R R32
+L footswitch-rescue:R R32
 U 1 1 5589B1B5
 P 8000 3800
@@
 $EndComp
 $Comp
-L R R33
+L footswitch-rescue:R R33
 U 1 1 5589B1BC
 P 8000 4000
@@
 $EndComp
 $Comp
-L +3.3V #PWR044
+L footswitch-rescue:+3.3V #PWR044
 U 1 1 5589B1DB
 P 8750 4500
@@
 $EndComp
 $Comp
-L R R34
+L footswitch-rescue:R R34
 U 1 1 5589B1E8
 P 8000 4600
@@
 $EndComp
 $Comp
-L LED_RGB D8
+L footswitch-rescue:LED_RGB D8
 U 1 1 5589B1EF
 P 8450 4800
@@
 $EndComp
 $Comp
-L R R35
+L footswitch-rescue:R R35
 U 1 1 5589B1F6
 P 8000 4800
@@
 $EndComp
 $Comp
-L R R36
+L footswitch-rescue:R R36
 U 1 1 5589B1FD
 P 8000 5000
@@
 $EndComp
 $Comp
-L R R11
+L footswitch-rescue:R R11
 U 1 1 5589C3DA
 P 2900 1850
@@
 $EndComp
 $Comp
-L GNDD #PWR045
+L footswitch-rescue:GNDD #PWR045
 U 1 1 5589C3E0
 P 2900 2350
@@
 $EndComp
 $Comp
-L CONN_01X02 P4
+L footswitch-rescue:CONN_01X02 P4
 U 1 1 5589C3E7
 P 2600 2150
@@
 F 3 "" H 2600 2150 60  0000 C CNN
 F 4 "M20-9960245" H 850 200 50  0001 C CNN "MPN"
+F 5 "place on the back side" H 2600 2150 50  0001 C CNN "Note"
 	1    2600 2150
 	-1   0    0    -1
 $EndComp
 $Comp
-L +3.3V #PWR046
+L footswitch-rescue:+3.3V #PWR046
 U 1 1 5589C3ED
 P 2900 1600
@@
 $EndComp
 $Comp
-L R R2
+L footswitch-rescue:R R2
 U 1 1 5589C484
 P 1850 3250
@@
 $EndComp
 $Comp
-L GNDD #PWR047
+L footswitch-rescue:GNDD #PWR047
 U 1 1 5589C48A
 P 1850 3750
@@
 $EndComp
 $Comp
-L CONN_01X02 P2
+L footswitch-rescue:CONN_01X02 P2
 U 1 1 5589C491
 P 1550 3550
@@
 F 3 "" H 1550 3550 60  0000 C CNN
 F 4 "M20-9960245" H -200 1600 50  0001 C CNN "MPN"
+F 5 "place on the back side" H 1550 3550 50  0001 C CNN "Note"
 	1    1550 3550
 	-1   0    0    -1
 $EndComp
 $Comp
-L +3.3V #PWR048
+L footswitch-rescue:+3.3V #PWR048
 U 1 1 5589C497
 P 1850 3000
@@
 $EndComp
 $Comp
-L R R12
+L footswitch-rescue:R R12
 U 1 1 5589C571
 P 2900 3250
@@
 $EndComp
 $Comp
-L GNDD #PWR049
+L footswitch-rescue:GNDD #PWR049
 U 1 1 5589C577
 P 2900 3750
@@
 $EndComp
 $Comp
-L CONN_01X02 P5
+L footswitch-rescue:CONN_01X02 P5
 U 1 1 5589C57E
 P 2600 3550
@@
 F 3 "" H 2600 3550 60  0000 C CNN
 F 4 "M20-9960245" H 850 1600 50  0001 C CNN "MPN"
+F 5 "place on the back side" H 2600 3550 50  0001 C CNN "Note"
 	1    2600 3550
 	-1   0    0    -1
 $EndComp
 $Comp
-L +3.3V #PWR050
+L footswitch-rescue:+3.3V #PWR050
 U 1 1 5589C584
 P 2900 3000
@@
 	1850 2000 1850 2100
 Wire Wire Line
-	1750 2100 1950 2100
+	1750 2100 1850 2100
 Wire Wire Line
 	1850 1600 1850 1700
@@
 	1850 2200 1850 2350
 Wire Wire Line
-	8750 1500 8750 2000
+	8750 1500 8750 1600
 Wire Wire Line
 	8750 2000 8650 2000
@@
 	8150 2000 8250 2000
 Wire Wire Line
-	8750 2500 8750 3000
+	8750 2500 8750 2600
 Wire Wire Line
 	8750 3000 8650 3000
@@
 	8150 3000 8250 3000
 Wire Wire Line
-	8750 3500 8750 4000
+	8750 3500 8750 3600
 Wire Wire Line
 	8750 4000 8650 4000
@@
 	8150 4000 8250 4000
 Wire Wire Line
-	8750 4500 8750 5000
+	8750 4500 8750 4600
 Wire Wire Line
 	8750 5000 8650 5000
@@
 	2900 2000 2900 2100
 Wire Wire Line
-	2800 2100 3000 2100
+	2800 2100 2900 2100
 Wire Wire Line
 	2900 1600 2900 1700
@@
 	1850 3400 1850 3500
 Wire Wire Line
-	1750 3500 1950 3500
+	1750 3500 1850 3500
 Wire Wire Line
 	1850 3000 1850 3100
@@
 	2900 3400 2900 3500
 Wire Wire Line
-	2800 3500 3000 3500
+	2800 3500 2900 3500
 Wire Wire Line
 	2900 3000 2900 3100
@@
 Wire Wire Line
 	8650 4600 8750 4600
+Wire Wire Line
+	1850 2100 1950 2100
+Wire Wire Line
+	8750 1800 8750 2000
+Wire Wire Line
+	8750 1600 8750 1800
+Wire Wire Line
+	8750 2800 8750 3000
+Wire Wire Line
+	8750 2600 8750 2800
+Wire Wire Line
+	8750 3800 8750 4000
+Wire Wire Line
+	8750 3600 8750 3800
+Wire Wire Line
+	8750 4800 8750 5000
+Wire Wire Line
+	8750 4600 8750 4800
+Wire Wire Line
+	2900 2100 3000 2100
+Wire Wire Line
+	1850 3500 1950 3500
+Wire Wire Line
+	2900 3500 3000 3500
 $EndSCHEMATC

Commit message: Changed R40 RE from pull-up to pull-down
Parts:
- D5, D6, D7, D8: symbol footswitch-rescue:LED_RGB -> footswitch-rescue:LED_RGB-footswitch-rescue
- P1, P2, P4, P5: symbol footswitch-rescue:CONN_01X02 -> footswitch-rescue:CONN_01X02-footswitch-rescue
- R1, R11, R12, R2, R23, R24, R25, R28, R29, R30, R31, R32, R33, R34, R35, R36: symbol footswitch-rescue:R -> footswitch-rescue:R-footswitch-rescue
Changed lines of the file:
@@
 $EndDescr
 $Comp
-L footswitch-rescue:R R1
+L footswitch-rescue:R-footswitch-rescue R1
 U 1 1 54CBEC53
 P 1850 1850
@@
 $EndComp
 $Comp
-L footswitch-rescue:GNDD #PWR039
+L footswitch-rescue:GNDD-footswitch-rescue #PWR039
 U 1 1 54E65047
 P 1850 2350
@@
 $EndComp
 $Comp
-L footswitch-rescue:CONN_01X02 P1
+L footswitch-rescue:CONN_01X02-footswitch-rescue P1
 U 1 1 54E6B5CA
 P 1550 2150
@@
 $EndComp
 $Comp
-L footswitch-rescue:+3.3V #PWR040
+L footswitch-rescue:+3.3V-footswitch-rescue #PWR040
 U 1 1 556F3C3C
 P 1850 1600
@@
 $EndComp
 $Comp
-L footswitch-rescue:+3.3V #PWR041
+L footswitch-rescue:+3.3V-footswitch-rescue #PWR041
 U 1 1 557A9EA8
 P 8750 1500
@@
 $EndComp
 $Comp
-L footswitch-rescue:R R23
+L footswitch-rescue:R-footswitch-rescue R23
 U 1 1 557AA39A
 P 8000 1600
@@
 $EndComp
 $Comp
-L footswitch-rescue:LED_RGB D5
+L footswitch-rescue:LED_RGB-footswitch-rescue D5
 U 1 1 557AAC2C
 P 8450 1800
@@
 $EndComp
 $Comp
-L footswitch-rescue:R R24
+L footswitch-rescue:R-footswitch-rescue R24
 U 1 1 557AADB8
 P 8000 1800
@@
 $EndComp
 $Comp
-L footswitch-rescue:R R25
+L footswitch-rescue:R-footswitch-rescue R25
 U 1 1 557AAE1B
 P 8000 2000
@@
 $EndComp
 $Comp
-L footswitch-rescue:+3.3V #PWR042
+L footswitch-rescue:+3.3V-footswitch-rescue #PWR042
 U 1 1 55899AA7
 P 8750 2500
@@
 $EndComp
 $Comp
-L footswitch-rescue:R R28
+L footswitch-rescue:R-footswitch-rescue R28
 U 1 1 55899AB4
 P 8000 2600
@@
 $EndComp
 $Comp
-L footswitch-rescue:LED_RGB D6
+L footswitch-rescue:LED_RGB-footswitch-rescue D6
 U 1 1 55899ABB
 P 8450 2800
@@
 $EndComp
 $Comp
-L footswitch-rescue:R R29
+L footswitch-rescue:R-footswitch-rescue R29
 U 1 1 55899AC2
 P 8000 2800
@@
 $EndComp
 $Comp
-L footswitch-rescue:R R30
+L footswitch-rescue:R-footswitch-rescue R30
 U 1 1 55899AC9
 P 8000 3000
@@
 $EndComp
 $Comp
-L footswitch-rescue:+3.3V #PWR043
+L footswitch-rescue:+3.3V-footswitch-rescue #PWR043
 U 1 1 5589B19A
 P 8750 3500
@@
 $EndComp
 $Comp
-L footswitch-rescue:R R31
+L footswitch-rescue:R-footswitch-rescue R31
 U 1 1 5589B1A7
 P 8000 3600
@@
 $EndComp
 $Comp
-L footswitch-rescue:LED_RGB D7
+L footswitch-rescue:LED_RGB-footswitch-rescue D7
 U 1 1 5589B1AE
 P 8450 3800
@@
 $EndComp
 $Comp
-L footswitch-rescue:R R32
+L footswitch-rescue:R-footswitch-rescue R32
 U 1 1 5589B1B5
 P 8000 3800
@@
 $EndComp
 $Comp
-L footswitch-rescue:R R33
+L footswitch-rescue:R-footswitch-rescue R33
 U 1 1 5589B1BC
 P 8000 4000
@@
 $EndComp
 $Comp
-L footswitch-rescue:+3.3V #PWR044
+L footswitch-rescue:+3.3V-footswitch-rescue #PWR044
 U 1 1 5589B1DB
 P 8750 4500
@@
 $EndComp
 $Comp
-L footswitch-rescue:R R34
+L footswitch-rescue:R-footswitch-rescue R34
 U 1 1 5589B1E8
 P 8000 4600
@@
 $EndComp
 $Comp
-L footswitch-rescue:LED_RGB D8
+L footswitch-rescue:LED_RGB-footswitch-rescue D8
 U 1 1 5589B1EF
 P 8450 4800
@@
 $EndComp
 $Comp
-L footswitch-rescue:R R35
+L footswitch-rescue:R-footswitch-rescue R35
 U 1 1 5589B1F6
 P 8000 4800
@@
 $EndComp
 $Comp
-L footswitch-rescue:R R36
+L footswitch-rescue:R-footswitch-rescue R36
 U 1 1 5589B1FD
 P 8000 5000
@@
 $EndComp
 $Comp
-L footswitch-rescue:R R11
+L footswitch-rescue:R-footswitch-rescue R11
 U 1 1 5589C3DA
 P 2900 1850
@@
 $EndComp
 $Comp
-L footswitch-rescue:GNDD #PWR045
+L footswitch-rescue:GNDD-footswitch-rescue #PWR045
 U 1 1 5589C3E0
 P 2900 2350
@@
 $EndComp
 $Comp
-L footswitch-rescue:CONN_01X02 P4
+L footswitch-rescue:CONN_01X02-footswitch-rescue P4
 U 1 1 5589C3E7
 P 2600 2150
@@
 $EndComp
 $Comp
-L footswitch-rescue:+3.3V #PWR046
+L footswitch-rescue:+3.3V-footswitch-rescue #PWR046
 U 1 1 5589C3ED
 P 2900 1600
@@
 $EndComp
 $Comp
-L footswitch-rescue:R R2
+L footswitch-rescue:R-footswitch-rescue R2
 U 1 1 5589C484
 P 1850 3250
@@
 $EndComp
 $Comp
-L footswitch-rescue:GNDD #PWR047
+L footswitch-rescue:GNDD-footswitch-rescue #PWR047
 U 1 1 5589C48A
 P 1850 3750
@@
 $EndComp
 $Comp
-L footswitch-rescue:CONN_01X02 P2
+L footswitch-rescue:CONN_01X02-footswitch-rescue P2
 U 1 1 5589C491
 P 1550 3550
@@
 $EndComp
 $Comp
-L footswitch-rescue:+3.3V #PWR048
+L footswitch-rescue:+3.3V-footswitch-rescue #PWR048
 U 1 1 5589C497
 P 1850 3000
@@
 $EndComp
 $Comp
-L footswitch-rescue:R R12
+L footswitch-rescue:R-footswitch-rescue R12
 U 1 1 5589C571
 P 2900 3250
@@
 $EndComp
 $Comp
-L footswitch-rescue:GNDD #PWR049
+L footswitch-rescue:GNDD-footswitch-rescue #PWR049
 U 1 1 5589C577
 P 2900 3750
@@
 $EndComp
 $Comp
-L footswitch-rescue:CONN_01X02 P5
+L footswitch-rescue:CONN_01X02-footswitch-rescue P5
 U 1 1 5589C57E
 P 2600 3550
@@
 $EndComp
 $Comp
-L footswitch-rescue:+3.3V #PWR050
+L footswitch-rescue:+3.3V-footswitch-rescue #PWR050
 U 1 1 5589C584
 P 2900 3000
