File: hw-design/board/display.sch (KiCad schematic (older format))
At the start: 12 parts, among them Q3 MMBT3904, U5 74HC245, U6 74HC245

Commit message: sch: schematic updated (missing displays circuit)
Parts:
- removed C14, C15, C17: 100nF_X7R, MOD_Footprints_Lib:SM0603, symbol C
- removed C16: 100uF, MOD_Footprints_Lib:CAP_RAD_5MM, symbol CP1
- removed LCD1: AGM-2004A-204, MOD_Footprints_Lib:LCD-AGM-2004A-204, symbol AGM-2004A-204
- removed Q3: MMBT3904, MOD_Footprints_Lib:SOT23, symbol NPN
- removed R34: 3k, MOD_Footprints_Lib:SM0805, symbol R
- removed R35: 330R, MOD_Footprints_Lib:SM0805, symbol R
- removed R36: 1k, MOD_Footprints_Lib:SM0603, symbol R
- removed R37: 0R, MOD_Footprints_Lib:SM0805, symbol R
- removed U5, U6: 74HC245, MOD_Footprints_Lib:TSSOP20, symbol 74HC245
Connections:
- net labels removed: +5V, DGND, LCD0, LCD1, LCD2, LCD3, LCD4, LCD5, LCD6, LCD7, LCD_E, LCD_RS, LCD_RW, UC_LCD0, UC_LCD1, UC_LCD2, UC_LCD3, UC_LCD4, UC_LCD5, UC_LCD6, UC_LCD7, UC_LCD_BACK, UC_LCD_DIR, UC_LCD_E, UC_LCD_RS, UC_LCD_RW
- wire segments 68 -> 0
- no-connect marks 10 -> 0

Commit message: sch: display circuit done
Parts:
- added C21, C24: 100nF, symbol C
- added C22, C25: 10uF, symbol C
- added C23: 47uF, symbol CP1
- added DS1, DS2: ERM1602FS-6 3.3V, Display:WC1602A, symbol RC1602A-GHW-ESX
- added Q10, Q8, Q9: 2N7002, symbol Q_NMOS_GSD
- added R41: 4K7, symbol R
- added R42: 680R, symbol R
- added R43, R44: 100K, symbol R
Connections:
- new net: DS1.16 (LED-), Q9.2 (S), R43.2
- new net: Q8.2 (S), R41.2, R42.1
- new net: DS2.16 (LED-), Q10.2 (S), R44.2
- new net +3V3: C21.1, C22.1, C24.1, C25.1, DS1.15 (LED+), DS1.2 (VDD), DS2.15 (LED+), DS2.2 (VDD), R41.1, R43.1, R44.1
- new net GNDD: C21.2, C22.2, C23.2, C24.2, C25.2, DS1.1 (VSS), DS1.10 (DB3), DS1.7 (DB0), DS1.8 (DB1), DS1.9 (DB2), DS2.1 (VSS), DS2.10 (DB3), DS2.7 (DB0), DS2.8 (DB1), DS2.9 (DB2), Q10.3 (D), Q8.3 (D), Q9.3 (D)
- new net LCD1_BL: Q9.1 (G)
- new net LCD1_EN: DS1.6 (E)
- new net LCD2_BL: Q10.1 (G)
- new net LCD2_EN: DS2.6 (E)
- new net LCD_CONTRAST: Q8.1 (G)
- new net LCD_D4: DS1.11 (DB4), DS2.11 (DB4)
- new net LCD_D5: DS1.12 (DB5), DS2.12 (DB5)
- new net LCD_D6: DS1.13 (DB6), DS2.13 (DB6)
- new net LCD_D7: DS1.14 (DB7), DS2.14 (DB7)
- new net LCD_RS: DS1.4 (RS), DS2.4 (RS)
- new net LCD_RW: DS1.5 (R/~W), DS2.5 (R/~W)
- new net LCD_VO: C23.1, DS1.3 (Vo), DS2.3 (Vo), R42.2
Other:
- note added: "LCD CONTRAST"

Commit message: sch: MPN added to all components
Parts:
- C21, C24: footprint (none) -> Capacitors_SMD:C_0603
- C22, C25: footprint (none) -> Capacitors_SMD:C_0805
- C23: footprint (none) -> Capacitors_SMD:c_elec_6.3x5.3; MPN (none) -> UWX1C470MCL1GB
- Q10, Q8, Q9: footprint (none) -> Housings_SOT-23_SOT-143_TSOT-6:SOT-23; MPN (none) -> 2N7002P,215
- R41: footprint (none) -> Resistors_SMD:R_0603; MPN (none) -> RMCF0603JT4K70
- R42: footprint (none) -> Resistors_SMD:R_0603; MPN (none) -> RMCF0603JT680R
- R43, R44: footprint (none) -> Resistors_SMD:R_0603; MPN (none) -> RMCF0603JT100K

Commit message: sch: fixing VBUS signal and FS1 I/O
Parts:
- renumbered R41 to R42, R42 to R43, R43 to R44, R44 to R45
Changed lines of the file:
@@
 $EndComp
 $Comp
-L +3.3V #PWR083
+L +3.3V #PWR82
 U 1 1 558A75D0
 P 2700 2600
-F 0 "#PWR083" H 2700 2450 50  0001 C CNN
+F 0 "#PWR82" H 2700 2450 50  0001 C CNN
 F 1 "+3.3V" H 2700 2740 50  0000 C CNN
 F 2 "" H 2700 2600 60  0000 C CNN
@@
 $EndComp
 $Comp
-L GNDD #PWR084
+L GNDD #PWR84
 U 1 1 558A75FC
 P 2950 2700
-F 0 "#PWR084" H 2950 2450 50  0001 C CNN
+F 0 "#PWR84" H 2950 2450 50  0001 C CNN
 F 1 "GNDD" H 2950 2550 50  0000 C CNN
 F 2 "" H 2950 2700 60  0000 C CNN
@@
 $EndComp
 $Comp
-L GNDD #PWR085
+L GNDD #PWR81
 U 1 1 558A7699
 P 2150 3300
-F 0 "#PWR085" H 2150 3050 50  0001 C CNN
+F 0 "#PWR81" H 2150 3050 50  0001 C CNN
 F 1 "GNDD" H 2150 3150 50  0000 C CNN
 F 2 "" H 2150 3300 60  0000 C CNN
@@
 $EndComp
 $Comp
-L GNDD #PWR086
+L GNDD #PWR85
 U 1 1 558A77CB
 P 3700 2700
-F 0 "#PWR086" H 3700 2450 50  0001 C CNN
+F 0 "#PWR85" H 3700 2450 50  0001 C CNN
 F 1 "GNDD" H 3700 2550 50  0000 C CNN
 F 2 "" H 3700 2700 60  0000 C CNN
@@
 $EndComp
 $Comp
-L GNDD #PWR087
+L GNDD #PWR88
 U 1 1 558A7B13
 P 4750 3250
-F 0 "#PWR087" H 4750 3000 50  0001 C CNN
+F 0 "#PWR88" H 4750 3000 50  0001 C CNN
 F 1 "GNDD" H 4750 3100 50  0000 C CNN
 F 2 "" H 4750 3250 60  0000 C CNN
@@
 $EndComp
 $Comp
-L R R43
+L R R44
 U 1 1 558A7C00
 P 4750 2400
-F 0 "R43" V 4830 2400 50  0000 C CNN
+F 0 "R44" V 4830 2400 50  0000 C CNN
 F 1 "100K" V 4750 2400 50  0000 C CNN
 F 2 "Resistors_SMD:R_0603" V 4680 2400 30  0000 C CNN
@@
 $EndComp
 $Comp
-L +3.3V #PWR088
+L +3.3V #PWR87
 U 1 1 558A7C5A
 P 4750 2150
-F 0 "#PWR088" H 4750 2000 50  0001 C CNN
+F 0 "#PWR87" H 4750 2000 50  0001 C CNN
 F 1 "+3.3V" H 4750 2290 50  0000 C CNN
 F 2 "" H 4750 2150 60  0000 C CNN
@@
 $EndComp
 $Comp
-L +3.3V #PWR089
+L +3.3V #PWR86
 U 1 1 558A7D34
 P 4550 2850
-F 0 "#PWR089" H 4550 2700 50  0001 C CNN
+F 0 "#PWR86" H 4550 2700 50  0001 C CNN
 F 1 "+3.3V" H 4550 2990 50  0000 C CNN
 F 2 "" H 4550 2850 60  0000 C CNN
@@
 $EndComp
 $Comp
-L GNDD #PWR090
+L GNDD #PWR80
 U 1 1 558A8A45
 P 2100 6500
-F 0 "#PWR090" H 2100 6250 50  0001 C CNN
+F 0 "#PWR80" H 2100 6250 50  0001 C CNN
 F 1 "GNDD" H 2100 6350 50  0000 C CNN
 F 2 "" H 2100 6500 60  0000 C CNN
@@
 $EndComp
 $Comp
-L R R41
+L R R42
 U 1 1 558A8A4C
 P 2100 5650
-F 0 "R41" V 2180 5650 50  0000 C CNN
+F 0 "R42" V 2180 5650 50  0000 C CNN
 F 1 "4K7" V 2100 5650 50  0000 C CNN
 F 2 "Resistors_SMD:R_0603" V 2030 5650 30  0000 C CNN
@@
 $EndComp
 $Comp
-L +3.3V #PWR091
+L +3.3V #PWR79
 U 1 1 558A8A52
 P 2100 5400
-F 0 "#PWR091" H 2100 5250 50  0001 C CNN
+F 0 "#PWR79" H 2100 5250 50  0001 C CNN
 F 1 "+3.3V" H 2100 5540 50  0000 C CNN
 F 2 "" H 2100 5400 60  0000 C CNN
@@
 $EndComp
 $Comp
-L R R42
+L R R43
 U 1 1 558A8AE2
 P 2400 5900
-F 0 "R42" V 2480 5900 50  0000 C CNN
+F 0 "R43" V 2480 5900 50  0000 C CNN
 F 1 "680R" V 2400 5900 50  0000 C CNN
 F 2 "Resistors_SMD:R_0603" V 2330 5900 30  0000 C CNN
@@
 $EndComp
 $Comp
-L GNDD #PWR092
+L GNDD #PWR83
 U 1 1 558A9218
 P 2700 6450
-F 0 "#PWR092" H 2700 6200 50  0001 C CNN
+F 0 "#PWR83" H 2700 6200 50  0001 C CNN
 F 1 "GNDD" H 2700 6300 50  0000 C CNN
 F 2 "" H 2700 6450 60  0000 C CNN
@@
 $EndComp
 $Comp
-L +3.3V #PWR093
+L +3.3V #PWR90
 U 1 1 558AA390
 P 6750 2600
-F 0 "#PWR093" H 6750 2450 50  0001 C CNN
+F 0 "#PWR90" H 6750 2450 50  0001 C CNN
 F 1 "+3.3V" H 6750 2740 50  0000 C CNN
 F 2 "" H 6750 2600 60  0000 C CNN
@@
 $EndComp
 $Comp
-L GNDD #PWR094
+L GNDD #PWR91
 U 1 1 558AA396
 P 7000 2700
-F 0 "#PWR094" H 7000 2450 50  0001 C CNN
+F 0 "#PWR91" H 7000 2450 50  0001 C CNN
 F 1 "GNDD" H 7000 2550 50  0000 C CNN
 F 2 "" H 7000 2700 60  0000 C CNN
@@
 $EndComp
 $Comp
-L GNDD #PWR095
+L GNDD #PWR89
 U 1 1 558AA3A8
 P 6200 3300
-F 0 "#PWR095" H 6200 3050 50  0001 C CNN
+F 0 "#PWR89" H 6200 3050 50  0001 C CNN
 F 1 "GNDD" H 6200 3150 50  0000 C CNN
 F 2 "" H 6200 3300 60  0000 C CNN
@@
 $EndComp
 $Comp
-L GNDD #PWR096
+L GNDD #PWR92
 U 1 1 558AA3AE
 P 7750 2700
-F 0 "#PWR096" H 7750 2450 50  0001 C CNN
+F 0 "#PWR92" H 7750 2450 50  0001 C CNN
 F 1 "GNDD" H 7750 2550 50  0000 C CNN
 F 2 "" H 7750 2700 60  0000 C CNN
@@
 $EndComp
 $Comp
-L GNDD #PWR097
+L GNDD #PWR95
 U 1 1 558AA3BA
 P 8800 3250
-F 0 "#PWR097" H 8800 3000 50  0001 C CNN
+F 0 "#PWR95" H 8800 3000 50  0001 C CNN
 F 1 "GNDD" H 8800 3100 50  0000 C CNN
 F 2 "" H 8800 3250 60  0000 C CNN
@@
 $EndComp
 $Comp
-L R R44
+L R R45
 U 1 1 558AA3C1
 P 8800 2400
-F 0 "R44" V 8880 2400 50  0000 C CNN
+F 0 "R45" V 8880 2400 50  0000 C CNN
 F 1 "100K" V 8800 2400 50  0000 C CNN
 F 2 "Resistors_SMD:R_0603" V 8730 2400 30  0000 C CNN
@@
 $EndComp
 $Comp
-L +3.3V #PWR098
+L +3.3V #PWR94
 U 1 1 558AA3C7
 P 8800 2150
-F 0 "#PWR098" H 8800 2000 50  0001 C CNN
+F 0 "#PWR94" H 8800 2000 50  0001 C CNN
 F 1 "+3.3V" H 8800 2290 50  0000 C CNN
 F 2 "" H 8800 2150 60  0000 C CNN
@@
 $EndComp
 $Comp
-L +3.3V #PWR099
+L +3.3V #PWR93
 U 1 1 558AA3CD
 P 8600 2850
-F 0 "#PWR099" H 8600 2700 50  0001 C CNN
+F 0 "#PWR93" H 8600 2700 50  0001 C CNN
 F 1 "+3.3V" H 8600 2990 50  0000 C CNN
 F 2 "" H 8600 2850 60  0000 C CNN

Commit message: sch: channel selector switch is no longer used
Parts:
- renumbered R42 to R39, R43 to R40, R44 to R41, R45 to R42
Changed lines of the file:
@@
 $EndComp
 $Comp
-L +3.3V #PWR084
+L +3.3V #PWR082
 U 1 1 558A75D0
 P 2700 2600
-F 0 "#PWR084" H 2700 2450 50  0001 C CNN
+F 0 "#PWR082" H 2700 2450 50  0001 C CNN
 F 1 "+3.3V" H 2700 2740 50  0000 C CNN
 F 2 "" H 2700 2600 60  0000 C CNN
@@
 $EndComp
 $Comp
-L GNDD #PWR085
+L GNDD #PWR083
 U 1 1 558A75FC
 P 2950 2700
-F 0 "#PWR085" H 2950 2450 50  0001 C CNN
+F 0 "#PWR083" H 2950 2450 50  0001 C CNN
 F 1 "GNDD" H 2950 2550 50  0000 C CNN
 F 2 "" H 2950 2700 60  0000 C CNN
@@
 $EndComp
 $Comp
-L GNDD #PWR086
+L GNDD #PWR084
 U 1 1 558A7699
 P 2150 3300
-F 0 "#PWR086" H 2150 3050 50  0001 C CNN
+F 0 "#PWR084" H 2150 3050 50  0001 C CNN
 F 1 "GNDD" H 2150 3150 50  0000 C CNN
 F 2 "" H 2150 3300 60  0000 C CNN
@@
 $EndComp
 $Comp
-L GNDD #PWR087
+L GNDD #PWR085
 U 1 1 558A77CB
 P 3700 2700
-F 0 "#PWR087" H 3700 2450 50  0001 C CNN
+F 0 "#PWR085" H 3700 2450 50  0001 C CNN
 F 1 "GNDD" H 3700 2550 50  0000 C CNN
 F 2 "" H 3700 2700 60  0000 C CNN
@@
 $EndComp
 $Comp
-L GNDD #PWR088
+L GNDD #PWR086
 U 1 1 558A7B13
 P 4750 3250
-F 0 "#PWR088" H 4750 3000 50  0001 C CNN
+F 0 "#PWR086" H 4750 3000 50  0001 C CNN
 F 1 "GNDD" H 4750 3100 50  0000 C CNN
 F 2 "" H 4750 3250 60  0000 C CNN
@@
 $EndComp
 $Comp
-L R R44
+L R R41
 U 1 1 558A7C00
 P 4750 2400
-F 0 "R44" V 4830 2400 50  0000 C CNN
+F 0 "R41" V 4830 2400 50  0000 C CNN
 F 1 "100K" V 4750 2400 50  0000 C CNN
 F 2 "Resistors_SMD:R_0603" V 4680 2400 30  0000 C CNN
@@
 $EndComp
 $Comp
-L +3.3V #PWR089
+L +3.3V #PWR087
 U 1 1 558A7C5A
 P 4750 2150
-F 0 "#PWR089" H 4750 2000 50  0001 C CNN
+F 0 "#PWR087" H 4750 2000 50  0001 C CNN
 F 1 "+3.3V" H 4750 2290 50  0000 C CNN
 F 2 "" H 4750 2150 60  0000 C CNN
@@
 $EndComp
 $Comp
-L +3.3V #PWR090
+L +3.3V #PWR088
 U 1 1 558A7D34
 P 4550 2850
-F 0 "#PWR090" H 4550 2700 50  0001 C CNN
+F 0 "#PWR088" H 4550 2700 50  0001 C CNN
 F 1 "+3.3V" H 4550 2990 50  0000 C CNN
 F 2 "" H 4550 2850 60  0000 C CNN
@@
 $EndComp
 $Comp
-L GNDD #PWR091
+L GNDD #PWR089
 U 1 1 558A8A45
 P 2100 6500
-F 0 "#PWR091" H 2100 6250 50  0001 C CNN
+F 0 "#PWR089" H 2100 6250 50  0001 C CNN
 F 1 "GNDD" H 2100 6350 50  0000 C CNN
 F 2 "" H 2100 6500 60  0000 C CNN
@@
 $EndComp
 $Comp
-L R R42
+L R R39
 U 1 1 558A8A4C
 P 2100 5650
-F 0 "R42" V 2180 5650 50  0000 C CNN
+F 0 "R39" V 2180 5650 50  0000 C CNN
 F 1 "4K7" V 2100 5650 50  0000 C CNN
 F 2 "Resistors_SMD:R_0603" V 2030 5650 30  0000 C CNN
@@
 $EndComp
 $Comp
-L +3.3V #PWR092
+L +3.3V #PWR090
 U 1 1 558A8A52
 P 2100 5400
-F 0 "#PWR092" H 2100 5250 50  0001 C CNN
+F 0 "#PWR090" H 2100 5250 50  0001 C CNN
 F 1 "+3.3V" H 2100 5540 50  0000 C CNN
 F 2 "" H 2100 5400 60  0000 C CNN
@@
 $EndComp
 $Comp
-L R R43
+L R R40
 U 1 1 558A8AE2
 P 2400 5900
-F 0 "R43" V 2480 5900 50  0000 C CNN
+F 0 "R40" V 2480 5900 50  0000 C CNN
 F 1 "680R" V 2400 5900 50  0000 C CNN
 F 2 "Resistors_SMD:R_0603" V 2330 5900 30  0000 C CNN
@@
 $EndComp
 $Comp
-L GNDD #PWR093
+L GNDD #PWR091
 U 1 1 558A9218
 P 2700 6450
-F 0 "#PWR093" H 2700 6200 50  0001 C CNN
+F 0 "#PWR091" H 2700 6200 50  0001 C CNN
 F 1 "GNDD" H 2700 6300 50  0000 C CNN
 F 2 "" H 2700 6450 60  0000 C CNN
@@
 $EndComp
 $Comp
-L +3.3V #PWR094
+L +3.3V #PWR092
 U 1 1 558AA390
 P 6750 2600
-F 0 "#PWR094" H 6750 2450 50  0001 C CNN
+F 0 "#PWR092" H 6750 2450 50  0001 C CNN
 F 1 "+3.3V" H 6750 2740 50  0000 C CNN
 F 2 "" H 6750 2600 60  0000 C CNN
@@
 $EndComp
 $Comp
-L GNDD #PWR095
+L GNDD #PWR093
 U 1 1 558AA396
 P 7000 2700
-F 0 "#PWR095" H 7000 2450 50  0001 C CNN
+F 0 "#PWR093" H 7000 2450 50  0001 C CNN
 F 1 "GNDD" H 7000 2550 50  0000 C CNN
 F 2 "" H 7000 2700 60  0000 C CNN
@@
 $EndComp
 $Comp
-L GNDD #PWR096
+L GNDD #PWR094
 U 1 1 558AA3A8
 P 6200 3300
-F 0 "#PWR096" H 6200 3050 50  0001 C CNN
+F 0 "#PWR094" H 6200 3050 50  0001 C CNN
 F 1 "GNDD" H 6200 3150 50  0000 C CNN
 F 2 "" H 6200 3300 60  0000 C CNN
@@
 $EndComp
 $Comp
-L GNDD #PWR097
+L GNDD #PWR095
 U 1 1 558AA3AE
 P 7750 2700
-F 0 "#PWR097" H 7750 2450 50  0001 C CNN
+F 0 "#PWR095" H 7750 2450 50  0001 C CNN
 F 1 "GNDD" H 7750 2550 50  0000 C CNN
 F 2 "" H 7750 2700 60  0000 C CNN
@@
 $EndComp
 $Comp
-L GNDD #PWR098
+L GNDD #PWR096
 U 1 1 558AA3BA
 P 8800 3250
-F 0 "#PWR098" H 8800 3000 50  0001 C CNN
+F 0 "#PWR096" H 8800 3000 50  0001 C CNN
 F 1 "GNDD" H 8800 3100 50  0000 C CNN
 F 2 "" H 8800 3250 60  0000 C CNN
@@
 $EndComp
 $Comp
-L R R45
+L R R42
 U 1 1 558AA3C1
 P 8800 2400
-F 0 "R45" V 8880 2400 50  0000 C CNN
+F 0 "R42" V 8880 2400 50  0000 C CNN
 F 1 "100K" V 8800 2400 50  0000 C CNN
 F 2 "Resistors_SMD:R_0603" V 8730 2400 30  0000 C CNN
@@
 $EndComp
 $Comp
-L +3.3V #PWR099
+L +3.3V #PWR097
 U 1 1 558AA3C7
 P 8800 2150
-F 0 "#PWR099" H 8800 2000 50  0001 C CNN
+F 0 "#PWR097" H 8800 2000 50  0001 C CNN
 F 1 "+3.3V" H 8800 2290 50  0000 C CNN
 F 2 "" H 8800 2150 60  0000 C CNN
@@
 $EndComp
 $Comp
-L +3.3V #PWR0100
+L +3.3V #PWR098
 U 1 1 558AA3CD
 P 8600 2850
-F 0 "#PWR0100" H 8600 2700 50  0001 C CNN
+F 0 "#PWR098" H 8600 2700 50  0001 C CNN
 F 1 "+3.3V" H 8600 2990 50  0000 C CNN
 F 2 "" H 8600 2850 60  0000 C CNN
