File: hw-design/board/display.sch (KiCad schematic (older format))
At the start: 14 parts, among them Q10 2N7002, Q8 2N7002, Q9 2N7002

Commit message: sch: increasing display holes
Parts:
- DS1, DS2: footprint Display:WC1602A -> local-footprints:WC1602A
Changed lines of the file:
@@
 F 0 "DS1" H 2900 2500 40  0000 C CNN
 F 1 "ERM1602FS-6 3.3V" H 4250 2500 40  0000 C CNN
-F 2 "Display:WC1602A" H 3700 2050 35  0000 C CIN
+F 2 "local-footprints:WC1602A" H 3700 2050 35  0000 C CIN
 F 3 "" H 3700 2100 60  0000 C CNN
 F 4 "ERM1602FS-6" H 3700 2100 60  0001 C CNN "MPN"
@@
 F 0 "DS2" H 6950 2500 40  0000 C CNN
 F 1 "ERM1602FS-6 3.3V" H 8300 2500 40  0000 C CNN
-F 2 "Display:WC1602A" H 7750 2050 35  0000 C CIN
+F 2 "local-footprints:WC1602A" H 7750 2050 35  0000 C CIN
 F 3 "" H 7750 2100 60  0000 C CNN
 F 4 "ERM1602FS-6" H 7750 2100 60  0001 C CNN "MPN"

Commit message: sch: schematic files reorganized, new sheets for usb and rear board
Parts:
- renumbered C21 to C18, C22 to C19, C23 to C20, C24 to C21, C25 to C22, Q8 to Q4, Q9 to Q5, Q10 to Q6, R39 to R23, R40 to R24, R41 to R25, R42 to R26
Changed lines of the file:
@@
 $Descr A4 11693 8268
 encoding utf-8
-Sheet 6 7
+Sheet 6 9
 Title "MOD Footswitch Extensor"
 Date "Tue 09 Dec 2014"
@@
 $EndComp
 $Comp
-L +3.3V #PWR082
+L +3.3V #PWR065
 U 1 1 558A75D0
 P 2700 2600
-F 0 "#PWR082" H 2700 2450 50  0001 C CNN
+F 0 "#PWR065" H 2700 2450 50  0001 C CNN
 F 1 "+3.3V" H 2700 2740 50  0000 C CNN
 F 2 "" H 2700 2600 60  0000 C CNN
@@
 $EndComp
 $Comp
-L GNDD #PWR083
+L GNDD #PWR066
 U 1 1 558A75FC
 P 2950 2700
-F 0 "#PWR083" H 2950 2450 50  0001 C CNN
+F 0 "#PWR066" H 2950 2450 50  0001 C CNN
 F 1 "GNDD" H 2950 2550 50  0000 C CNN
 F 2 "" H 2950 2700 60  0000 C CNN
@@
 $EndComp
 $Comp
-L C C21
+L C C18
 U 1 1 558A7629
 P 2150 2950
-F 0 "C21" H 2175 3050 50  0000 L CNN
+F 0 "C18" H 2175 3050 50  0000 L CNN
 F 1 "100nF" H 2175 2850 50  0000 L CNN
 F 2 "Capacitors_SMD:C_0603" H 2188 2800 30  0000 C CNN
@@
 $EndComp
 $Comp
-L GNDD #PWR084
+L GNDD #PWR067
 U 1 1 558A7699
 P 2150 3300
-F 0 "#PWR084" H 2150 3050 50  0001 C CNN
+F 0 "#PWR067" H 2150 3050 50  0001 C CNN
 F 1 "GNDD" H 2150 3150 50  0000 C CNN
 F 2 "" H 2150 3300 60  0000 C CNN
@@
 $EndComp
 $Comp
-L GNDD #PWR085
+L GNDD #PWR068
 U 1 1 558A77CB
 P 3700 2700
-F 0 "#PWR085" H 3700 2450 50  0001 C CNN
+F 0 "#PWR068" H 3700 2450 50  0001 C CNN
 F 1 "GNDD" H 3700 2550 50  0000 C CNN
 F 2 "" H 3700 2700 60  0000 C CNN
@@
 $EndComp
 $Comp
-L Q_NMOS_GSD Q9
+L Q_NMOS_GSD Q5
 U 1 1 558A78F3
 P 4850 2950
-F 0 "Q9" H 4750 2900 50  0000 R CNN
+F 0 "Q5" H 4750 2900 50  0000 R CNN
 F 1 "2N7002" H 4800 2800 50  0000 R CNN
 F 2 "Housings_SOT-23_SOT-143_TSOT-6:SOT-23" H 5050 3050 29  0000 C CNN
@@
 $EndComp
 $Comp
-L GNDD #PWR086
+L GNDD #PWR069
 U 1 1 558A7B13
 P 4750 3250
-F 0 "#PWR086" H 4750 3000 50  0001 C CNN
+F 0 "#PWR069" H 4750 3000 50  0001 C CNN
 F 1 "GNDD" H 4750 3100 50  0000 C CNN
 F 2 "" H 4750 3250 60  0000 C CNN
@@
 $EndComp
 $Comp
-L R R41
+L R R25
 U 1 1 558A7C00
 P 4750 2400
-F 0 "R41" V 4830 2400 50  0000 C CNN
+F 0 "R25" V 4830 2400 50  0000 C CNN
 F 1 "100K" V 4750 2400 50  0000 C CNN
 F 2 "Resistors_SMD:R_0603" V 4680 2400 30  0000 C CNN
@@
 $EndComp
 $Comp
-L +3.3V #PWR087
+L +3.3V #PWR070
 U 1 1 558A7C5A
 P 4750 2150
-F 0 "#PWR087" H 4750 2000 50  0001 C CNN
+F 0 "#PWR070" H 4750 2000 50  0001 C CNN
 F 1 "+3.3V" H 4750 2290 50  0000 C CNN
 F 2 "" H 4750 2150 60  0000 C CNN
@@
 $EndComp
 $Comp
-L +3.3V #PWR088
+L +3.3V #PWR071
 U 1 1 558A7D34
 P 4550 2850
-F 0 "#PWR088" H 4550 2700 50  0001 C CNN
+F 0 "#PWR071" H 4550 2700 50  0001 C CNN
 F 1 "+3.3V" H 4550 2990 50  0000 C CNN
 F 2 "" H 4550 2850 60  0000 C CNN
@@
 $EndComp
 $Comp
-L Q_NMOS_GSD Q8
+L Q_NMOS_GSD Q4
 U 1 1 558A8A3F
 P 2000 6200
-F 0 "Q8" H 1900 6150 50  0000 R CNN
+F 0 "Q4" H 1900 6150 50  0000 R CNN
 F 1 "2N7002" H 1950 6050 50  0000 R CNN
 F 2 "Housings_SOT-23_SOT-143_TSOT-6:SOT-23" H 2200 6300 29  0000 C CNN
@@
 $EndComp
 $Comp
-L GNDD #PWR089
+L GNDD #PWR072
 U 1 1 558A8A45
 P 2100 6500
-F 0 "#PWR089" H 2100 6250 50  0001 C CNN
+F 0 "#PWR072" H 2100 6250 50  0001 C CNN
 F 1 "GNDD" H 2100 6350 50  0000 C CNN
 F 2 "" H 2100 6500 60  0000 C CNN
@@
 $EndComp
 $Comp
-L R R39
+L R R23
 U 1 1 558A8A4C
 P 2100 5650
-F 0 "R39" V 2180 5650 50  0000 C CNN
+F 0 "R23" V 2180 5650 50  0000 C CNN
 F 1 "4K7" V 2100 5650 50  0000 C CNN
 F 2 "Resistors_SMD:R_0603" V 2030 5650 30  0000 C CNN
@@
 $EndComp
 $Comp
-L +3.3V #PWR090
+L +3.3V #PWR073
 U 1 1 558A8A52
 P 2100 5400
-F 0 "#PWR090" H 2100 5250 50  0001 C CNN
+F 0 "#PWR073" H 2100 5250 50  0001 C CNN
 F 1 "+3.3V" H 2100 5540 50  0000 C CNN
 F 2 "" H 2100 5400 60  0000 C CNN
@@
 $EndComp
 $Comp
-L R R40
+L R R24
 U 1 1 558A8AE2
 P 2400 5900
-F 0 "R40" V 2480 5900 50  0000 C CNN
+F 0 "R24" V 2480 5900 50  0000 C CNN
 F 1 "680R" V 2400 5900 50  0000 C CNN
 F 2 "Resistors_SMD:R_0603" V 2330 5900 30  0000 C CNN
@@
 $EndComp
 $Comp
-L CP1 C23
+L CP1 C20
 U 1 1 558A8E3B
 P 2700 6200
-F 0 "C23" H 2725 6300 50  0000 L CNN
+F 0 "C20" H 2725 6300 50  0000 L CNN
 F 1 "47uF" H 2725 6100 50  0000 L CNN
 F 2 "Capacitors_SMD:c_elec_6.3x5.3" H 2700 6200 60  0000 C CNN
@@
 $EndComp
 $Comp
-L GNDD #PWR091
+L GNDD #PWR074
 U 1 1 558A9218
 P 2700 6450
-F 0 "#PWR091" H 2700 6200 50  0001 C CNN
+F 0 "#PWR074" H 2700 6200 50  0001 C CNN
 F 1 "GNDD" H 2700 6300 50  0000 C CNN
 F 2 "" H 2700 6450 60  0000 C CNN
@@
 $EndComp
 $Comp
-L +3.3V #PWR092
+L +3.3V #PWR075
 U 1 1 558AA390
 P 6750 2600
-F 0 "#PWR092" H 6750 2450 50  0001 C CNN
+F 0 "#PWR075" H 6750 2450 50  0001 C CNN
 F 1 "+3.3V" H 6750 2740 50  0000 C CNN
 F 2 "" H 6750 2600 60  0000 C CNN
@@
 $EndComp
 $Comp
-L GNDD #PWR093
+L GNDD #PWR076
 U 1 1 558AA396
 P 7000 2700
-F 0 "#PWR093" H 7000 2450 50  0001 C CNN
+F 0 "#PWR076" H 7000 2450 50  0001 C CNN
 F 1 "GNDD" H 7000 2550 50  0000 C CNN
 F 2 "" H 7000 2700 60  0000 C CNN
@@
 $EndComp
 $Comp
-L C C24
+L C C21
 U 1 1 558AA39C
 P 6200 2950
-F 0 "C24" H 6225 3050 50  0000 L CNN
+F 0 "C21" H 6225 3050 50  0000 L CNN
 F 1 "100nF" H 6225 2850 50  0000 L CNN
 F 2 "Capacitors_SMD:C_0603" H 6238 2800 30  0000 C CNN
@@
 $EndComp
 $Comp
-L GNDD #PWR094
+L GNDD #PWR077
 U 1 1 558AA3A8
 P 6200 3300
-F 0 "#PWR094" H 6200 3050 50  0001 C CNN
+F 0 "#PWR077" H 6200 3050 50  0001 C CNN
 F 1 "GNDD" H 6200 3150 50  0000 C CNN
 F 2 "" H 6200 3300 60  0000 C CNN
@@
 $EndComp
 $Comp
-L GNDD #PWR095
+L GNDD #PWR078
 U 1 1 558AA3AE
 P 7750 2700
-F 0 "#PWR095" H 7750 2450 50  0001 C CNN
+F 0 "#PWR078" H 7750 2450 50  0001 C CNN
 F 1 "GNDD" H 7750 2550 50  0000 C CNN
 F 2 "" H 7750 2700 60  0000 C CNN
@@
 $EndComp
 $Comp
-L Q_NMOS_GSD Q10
+L Q_NMOS_GSD Q6
 U 1 1 558AA3B4
 P 8900 2950
-F 0 "Q10" H 8800 2900 50  0000 R CNN
+F 0 "Q6" H 8800 2900 50  0000 R CNN
 F 1 "2N7002" H 8850 2800 50  0000 R CNN
 F 2 "Housings_SOT-23_SOT-143_TSOT-6:SOT-23" H 9100 3050 29  0000 C CNN
@@
 $EndComp
 $Comp
-L GNDD #PWR096
+L GNDD #PWR079
 U 1 1 558AA3BA
 P 8800 3250
-F 0 "#PWR096" H 8800 3000 50  0001 C CNN
+F 0 "#PWR079" H 8800 3000 50  0001 C CNN
 F 1 "GNDD" H 8800 3100 50  0000 C CNN
 F 2 "" H 8800 3250 60  0000 C CNN
@@
 $EndComp
 $Comp
-L R R42
+L R R26
 U 1 1 558AA3C1
 P 8800 2400
-F 0 "R42" V 8880 2400 50  0000 C CNN
+F 0 "R26" V 8880 2400 50  0000 C CNN
 F 1 "100K" V 8800 2400 50  0000 C CNN
 F 2 "Resistors_SMD:R_0603" V 8730 2400 30  0000 C CNN
@@
 $EndComp
 $Comp
-L +3.3V #PWR097
+L +3.3V #PWR080
 U 1 1 558AA3C7
 P 8800 2150
-F 0 "#PWR097" H 8800 2000 50  0001 C CNN
+F 0 "#PWR080" H 8800 2000 50  0001 C CNN
 F 1 "+3.3V" H 8800 2290 50  0000 C CNN
 F 2 "" H 8800 2150 60  0000 C CNN
@@
 $EndComp
 $Comp
-L +3.3V #PWR098
+L +3.3V #PWR081
 U 1 1 558AA3CD
 P 8600 2850
-F 0 "#PWR098" H 8600 2700 50  0001 C CNN
+F 0 "#PWR081" H 8600 2700 50  0001 C CNN
 F 1 "+3.3V" H 8600 2990 50  0000 C CNN
 F 2 "" H 8600 2850 60  0000 C CNN
@@
 $EndComp
 $Comp
-L C C22
+L C C19
 U 1 1 558AACB8
 P 2500 2950
-F 0 "C22" H 2525 3050 50  0000 L CNN
+F 0 "C19" H 2525 3050 50  0000 L CNN
 F 1 "10uF" H 2525 2850 50  0000 L CNN
 F 2 "Capacitors_SMD:C_0805" H 2538 2800 30  0000 C CNN
@@
 $EndComp
 $Comp
-L C C25
+L C C22
 U 1 1 558AACEE
 P 6550 2950
-F 0 "C25" H 6575 3050 50  0000 L CNN
+F 0 "C22" H 6575 3050 50  0000 L CNN
 F 1 "10uF" H 6575 2850 50  0000 L CNN
 F 2 "Capacitors_SMD:C_0805" H 6588 2800 30  0000 C CNN

Commit message: annotation and ERC
Parts:
- renumbered C18 to C1, C21 to C15, C22 to C16, C19 to C2, C20 to C3, Q4 to Q1, Q5 to Q7, Q6 to Q8, R25 to R19, R26 to R35, R23 to R5, R24 to R8
Changed lines of the file:
@@
 $EndComp
 $Comp
-L +3.3V #PWR065
+L +3.3V #PWR15
 U 1 1 558A75D0
 P 2700 2600
-F 0 "#PWR065" H 2700 2450 50  0001 C CNN
+F 0 "#PWR15" H 2700 2450 50  0001 C CNN
 F 1 "+3.3V" H 2700 2740 50  0000 C CNN
 F 2 "" H 2700 2600 60  0000 C CNN
@@
 $EndComp
 $Comp
-L GNDD #PWR066
+L GNDD #PWR21
 U 1 1 558A75FC
 P 2950 2700
-F 0 "#PWR066" H 2950 2450 50  0001 C CNN
+F 0 "#PWR21" H 2950 2450 50  0001 C CNN
 F 1 "GNDD" H 2950 2550 50  0000 C CNN
 F 2 "" H 2950 2700 60  0000 C CNN
@@
 $EndComp
 $Comp
-L C C18
+L C C1
 U 1 1 558A7629
 P 2150 2950
-F 0 "C18" H 2175 3050 50  0000 L CNN
+F 0 "C1" H 2175 3050 50  0000 L CNN
 F 1 "100nF" H 2175 2850 50  0000 L CNN
-F 2 "Capacitors_SMD:C_0603" H 2188 2800 30  0000 C CNN
+F 2 "Capacitors_SMD:C_0603" H 2188 2800 30  0001 C CNN
 F 3 "" H 2150 2950 60  0000 C CNN
 F 4 "C1608X7R1E104K080AA" H 2150 2950 60  0001 C CNN "MPN"
@@
 $EndComp
 $Comp
-L GNDD #PWR067
+L GNDD #PWR11
 U 1 1 558A7699
 P 2150 3300
-F 0 "#PWR067" H 2150 3050 50  0001 C CNN
+F 0 "#PWR11" H 2150 3050 50  0001 C CNN
 F 1 "GNDD" H 2150 3150 50  0000 C CNN
 F 2 "" H 2150 3300 60  0000 C CNN
@@
 $EndComp
 $Comp
-L GNDD #PWR068
+L GNDD #PWR34
 U 1 1 558A77CB
 P 3700 2700
-F 0 "#PWR068" H 3700 2450 50  0001 C CNN
+F 0 "#PWR34" H 3700 2450 50  0001 C CNN
 F 1 "GNDD" H 3700 2550 50  0000 C CNN
 F 2 "" H 3700 2700 60  0000 C CNN
@@
 $EndComp
 $Comp
-L Q_NMOS_GSD Q5
+L Q_NMOS_GSD Q7
 U 1 1 558A78F3
 P 4850 2950
-F 0 "Q5" H 4750 2900 50  0000 R CNN
+F 0 "Q7" H 4750 2900 50  0000 R CNN
 F 1 "2N7002" H 4800 2800 50  0000 R CNN
-F 2 "Housings_SOT-23_SOT-143_TSOT-6:SOT-23" H 5050 3050 29  0000 C CNN
+F 2 "Housings_SOT-23_SOT-143_TSOT-6:SOT-23" H 5050 3050 29  0001 C CNN
 F 3 "" H 4850 2950 60  0000 C CNN
 F 4 "2N7002P,215" H 0   0   50  0001 C CNN "MPN"
@@
 $EndComp
 $Comp
-L GNDD #PWR069
+L GNDD #PWR43
 U 1 1 558A7B13
 P 4750 3250
-F 0 "#PWR069" H 4750 3000 50  0001 C CNN
+F 0 "#PWR43" H 4750 3000 50  0001 C CNN
 F 1 "GNDD" H 4750 3100 50  0000 C CNN
 F 2 "" H 4750 3250 60  0000 C CNN
@@
 $EndComp
 $Comp
-L R R25
+L R R19
 U 1 1 558A7C00
 P 4750 2400
-F 0 "R25" V 4830 2400 50  0000 C CNN
+F 0 "R19" V 4830 2400 50  0000 C CNN
 F 1 "100K" V 4750 2400 50  0000 C CNN
-F 2 "Resistors_SMD:R_0603" V 4680 2400 30  0000 C CNN
+F 2 "Resistors_SMD:R_0603" V 4680 2400 30  0001 C CNN
 F 3 "" H 4750 2400 30  0000 C CNN
 F 4 "RMCF0603JT100K" H 0   0   50  0001 C CNN "MPN"
@@
 $EndComp
 $Comp
-L +3.3V #PWR070
+L +3.3V #PWR42
 U 1 1 558A7C5A
 P 4750 2150
-F 0 "#PWR070" H 4750 2000 50  0001 C CNN
+F 0 "#PWR42" H 4750 2000 50  0001 C CNN
 F 1 "+3.3V" H 4750 2290 50  0000 C CNN
 F 2 "" H 4750 2150 60  0000 C CNN
@@
 $EndComp
 $Comp
-L +3.3V #PWR071
+L +3.3V #PWR40
 U 1 1 558A7D34
 P 4550 2850
-F 0 "#PWR071" H 4550 2700 50  0001 C CNN
+F 0 "#PWR40" H 4550 2700 50  0001 C CNN
 F 1 "+3.3V" H 4550 2990 50  0000 C CNN
 F 2 "" H 4550 2850 60  0000 C CNN
@@
 $EndComp
 $Comp
-L Q_NMOS_GSD Q4
+L Q_NMOS_GSD Q1
 U 1 1 558A8A3F
 P 2000 6200
-F 0 "Q4" H 1900 6150 50  0000 R CNN
+F 0 "Q1" H 1900 6150 50  0000 R CNN
 F 1 "2N7002" H 1950 6050 50  0000 R CNN
-F 2 "Housings_SOT-23_SOT-143_TSOT-6:SOT-23" H 2200 6300 29  0000 C CNN
+F 2 "Housings_SOT-23_SOT-143_TSOT-6:SOT-23" H 2200 6300 29  0001 C CNN
 F 3 "" H 2000 6200 60  0000 C CNN
 F 4 "2N7002P,215" H 0   0   50  0001 C CNN "MPN"
@@
 $EndComp
 $Comp
-L GNDD #PWR072
+L GNDD #PWR10
 U 1 1 558A8A45
 P 2100 6500
-F 0 "#PWR072" H 2100 6250 50  0001 C CNN
+F 0 "#PWR10" H 2100 6250 50  0001 C CNN
 F 1 "GNDD" H 2100 6350 50  0000 C CNN
 F 2 "" H 2100 6500 60  0000 C CNN
@@
 $EndComp
 $Comp
-L R R23
+L R R5
 U 1 1 558A8A4C
 P 2100 5650
-F 0 "R23" V 2180 5650 50  0000 C CNN
+F 0 "R5" V 2180 5650 50  0000 C CNN
 F 1 "4K7" V 2100 5650 50  0000 C CNN
-F 2 "Resistors_SMD:R_0603" V 2030 5650 30  0000 C CNN
+F 2 "Resistors_SMD:R_0603" V 2030 5650 30  0001 C CNN
 F 3 "" H 2100 5650 30  0000 C CNN
 F 4 "RMCF0603JT4K70" H 0   0   50  0001 C CNN "MPN"
@@
 $EndComp
 $Comp
-L +3.3V #PWR073
+L +3.3V #PWR9
 U 1 1 558A8A52
 P 2100 5400
-F 0 "#PWR073" H 2100 5250 50  0001 C CNN
+F 0 "#PWR9" H 2100 5250 50  0001 C CNN
 F 1 "+3.3V" H 2100 5540 50  0000 C CNN
 F 2 "" H 2100 5400 60  0000 C CNN
@@
 $EndComp
 $Comp
-L R R24
+L R R8
 U 1 1 558A8AE2
 P 2400 5900
-F 0 "R24" V 2480 5900 50  0000 C CNN
+F 0 "R8" V 2480 5900 50  0000 C CNN
 F 1 "680R" V 2400 5900 50  0000 C CNN
-F 2 "Resistors_SMD:R_0603" V 2330 5900 30  0000 C CNN
+F 2 "Resistors_SMD:R_0603" V 2330 5900 30  0001 C CNN
 F 3 "" H 2400 5900 30  0000 C CNN
 F 4 "RMCF0603JT680R" H 0   0   50  0001 C CNN "MPN"
@@
 $EndComp
 $Comp
-L CP1 C20
+L CP1 C3
 U 1 1 558A8E3B
 P 2700 6200
-F 0 "C20" H 2725 6300 50  0000 L CNN
+F 0 "C3" H 2725 6300 50  0000 L CNN
 F 1 "47uF" H 2725 6100 50  0000 L CNN
-F 2 "Capacitors_SMD:c_elec_6.3x5.3" H 2700 6200 60  0000 C CNN
+F 2 "Capacitors_SMD:c_elec_6.3x5.3" H 2700 6200 60  0001 C CNN
 F 3 "" H 2700 6200 60  0000 C CNN
 F 4 "UWX1C470MCL1GB" H 0   0   50  0001 C CNN "MPN"
@@
 $EndComp
 $Comp
-L GNDD #PWR074
+L GNDD #PWR16
 U 1 1 558A9218
 P 2700 6450
-F 0 "#PWR074" H 2700 6200 50  0001 C CNN
+F 0 "#PWR16" H 2700 6200 50  0001 C CNN
 F 1 "GNDD" H 2700 6300 50  0000 C CNN
 F 2 "" H 2700 6450 60  0000 C CNN
@@
 $EndComp
 $Comp
-L +3.3V #PWR075
+L +3.3V #PWR55
 U 1 1 558AA390
 P 6750 2600
-F 0 "#PWR075" H 6750 2450 50  0001 C CNN
+F 0 "#PWR55" H 6750 2450 50  0001 C CNN
 F 1 "+3.3V" H 6750 2740 50  0000 C CNN
 F 2 "" H 6750 2600 60  0000 C CNN
@@
 $EndComp
 $Comp
-L GNDD #PWR076
+L GNDD #PWR56
 U 1 1 558AA396
 P 7000 2700
-F 0 "#PWR076" H 7000 2450 50  0001 C CNN
+F 0 "#PWR56" H 7000 2450 50  0001 C CNN
 F 1 "GNDD" H 7000 2550 50  0000 C CNN
 F 2 "" H 7000 2700 60  0000 C CNN
@@
 $EndComp
 $Comp
-L C C21
+L C C15
 U 1 1 558AA39C
 P 6200 2950
-F 0 "C21" H 6225 3050 50  0000 L CNN
+F 0 "C15" H 6225 3050 50  0000 L CNN
 F 1 "100nF" H 6225 2850 50  0000 L CNN
-F 2 "Capacitors_SMD:C_0603" H 6238 2800 30  0000 C CNN
+F 2 "Capacitors_SMD:C_0603" H 6238 2800 30  0001 C CNN
 F 3 "" H 6200 2950 60  0000 C CNN
 F 4 "C1608X7R1E104K080AA" H 6200 2950 60  0001 C CNN "MPN"
@@
 $EndComp
 $Comp
-L GNDD #PWR077
+L GNDD #PWR53
 U 1 1 558AA3A8
 P 6200 3300
-F 0 "#PWR077" H 6200 3050 50  0001 C CNN
+F 0 "#PWR53" H 6200 3050 50  0001 C CNN
 F 1 "GNDD" H 6200 3150 50  0000 C CNN
 F 2 "" H 6200 3300 60  0000 C CNN
@@
 $EndComp
 $Comp
-L GNDD #PWR078
+L GNDD #PWR58
 U 1 1 558AA3AE
 P 7750 2700
-F 0 "#PWR078" H 7750 2450 50  0001 C CNN
+F 0 "#PWR58" H 7750 2450 50  0001 C CNN
 F 1 "GNDD" H 7750 2550 50  0000 C CNN
 F 2 "" H 7750 2700 60  0000 C CNN
@@
 $EndComp
 $Comp
-L Q_NMOS_GSD Q6
+L Q_NMOS_GSD Q8
 U 1 1 558AA3B4
 P 8900 2950
-F 0 "Q6" H 8800 2900 50  0000 R CNN
+F 0 "Q8" H 8800 2900 50  0000 R CNN
 F 1 "2N7002" H 8850 2800 50  0000 R CNN
-F 2 "Housings_SOT-23_SOT-143_TSOT-6:SOT-23" H 9100 3050 29  0000 C CNN
+F 2 "Housings_SOT-23_SOT-143_TSOT-6:SOT-23" H 9100 3050 29  0001 C CNN
 F 3 "" H 8900 2950 60  0000 C CNN
 F 4 "2N7002P,215" H 0   0   50  0001 C CNN "MPN"
@@
 $EndComp
 $Comp
-L GNDD #PWR079
+L GNDD #PWR73
 U 1 1 558AA3BA
 P 8800 3250
-F 0 "#PWR079" H 8800 3000 50  0001 C CNN
+F 0 "#PWR73" H 8800 3000 50  0001 C CNN
 F 1 "GNDD" H 8800 3100 50  0000 C CNN
 F 2 "" H 8800 3250 60  0000 C CNN
@@
 $EndComp
 $Comp
-L R R26
+L R R35
 U 1 1 558AA3C1
 P 8800 2400
-F 0 "R26" V 8880 2400 50  0000 C CNN
+F 0 "R35" V 8880 2400 50  0000 C CNN
 F 1 "100K" V 8800 2400 50  0000 C CNN
-F 2 "Resistors_SMD:R_0603" V 8730 2400 30  0000 C CNN
+F 2 "Resistors_SMD:R_0603" V 8730 2400 30  0001 C CNN
 F 3 "" H 8800 2400 30  0000 C CNN
 F 4 "RMCF0603JT100K" H 0   0   50  0001 C CNN "MPN"
@@
 $EndComp
 $Comp
-L +3.3V #PWR080
+L +3.3V #PWR72
 U 1 1 558AA3C7
 P 8800 2150
-F 0 "#PWR080" H 8800 2000 50  0001 C CNN
+F 0 "#PWR72" H 8800 2000 50  0001 C CNN
 F 1 "+3.3V" H 8800 2290 50  0000 C CNN
 F 2 "" H 8800 2150 60  0000 C CNN
@@
 $EndComp
 $Comp
-L +3.3V #PWR081
+L +3.3V #PWR67
 U 1 1 558AA3CD
 P 8600 2850
-F 0 "#PWR081" H 8600 2700 50  0001 C CNN
+F 0 "#PWR67" H 8600 2700 50  0001 C CNN
 F 1 "+3.3V" H 8600 2990 50  0000 C CNN
 F 2 "" H 8600 2850 60  0000 C CNN
@@
 $EndComp
 $Comp
-L C C19
+L C C2
 U 1 1 558AACB8
 P 2500 2950
-F 0 "C19" H 2525 3050 50  0000 L CNN
+F 0 "C2" H 2525 3050 50  0000 L CNN
 F 1 "10uF" H 2525 2850 50  0000 L CNN
-F 2 "Capacitors_SMD:C_0805" H 2538 2800 30  0000 C CNN
+F 2 "Capacitors_SMD:C_0805" H 2538 2800 30  0001 C CNN
 F 3 "" H 2500 2950 60  0000 C CNN
 F 4 "GRM219R61E106KA12D" H 2500 2950 60  0001 C CNN "MPN"
@@
 $EndComp
 $Comp
-L C C22
+L C C16
 U 1 1 558AACEE
 P 6550 2950
-F 0 "C22" H 6575 3050 50  0000 L CNN
+F 0 "C16" H 6575 3050 50  0000 L CNN
 F 1 "10uF" H 6575 2850 50  0000 L CNN
-F 2 "Capacitors_SMD:C_0805" H 6588 2800 30  0000 C CNN
+F 2 "Capacitors_SMD:C_0805" H 6588 2800 30  0001 C CNN
 F 3 "" H 6550 2950 60  0000 C CNN
 F 4 "GRM219R61E106KA12D" H 6550 2950 60  0001 C CNN "MPN"

Commit message: point the LCD voltage in the MPN
Parts:
- DS1, DS2: MPN ERM1602FS-6 -> ERM1602FS-6 3.3V
Changed lines of the file:
@@
 F 2 "local-footprints:WC1602A" H 3700 2050 35  0000 C CIN
 F 3 "" H 3700 2100 60  0000 C CNN
-F 4 "ERM1602FS-6" H 3700 2100 60  0001 C CNN "MPN"
+F 4 "ERM1602FS-6 3.3V" H 3700 2100 60  0001 C CNN "MPN"
 	1    3700 2100
 	1    0    0    -1
@@
 F 2 "local-footprints:WC1602A" H 7750 2050 35  0000 C CIN
 F 3 "" H 7750 2100 60  0000 C CNN
-F 4 "ERM1602FS-6" H 7750 2100 60  0001 C CNN "MPN"
+F 4 "ERM1602FS-6 3.3V" H 7750 2100 60  0001 C CNN "MPN"
 	1    7750 2100
 	1    0    0    -1

Commit message: use fixed contrast to displays
Parts:
- removed C3: 47uF, Capacitors_SMD:c_elec_6.3x5.3, symbol CP1
- removed Q1: 2N7002, Housings_SOT-23_SOT-143_TSOT-6:SOT-23, symbol Q_NMOS_GSD
- removed R5: 4K7, Resistors_SMD:R_0603, symbol R
- added C17, C3: 1uF, Capacitors_SMD:C_0805, symbol C
- added R13, R20: 2K, Resistors_SMD:R_0603, symbol R
- added R19: 2K4, Resistors_SMD:R_0603, symbol R
- R8: value 680R -> 2K4; MPN RMCF0603JT680R -> (none)
- renumbered Q7 to Q6, Q8 to Q7, R19 to R17, R35 to R36
Connections:
- net +3V3: now also R8.2, R19.2
- net GNDD: now also C17.2, C3.2, R13.2, R20.2
- net at R8.1: now also DS1.3 (Vo), C3.1, R13.1
- removed net LCD_VO: DS1.3 (Vo), DS2.3 (Vo), R8.2
- new net: C17.1, DS2.3 (Vo), R19.1, R20.1
Other:
- note removed: "LCD CONTRAST"
