File: hw-design/board/display.sch (KiCad schematic (older format))
At the start: 16 parts, among them Q6 2N7002, Q7 2N7002

Commit message: update netlist
Parts:
- renumbered Q6 to Q7, Q7 to Q8, R13 to R15, R17 to R19, R19 to R21, R20 to R22, R36 to R38, R8 to R9
Changed lines of the file:
@@
 $EndComp
 $Comp
-L +3.3V #PWR14
+L +3.3V #PWR15
 U 1 1 558A75D0
 P 2700 2600
-F 0 "#PWR14" H 2700 2450 50  0001 C CNN
+F 0 "#PWR15" H 2700 2450 50  0001 C CNN
 F 1 "+3.3V" H 2700 2740 50  0000 C CNN
 F 2 "" H 2700 2600 60  0000 C CNN
@@
 $EndComp
 $Comp
-L GNDD #PWR19
+L GNDD #PWR21
 U 1 1 558A75FC
 P 2950 2700
-F 0 "#PWR19" H 2950 2450 50  0001 C CNN
+F 0 "#PWR21" H 2950 2450 50  0001 C CNN
 F 1 "GNDD" H 2950 2550 50  0000 C CNN
 F 2 "" H 2950 2700 60  0000 C CNN
@@
 $EndComp
 $Comp
-L GNDD #PWR31
+L GNDD #PWR33
 U 1 1 558A77CB
 P 3700 2700
-F 0 "#PWR31" H 3700 2450 50  0001 C CNN
+F 0 "#PWR33" H 3700 2450 50  0001 C CNN
 F 1 "GNDD" H 3700 2550 50  0000 C CNN
 F 2 "" H 3700 2700 60  0000 C CNN
@@
 $EndComp
 $Comp
-L Q_NMOS_GSD Q6
+L Q_NMOS_GSD Q7
 U 1 1 558A78F3
 P 4850 2950
-F 0 "Q6" H 4750 2900 50  0000 R CNN
+F 0 "Q7" H 4750 2900 50  0000 R CNN
 F 1 "2N7002" H 4800 2800 50  0000 R CNN
 F 2 "Housings_SOT-23_SOT-143_TSOT-6:SOT-23" H 5050 3050 29  0001 C CNN
@@
 $EndComp
 $Comp
-L GNDD #PWR39
+L GNDD #PWR41
 U 1 1 558A7B13
 P 4750 3250
-F 0 "#PWR39" H 4750 3000 50  0001 C CNN
+F 0 "#PWR41" H 4750 3000 50  0001 C CNN
 F 1 "GNDD" H 4750 3100 50  0000 C CNN
 F 2 "" H 4750 3250 60  0000 C CNN
@@
 $EndComp
 $Comp
-L R R17
+L R R19
 U 1 1 558A7C00
 P 4750 2400
-F 0 "R17" V 4830 2400 50  0000 C CNN
+F 0 "R19" V 4830 2400 50  0000 C CNN
 F 1 "100K" V 4750 2400 50  0000 C CNN
 F 2 "Resistors_SMD:R_0603" V 4680 2400 30  0001 C CNN
@@
 $EndComp
 $Comp
-L +3.3V #PWR38
+L +3.3V #PWR40
 U 1 1 558A7C5A
 P 4750 2150
-F 0 "#PWR38" H 4750 2000 50  0001 C CNN
+F 0 "#PWR40" H 4750 2000 50  0001 C CNN
 F 1 "+3.3V" H 4750 2290 50  0000 C CNN
 F 2 "" H 4750 2150 60  0000 C CNN
@@
 $EndComp
 $Comp
-L +3.3V #PWR36
+L +3.3V #PWR38
 U 1 1 558A7D34
 P 4550 2850
-F 0 "#PWR36" H 4550 2700 50  0001 C CNN
+F 0 "#PWR38" H 4550 2700 50  0001 C CNN
 F 1 "+3.3V" H 4550 2990 50  0000 C CNN
 F 2 "" H 4550 2850 60  0000 C CNN
@@
 $EndComp
 $Comp
-L +3.3V #PWR51
+L +3.3V #PWR53
 U 1 1 558AA390
 P 6750 2600
-F 0 "#PWR51" H 6750 2450 50  0001 C CNN
+F 0 "#PWR53" H 6750 2450 50  0001 C CNN
 F 1 "+3.3V" H 6750 2740 50  0000 C CNN
 F 2 "" H 6750 2600 60  0000 C CNN
@@
 $EndComp
 $Comp
-L GNDD #PWR52
+L GNDD #PWR54
 U 1 1 558AA396
 P 7000 2700
-F 0 "#PWR52" H 7000 2450 50  0001 C CNN
+F 0 "#PWR54" H 7000 2450 50  0001 C CNN
 F 1 "GNDD" H 7000 2550 50  0000 C CNN
 F 2 "" H 7000 2700 60  0000 C CNN
@@
 $EndComp
 $Comp
-L GNDD #PWR49
+L GNDD #PWR51
 U 1 1 558AA3A8
 P 6200 3300
-F 0 "#PWR49" H 6200 3050 50  0001 C CNN
+F 0 "#PWR51" H 6200 3050 50  0001 C CNN
 F 1 "GNDD" H 6200 3150 50  0000 C CNN
 F 2 "" H 6200 3300 60  0000 C CNN
@@
 $EndComp
 $Comp
-L GNDD #PWR55
+L GNDD #PWR57
 U 1 1 558AA3AE
 P 7750 2700
-F 0 "#PWR55" H 7750 2450 50  0001 C CNN
+F 0 "#PWR57" H 7750 2450 50  0001 C CNN
 F 1 "GNDD" H 7750 2550 50  0000 C CNN
 F 2 "" H 7750 2700 60  0000 C CNN
@@
 $EndComp
 $Comp
-L Q_NMOS_GSD Q7
+L Q_NMOS_GSD Q8
 U 1 1 558AA3B4
 P 8900 2950
-F 0 "Q7" H 8800 2900 50  0000 R CNN
+F 0 "Q8" H 8800 2900 50  0000 R CNN
 F 1 "2N7002" H 8850 2800 50  0000 R CNN
 F 2 "Housings_SOT-23_SOT-143_TSOT-6:SOT-23" H 9100 3050 29  0001 C CNN
@@
 $EndComp
 $Comp
-L GNDD #PWR69
+L GNDD #PWR71
 U 1 1 558AA3BA
 P 8800 3250
-F 0 "#PWR69" H 8800 3000 50  0001 C CNN
+F 0 "#PWR71" H 8800 3000 50  0001 C CNN
 F 1 "GNDD" H 8800 3100 50  0000 C CNN
 F 2 "" H 8800 3250 60  0000 C CNN
@@
 $EndComp
 $Comp
-L R R36
+L R R38
 U 1 1 558AA3C1
 P 8800 2400
-F 0 "R36" V 8880 2400 50  0000 C CNN
+F 0 "R38" V 8880 2400 50  0000 C CNN
 F 1 "100K" V 8800 2400 50  0000 C CNN
 F 2 "Resistors_SMD:R_0603" V 8730 2400 30  0001 C CNN
@@
 $EndComp
 $Comp
-L +3.3V #PWR68
+L +3.3V #PWR70
 U 1 1 558AA3C7
 P 8800 2150
-F 0 "#PWR68" H 8800 2000 50  0001 C CNN
+F 0 "#PWR70" H 8800 2000 50  0001 C CNN
 F 1 "+3.3V" H 8800 2290 50  0000 C CNN
 F 2 "" H 8800 2150 60  0000 C CNN
@@
 $EndComp
 $Comp
-L +3.3V #PWR63
+L +3.3V #PWR65
 U 1 1 558AA3CD
 P 8600 2850
-F 0 "#PWR63" H 8600 2700 50  0001 C CNN
+F 0 "#PWR65" H 8600 2700 50  0001 C CNN
 F 1 "+3.3V" H 8600 2990 50  0000 C CNN
 F 2 "" H 8600 2850 60  0000 C CNN
@@
 $EndComp
 $Comp
-L R R13
+L R R15
 U 1 1 578CCDA0
 P 3150 3900
-F 0 "R13" V 3230 3900 50  0000 C CNN
+F 0 "R15" V 3230 3900 50  0000 C CNN
 F 1 "2K" V 3150 3900 50  0000 C CNN
 F 2 "Resistors_SMD:R_0603" V 3080 3900 30  0001 C CNN
@@
 $EndComp
 $Comp
-L R R8
+L R R9
 U 1 1 578CDA36
 P 2700 3650
-F 0 "R8" V 2600 3650 50  0000 C CNN
+F 0 "R9" V 2600 3650 50  0000 C CNN
 F 1 "2K4" V 2700 3650 50  0000 C CNN
 F 2 "Resistors_SMD:R_0603" V 2630 3650 30  0001 C CNN
@@
 $EndComp
 $Comp
-L GNDD #PWR25
+L GNDD #PWR27
 U 1 1 578CDB27
 P 3050 4150
-F 0 "#PWR25" H 3050 3900 50  0001 C CNN
+F 0 "#PWR27" H 3050 3900 50  0001 C CNN
 F 1 "GNDD" H 3050 4000 50  0000 C CNN
 F 2 "" H 3050 4150 60  0000 C CNN
@@
 Connection ~ 2950 3650
 $Comp
-L +3.3V #PWR11
+L +3.3V #PWR12
 U 1 1 578CEAAB
 P 2450 3550
-F 0 "#PWR11" H 2450 3400 50  0001 C CNN
+F 0 "#PWR12" H 2450 3400 50  0001 C CNN
 F 1 "+3.3V" H 2450 3690 50  0000 C CNN
 F 2 "" H 2450 3550 60  0000 C CNN
@@
 $EndComp
 $Comp
-L R R20
+L R R22
 U 1 1 578CEDFE
 P 7200 3900
-F 0 "R20" V 7280 3900 50  0000 C CNN
+F 0 "R22" V 7280 3900 50  0000 C CNN
 F 1 "2K" V 7200 3900 50  0000 C CNN
 F 2 "Resistors_SMD:R_0603" V 7130 3900 30  0001 C CNN
@@
 $EndComp
 $Comp
-L R R19
+L R R21
 U 1 1 578CEE04
 P 6750 3650
-F 0 "R19" V 6650 3650 50  0000 C CNN
+F 0 "R21" V 6650 3650 50  0000 C CNN
 F 1 "2K4" V 6750 3650 50  0000 C CNN
 F 2 "Resistors_SMD:R_0603" V 6680 3650 30  0001 C CNN
@@
 $EndComp
 $Comp
-L GNDD #PWR53
+L GNDD #PWR55
 U 1 1 578CEE0A
 P 7100 4150
-F 0 "#PWR53" H 7100 3900 50  0001 C CNN
+F 0 "#PWR55" H 7100 3900 50  0001 C CNN
 F 1 "GNDD" H 7100 4000 50  0000 C CNN
 F 2 "" H 7100 4150 60  0000 C CNN
@@
 Connection ~ 7000 3650
 $Comp
-L +3.3V #PWR50
+L +3.3V #PWR52
 U 1 1 578CEE1D
 P 6500 3550
-F 0 "#PWR50" H 6500 3400 50  0001 C CNN
+F 0 "#PWR52" H 6500 3400 50  0001 C CNN
 F 1 "+3.3V" H 6500 3690 50  0000 C CNN
 F 2 "" H 6500 3550 60  0000 C CNN
