File: hw-design/board/display.sch (KiCad schematic (older format))
At the start: 16 parts, among them Q7 2N7002, Q8 2N7002

Commit message: update files to KiCAD 5
Parts:
- C1, C15, C16, C17, C2, C3: symbol C -> footswitch-rescue:C
- DS1, DS2: symbol RC1602A-GHW-ESX -> footswitch-rescue:RC1602A-GHW-ESX; Note (none) -> 3.3V display
- Q7, Q8: symbol Q_NMOS_GSD -> footswitch-rescue:Q_NMOS_GSD
- R15, R19, R22, R38: symbol R -> footswitch-rescue:R
- R21, R9: symbol R -> footswitch-rescue:R; Note (none) -> do not place
Changed lines of the file:
@@
-EESchema Schematic File Version 2
-LIBS:conn
-LIBS:device
-LIBS:interface
-LIBS:power
-LIBS:regul
-LIBS:transistors
-LIBS:display
-LIBS:nxp_armmcu
-LIBS:philips
-LIBS:graphic_symbols
+EESchema Schematic File Version 4
 LIBS:footswitch-cache
 EELAYER 26 0
@@
 $EndDescr
 $Comp
-L RC1602A-GHW-ESX DS1
+L footswitch-rescue:RC1602A-GHW-ESX DS1
 U 1 1 558A7276
 P 3700 2100
@@
 F 3 "" H 3700 2100 60  0000 C CNN
 F 4 "ERM1602FS-6 3.3V" H 3700 2100 60  0001 C CNN "MPN"
+F 5 "3.3V display" H 3700 2100 50  0001 C CNN "Note"
 	1    3700 2100
 	1    0    0    -1
 $EndComp
 $Comp
-L +3.3V #PWR051
+L footswitch-rescue:+3.3V #PWR051
 U 1 1 558A75D0
 P 2700 2600
@@
 $EndComp
 $Comp
-L GNDD #PWR052
+L footswitch-rescue:GNDD #PWR052
 U 1 1 558A75FC
 P 2950 2700
@@
 $EndComp
 $Comp
-L C C1
+L footswitch-rescue:C C1
 U 1 1 558A7629
 P 2150 2950
@@
 $EndComp
 $Comp
-L GNDD #PWR053
+L footswitch-rescue:GNDD #PWR053
 U 1 1 558A7699
 P 2150 3300
@@
 $EndComp
 $Comp
-L GNDD #PWR054
+L footswitch-rescue:GNDD #PWR054
 U 1 1 558A77CB
 P 3700 2700
@@
 $EndComp
 $Comp
-L Q_NMOS_GSD Q7
+L footswitch-rescue:Q_NMOS_GSD Q7
 U 1 1 558A78F3
 P 4850 2950
@@
 $EndComp
 $Comp
-L GNDD #PWR055
+L footswitch-rescue:GNDD #PWR055
 U 1 1 558A7B13
 P 4750 3250
@@
 $EndComp
 $Comp
-L R R19
+L footswitch-rescue:R R19
 U 1 1 558A7C00
 P 4750 2400
@@
 $EndComp
 $Comp
-L +3.3V #PWR056
+L footswitch-rescue:+3.3V #PWR056
 U 1 1 558A7C5A
 P 4750 2150
@@
 $EndComp
 $Comp
-L +3.3V #PWR057
+L footswitch-rescue:+3.3V #PWR057
 U 1 1 558A7D34
 P 4550 2850
@@
 $EndComp
 $Comp
-L RC1602A-GHW-ESX DS2
+L footswitch-rescue:RC1602A-GHW-ESX DS2
 U 1 1 558AA38A
 P 7750 2100
@@
 F 3 "" H 7750 2100 60  0000 C CNN
 F 4 "ERM1602FS-6 3.3V" H 7750 2100 60  0001 C CNN "MPN"
+F 5 "3.3V display" H 7750 2100 50  0001 C CNN "Note"
 	1    7750 2100
 	1    0    0    -1
 $EndComp
 $Comp
-L +3.3V #PWR058
+L footswitch-rescue:+3.3V #PWR058
 U 1 1 558AA390
 P 6750 2600
@@
 $EndComp
 $Comp
-L GNDD #PWR059
+L footswitch-rescue:GNDD #PWR059
 U 1 1 558AA396
 P 7000 2700
@@
 $EndComp
 $Comp
-L C C15
+L footswitch-rescue:C C15
 U 1 1 558AA39C
 P 6200 2950
@@
 $EndComp
 $Comp
-L GNDD #PWR060
+L footswitch-rescue:GNDD #PWR060
 U 1 1 558AA3A8
 P 6200 3300
@@
 $EndComp
 $Comp
-L GNDD #PWR061
+L footswitch-rescue:GNDD #PWR061
 U 1 1 558AA3AE
 P 7750 2700
@@
 $EndComp
 $Comp
-L Q_NMOS_GSD Q8
+L footswitch-rescue:Q_NMOS_GSD Q8
 U 1 1 558AA3B4
 P 8900 2950
@@
 $EndComp
 $Comp
-L GNDD #PWR062
+L footswitch-rescue:GNDD #PWR062
 U 1 1 558AA3BA
 P 8800 3250
@@
 $EndComp
 $Comp
-L R R38
+L footswitch-rescue:R R38
 U 1 1 558AA3C1
 P 8800 2400
@@
 $EndComp
 $Comp
-L +3.3V #PWR063
+L footswitch-rescue:+3.3V #PWR063
 U 1 1 558AA3C7
 P 8800 2150
@@
 $EndComp
 $Comp
-L +3.3V #PWR064
+L footswitch-rescue:+3.3V #PWR064
 U 1 1 558AA3CD
 P 8600 2850
@@
 $EndComp
 $Comp
-L C C2
+L footswitch-rescue:C C2
 U 1 1 558AACB8
 P 2500 2950
@@
 $EndComp
 $Comp
-L C C16
+L footswitch-rescue:C C16
 U 1 1 558AACEE
 P 6550 2950
@@
 LCD_D4
 $Comp
-L C C3
+L footswitch-rescue:C C3
 U 1 1 578CBDC0
 P 2950 3900
@@
 $EndComp
 $Comp
-L R R15
+L footswitch-rescue:R R15
 U 1 1 578CCDA0
 P 3150 3900
@@
 $EndComp
 $Comp
-L R R9
+L footswitch-rescue:R R9
 U 1 1 578CDA36
 P 2700 3650
@@
 F 2 "Resistors_SMD:R_0603" V 2630 3650 30  0001 C CNN
 F 3 "" H 2700 3650 30  0000 C CNN
+F 4 "do not place" V 2700 3650 50  0001 C CNN "Note"
 	1    2700 3650
 	0    1    1    0
 $EndComp
 $Comp
-L GNDD #PWR065
+L footswitch-rescue:GNDD #PWR065
 U 1 1 578CDB27
 P 3050 4150
@@
 	2950 2600 2950 2700
 Wire Wire Line
-	2700 2600 2700 3150
+	2700 2600 2700 2700
 Wire Wire Line
 	2700 3150 3050 3150
@@
 	2150 2800 2150 2700
 Wire Wire Line
-	2150 2700 2700 2700
+	2150 2700 2500 2700
 Wire Wire Line
 	2500 2800 2500 2700
 Wire Wire Line
-	2150 3100 2150 3300
+	2150 3100 2150 3200
 Wire Wire Line
 	2500 3100 2500 3200
@@
 	3550 2600 3550 2650
 Wire Wire Line
-	3550 2650 3850 2650
+	3550 2650 3650 2650
 Wire Wire Line
 	3850 2650 3850 2600
@@
 	4450 2650 4750 2650
 Wire Wire Line
-	4750 2550 4750 2750
+	4750 2550 4750 2650
 Wire Wire Line
 	4750 3150 4750 3250
@@
 	7000 2600 7000 2700
 Wire Wire Line
-	6750 2600 6750 3150
+	6750 2600 6750 2700
 Wire Wire Line
 	6750 3150 7100 3150
@@
 	6200 2800 6200 2700
 Wire Wire Line
-	6200 2700 6750 2700
+	6200 2700 6550 2700
 Wire Wire Line
 	6550 2800 6550 2700
 Wire Wire Line
-	6200 3100 6200 3300
+	6200 3100 6200 3200
 Wire Wire Line
 	6550 3100 6550 3200
@@
 	7600 2600 7600 2650
 Wire Wire Line
-	7600 2650 7900 2650
+	7600 2650 7700 2650
 Wire Wire Line
 	7900 2650 7900 2600
@@
 	8500 2650 8800 2650
 Wire Wire Line
-	8800 2550 8800 2750
+	8800 2550 8800 2650
 Wire Wire Line
 	8800 3150 8800 3250
@@
 	2950 4050 2950 4100
 Wire Wire Line
-	2950 4100 3150 4100
+	2950 4100 3050 4100
 Wire Wire Line
 	3150 4100 3150 4050
@@
 Connection ~ 3050 4100
 Wire Wire Line
-	3150 2600 3150 3750
+	3150 2600 3150 3650
 Connection ~ 3150 3650
 Wire Wire Line
-	2850 3650 3150 3650
+	2850 3650 2950 3650
 Wire Wire Line
 	2950 3750 2950 3650
 Connection ~ 2950 3650
 $Comp
-L +3.3V #PWR066
+L footswitch-rescue:+3.3V #PWR066
 U 1 1 578CEAAB
 P 2450 3550
@@
 	2450 3650 2450 3550
 $Comp
-L C C17
+L footswitch-rescue:C C17
 U 1 1 578CEDF7
 P 7000 3900
@@
 $EndComp
 $Comp
-L R R22
+L footswitch-rescue:R R22
 U 1 1 578CEDFE
 P 7200 3900
@@
 $EndComp
 $Comp
-L R R21
+L footswitch-rescue:R R21
 U 1 1 578CEE04
 P 6750 3650
@@
 F 2 "Resistors_SMD:R_0603" V 6680 3650 30  0001 C CNN
 F 3 "" H 6750 3650 30  0000 C CNN
+F 4 "do not place" V 6750 3650 50  0001 C CNN "Note"
 	1    6750 3650
 	0    1    1    0
 $EndComp
 $Comp
-L GNDD #PWR067
+L footswitch-rescue:GNDD #PWR067
 U 1 1 578CEE0A
 P 7100 4150
@@
 	7000 4050 7000 4100
 Wire Wire Line
-	7000 4100 7200 4100
+	7000 4100 7100 4100
 Wire Wire Line
 	7200 4100 7200 4050
@@
 Connection ~ 7100 4100
 Wire Wire Line
-	7200 2600 7200 3750
+	7200 2600 7200 3650
 Connection ~ 7200 3650
 Wire Wire Line
-	6900 3650 7200 3650
+	6900 3650 7000 3650
 Wire Wire Line
 	7000 3750 7000 3650
 Connection ~ 7000 3650
 $Comp
-L +3.3V #PWR068
+L footswitch-rescue:+3.3V #PWR068
 U 1 1 578CEE1D
 P 6500 3550
@@
 Wire Wire Line
 	7300 3600 7300 2600
+Wire Wire Line
+	2700 2700 2700 3150
+Wire Wire Line
+	2500 2700 2700 2700
+Wire Wire Line
+	2150 3200 2150 3300
+Wire Wire Line
+	3650 2650 3700 2650
+Wire Wire Line
+	3750 2650 3850 2650
+Wire Wire Line
+	3700 2650 3750 2650
+Wire Wire Line
+	4750 2650 4750 2750
+Wire Wire Line
+	6750 2700 6750 3150
+Wire Wire Line
+	6550 2700 6750 2700
+Wire Wire Line
+	6200 3200 6200 3300
+Wire Wire Line
+	7700 2650 7750 2650
+Wire Wire Line
+	7800 2650 7900 2650
+Wire Wire Line
+	7750 2650 7800 2650
+Wire Wire Line
+	8800 2650 8800 2750
+Wire Wire Line
+	3050 4100 3150 4100
+Wire Wire Line
+	3150 3650 3150 3750
+Wire Wire Line
+	2950 3650 3150 3650
+Wire Wire Line
+	7100 4100 7200 4100
+Wire Wire Line
+	7200 3650 7200 3750
+Wire Wire Line
+	7000 3650 7200 3650
 $EndSCHEMATC

Commit message: decrease res value of display backlight (same footprint); bom updated
Parts:
- R15, R22: value 2K -> 1.2K; MPN RMCF0603JT2K00 -> RMCF0603JT1K20
Changed lines of the file:
@@
 P 3150 3900
 F 0 "R15" V 3230 3900 50  0000 C CNN
-F 1 "2K" V 3150 3900 50  0000 C CNN
+F 1 "1.2K" V 3150 3900 50  0000 C CNN
 F 2 "Resistors_SMD:R_0603" V 3080 3900 30  0001 C CNN
 F 3 "" H 3150 3900 30  0000 C CNN
-F 4 "RMCF0603JT2K00" H -1600 1500 50  0001 C CNN "MPN"
+F 4 "RMCF0603JT1K20" H -1600 1500 50  0001 C CNN "MPN"
 	1    3150 3900
 	1    0    0    -1
@@
 P 7200 3900
 F 0 "R22" V 7280 3900 50  0000 C CNN
-F 1 "2K" V 7200 3900 50  0000 C CNN
+F 1 "1.2K" V 7200 3900 50  0000 C CNN
 F 2 "Resistors_SMD:R_0603" V 7130 3900 30  0001 C CNN
 F 3 "" H 7200 3900 30  0000 C CNN
-F 4 "RMCF0603JT2K00" H 2450 1500 50  0001 C CNN "MPN"
+F 4 "RMCF0603JT1K20" H 2450 1500 50  0001 C CNN "MPN"
 	1    7200 3900
 	1    0    0    -1

Commit message: Changed R40 RE from pull-up to pull-down
Parts:
- C1, C15, C16, C17, C2, C3: symbol footswitch-rescue:C -> footswitch-rescue:C-footswitch-rescue
- DS1, DS2: symbol footswitch-rescue:RC1602A-GHW-ESX -> footswitch-rescue:RC1602A-GHW-ESX-footswitch-rescue
- Q7, Q8: symbol footswitch-rescue:Q_NMOS_GSD -> footswitch-rescue:Q_NMOS_GSD-footswitch-rescue
- R15, R19, R21, R22, R38, R9: symbol footswitch-rescue:R -> footswitch-rescue:R-footswitch-rescue
Changed lines of the file:
@@
 $EndDescr
 $Comp
-L footswitch-rescue:RC1602A-GHW-ESX DS1
+L footswitch-rescue:RC1602A-GHW-ESX-footswitch-rescue DS1
 U 1 1 558A7276
 P 3700 2100
@@
 $EndComp
 $Comp
-L footswitch-rescue:+3.3V #PWR051
+L footswitch-rescue:+3.3V-footswitch-rescue #PWR051
 U 1 1 558A75D0
 P 2700 2600
@@
 $EndComp
 $Comp
-L footswitch-rescue:GNDD #PWR052
+L footswitch-rescue:GNDD-footswitch-rescue #PWR052
 U 1 1 558A75FC
 P 2950 2700
@@
 $EndComp
 $Comp
-L footswitch-rescue:C C1
+L footswitch-rescue:C-footswitch-rescue C1
 U 1 1 558A7629
 P 2150 2950
@@
 $EndComp
 $Comp
-L footswitch-rescue:GNDD #PWR053
+L footswitch-rescue:GNDD-footswitch-rescue #PWR053
 U 1 1 558A7699
 P 2150 3300
@@
 $EndComp
 $Comp
-L footswitch-rescue:GNDD #PWR054
+L footswitch-rescue:GNDD-footswitch-rescue #PWR054
 U 1 1 558A77CB
 P 3700 2700
@@
 $EndComp
 $Comp
-L footswitch-rescue:Q_NMOS_GSD Q7
+L footswitch-rescue:Q_NMOS_GSD-footswitch-rescue Q7
 U 1 1 558A78F3
 P 4850 2950
@@
 $EndComp
 $Comp
-L footswitch-rescue:GNDD #PWR055
+L footswitch-rescue:GNDD-footswitch-rescue #PWR055
 U 1 1 558A7B13
 P 4750 3250
@@
 $EndComp
 $Comp
-L footswitch-rescue:R R19
+L footswitch-rescue:R-footswitch-rescue R19
 U 1 1 558A7C00
 P 4750 2400
@@
 $EndComp
 $Comp
-L footswitch-rescue:+3.3V #PWR056
+L footswitch-rescue:+3.3V-footswitch-rescue #PWR056
 U 1 1 558A7C5A
 P 4750 2150
@@
 $EndComp
 $Comp
-L footswitch-rescue:+3.3V #PWR057
+L footswitch-rescue:+3.3V-footswitch-rescue #PWR057
 U 1 1 558A7D34
 P 4550 2850
@@
 $EndComp
 $Comp
-L footswitch-rescue:RC1602A-GHW-ESX DS2
+L footswitch-rescue:RC1602A-GHW-ESX-footswitch-rescue DS2
 U 1 1 558AA38A
 P 7750 2100
@@
 $EndComp
 $Comp
-L footswitch-rescue:+3.3V #PWR058
+L footswitch-rescue:+3.3V-footswitch-rescue #PWR058
 U 1 1 558AA390
 P 6750 2600
@@
 $EndComp
 $Comp
-L footswitch-rescue:GNDD #PWR059
+L footswitch-rescue:GNDD-footswitch-rescue #PWR059
 U 1 1 558AA396
 P 7000 2700
@@
 $EndComp
 $Comp
-L footswitch-rescue:C C15
+L footswitch-rescue:C-footswitch-rescue C15
 U 1 1 558AA39C
 P 6200 2950
@@
 $EndComp
 $Comp
-L footswitch-rescue:GNDD #PWR060
+L footswitch-rescue:GNDD-footswitch-rescue #PWR060
 U 1 1 558AA3A8
 P 6200 3300
@@
 $EndComp
 $Comp
-L footswitch-rescue:GNDD #PWR061
+L footswitch-rescue:GNDD-footswitch-rescue #PWR061
 U 1 1 558AA3AE
 P 7750 2700
@@
 $EndComp
 $Comp
-L footswitch-rescue:Q_NMOS_GSD Q8
+L footswitch-rescue:Q_NMOS_GSD-footswitch-rescue Q8
 U 1 1 558AA3B4
 P 8900 2950
@@
 $EndComp
 $Comp
-L footswitch-rescue:GNDD #PWR062
+L footswitch-rescue:GNDD-footswitch-rescue #PWR062
 U 1 1 558AA3BA
 P 8800 3250
@@
 $EndComp
 $Comp
-L footswitch-rescue:R R38
+L footswitch-rescue:R-footswitch-rescue R38
 U 1 1 558AA3C1
 P 8800 2400
@@
 $EndComp
 $Comp
-L footswitch-rescue:+3.3V #PWR063
+L footswitch-rescue:+3.3V-footswitch-rescue #PWR063
 U 1 1 558AA3C7
 P 8800 2150
@@
 $EndComp
 $Comp
-L footswitch-rescue:+3.3V #PWR064
+L footswitch-rescue:+3.3V-footswitch-rescue #PWR064
 U 1 1 558AA3CD
 P 8600 2850
@@
 $EndComp
 $Comp
-L footswitch-rescue:C C2
+L footswitch-rescue:C-footswitch-rescue C2
 U 1 1 558AACB8
 P 2500 2950
@@
 $EndComp
 $Comp
-L footswitch-rescue:C C16
+L footswitch-rescue:C-footswitch-rescue C16
 U 1 1 558AACEE
 P 6550 2950
@@
 LCD_D4
 $Comp
-L footswitch-rescue:C C3
+L footswitch-rescue:C-footswitch-rescue C3
 U 1 1 578CBDC0
 P 2950 3900
@@
 $EndComp
 $Comp
-L footswitch-rescue:R R15
+L footswitch-rescue:R-footswitch-rescue R15
 U 1 1 578CCDA0
 P 3150 3900
@@
 $EndComp
 $Comp
-L footswitch-rescue:R R9
+L footswitch-rescue:R-footswitch-rescue R9
 U 1 1 578CDA36
 P 2700 3650
@@
 $EndComp
 $Comp
-L footswitch-rescue:GNDD #PWR065
+L footswitch-rescue:GNDD-footswitch-rescue #PWR065
 U 1 1 578CDB27
 P 3050 4150
@@
 Connection ~ 2950 3650
 $Comp
-L footswitch-rescue:+3.3V #PWR066
+L footswitch-rescue:+3.3V-footswitch-rescue #PWR066
 U 1 1 578CEAAB
 P 2450 3550
@@
 	2450 3650 2450 3550
 $Comp
-L footswitch-rescue:C C17
+L footswitch-rescue:C-footswitch-rescue C17
 U 1 1 578CEDF7
 P 7000 3900
@@
 $EndComp
 $Comp
-L footswitch-rescue:R R22
+L footswitch-rescue:R-footswitch-rescue R22
 U 1 1 578CEDFE
 P 7200 3900
@@
 $EndComp
 $Comp
-L footswitch-rescue:R R21
+L footswitch-rescue:R-footswitch-rescue R21
 U 1 1 578CEE04
 P 6750 3650
@@
 $EndComp
 $Comp
-L footswitch-rescue:GNDD #PWR067
+L footswitch-rescue:GNDD-footswitch-rescue #PWR067
 U 1 1 578CEE0A
 P 7100 4150
@@
 Connection ~ 7000 3650
 $Comp
-L footswitch-rescue:+3.3V #PWR068
+L footswitch-rescue:+3.3V-footswitch-rescue #PWR068
 U 1 1 578CEE1D
 P 6500 3550
