File: hw-design/board/footswitch.sch (KiCad schematic (older format))
At the start: 0 parts

Commit message: sch: schematic updated (missing displays circuit)
Changed lines of the file:
@@
 LIBS:transistors
 LIBS:nxp_armmcu
+LIBS:philips
 LIBS:footswitch-cache
 EELAYER 25 0
@@
 $EndSheet
 $Sheet
-S 800  4050 1450 550
+S 800  4150 1450 550
 U 53485BBD
 F0 "Display" 60

Commit message: sch: added mechanic sheet
Changed lines of the file:
@@
 $Descr A4 11693 8268
 encoding utf-8
-Sheet 1 6
+Sheet 1 7
 Title "MOD Footswitch Extensor"
 Date "Tue 09 Dec 2014"
@@
 F1 "display.sch" 60
 $EndSheet
+$Sheet
+S 800  5050 1450 550
+U 55B0CAF6
+F0 "Mechanic" 60
+F1 "Mechanic.sch" 60
+$EndSheet
 $EndSCHEMATC

Commit message: sch: fixing mechanic sheet
Changed lines of the file:
@@
 U 55B0CAF6
 F0 "Mechanic" 60
-F1 "Mechanic.sch" 60
+F1 "mechanic.sch" 60
 $EndSheet
 $EndSCHEMATC

Commit message: sch: schematic files reorganized, new sheets for usb and rear board
Changed lines of the file:
@@
 $Descr A4 11693 8268
 encoding utf-8
-Sheet 1 7
+Sheet 1 9
 Title "MOD Footswitch Extensor"
 Date "Tue 09 Dec 2014"
@@
 $EndSheet
 $Sheet
-S 800  4150 1450 550
+S 2500 800  1450 550
 U 53485BBD
 F0 "Display" 60
@@
 $EndSheet
 $Sheet
-S 800  5050 1450 550
+S 2500 1600 1450 550
 U 55B0CAF6
 F0 "Mechanic" 60
 F1 "mechanic.sch" 60
 $EndSheet
+$Sheet
+S 2500 2400 1450 550
+U 55B25118
+F0 "Rear Board" 60
+F1 "rear-board.sch" 60
+$EndSheet
+$Sheet
+S 2500 3250 1450 550
+U 55B4D84D
+F0 "USB" 60
+F1 "usb.sch" 60
+$EndSheet
 $EndSCHEMATC
