File: hw-design/board/power.sch (KiCad schematic (older format))
At the start: 16 parts, among them U2 MC7805, U3 NCP1117DT33G

Commit message: importing common sheets from expression-pedal project
Parts:
- removed C3, C6: 100uF, MOD_Footprints_Lib:CAP_RAD_5MM, symbol CP1
- removed C4, C7: 100nF_X7R, MOD_Footprints_Lib:SM0603, symbol C
- removed D1: CGRA4007-G, MOD_Footprints_Lib:DO-214AC(SMA), symbol DIODE
- removed R26, R38: 0R, MOD_Footprints_Lib:SM0805, symbol R
- removed RT2: PTC_FUSE_500mA, MOD_Footprints_Lib:SM1210, symbol FUSE
- removed TP1, TP2, TP3: CONN_1, MOD_Footprints_Lib:SIL-1, symbol CONN_1
- removed U2: MC7805, MOD_Footprints_Lib:DPAK(369C), symbol LINEAR_REGULATOR_DPAK_3P
- removed U3: NCP1117DT33G, MOD_Footprints_Lib:DPAK(369C), symbol NCP1117DT33G
- added C3, C5, C6, C8: 100nF, Capacitors_SMD:C_0603, symbol C
- added C4, C7: 100uF, Capacitors_SMD:c_elec_6.3x5.3, symbol CP1
- added D1: CGRA4007-G, Diodes_SMD:Diode-SMA_Standard, symbol D
- added D2, D3: 1N5819, Diodes_SMD:SOD-123, symbol D_Schottky
- added Q1, Q2: 2N7002, Housings_SOT-23_SOT-143_TSOT-6:SOT-23, symbol Q_NMOS_GSD
- added Q3: FDN306P, local-footprints:SOT-23-fairchild, symbol Q_PMOS_GSD
- added R1: 3K6, Resistors_SMD:R_0603, symbol R
- added R2: 5K6, Resistors_SMD:R_0603, symbol R
- added R3, R4: 10k, Resistors_SMD:R_0603, symbol R
- added U1: NCP1117DT50G, SMD_Packages:DPAK-2, symbol NCP1117ST50T3G
- added U2: NCP1117DT33G, SMD_Packages:DPAK-2, symbol NCP1117ST33T3G
- C1: value 100uF -> 10uF; footprint MOD_Footprints_Lib:CAP_RAD_5MM -> Capacitors_SMD:c_elec_5x5.3; MPN (none) -> UWX1E100MCL1GB
- C2: value 100nF_X7R -> 10uF; footprint MOD_Footprints_Lib:SM0603 -> Capacitors_SMD:C_0805; MPN (none) -> GRM219R61E106KA12D
- RT1: value PTC_FUSE_500mA -> PTC_FUSE; footprint MOD_Footprints_Lib:SM2920 -> Resistors_SMD:R_1210; MPN (none) -> 0ZCB0050FF2G
Connections:
- net labels added: GNDD, POWER_INPUT
- net labels removed: DGND
- wire segments 32 -> 51
Other:
- note added: "CONTROL CHAIN POWER"
- note added: "USB POWER"

Commit message: sch: schematic files reorganized, new sheets for usb and rear board
Changed lines of the file:
@@
 $Descr A4 11693 8268
 encoding utf-8
-Sheet 2 7
+Sheet 2 9
 Title ""
 Date ""
@@
 Connection ~ 1600 5100
 Connection ~ 3300 1600
+$Comp
+L VCC #PWR027
+U 1 1 55B522FD
+P 8800 3250
+F 0 "#PWR027" H 8800 3100 50  0001 C CNN
+F 1 "VCC" H 8800 3400 50  0000 C CNN
+F 2 "" H 8800 3250 60  0000 C CNN
+F 3 "" H 8800 3250 60  0000 C CNN
+	1    8800 3250
+	1    0    0    -1
+$EndComp
+$Comp
+L PWR_FLAG #FLG028
+U 1 1 55B523DA
+P 8800 3400
+F 0 "#FLG028" H 8800 3495 30  0001 C CNN
+F 1 "PWR_FLAG" H 8800 3580 30  0000 C CNN
+F 2 "" H 8800 3400 60  0000 C CNN
+F 3 "" H 8800 3400 60  0000 C CNN
+	1    8800 3400
+	-1   0    0    1
+$EndComp
+Wire Wire Line
+	8800 3250 8800 3400
 $EndSCHEMATC
