File: hw-design/board/power.sch (KiCad schematic (older format))
At the start: 21 parts, among them Q1 2N7002, Q2 2N7002, Q3 FDN306P, U1 NCP1117DT50G, U2 NCP1117DT33G

Commit message: fix power voltage
Parts:
- R1: value 3K6 -> 10K; MPN RMCF0603JT3K60 -> RMCF0603JT10K0
- R2: value 5K6 -> 10K; MPN RMCF0603JT5K60 -> RMCF0603JT10K0
Connections:
- net POWER_INPUT renamed +12V
Other:
- note added: "CPU POWER"
- moved on the sheet: C2, D2, Q1, Q2, Q3, R1, R2, R3, R4

Commit message: annotation and ERC
Parts:
- renumbered C4 to C10, C5 to C11, C6 to C17, C7 to C19, C8 to C20, C1 to C5, C3 to C7, C2 to C8, D2 to D3, D3 to D4, Q1 to Q2, Q2 to Q4, Q3 to Q5, R4 to R12, R1 to R3, R2 to R4, R3 to R9, U1 to U2, U2 to U4

Commit message: update MPN
Parts:
- R12, R9: value 10k -> 10K
Changed lines of the file:
@@
 P 2950 4100
 F 0 "R12" V 3030 4100 50  0000 C CNN
-F 1 "10k" V 2950 4100 50  0000 C CNN
+F 1 "10K" V 2950 4100 50  0000 C CNN
 F 2 "Resistors_SMD:R_0603" V 2880 4100 30  0001 C CNN
 F 3 "" H 2950 4100 30  0000 C CNN
@@
 P 2500 4450
 F 0 "R9" V 2580 4450 50  0000 C CNN
-F 1 "10k" V 2500 4450 50  0000 C CNN
+F 1 "10K" V 2500 4450 50  0000 C CNN
 F 2 "Resistors_SMD:R_0603" V 2430 4450 30  0001 C CNN
 F 3 "" H 2500 4450 30  0000 C CNN

Commit message: DRC done
Parts:
- renumbered C11 to C12, C17 to C18, C19 to C20, C20 to C22, Q2 to Q1, Q4 to Q3, Q5 to Q4, R12 to R11, R9 to R7
Changed lines of the file:
@@
 $EndDescr
 $Comp
-L CP1 C19
+L CP1 C20
 U 1 1 548B65E4
 P 9200 1850
-F 0 "C19" V 9300 1950 50  0000 L CNN
+F 0 "C20" V 9300 1950 50  0000 L CNN
 F 1 "100uF" V 9050 1750 50  0000 L CNN
 F 2 "Capacitors_SMD:c_elec_6.3x5.3" H 9200 1850 60  0001 C CNN
@@
 $EndComp
 $Comp
-L C C20
+L C C22
 U 1 1 548B660A
 P 9550 1850
-F 0 "C20" V 9500 1950 50  0000 L CNN
+F 0 "C22" V 9500 1950 50  0000 L CNN
 F 1 "100nF" V 9700 1700 50  0000 L CNN
 F 2 "Capacitors_SMD:C_0603" H 9588 1700 30  0001 C CNN
@@
 $EndComp
 $Comp
-L C C11
+L C C12
 U 1 1 548B6624
 P 5200 1850
-F 0 "C11" V 5150 1950 50  0000 L CNN
+F 0 "C12" V 5150 1950 50  0000 L CNN
 F 1 "100nF" V 5350 1800 50  0000 L CNN
 F 2 "Capacitors_SMD:C_0603" H 5238 1700 30  0001 C CNN
@@
 $EndComp
 $Comp
-L GNDD #PWR27
+L GNDD #PWR26
 U 1 1 54E7EE6C
 P 3150 2100
-F 0 "#PWR27" H 3150 1850 60  0001 C CNN
+F 0 "#PWR26" H 3150 1850 60  0001 C CNN
 F 1 "GNDD" H 3150 1950 60  0000 C CNN
 F 2 "" H 3150 2100 60  0000 C CNN
@@
 $EndComp
 $Comp
-L GNDD #PWR30
+L GNDD #PWR29
 U 1 1 54E7EE80
 P 3450 2100
-F 0 "#PWR30" H 3450 1850 60  0001 C CNN
+F 0 "#PWR29" H 3450 1850 60  0001 C CNN
 F 1 "GNDD" H 3450 1950 60  0000 C CNN
 F 2 "" H 3450 2100 60  0000 C CNN
@@
 $EndComp
 $Comp
-L GNDD #PWR44
+L GNDD #PWR40
 U 1 1 54E7F9F2
 P 4850 2100
-F 0 "#PWR44" H 4850 1850 60  0001 C CNN
+F 0 "#PWR40" H 4850 1850 60  0001 C CNN
 F 1 "GNDD" H 4850 1950 60  0000 C CNN
 F 2 "" H 4850 2100 60  0000 C CNN
@@
 $EndComp
 $Comp
-L GNDD #PWR45
+L GNDD #PWR43
 U 1 1 54E7FA28
 P 5200 2100
-F 0 "#PWR45" H 5200 1850 60  0001 C CNN
+F 0 "#PWR43" H 5200 1850 60  0001 C CNN
 F 1 "GNDD" H 5200 1950 60  0000 C CNN
 F 2 "" H 5200 2100 60  0000 C CNN
@@
 $EndComp
 $Comp
-L GNDD #PWR75
+L GNDD #PWR71
 U 1 1 54E7FA3C
 P 9200 2100
-F 0 "#PWR75" H 9200 1850 60  0001 C CNN
+F 0 "#PWR71" H 9200 1850 60  0001 C CNN
 F 1 "GNDD" H 9200 1950 60  0000 C CNN
 F 2 "" H 9200 2100 60  0000 C CNN
@@
 $EndComp
 $Comp
-L GNDD #PWR77
+L GNDD #PWR75
 U 1 1 54E7FA50
 P 9550 2100
-F 0 "#PWR77" H 9550 1850 60  0001 C CNN
+F 0 "#PWR75" H 9550 1850 60  0001 C CNN
 F 1 "GNDD" H 9550 1950 60  0000 C CNN
 F 2 "" H 9550 2100 60  0000 C CNN
@@
 $EndComp
 $Comp
-L GNDD #PWR35
+L GNDD #PWR32
 U 1 1 54E80258
 P 4100 1950
-F 0 "#PWR35" H 4100 1700 60  0001 C CNN
+F 0 "#PWR32" H 4100 1700 60  0001 C CNN
 F 1 "GNDD" H 4100 1800 60  0000 C CNN
 F 2 "" H 4100 1950 60  0000 C CNN
@@
 $EndComp
 $Comp
-L GNDD #PWR66
+L GNDD #PWR62
 U 1 1 54E876DB
 P 8600 1950
-F 0 "#PWR66" H 8600 1700 60  0001 C CNN
+F 0 "#PWR62" H 8600 1700 60  0001 C CNN
 F 1 "GNDD" H 8600 1800 60  0000 C CNN
 F 2 "" H 8600 1950 60  0000 C CNN
@@
 $EndComp
 $Comp
-L +3.3V #PWR81
+L +3.3V #PWR78
 U 1 1 556EF2E1
 P 9800 1450
-F 0 "#PWR81" H 9800 1300 50  0001 C CNN
+F 0 "#PWR78" H 9800 1300 50  0001 C CNN
 F 1 "+3.3V" H 9800 1590 50  0000 C CNN
 F 2 "" H 9800 1450 60  0000 C CNN
@@
 $EndComp
 $Comp
-L Q_PMOS_GSD Q5
+L Q_PMOS_GSD Q4
 U 1 1 5576EC7B
 P 3450 3950
-F 0 "Q5" V 3350 3900 50  0000 R CNN
+F 0 "Q4" V 3350 3900 50  0000 R CNN
 F 1 "FDN306P" V 3650 4100 50  0000 R CNN
 F 2 "local-footprints:SOT-23-fairchild" H 3650 4050 29  0001 C CNN
@@
 $EndComp
 $Comp
-L R R12
+L R R11
 U 1 1 5576FA4A
 P 2950 4100
-F 0 "R12" V 3030 4100 50  0000 C CNN
+F 0 "R11" V 3030 4100 50  0000 C CNN
 F 1 "10K" V 2950 4100 50  0000 C CNN
 F 2 "Resistors_SMD:R_0603" V 2880 4100 30  0001 C CNN
@@
 $EndComp
 $Comp
-L VCC #PWR22
+L VCC #PWR20
 U 1 1 55770535
 P 2950 3750
-F 0 "#PWR22" H 2950 3600 50  0001 C CNN
+F 0 "#PWR20" H 2950 3600 50  0001 C CNN
 F 1 "VCC" H 2950 3900 50  0000 C CNN
 F 2 "" H 2950 3750 60  0000 C CNN
@@
 $EndComp
 $Comp
-L Q_NMOS_GSD Q4
+L Q_NMOS_GSD Q3
 U 1 1 55771A8F
 P 2850 4750
-F 0 "Q4" H 2750 4800 50  0000 R CNN
+F 0 "Q3" H 2750 4800 50  0000 R CNN
 F 1 "2N7002" V 3050 4850 50  0000 R CNN
 F 2 "Housings_SOT-23_SOT-143_TSOT-6:SOT-23" H 3050 4850 29  0001 C CNN
@@
 $EndComp
 $Comp
-L Q_NMOS_GSD Q2
+L Q_NMOS_GSD Q1
 U 1 1 55771C8E
 P 2400 5100
-F 0 "Q2" H 2300 5150 50  0000 R CNN
+F 0 "Q1" H 2300 5150 50  0000 R CNN
 F 1 "2N7002" V 2600 5200 50  0000 R CNN
 F 2 "Housings_SOT-23_SOT-143_TSOT-6:SOT-23" H 2600 5200 29  0001 C CNN
@@
 $EndComp
 $Comp
-L GNDD #PWR14
+L GNDD #PWR13
 U 1 1 557724D6
 P 2500 5400
-F 0 "#PWR14" H 2500 5150 60  0001 C CNN
+F 0 "#PWR13" H 2500 5150 60  0001 C CNN
 F 1 "GNDD" H 2500 5250 60  0000 C CNN
 F 2 "" H 2500 5400 60  0000 C CNN
@@
 $EndComp
 $Comp
-L GNDD #PWR23
+L GNDD #PWR21
 U 1 1 55772F70
 P 2950 5050
-F 0 "#PWR23" H 2950 4800 60  0001 C CNN
+F 0 "#PWR21" H 2950 4800 60  0001 C CNN
 F 1 "GNDD" H 2950 4900 60  0000 C CNN
 F 2 "" H 2950 5050 60  0000 C CNN
@@
 $EndComp
 $Comp
-L R R9
+L R R7
 U 1 1 55773BAE
 P 2500 4450
-F 0 "R9" V 2580 4450 50  0000 C CNN
+F 0 "R7" V 2580 4450 50  0000 C CNN
 F 1 "10K" V 2500 4450 50  0000 C CNN
 F 2 "Resistors_SMD:R_0603" V 2430 4450 30  0001 C CNN
@@
 $EndComp
 $Comp
-L VCC #PWR13
+L VCC #PWR12
 U 1 1 55774D84
 P 2500 4200
-F 0 "#PWR13" H 2500 4050 50  0001 C CNN
+F 0 "#PWR12" H 2500 4050 50  0001 C CNN
 F 1 "VCC" H 2500 4350 50  0000 C CNN
 F 2 "" H 2500 4200 60  0000 C CNN
@@
 $EndComp
 $Comp
-L C C17
+L C C18
 U 1 1 557CA3A5
 P 7950 1850
-F 0 "C17" V 7900 1950 40  0000 L CNN
+F 0 "C18" V 7900 1950 40  0000 L CNN
 F 1 "100nF" V 8100 1700 50  0000 L CNN
 F 2 "Capacitors_SMD:C_0603" H 7988 1700 30  0001 C CNN
@@
 $EndComp
 $Comp
-L GNDD #PWR60
+L GNDD #PWR57
 U 1 1 557CA58F
 P 7950 2100
-F 0 "#PWR60" H 7950 1850 60  0001 C CNN
+F 0 "#PWR57" H 7950 1850 60  0001 C CNN
 F 1 "GNDD" H 7950 1950 60  0000 C CNN
 F 2 "" H 7950 2100 60  0000 C CNN
@@
 $EndComp
 $Comp
-L +5V #PWR57
+L +5V #PWR54
 U 1 1 557CCB1A
 P 7650 1450
-F 0 "#PWR57" H 7650 1300 50  0001 C CNN
+F 0 "#PWR54" H 7650 1300 50  0001 C CNN
 F 1 "+5V" H 7650 1590 50  0000 C CNN
 F 2 "" H 7650 1450 60  0000 C CNN
@@
 $EndComp
 $Comp
-L +5V #PWR41
+L +5V #PWR37
 U 1 1 557CDFF5
 P 4600 3750
-F 0 "#PWR41" H 4600 3600 50  0001 C CNN
+F 0 "#PWR37" H 4600 3600 50  0001 C CNN
 F 1 "+5V" H 4600 3890 50  0000 C CNN
 F 2 "" H 4600 3750 60  0000 C CNN
@@
 $EndComp
 $Comp
-L +5V #PWR52
+L +5V #PWR48
 U 1 1 557CC20F
 P 6150 1500
-F 0 "#PWR52" H 6150 1350 50  0001 C CNN
+F 0 "#PWR48" H 6150 1350 50  0001 C CNN
 F 1 "+5V" H 6150 1640 50  0000 C CNN
 F 2 "" H 6150 1500 60  0000 C CNN
@@
 $EndComp
 $Comp
-L +5V #PWR61
+L +5V #PWR58
 U 1 1 557B3200
 P 8200 3250
-F 0 "#PWR61" H 8200 3100 50  0001 C CNN
+F 0 "#PWR58" H 8200 3100 50  0001 C CNN
 F 1 "+5V" H 8200 3390 50  0000 C CNN
 F 2 "" H 8200 3250 60  0000 C CNN
@@
 USB POWER
 $Comp
-L VCC #PWR64
+L VCC #PWR60
 U 1 1 55B522FD
 P 8450 3250
-F 0 "#PWR64" H 8450 3100 50  0001 C CNN
+F 0 "#PWR60" H 8450 3100 50  0001 C CNN
 F 1 "VCC" H 8450 3400 50  0000 C CNN
 F 2 "" H 8450 3250 60  0000 C CNN
@@
 	7900 3250 7900 3400
 $Comp
-L GNDD #PWR59
+L GNDD #PWR56
 U 1 1 54E7EDE1
 P 7900 3400
-F 0 "#PWR59" H 7900 3150 60  0001 C CNN
+F 0 "#PWR56" H 7900 3150 60  0001 C CNN
 F 1 "GNDD" H 7900 3250 60  0000 C CNN
 F 2 "" H 7900 3400 60  0000 C CNN

Commit message: update netlist
Parts:
- renumbered Q3 to Q4, Q4 to Q5, R11 to R13, R7 to R8
Changed lines of the file:
@@
 $EndComp
 $Comp
-L GNDD #PWR26
+L GNDD #PWR28
 U 1 1 54E7EE6C
 P 3150 2100
-F 0 "#PWR26" H 3150 1850 60  0001 C CNN
+F 0 "#PWR28" H 3150 1850 60  0001 C CNN
 F 1 "GNDD" H 3150 1950 60  0000 C CNN
 F 2 "" H 3150 2100 60  0000 C CNN
@@
 $EndComp
 $Comp
-L GNDD #PWR29
+L GNDD #PWR31
 U 1 1 54E7EE80
 P 3450 2100
-F 0 "#PWR29" H 3450 1850 60  0001 C CNN
+F 0 "#PWR31" H 3450 1850 60  0001 C CNN
 F 1 "GNDD" H 3450 1950 60  0000 C CNN
 F 2 "" H 3450 2100 60  0000 C CNN
@@
 $EndComp
 $Comp
-L GNDD #PWR40
+L GNDD #PWR42
 U 1 1 54E7F9F2
 P 4850 2100
-F 0 "#PWR40" H 4850 1850 60  0001 C CNN
+F 0 "#PWR42" H 4850 1850 60  0001 C CNN
 F 1 "GNDD" H 4850 1950 60  0000 C CNN
 F 2 "" H 4850 2100 60  0000 C CNN
@@
 $EndComp
 $Comp
-L GNDD #PWR43
+L GNDD #PWR45
 U 1 1 54E7FA28
 P 5200 2100
-F 0 "#PWR43" H 5200 1850 60  0001 C CNN
+F 0 "#PWR45" H 5200 1850 60  0001 C CNN
 F 1 "GNDD" H 5200 1950 60  0000 C CNN
 F 2 "" H 5200 2100 60  0000 C CNN
@@
 $EndComp
 $Comp
-L GNDD #PWR71
+L GNDD #PWR73
 U 1 1 54E7FA3C
 P 9200 2100
-F 0 "#PWR71" H 9200 1850 60  0001 C CNN
+F 0 "#PWR73" H 9200 1850 60  0001 C CNN
 F 1 "GNDD" H 9200 1950 60  0000 C CNN
 F 2 "" H 9200 2100 60  0000 C CNN
@@
 $EndComp
 $Comp
-L GNDD #PWR75
+L GNDD #PWR77
 U 1 1 54E7FA50
 P 9550 2100
-F 0 "#PWR75" H 9550 1850 60  0001 C CNN
+F 0 "#PWR77" H 9550 1850 60  0001 C CNN
 F 1 "GNDD" H 9550 1950 60  0000 C CNN
 F 2 "" H 9550 2100 60  0000 C CNN
@@
 $EndComp
 $Comp
-L GNDD #PWR32
+L GNDD #PWR34
 U 1 1 54E80258
 P 4100 1950
-F 0 "#PWR32" H 4100 1700 60  0001 C CNN
+F 0 "#PWR34" H 4100 1700 60  0001 C CNN
 F 1 "GNDD" H 4100 1800 60  0000 C CNN
 F 2 "" H 4100 1950 60  0000 C CNN
@@
 $EndComp
 $Comp
-L GNDD #PWR62
+L GNDD #PWR64
 U 1 1 54E876DB
 P 8600 1950
-F 0 "#PWR62" H 8600 1700 60  0001 C CNN
+F 0 "#PWR64" H 8600 1700 60  0001 C CNN
 F 1 "GNDD" H 8600 1800 60  0000 C CNN
 F 2 "" H 8600 1950 60  0000 C CNN
@@
 $EndComp
 $Comp
-L +3.3V #PWR78
+L +3.3V #PWR80
 U 1 1 556EF2E1
 P 9800 1450
-F 0 "#PWR78" H 9800 1300 50  0001 C CNN
+F 0 "#PWR80" H 9800 1300 50  0001 C CNN
 F 1 "+3.3V" H 9800 1590 50  0000 C CNN
 F 2 "" H 9800 1450 60  0000 C CNN
@@
 $EndComp
 $Comp
-L Q_PMOS_GSD Q4
+L Q_PMOS_GSD Q5
 U 1 1 5576EC7B
 P 3450 3950
-F 0 "Q4" V 3350 3900 50  0000 R CNN
+F 0 "Q5" V 3350 3900 50  0000 R CNN
 F 1 "FDN306P" V 3650 4100 50  0000 R CNN
 F 2 "local-footprints:SOT-23-fairchild" H 3650 4050 29  0001 C CNN
@@
 $EndComp
 $Comp
-L R R11
+L R R13
 U 1 1 5576FA4A
 P 2950 4100
-F 0 "R11" V 3030 4100 50  0000 C CNN
+F 0 "R13" V 3030 4100 50  0000 C CNN
 F 1 "10K" V 2950 4100 50  0000 C CNN
 F 2 "Resistors_SMD:R_0603" V 2880 4100 30  0001 C CNN
@@
 $EndComp
 $Comp
-L VCC #PWR20
+L VCC #PWR22
 U 1 1 55770535
 P 2950 3750
-F 0 "#PWR20" H 2950 3600 50  0001 C CNN
+F 0 "#PWR22" H 2950 3600 50  0001 C CNN
 F 1 "VCC" H 2950 3900 50  0000 C CNN
 F 2 "" H 2950 3750 60  0000 C CNN
@@
 $EndComp
 $Comp
-L Q_NMOS_GSD Q3
+L Q_NMOS_GSD Q4
 U 1 1 55771A8F
 P 2850 4750
-F 0 "Q3" H 2750 4800 50  0000 R CNN
+F 0 "Q4" H 2750 4800 50  0000 R CNN
 F 1 "2N7002" V 3050 4850 50  0000 R CNN
 F 2 "Housings_SOT-23_SOT-143_TSOT-6:SOT-23" H 3050 4850 29  0001 C CNN
@@
 $EndComp
 $Comp
-L GNDD #PWR13
+L GNDD #PWR14
 U 1 1 557724D6
 P 2500 5400
-F 0 "#PWR13" H 2500 5150 60  0001 C CNN
+F 0 "#PWR14" H 2500 5150 60  0001 C CNN
 F 1 "GNDD" H 2500 5250 60  0000 C CNN
 F 2 "" H 2500 5400 60  0000 C CNN
@@
 $EndComp
 $Comp
-L GNDD #PWR21
+L GNDD #PWR23
 U 1 1 55772F70
 P 2950 5050
-F 0 "#PWR21" H 2950 4800 60  0001 C CNN
+F 0 "#PWR23" H 2950 4800 60  0001 C CNN
 F 1 "GNDD" H 2950 4900 60  0000 C CNN
 F 2 "" H 2950 5050 60  0000 C CNN
@@
 $EndComp
 $Comp
-L R R7
+L R R8
 U 1 1 55773BAE
 P 2500 4450
-F 0 "R7" V 2580 4450 50  0000 C CNN
+F 0 "R8" V 2580 4450 50  0000 C CNN
 F 1 "10K" V 2500 4450 50  0000 C CNN
 F 2 "Resistors_SMD:R_0603" V 2430 4450 30  0001 C CNN
@@
 $EndComp
 $Comp
-L VCC #PWR12
+L VCC #PWR13
 U 1 1 55774D84
 P 2500 4200
-F 0 "#PWR12" H 2500 4050 50  0001 C CNN
+F 0 "#PWR13" H 2500 4050 50  0001 C CNN
 F 1 "VCC" H 2500 4350 50  0000 C CNN
 F 2 "" H 2500 4200 60  0000 C CNN
@@
 $EndComp
 $Comp
-L GNDD #PWR57
+L GNDD #PWR59
 U 1 1 557CA58F
 P 7950 2100
-F 0 "#PWR57" H 7950 1850 60  0001 C CNN
+F 0 "#PWR59" H 7950 1850 60  0001 C CNN
 F 1 "GNDD" H 7950 1950 60  0000 C CNN
 F 2 "" H 7950 2100 60  0000 C CNN
@@
 $EndComp
 $Comp
-L +5V #PWR54
+L +5V #PWR56
 U 1 1 557CCB1A
 P 7650 1450
-F 0 "#PWR54" H 7650 1300 50  0001 C CNN
+F 0 "#PWR56" H 7650 1300 50  0001 C CNN
 F 1 "+5V" H 7650 1590 50  0000 C CNN
 F 2 "" H 7650 1450 60  0000 C CNN
@@
 $EndComp
 $Comp
-L +5V #PWR37
+L +5V #PWR39
 U 1 1 557CDFF5
 P 4600 3750
-F 0 "#PWR37" H 4600 3600 50  0001 C CNN
+F 0 "#PWR39" H 4600 3600 50  0001 C CNN
 F 1 "+5V" H 4600 3890 50  0000 C CNN
 F 2 "" H 4600 3750 60  0000 C CNN
@@
 $EndComp
 $Comp
-L +5V #PWR48
+L +5V #PWR50
 U 1 1 557CC20F
 P 6150 1500
-F 0 "#PWR48" H 6150 1350 50  0001 C CNN
+F 0 "#PWR50" H 6150 1350 50  0001 C CNN
 F 1 "+5V" H 6150 1640 50  0000 C CNN
 F 2 "" H 6150 1500 60  0000 C CNN
@@
 $EndComp
 $Comp
-L +5V #PWR58
+L +5V #PWR60
 U 1 1 557B3200
 P 8200 3250
-F 0 "#PWR58" H 8200 3100 50  0001 C CNN
+F 0 "#PWR60" H 8200 3100 50  0001 C CNN
 F 1 "+5V" H 8200 3390 50  0000 C CNN
 F 2 "" H 8200 3250 60  0000 C CNN
@@
 USB POWER
 $Comp
-L VCC #PWR60
+L VCC #PWR62
 U 1 1 55B522FD
 P 8450 3250
-F 0 "#PWR60" H 8450 3100 50  0001 C CNN
+F 0 "#PWR62" H 8450 3100 50  0001 C CNN
 F 1 "VCC" H 8450 3400 50  0000 C CNN
 F 2 "" H 8450 3250 60  0000 C CNN
@@
 	7900 3250 7900 3400
 $Comp
-L GNDD #PWR56
+L GNDD #PWR58
 U 1 1 54E7EDE1
 P 7900 3400
-F 0 "#PWR56" H 7900 3150 60  0001 C CNN
+F 0 "#PWR58" H 7900 3150 60  0001 C CNN
 F 1 "GNDD" H 7900 3250 60  0000 C CNN
 F 2 "" H 7900 3400 60  0000 C CNN
