File: hw-design/board/power.sch (KiCad schematic (older format))
At the start: 21 parts, among them Q1 2N7002, Q4 2N7002, Q5 FDN306P, U2 NCP1117DT50G, U4 NCP1117DT33G

Commit message: sch: remove 5V regulator
Parts:
- removed C18, C22: 100nF, Capacitors_SMD:C_0603, symbol C
- removed C20: 100uF, Capacitors_SMD:c_elec_6.3x5.3, symbol CP1
- removed D4: 1N5819, Diodes_SMD:SOD-123, symbol D_Schottky
- removed U2: NCP1117DT50G, SMD_Packages:DPAK-2, symbol NCP1117ST50T3G
- renumbered U4 to U2
Connections:
- net +3V3: now also C10.1, C12.1
- net +5V: now also D1.1 (K), RT1.1; no longer U2.3 (VI)
- net at C5.1, C7.1, RT1.2: now also U2.3 (VI)
Other:
- note added: "+5V power comes from USB and it's activated\nonly if +12V is not present, i.e. when the control\nchain cable is not plugged in"
- note removed: "CPU POWER"
- moved on the sheet: C10, C12, C5, C7, D1, RT1, U2

Commit message: update files to KiCAD 5
Parts:
- C10, C5: symbol CP1 -> footswitch-rescue:CP1
- C12, C7, C8: symbol C -> footswitch-rescue:C
- D1: symbol D -> footswitch-rescue:D
- D3: symbol D_Schottky -> footswitch-rescue:D_Schottky
- Q1, Q4: symbol Q_NMOS_GSD -> footswitch-rescue:Q_NMOS_GSD
- Q5: symbol Q_PMOS_GSD -> footswitch-rescue:Q_PMOS_GSD
- R13, R3, R4, R8: symbol R -> footswitch-rescue:R
- RT1: symbol FUSE -> footswitch-rescue:FUSE
- U2: symbol NCP1117ST33T3G -> footswitch-rescue:NCP1117ST33T3G
Changed lines of the file:
@@
-EESchema Schematic File Version 2
-LIBS:conn
-LIBS:device
-LIBS:interface
-LIBS:power
-LIBS:regul
-LIBS:transistors
-LIBS:display
-LIBS:nxp_armmcu
-LIBS:philips
-LIBS:graphic_symbols
+EESchema Schematic File Version 4
 LIBS:footswitch-cache
 EELAYER 26 0
@@
 $EndDescr
 $Comp
-L CP1 C10
+L footswitch-rescue:CP1 C10
 U 1 1 548B65F7
 P 5100 1850
@@
 $EndComp
 $Comp
-L C C12
+L footswitch-rescue:C C12
 U 1 1 548B6624
 P 5450 1850
@@
 $EndComp
 $Comp
-L CP1 C5
+L footswitch-rescue:CP1 C5
 U 1 1 548B663E
 P 3500 1850
@@
 $EndComp
 $Comp
-L D D1
+L footswitch-rescue:D D1
 U 1 1 548B6651
 P 2300 1600
@@
 $EndComp
 $Comp
-L FUSE RT1
+L footswitch-rescue:FUSE RT1
 U 1 1 548B6658
 P 3050 1600
@@
 $EndComp
 $Comp
-L C C7
+L footswitch-rescue:C C7
 U 1 1 548B665F
 P 3800 1850
@@
 $EndComp
 $Comp
-L GNDD #PWR01
+L footswitch-rescue:GNDD #PWR01
 U 1 1 54E7EE6C
 P 3500 2100
@@
 $EndComp
 $Comp
-L GNDD #PWR02
+L footswitch-rescue:GNDD #PWR02
 U 1 1 54E7EE80
 P 3800 2100
@@
 $EndComp
 $Comp
-L GNDD #PWR03
+L footswitch-rescue:GNDD #PWR03
 U 1 1 54E7F9F2
 P 5100 2100
@@
 $EndComp
 $Comp
-L GNDD #PWR04
+L footswitch-rescue:GNDD #PWR04
 U 1 1 54E7FA28
 P 5450 2100
@@
 $EndComp
 $Comp
-L GNDD #PWR05
+L footswitch-rescue:GNDD #PWR05
 U 1 1 54E80258
 P 4450 1950
@@
 $EndComp
 $Comp
-L +3.3V #PWR06
+L footswitch-rescue:+3.3V #PWR06
 U 1 1 556EF2E1
 P 5700 1500
@@
 $EndComp
 $Comp
-L Q_PMOS_GSD Q5
+L footswitch-rescue:Q_PMOS_GSD Q5
 U 1 1 5576EC7B
 P 3450 3950
@@
 $EndComp
 $Comp
-L D_Schottky D3
+L footswitch-rescue:D_Schottky D3
 U 1 1 5576EF8F
 P 4250 3850
@@
 $EndComp
 $Comp
-L R R13
+L footswitch-rescue:R R13
 U 1 1 5576FA4A
 P 2950 4100
@@
 $EndComp
 $Comp
-L VCC #PWR07
+L footswitch-rescue:VCC #PWR07
 U 1 1 55770535
 P 2950 3750
@@
 $EndComp
 $Comp
-L Q_NMOS_GSD Q4
+L footswitch-rescue:Q_NMOS_GSD Q4
 U 1 1 55771A8F
 P 2850 4750
@@
 $EndComp
 $Comp
-L Q_NMOS_GSD Q1
+L footswitch-rescue:Q_NMOS_GSD Q1
 U 1 1 55771C8E
 P 2400 5100
@@
 $EndComp
 $Comp
-L GNDD #PWR08
+L footswitch-rescue:GNDD #PWR08
 U 1 1 557724D6
 P 2500 5400
@@
 $EndComp
 $Comp
-L GNDD #PWR09
+L footswitch-rescue:GNDD #PWR09
 U 1 1 55772F70
 P 2950 5050
@@
 $EndComp
 $Comp
-L R R8
+L footswitch-rescue:R R8
 U 1 1 55773BAE
 P 2500 4450
@@
 $EndComp
 $Comp
-L VCC #PWR010
+L footswitch-rescue:VCC #PWR010
 U 1 1 55774D84
 P 2500 4200
@@
 $EndComp
 $Comp
-L C C8
+L footswitch-rescue:C C8
 U 1 1 55779079
 P 3800 4100
@@
 $EndComp
 $Comp
-L NCP1117ST33T3G U2
+L footswitch-rescue:NCP1117ST33T3G U2
 U 1 1 557C3298
 P 4450 1650
@@
 $EndComp
 $Comp
-L R R4
+L footswitch-rescue:R R4
 U 1 1 557CABF6
 P 2050 5400
@@
 $EndComp
 $Comp
-L GNDD #PWR011
+L footswitch-rescue:GNDD #PWR011
 U 1 1 557CAF87
 P 2050 5650
@@
 $EndComp
 $Comp
-L +5V #PWR012
+L footswitch-rescue:+5V #PWR012
 U 1 1 557CDFF5
 P 4600 3750
@@
 $EndComp
 $Comp
-L +5V #PWR013
+L footswitch-rescue:+5V #PWR013
 U 1 1 557CC20F
 P 2650 1500
@@
 $EndComp
 $Comp
-L R R3
+L footswitch-rescue:R R3
 U 1 1 557CFF3F
 P 2050 4800
@@
 $EndComp
 $Comp
-L PWR_FLAG #FLG014
+L footswitch-rescue:PWR_FLAG #FLG014
 U 1 1 557B3123
 P 6950 1700
@@
 $EndComp
 $Comp
-L +5V #PWR015
+L footswitch-rescue:+5V #PWR015
 U 1 1 557B3200
 P 6950 1550
@@
 USB POWER
 $Comp
-L VCC #PWR016
+L footswitch-rescue:VCC #PWR016
 U 1 1 55B522FD
 P 7200 1550
@@
 $EndComp
 $Comp
-L PWR_FLAG #FLG017
+L footswitch-rescue:PWR_FLAG #FLG017
 U 1 1 55B523DA
 P 7200 1700
@@
 $EndComp
 $Comp
-L +12V #PWR018
+L footswitch-rescue:+12V #PWR018
 U 1 1 575EB4B7
 P 1600 1500
+AR Path="/575EB4B7" Ref="#PWR018"  Part="1"
+AR Path="/54830571/575EB4B7" Ref="#PWR018"  Part="1"
 F 0 "#PWR018" H 1600 1350 50  0001 C CNN
 F 1 "+12V" H 1618 1674 50  0000 C CNN
@@
 $EndComp
 $Comp
-L PWR_FLAG #FLG019
+L footswitch-rescue:PWR_FLAG #FLG019
 U 1 1 54B50E4C
 P 1950 1500
@@
 $EndComp
 $Comp
-L +12V #PWR020
+L footswitch-rescue:+12V #PWR020
 U 1 1 575EFB81
 P 2050 4550
+AR Path="/575EFB81" Ref="#PWR020"  Part="1"
+AR Path="/54830571/575EFB81" Ref="#PWR020"  Part="1"
 F 0 "#PWR020" H 2050 4400 50  0001 C CNN
 F 1 "+12V" H 2050 4700 50  0000 C CNN
@@
 $EndComp
 $Comp
-L PWR_FLAG #FLG021
+L footswitch-rescue:PWR_FLAG #FLG021
 U 1 1 5760D14C
 P 6650 1550
@@
 $EndComp
 $Comp
-L GNDD #PWR022
+L footswitch-rescue:GNDD #PWR022
 U 1 1 54E7EDE1
 P 6650 1700
@@
 +5V power comes from USB and it's activated\nonly if +12V is not present, i.e. when the control\nchain cable is not plugged in
 $Comp
-L PWR_FLAG #FLG023
+L footswitch-rescue:PWR_FLAG #FLG023
 U 1 1 59675A29
 P 3950 1500

Commit message: Changed R40 RE from pull-up to pull-down
Parts:
- C10, C5: symbol footswitch-rescue:CP1 -> footswitch-rescue:CP1-footswitch-rescue
- C12, C7, C8: symbol footswitch-rescue:C -> footswitch-rescue:C-footswitch-rescue
- D1: symbol footswitch-rescue:D -> footswitch-rescue:D-footswitch-rescue
- D3: symbol footswitch-rescue:D_Schottky -> footswitch-rescue:D_Schottky-footswitch-rescue
- Q1, Q4: symbol footswitch-rescue:Q_NMOS_GSD -> footswitch-rescue:Q_NMOS_GSD-footswitch-rescue
- Q5: symbol footswitch-rescue:Q_PMOS_GSD -> footswitch-rescue:Q_PMOS_GSD-footswitch-rescue
- R13, R3, R4, R8: symbol footswitch-rescue:R -> footswitch-rescue:R-footswitch-rescue
- RT1: symbol footswitch-rescue:FUSE -> footswitch-rescue:FUSE-footswitch-rescue
- U2: symbol footswitch-rescue:NCP1117ST33T3G -> footswitch-rescue:NCP1117ST33T3G-footswitch-rescue
Changed lines of the file:
@@
 $EndDescr
 $Comp
-L footswitch-rescue:CP1 C10
+L footswitch-rescue:CP1-footswitch-rescue C10
 U 1 1 548B65F7
 P 5100 1850
@@
 $EndComp
 $Comp
-L footswitch-rescue:C C12
+L footswitch-rescue:C-footswitch-rescue C12
 U 1 1 548B6624
 P 5450 1850
@@
 $EndComp
 $Comp
-L footswitch-rescue:CP1 C5
+L footswitch-rescue:CP1-footswitch-rescue C5
 U 1 1 548B663E
 P 3500 1850
@@
 $EndComp
 $Comp
-L footswitch-rescue:D D1
+L footswitch-rescue:D-footswitch-rescue D1
 U 1 1 548B6651
 P 2300 1600
@@
 $EndComp
 $Comp
-L footswitch-rescue:FUSE RT1
+L footswitch-rescue:FUSE-footswitch-rescue RT1
 U 1 1 548B6658
 P 3050 1600
@@
 $EndComp
 $Comp
-L footswitch-rescue:C C7
+L footswitch-rescue:C-footswitch-rescue C7
 U 1 1 548B665F
 P 3800 1850
@@
 $EndComp
 $Comp
-L footswitch-rescue:GNDD #PWR01
+L footswitch-rescue:GNDD-footswitch-rescue #PWR01
 U 1 1 54E7EE6C
 P 3500 2100
@@
 $EndComp
 $Comp
-L footswitch-rescue:GNDD #PWR02
+L footswitch-rescue:GNDD-footswitch-rescue #PWR02
 U 1 1 54E7EE80
 P 3800 2100
@@
 $EndComp
 $Comp
-L footswitch-rescue:GNDD #PWR03
+L footswitch-rescue:GNDD-footswitch-rescue #PWR03
 U 1 1 54E7F9F2
 P 5100 2100
@@
 $EndComp
 $Comp
-L footswitch-rescue:GNDD #PWR04
+L footswitch-rescue:GNDD-footswitch-rescue #PWR04
 U 1 1 54E7FA28
 P 5450 2100
@@
 $EndComp
 $Comp
-L footswitch-rescue:GNDD #PWR05
+L footswitch-rescue:GNDD-footswitch-rescue #PWR05
 U 1 1 54E80258
 P 4450 1950
@@
 $EndComp
 $Comp
-L footswitch-rescue:+3.3V #PWR06
+L footswitch-rescue:+3.3V-footswitch-rescue #PWR06
 U 1 1 556EF2E1
 P 5700 1500
@@
 $EndComp
 $Comp
-L footswitch-rescue:Q_PMOS_GSD Q5
+L footswitch-rescue:Q_PMOS_GSD-footswitch-rescue Q5
 U 1 1 5576EC7B
 P 3450 3950
@@
 $EndComp
 $Comp
-L footswitch-rescue:D_Schottky D3
+L footswitch-rescue:D_Schottky-footswitch-rescue D3
 U 1 1 5576EF8F
 P 4250 3850
@@
 $EndComp
 $Comp
-L footswitch-rescue:R R13
+L footswitch-rescue:R-footswitch-rescue R13
 U 1 1 5576FA4A
 P 2950 4100
@@
 $EndComp
 $Comp
-L footswitch-rescue:VCC #PWR07
+L footswitch-rescue:VCC-footswitch-rescue #PWR07
 U 1 1 55770535
 P 2950 3750
@@
 $EndComp
 $Comp
-L footswitch-rescue:Q_NMOS_GSD Q4
+L footswitch-rescue:Q_NMOS_GSD-footswitch-rescue Q4
 U 1 1 55771A8F
 P 2850 4750
@@
 $EndComp
 $Comp
-L footswitch-rescue:Q_NMOS_GSD Q1
+L footswitch-rescue:Q_NMOS_GSD-footswitch-rescue Q1
 U 1 1 55771C8E
 P 2400 5100
@@
 $EndComp
 $Comp
-L footswitch-rescue:GNDD #PWR08
+L footswitch-rescue:GNDD-footswitch-rescue #PWR08
 U 1 1 557724D6
 P 2500 5400
@@
 $EndComp
 $Comp
-L footswitch-rescue:GNDD #PWR09
+L footswitch-rescue:GNDD-footswitch-rescue #PWR09
 U 1 1 55772F70
 P 2950 5050
@@
 $EndComp
 $Comp
-L footswitch-rescue:R R8
+L footswitch-rescue:R-footswitch-rescue R8
 U 1 1 55773BAE
 P 2500 4450
@@
 $EndComp
 $Comp
-L footswitch-rescue:VCC #PWR010
+L footswitch-rescue:VCC-footswitch-rescue #PWR010
 U 1 1 55774D84
 P 2500 4200
@@
 $EndComp
 $Comp
-L footswitch-rescue:C C8
+L footswitch-rescue:C-footswitch-rescue C8
 U 1 1 55779079
 P 3800 4100
@@
 $EndComp
 $Comp
-L footswitch-rescue:NCP1117ST33T3G U2
+L footswitch-rescue:NCP1117ST33T3G-footswitch-rescue U2
 U 1 1 557C3298
 P 4450 1650
@@
 $EndComp
 $Comp
-L footswitch-rescue:R R4
+L footswitch-rescue:R-footswitch-rescue R4
 U 1 1 557CABF6
 P 2050 5400
@@
 $EndComp
 $Comp
-L footswitch-rescue:GNDD #PWR011
+L footswitch-rescue:GNDD-footswitch-rescue #PWR011
 U 1 1 557CAF87
 P 2050 5650
@@
 $EndComp
 $Comp
-L footswitch-rescue:+5V #PWR012
+L footswitch-rescue:+5V-footswitch-rescue #PWR012
 U 1 1 557CDFF5
 P 4600 3750
@@
 $EndComp
 $Comp
-L footswitch-rescue:+5V #PWR013
+L footswitch-rescue:+5V-footswitch-rescue #PWR013
 U 1 1 557CC20F
 P 2650 1500
@@
 $EndComp
 $Comp
-L footswitch-rescue:R R3
+L footswitch-rescue:R-footswitch-rescue R3
 U 1 1 557CFF3F
 P 2050 4800
@@
 $EndComp
 $Comp
-L footswitch-rescue:PWR_FLAG #FLG014
+L footswitch-rescue:PWR_FLAG-footswitch-rescue #FLG014
 U 1 1 557B3123
 P 6950 1700
@@
 $EndComp
 $Comp
-L footswitch-rescue:+5V #PWR015
+L footswitch-rescue:+5V-footswitch-rescue #PWR015
 U 1 1 557B3200
 P 6950 1550
@@
 USB POWER
 $Comp
-L footswitch-rescue:VCC #PWR016
+L footswitch-rescue:VCC-footswitch-rescue #PWR016
 U 1 1 55B522FD
 P 7200 1550
@@
 $EndComp
 $Comp
-L footswitch-rescue:PWR_FLAG #FLG017
+L footswitch-rescue:PWR_FLAG-footswitch-rescue #FLG017
 U 1 1 55B523DA
 P 7200 1700
@@
 $EndComp
 $Comp
-L footswitch-rescue:+12V #PWR018
+L footswitch-rescue:+12V-footswitch-rescue #PWR018
 U 1 1 575EB4B7
 P 1600 1500
@@
 $EndComp
 $Comp
-L footswitch-rescue:PWR_FLAG #FLG019
+L footswitch-rescue:PWR_FLAG-footswitch-rescue #FLG019
 U 1 1 54B50E4C
 P 1950 1500
@@
 $EndComp
 $Comp
-L footswitch-rescue:+12V #PWR020
+L footswitch-rescue:+12V-footswitch-rescue #PWR020
 U 1 1 575EFB81
 P 2050 4550
@@
 $EndComp
 $Comp
-L footswitch-rescue:PWR_FLAG #FLG021
+L footswitch-rescue:PWR_FLAG-footswitch-rescue #FLG021
 U 1 1 5760D14C
 P 6650 1550
@@
 $EndComp
 $Comp
-L footswitch-rescue:GNDD #PWR022
+L footswitch-rescue:GNDD-footswitch-rescue #PWR022
 U 1 1 54E7EDE1
 P 6650 1700
@@
 +5V power comes from USB and it's activated\nonly if +12V is not present, i.e. when the control\nchain cable is not plugged in
 $Comp
-L footswitch-rescue:PWR_FLAG #FLG023
+L footswitch-rescue:PWR_FLAG-footswitch-rescue #FLG023
 U 1 1 59675A29
 P 3950 1500
