File: hw-design/board/control-chain.sch (KiCad schematic (older format))
At the start: 37 parts, among them J1 RJ45_CHAIN_MAIN, J2 RJ45_CHAIN_EXTENSION, Q1 MMBT3904, Q2 MMBT3906, Q4 MMBT3904, Q5 MMBT3904, Q6 MMBT3904, U4 MAX13450E

Commit message: importing common sheets from expression-pedal project
Parts:
- removed C18, C20, C8: 100nF_X7R, MOD_Footprints_Lib:SM0603, symbol C
- removed C19, C5: 100uF, MOD_Footprints_Lib:CAP_RAD_5MM, symbol CP1
- removed D2, D3: MMSZ5242B, MOD_Footprints_Lib:SOD123, symbol ZENERsmall
- removed J1: RJ45_CHAIN_MAIN, MOD_Footprints_Lib:RJ45-RJHSE5084, symbol RJ45_CHAIN
- removed J2: RJ45_CHAIN_EXTENSION, MOD_Footprints_Lib:RJ45-RJHSE5084, symbol RJ45_CHAIN
- removed Q1, Q4, Q5, Q6: MMBT3904, MOD_Footprints_Lib:SOT23, symbol NPN
- removed Q2: MMBT3906, MOD_Footprints_Lib:SOT23, symbol MMBT3906
- removed R1, R28, R29, R30, R31, R50, R51, R54: 10k, MOD_Footprints_Lib:SM0603, symbol R
- removed R2: 100R 0.5W, MOD_Footprints_Lib:SM1210, symbol R
- removed R27, R48, R49, R52: 100k, MOD_Footprints_Lib:SM0603, symbol R
- removed R3, R4: 1K2, MOD_Footprints_Lib:SM0805, symbol R
- removed R44: 0R/NC, MOD_Footprints_Lib:SM0805, symbol R
- removed R53: 1k, MOD_Footprints_Lib:SM0603, symbol R
- removed U4: MAX13450E, TSSOP-14EP, symbol MAX13450E
- added C9: 100nF X7R, Capacitors_SMD:C_0603, symbol C
- added D4: 1N4148, Diodes_SMD:SOD-323, symbol D
- added J1: CC_INPUT, Connect:RJHSE538X, symbol RJ45_LEDS
- added J2: CC_OUTPUT, Connect:RJHSE538X, symbol RJ45_LEDS
- added Q4, Q5: 2N7002, Housings_SOT-23_SOT-143_TSOT-6:SOT-23, symbol Q_NMOS_GSD
- added Q6: IRFML8244TRPBF, Housings_SOT-23_SOT-143_TSOT-6:SOT-23, symbol Q_NMOS_GSD
- added R10, R9: 10k, Resistors_SMD:R_0603, symbol R
- added R7, R8: 820R, Resistors_SMD:R_0603, symbol R
- added U3: ISL83491, Housings_SOIC:SOIC-14_3.9x8.7mm_Pitch1.27mm, symbol ISL83491
- R11: value 100R 0.5W -> 10k; footprint MOD_Footprints_Lib:SM1210 -> Resistors_SMD:R_0603; MPN (none) -> RMCF0603JT10K0
- R12: value 100k -> 100R; footprint MOD_Footprints_Lib:SM0603 -> Resistors_SMD:R_0805; MPN (none) -> ERJ-P06F1000V
- R13: footprint MOD_Footprints_Lib:SM0603 -> Resistors_SMD:R_0603; MPN (none) -> RMCF0603JT10K0
- R5, R6: value 1K2 -> 820R; footprint MOD_Footprints_Lib:SM0805 -> Resistors_SMD:R_0603; MPN (none) -> ESR03EZPJ821
Connections:
- net labels added: +9V, CC_OUTPUT_DET, CHAIN_DE, CHAIN_RX, CHAIN_TX, GNDD, POWER_INPUT, RS485_RX+, RS485_RX-, RS485_RX_LED, RS485_TX+, RS485_TX-, RS485_TX_LED, RX_LED, TX_LED
- net labels removed: +5V, DGND, GND_FB, LED_STATUS, RS422_RX+, RS422_RX-, RS422_TX+, RS422_TX-, RTERM_CHAIN, RX_CHAIN, TX_CHAIN, TX_CHAIN_EN, VCC, VCC_FB
- wire segments 133 -> 76
Other:
- note added: "CONNECTORS"
- note added: "INTERFACE"
- note added: "STATUS LEDS"
- note added: "TERMINATION RESISTOR"
- note removed: "PCB consideration: \nThis capacitor must \nbe placed as close as \npossible to the IC"

Commit message: sch: schematic files reorganized, new sheets for usb and rear board
Parts:
- removed C9: 100nF X7R, Capacitors_SMD:C_0603, symbol C
- removed D4: 1N4148, Diodes_SMD:SOD-323, symbol D
- removed J1: CC_INPUT, Connect:RJHSE538X, symbol RJ45_LEDS
- removed J2: CC_OUTPUT, Connect:RJHSE538X, symbol RJ45_LEDS
- removed Q4, Q5: 2N7002, Housings_SOT-23_SOT-143_TSOT-6:SOT-23, symbol Q_NMOS_GSD
- removed Q6: IRFML8244TRPBF, Housings_SOT-23_SOT-143_TSOT-6:SOT-23, symbol Q_NMOS_GSD
- removed R10, R11, R9: 10k, Resistors_SMD:R_0603, symbol R
- removed R12: 100R, Resistors_SMD:R_0805, symbol R
- removed R5, R6, R7, R8: 820R, Resistors_SMD:R_0603, symbol R
- renumbered R13 to R5
Other:
- note removed: "CONNECTORS"
- note removed: "STATUS LEDS"
- note removed: "TERMINATION RESISTOR"
- moved on the sheet: R5, U3

Commit message: annotation and ERC
Parts:
- renumbered R5 to R15, U3 to U1
Changed lines of the file:
@@
 $EndDescr
 $Comp
-L ISL83491 U3
+L ISL83491 U1
 U 1 1 557A059C
 P 3450 2200
-F 0 "U3" H 3150 1600 50  0000 L CNN
+F 0 "U1" H 3150 1600 50  0000 L CNN
 F 1 "ISL83491" H 3450 2800 50  0000 L CNN
 F 2 "Housings_SOIC:SOIC-14_3.9x8.7mm_Pitch1.27mm" H 3450 2200 50  0001 C CIN
@@
 $EndComp
 $Comp
-L GNDD #PWR029
+L GNDD #PWR29
 U 1 1 557D6D91
 P 3300 3000
-F 0 "#PWR029" H 3300 2750 60  0001 C CNN
+F 0 "#PWR29" H 3300 2750 60  0001 C CNN
 F 1 "GNDD" H 3300 2850 60  0000 C CNN
 F 2 "" H 3300 3000 60  0000 C CNN
@@
 $EndComp
 $Comp
-L +3.3V #PWR030
+L +3.3V #PWR33
 U 1 1 557D9E83
 P 3600 1400
-F 0 "#PWR030" H 3600 1250 50  0001 C CNN
+F 0 "#PWR33" H 3600 1250 50  0001 C CNN
 F 1 "+3.3V" H 3600 1540 50  0000 C CNN
 F 2 "" H 3600 1400 60  0000 C CNN
@@
 $EndComp
 $Comp
-L R R5
+L R R15
 U 1 1 557DF2C0
 P 4100 2850
-F 0 "R5" V 4180 2850 50  0000 C CNN
+F 0 "R15" V 4180 2850 50  0000 C CNN
 F 1 "10k" V 4100 2850 50  0000 C CNN
 F 2 "Resistors_SMD:R_0603" V 4030 2850 30  0001 C CNN
@@
 $EndComp
 $Comp
-L GNDD #PWR031
+L GNDD #PWR37
 U 1 1 557DFB58
 P 4100 3100
-F 0 "#PWR031" H 4100 2850 60  0001 C CNN
+F 0 "#PWR37" H 4100 2850 60  0001 C CNN
 F 1 "GNDD" H 4100 2950 60  0000 C CNN
 F 2 "" H 4100 3100 60  0000 C CNN
@@
 $EndComp
 $Comp
-L GNDD #PWR032
+L GNDD #PWR36
 U 1 1 557F118D
 P 4100 2150
-F 0 "#PWR032" H 4100 1900 60  0001 C CNN
+F 0 "#PWR36" H 4100 1900 60  0001 C CNN
 F 1 "GNDD" H 4100 2000 60  0000 C CNN
 F 2 "" H 4100 2150 60  0000 C CNN
@@
 Text GLabel 4250 2600 2    50   Input ~ 0
 CHAIN_DE
-Text Notes 3050 1000 0    100  ~ 0
+Text Notes 3100 1000 0    100  ~ 0
 INTERFACE
 Wire Wire Line
