File: hw-design/board/control-chain.sch (KiCad schematic (older format))
At the start: 2 parts, among them U1 ISL83491

Commit message: update MPN
Parts:
- R15: value 10k -> 10K
Changed lines of the file:
@@
 P 4100 2850
 F 0 "R15" V 4180 2850 50  0000 C CNN
-F 1 "10k" V 4100 2850 50  0000 C CNN
+F 1 "10K" V 4100 2850 50  0000 C CNN
 F 2 "Resistors_SMD:R_0603" V 4030 2850 30  0001 C CNN
 F 3 "" H 4100 2850 30  0000 C CNN

Commit message: update netlist
Parts:
- renumbered R15 to R17
Changed lines of the file:
@@
 $EndComp
 $Comp
-L GNDD #PWR28
+L GNDD #PWR30
 U 1 1 557D6D91
 P 3300 3000
-F 0 "#PWR28" H 3300 2750 60  0001 C CNN
+F 0 "#PWR30" H 3300 2750 60  0001 C CNN
 F 1 "GNDD" H 3300 2850 60  0000 C CNN
 F 2 "" H 3300 3000 60  0000 C CNN
@@
 $EndComp
 $Comp
-L +3.3V #PWR30
+L +3.3V #PWR32
 U 1 1 557D9E83
 P 3600 1400
-F 0 "#PWR30" H 3600 1250 50  0001 C CNN
+F 0 "#PWR32" H 3600 1250 50  0001 C CNN
 F 1 "+3.3V" H 3600 1540 50  0000 C CNN
 F 2 "" H 3600 1400 60  0000 C CNN
@@
 $EndComp
 $Comp
-L R R15
+L R R17
 U 1 1 557DF2C0
 P 4100 2850
-F 0 "R15" V 4180 2850 50  0000 C CNN
+F 0 "R17" V 4180 2850 50  0000 C CNN
 F 1 "10K" V 4100 2850 50  0000 C CNN
 F 2 "Resistors_SMD:R_0603" V 4030 2850 30  0001 C CNN
@@
 $EndComp
 $Comp
-L GNDD #PWR34
+L GNDD #PWR36
 U 1 1 557DFB58
 P 4100 3100
-F 0 "#PWR34" H 4100 2850 60  0001 C CNN
+F 0 "#PWR36" H 4100 2850 60  0001 C CNN
 F 1 "GNDD" H 4100 2950 60  0000 C CNN
 F 2 "" H 4100 3100 60  0000 C CNN
@@
 $EndComp
 $Comp
-L GNDD #PWR33
+L GNDD #PWR35
 U 1 1 557F118D
 P 4100 2150
-F 0 "#PWR33" H 4100 1900 60  0001 C CNN
+F 0 "#PWR35" H 4100 1900 60  0001 C CNN
 F 1 "GNDD" H 4100 2000 60  0000 C CNN
 F 2 "" H 4100 2150 60  0000 C CNN
