File: hw-design/board/control-chain.sch (KiCad schematic (older format))
At the start: 2 parts, among them U1 ISL83491

Commit message: sch: control RE pin via uC I/O
Parts:
- added R40: 10K, Resistors_SMD:R_0603, symbol R
Connections:
- net +3V3: now also R40.2
- net GNDD: no longer U1.3 (~RE)
- new net CHAIN_RE: R40.1, U1.3 (~RE)
Changed lines of the file:
@@
 LIBS:nxp_armmcu
 LIBS:philips
+LIBS:graphic_symbols
 LIBS:footswitch-cache
 EELAYER 26 0
@@
 	1    0    0    -1
 $EndComp
-$Comp
-L GNDD #PWR027
-U 1 1 557F118D
-P 4100 2150
-F 0 "#PWR027" H 4100 1900 60  0001 C CNN
-F 1 "GNDD" H 4100 2000 60  0000 C CNN
-F 2 "" H 4100 2150 60  0000 C CNN
-F 3 "" H 4100 2150 60  0000 C CNN
-	1    4100 2150
-	1    0    0    -1
-$EndComp
 Text GLabel 2800 1800 0    50   Input ~ 0
 RS485_RX+
@@
 	4250 2400 3950 2400
 Wire Wire Line
-	3950 2100 4100 2100
-Wire Wire Line
-	4100 2100 4100 2150
+	3950 2100 4250 2100
 Connection ~ 3300 2950
 Connection ~ 3600 1450
 Connection ~ 4100 2600
+$Comp
+L R R40
+U 1 1 59678A04
+P 4100 1650
+F 0 "R40" V 4180 1650 50  0000 C CNN
+F 1 "10K" V 4100 1650 50  0000 C CNN
+F 2 "Resistors_SMD:R_0603" V 4030 1650 30  0001 C CNN
+F 3 "" H 4100 1650 30  0000 C CNN
+F 4 "RMCF0603JT10K0" H -4550 -1400 50  0001 C CNN "MPN"
+	1    4100 1650
+	-1   0    0    1
+$EndComp
+$Comp
+L +3.3V #PWR027
+U 1 1 59678AAB
+P 4100 1400
+F 0 "#PWR027" H 4100 1250 50  0001 C CNN
+F 1 "+3.3V" H 4100 1540 50  0000 C CNN
+F 2 "" H 4100 1400 60  0000 C CNN
+F 3 "" H 4100 1400 60  0000 C CNN
+	1    4100 1400
+	1    0    0    -1
+$EndComp
+Wire Wire Line
+	4100 1400 4100 1500
+Text GLabel 4250 2100 2    50   Input ~ 0
+CHAIN_RE
+Wire Wire Line
+	4100 1800 4100 2100
+Connection ~ 4100 2100
 $EndSCHEMATC

Commit message: update files to KiCAD 5
Parts:
- R17, R40: symbol R -> footswitch-rescue:R
- U1: symbol ISL83491 -> footswitch-rescue:ISL83491
Changed lines of the file:
@@
-EESchema Schematic File Version 2
-LIBS:conn
-LIBS:device
-LIBS:interface
-LIBS:power
-LIBS:regul
-LIBS:transistors
-LIBS:display
-LIBS:nxp_armmcu
-LIBS:philips
-LIBS:graphic_symbols
+EESchema Schematic File Version 4
 LIBS:footswitch-cache
 EELAYER 26 0
@@
 $EndDescr
 $Comp
-L ISL83491 U1
+L footswitch-rescue:ISL83491 U1
 U 1 1 557A059C
 P 3450 2200
@@
 $EndComp
 $Comp
-L GNDD #PWR024
+L footswitch-rescue:GNDD #PWR024
 U 1 1 557D6D91
 P 3300 3000
@@
 $EndComp
 $Comp
-L +3.3V #PWR025
+L footswitch-rescue:+3.3V #PWR025
 U 1 1 557D9E83
 P 3600 1400
@@
 $EndComp
 $Comp
-L R R17
+L footswitch-rescue:R R17
 U 1 1 557DF2C0
 P 4100 2850
@@
 $EndComp
 $Comp
-L GNDD #PWR026
+L footswitch-rescue:GNDD #PWR026
 U 1 1 557DFB58
 P 4100 3100
@@
 Connection ~ 4100 2600
 $Comp
-L R R40
+L footswitch-rescue:R R40
 U 1 1 59678A04
 P 4100 1650
@@
 $EndComp
 $Comp
-L +3.3V #PWR027
+L footswitch-rescue:+3.3V #PWR027
 U 1 1 59678AAB
 P 4100 1400

Commit message: Changed R40 RE from pull-up to pull-down
Parts:
- R17, R40: symbol footswitch-rescue:R -> footswitch-rescue:R-footswitch-rescue
- U1: symbol footswitch-rescue:ISL83491 -> footswitch-rescue:ISL83491-footswitch-rescue
Connections:
- net +3V3: no longer R40.2
- net GNDD: now also R40.2
Changed lines of the file:
@@
 $EndDescr
 $Comp
-L footswitch-rescue:ISL83491 U1
+L footswitch-rescue:ISL83491-footswitch-rescue U1
 U 1 1 557A059C
 P 3450 2200
@@
 $EndComp
 $Comp
-L footswitch-rescue:GNDD #PWR024
+L footswitch-rescue:GNDD-footswitch-rescue #PWR024
 U 1 1 557D6D91
 P 3300 3000
@@
 $EndComp
 $Comp
-L footswitch-rescue:+3.3V #PWR025
+L footswitch-rescue:+3.3V-footswitch-rescue #PWR025
 U 1 1 557D9E83
 P 3600 1400
@@
 $EndComp
 $Comp
-L footswitch-rescue:R R17
+L footswitch-rescue:R-footswitch-rescue R17
 U 1 1 557DF2C0
 P 4100 2850
@@
 $EndComp
 $Comp
-L footswitch-rescue:GNDD #PWR026
+L footswitch-rescue:GNDD-footswitch-rescue #PWR026
 U 1 1 557DFB58
 P 4100 3100
@@
 	3250 2900 3250 2950
 Wire Wire Line
-	3250 2950 3350 2950
+	3250 2950 3300 2950
 Wire Wire Line
 	3350 2950 3350 2900
@@
 	3550 1500 3550 1450
 Wire Wire Line
-	3550 1450 3650 1450
+	3550 1450 3600 1450
 Wire Wire Line
 	3650 1450 3650 1500
@@
 	3600 1400 3600 1450
 Wire Wire Line
-	3950 2600 4250 2600
+	3950 2600 4100 2600
 Wire Wire Line
 	4100 2700 4100 2600
@@
 	4250 2400 3950 2400
 Wire Wire Line
-	3950 2100 4250 2100
+	3950 2100 4100 2100
 Connection ~ 3300 2950
 Connection ~ 3600 1450
 Connection ~ 4100 2600
 $Comp
-L footswitch-rescue:R R40
+L footswitch-rescue:R-footswitch-rescue R40
 U 1 1 59678A04
 P 4100 1650
@@
 	-1   0    0    1
 $EndComp
-$Comp
-L footswitch-rescue:+3.3V #PWR027
-U 1 1 59678AAB
-P 4100 1400
-F 0 "#PWR027" H 4100 1250 50  0001 C CNN
-F 1 "+3.3V" H 4100 1540 50  0000 C CNN
-F 2 "" H 4100 1400 60  0000 C CNN
-F 3 "" H 4100 1400 60  0000 C CNN
-	1    4100 1400
-	1    0    0    -1
-$EndComp
-Wire Wire Line
-	4100 1400 4100 1500
 Text GLabel 4250 2100 2    50   Input ~ 0
 CHAIN_RE
@@
 	4100 1800 4100 2100
 Connection ~ 4100 2100
+Wire Wire Line
+	3300 2950 3350 2950
+Wire Wire Line
+	3600 1450 3650 1450
+Wire Wire Line
+	4100 2600 4250 2600
+Wire Wire Line
+	4100 2100 4250 2100
+$Comp
+L footswitch-rescue:GNDD-footswitch-rescue #PWR0101
+U 1 1 5C8F8154
+P 4100 1400
+F 0 "#PWR0101" H 4100 1150 60  0001 C CNN
+F 1 "GNDD" H 4100 1250 60  0000 C CNN
+F 2 "" H 4100 1400 60  0000 C CNN
+F 3 "" H 4100 1400 60  0000 C CNN
+	1    4100 1400
+	-1   0    0    1
+$EndComp
+Wire Wire Line
+	4100 1500 4100 1400
 $EndSCHEMATC
