File: hw-design/board/footswitch.kicad_pcb (KiCad board)
At the start: 2 copper layers, 248.9 x 74.2 mm, 99 parts, among them CN1 CONN_PANNEL_2X2, CN2 CONN_PANNEL_2X2, J1 RJ45_CHAIN_MAIN, J2 RJ45_CHAIN_EXTENSION, P1 HEADER_5X2, P2 HEADER_5X2, Q1 MMBT3904, Q2 MMBT3906, Q3 MMBT3904, U1 LPC111X_LQFP48, U2 MC7805, U3 NCP1117DT33G, U4 MAX13450E, U5 74HC245, U6 74HC245, X1 10MHz

Commit message: sch: added mechanic sheet
Parts:
- removed C1, C16, C3, C5, C6: 100uF, MOD_Footprints_Lib:CAP_RAD_5MM
- removed C10, C11: 18pF_NP0, MOD_Footprints_Lib:SM0603
- removed C12, C13, C14, C15, C17, C18, C2, C4, C7, C8, C9: 100nF_X7R, MOD_Footprints_Lib:SM0603
- removed CN1, CN2: CONN_PANNEL_2X2, MOD_Footprints_Lib:CONN_PANNEL
- removed D1: CGRA4007-G, MOD_Footprints_Lib:DO-214AC(SMA)
- removed D2, D3: MMSZ5242B, MOD_Footprints_Lib:SOD123
- removed FOOT1, FOOT2, FOOT3, FOOT4: HEADER_2X1_180, MOD_Footprints_Lib:PIN_ARRAY_2X1
- removed G***: LOGO, MOD_Footprints_Lib:MOD_Logo
- removed J1: RJ45_CHAIN_MAIN, MOD_Footprints_Lib:RJ45-RJHSE5084
- removed J2: RJ45_CHAIN_EXTENSION, MOD_Footprints_Lib:RJ45-RJHSE5084
- removed LCD1: AGM-2004A-204, MOD_Footprints_Lib:LCD-AGM-2004A-204
- removed LED1, LED2, LED3, LED4: LED_RGB, MOD_Footprints_Lib:LED_CLRTB_GFSF_1
- removed P1, P2: HEADER_5X2, MOD_Footprints_Lib:PIN_ARRAY_5x2
- removed Q1, Q3: MMBT3904, MOD_Footprints_Lib:SOT23
- removed Q2: MMBT3906, MOD_Footprints_Lib:SOT23
- removed R1, R14, R15, R16, R17, R18, R19, R20, R21, R22, R23, R24, R25, R27, R36: 1k, MOD_Footprints_Lib:SM0603
- removed R10, R13, R28, R29, R30, R31, R32, R33, R46, R47, R7, R8, R9: 10k, MOD_Footprints_Lib:SM0603
- removed R11, R2: 100R 0.5W, MOD_Footprints_Lib:SM1210
- removed R12: 100k, MOD_Footprints_Lib:SM0603
- removed R26, R37, R38, R39, R42, R43, R45: 0R, MOD_Footprints_Lib:SM0805
- removed R3, R4, R5, R6: 470R, MOD_Footprints_Lib:SM0805
- removed R34: 3k, MOD_Footprints_Lib:SM0805
- removed R35: 330R, MOD_Footprints_Lib:SM0805
- removed R40, R41: 100R, MOD_Footprints_Lib:SM0603
- removed R44: 0R/NC, MOD_Footprints_Lib:SM0805
- removed RT1: PTC_FUSE_500mA, MOD_Footprints_Lib:SM2920
- removed RT2: PTC_FUSE_500mA, MOD_Footprints_Lib:SM1210
- removed TP1, TP2, TP3: CONN_1, MOD_Footprints_Lib:SIL-1
- removed U1: LPC111X_LQFP48, MOD_Footprints_Lib:LQFP48
- removed U2: MC7805, MOD_Footprints_Lib:DPAK(369C)
- removed U3: NCP1117DT33G, MOD_Footprints_Lib:DPAK(369C)
- removed U4: MAX13450E, MOD_Footprints_Lib:TSSOP14
- removed U5, U6: 74HC245, MOD_Footprints_Lib:TSSOP20
- removed X1: 10MHz, MOD_Footprints_Lib:HC_49US
Routing:
- net +3.3V: track 538.0 -> 0.00 mm, vias 22 -> 0
- net FOOT_4: track 203.3 -> 0.00 mm
- net LED4_B: track 199.0 -> 0.00 mm, vias 2 -> 0
- net LED4_R: track 198.7 -> 0.00 mm, vias 2 -> 0
- net LED4_G: track 196.4 -> 0.00 mm
- net DGND: track 166.9 -> 0.00 mm, vias 58 -> 0
- net +5V: track 151.3 -> 0.00 mm, vias 5 -> 0
- net FOOT_3: track 129.6 -> 0.00 mm
- net LED3_G: track 124.0 -> 0.00 mm
- net LED3_R: track 123.9 -> 0.00 mm
- net LED3_B: track 123.5 -> 0.00 mm
- net Net-(C6-Pad1): track 105.3 -> 0.00 mm, vias 33 -> 0
- net LCD_RS: track 58.6 -> 0.00 mm
- net RS422_TX+: track 58.5 -> 0.00 mm, vias 4 -> 0
- net FOOT_2: track 55.8 -> 0.00 mm
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- removed copper zone on B.Cu, net DGND
- removed copper zone on F.Cu, net DGND
- removed copper zone on B.Cu, net N-0000012
- removed copper zone on F.Cu, net N-0000012
Other:
- board outline removed
- net class Default: clearance 0.2032 -> 0.2; trace_width 0.254 -> 0.25; via_dia 0.889 -> 0.6; via_drill 0.635 -> 0.4
- rule pad_to_mask_clearance: 0 -> 0.2
- rule trace_clearance: 0.2032 -> 0.2
- rule trace_min: 0.2032 -> 0.2
- rule via_min_drill: 0.3048 -> 0.3
- rule via_min_size: 0.508 -> 0.4
- board text removed: "(c) 2014 Musical Operating Devices Licensed under CC By-SA https://github.com/portalmod/mod-hw-footswitch/"
- board text removed: "+3.3V"
- board text removed: "+5V"
- board text removed: "12"
- board text removed: "24"
- board text removed: "36"
- board text removed: "GND"
- board text removed: "UART DEBUGGER"

Commit message: pcb: importing board dxf files
Other:
- board outline added: 249.4 x 87.7 mm

Commit message: pcb: importing netlist
Parts:
- added C1: 10uF, Capacitors_SMD:c_elec_5x5.3, F.Cu at (501.0, 48.1)
- added C10: 10nF 500V, Capacitors_SMD:C_1206, F.Cu at (415.5, 107.3)
- added C11: 18pF, Capacitors_SMD:C_0603, F.Cu at (432.3, 103.6)
- added C12: 18pF, Capacitors_SMD:C_0603, F.Cu at (416.8, 113.6)
- added C13: 10nF, Capacitors_SMD:C_0603, F.Cu at (430.6, 97.7)
- added C14: 100nF X7R, Capacitors_SMD:C_0603, F.Cu at (403.4, 113.1)
- added C15: 100nF X7R, Capacitors_SMD:C_0603, F.Cu at (424.1, 97.0)
- added C16: 100nF X7R, Capacitors_SMD:C_0603, F.Cu at (424.1, 91.1)
- added C17: 100nF X7R, Capacitors_SMD:C_0603, F.Cu at (355.2, 101.8)
- added C18: 100nF X7R, Capacitors_SMD:C_0603, F.Cu at (346.4, 101.8)
- added C19: 100nF X7R, Capacitors_SMD:C_0603, F.Cu at (365.8, 91.1)
- added C2: 10uF, Capacitors_SMD:C_0805, F.Cu at (507.0, 50.4)
- added C20: 100nF X7R, Capacitors_SMD:C_0603, F.Cu at (338.7, 112.6)
- added C21: 100nF, Capacitors_SMD:C_0603, F.Cu at (404.4, 20.0)
- added C22: 10uF, Capacitors_SMD:C_0805, F.Cu at (413.4, 3.68)
- added C23: 47uF, Capacitors_SMD:c_elec_6.3x5.3, F.Cu at (406.5, 5.52)
- added C24: 100nF, Capacitors_SMD:C_0603, F.Cu at (340.7, 80.5)
- added C25: 10uF, Capacitors_SMD:C_0805, F.Cu at (336.0, 80.7)
- added C3: 100nF, Capacitors_SMD:C_0603, F.Cu at (511.7, 50.2)
- added C4: 100uF, Capacitors_SMD:c_elec_6.3x5.3, F.Cu at (491.4, 49.2)
- added C5: 100nF, Capacitors_SMD:C_0603, F.Cu at (505.1, 56.5)
- added C6: 100nF, Capacitors_SMD:C_0603, F.Cu at (521.9, 43.6)
- added C7: 100uF, Capacitors_SMD:c_elec_6.3x5.3, F.Cu at (501.9, 39.0)
- added C8: 100nF, Capacitors_SMD:C_0603, F.Cu at (516.8, 50.2)
- added C9: 100nF X7R, Capacitors_SMD:C_0603, F.Cu at (492.3, 22.3)
- added D1: CGRA4007-G, Diodes_SMD:Diode-SMA_Standard, F.Cu at (491.9, 38.9)
- added D2: 1N5819, Diodes_SMD:SOD-123, F.Cu at (516.1, 44.1)
- added D3: 1N5819, Diodes_SMD:SOD-123, F.Cu at (509.8, 44.1)
- added D4: 1N4148, Diodes_SMD:SOD-323, F.Cu at (523.8, 3.43)
- added D5: LED_RGB, LEDs:LED-RGB_PLLC-6, F.Cu at (353.6, 108.4)
- added D6: LED_RGB, LEDs:LED-RGB_PLLC-6, F.Cu at (364.8, 97.6)
- added D7: LED_RGB, LEDs:LED-RGB_PLLC-6, F.Cu at (346.6, 108.4)
- added D8: LED_RGB, LEDs:LED-RGB_PLLC-6, F.Cu at (346.6, 115.8)
- added DS1: ERM1602FS-6 3.3V, Display:WC1602A, F.Cu at (329.5, 5.18)
- added DS2: ERM1602FS-6 3.3V, Display:WC1602A, F.Cu at (329.5, 43.7)
- added J1: CC_INPUT, Connect:RJHSE538X, F.Cu at (480.6, 9.13)
- added J2: CC_OUTPUT, Connect:RJHSE538X, F.Cu at (499.8, 9.13)
- added P1: CHAIN, Pin_Headers:Pin_Header_Straight_1x04, F.Cu at (412.8, 94.3)
- added P2: USB_OTG, Connect:USB_Mini-B, F.Cu at (405.2, 96.3)
- added P3: SWD, Pin_Headers:Pin_Header_Straight_2x05_Pitch1.27mm, F.Cu at (417.1, 90.9)
- added P4: FOOT, Pin_Headers:Pin_Header_Angled_1x02, F.Cu at (350.5, 94.3)
- added P5: FOOT, Pin_Headers:Pin_Header_Angled_1x02, F.Cu at (331.1, 105.0)
- added P6: FOOT, Pin_Headers:Pin_Header_Angled_1x02, F.Cu at (323.4, 116.3)
- added P7: FOOT, Pin_Headers:Pin_Header_Angled_1x02, F.Cu at (337.5, 94.3)
- added Q1: 2N7002, Housings_SOT-23_SOT-143_TSOT-6:SOT-23, F.Cu at (517.1, 37.3)
- added Q10: 2N7002, Housings_SOT-23_SOT-143_TSOT-6:SOT-23, F.Cu at (324.4, 80.8)
- added Q2: 2N7002, Housings_SOT-23_SOT-143_TSOT-6:SOT-23, F.Cu at (499.3, 55.6)
- added Q3: FDN306P, local-footprints:SOT-23-fairchild, F.Cu at (510.3, 37.7)
- added Q4: 2N7002, Housings_SOT-23_SOT-143_TSOT-6:SOT-23, F.Cu at (499.9, 22.7)
- added Q5: 2N7002, Housings_SOT-23_SOT-143_TSOT-6:SOT-23, F.Cu at (516.1, 16.7)
- added Q6: IRFML8244TRPBF, Housings_SOT-23_SOT-143_TSOT-6:SOT-23, F.Cu at (481.2, 22.7)
- added Q7: BC857, Housings_SOT-23_SOT-143_TSOT-6:SOT-23, F.Cu at (431.2, 91.4)
- added Q8: 2N7002, Housings_SOT-23_SOT-143_TSOT-6:SOT-23, F.Cu at (330.8, 80.8)
- added Q9: 2N7002, Housings_SOT-23_SOT-143_TSOT-6:SOT-23, F.Cu at (405.0, 13.7)
- added R1: 3K6, Resistors_SMD:R_0603, F.Cu at (521.2, 49.5)
- added R10: 10k, Resistors_SMD:R_0603, F.Cu at (525.9, 9.33)
- added R11: 10k, Resistors_SMD:R_0603, F.Cu at (521.0, 16.3)
- added R12: 100R, Resistors_SMD:R_0805, F.Cu at (505.2, 23.2)
- added R13: 10k, Resistors_SMD:R_0603, F.Cu at (522.5, 9.33)
- added R14: 3k, Resistors_SMD:R_0603, F.Cu at (434.4, 97.7)
- added R15: 24k, Resistors_SMD:R_0603, F.Cu at (421.6, 108.8)
- added R16: 1k5, Resistors_SMD:R_0603, F.Cu at (428.5, 103.6)
- added R17: 1M, Resistors_SMD:R_0603, F.Cu at (425.0, 108.8)
- added R18: 33R, Resistors_SMD:R_0603, F.Cu at (428.5, 109.5)
- added R19: 33R, Resistors_SMD:R_0603, F.Cu at (421.6, 102.9)
- added R2: 5K6, Resistors_SMD:R_0603, F.Cu at (514.1, 56.1)
- added R20: 2K, Resistors_SMD:R_0603, F.Cu at (413.0, 113.6)
- added R21: 3K3, Resistors_SMD:R_0603, F.Cu at (409.5, 113.6)
- added R22: 10k, Resistors_SMD:R_0603, F.Cu at (425.0, 102.9)
- added R23: 10k, Resistors_SMD:R_0603, F.Cu at (374.5, 102.9)
- added R24: 10k, Resistors_SMD:R_0603, F.Cu at (363.2, 110.3)
- added R25: 10k, Resistors_SMD:R_0603, F.Cu at (377.9, 97.0)
- added R26: 10k, Resistors_SMD:R_0603, F.Cu at (356.2, 116.2)
- added R27: 10k, Resistors_SMD:R_0603, F.Cu at (377.9, 102.9)
- added R28: 10k, Resistors_SMD:R_0603, F.Cu at (365.8, 104.4)
- added R29: 10k, Resistors_SMD:R_0603, F.Cu at (374.5, 97.0)
- added R3: 10k, Resistors_SMD:R_0603, F.Cu at (510.7, 56.1)
- added R30: 220R, Resistors_SMD:R_0603, F.Cu at (359.3, 110.3)
- added R31: 220R, Resistors_SMD:R_0603, F.Cu at (370.6, 97.0)
- added R32: 220R, Resistors_SMD:R_0603, F.Cu at (352.3, 115.2)
- added R33: 220R, Resistors_SMD:R_0603, F.Cu at (376.8, 91.1)
- added R34: 220R, Resistors_SMD:R_0603, F.Cu at (361.8, 104.4)
- added R35: 220R, Resistors_SMD:R_0603, F.Cu at (372.4, 91.1)
- added R36: 220R, Resistors_SMD:R_0603, F.Cu at (370.6, 102.9)
- added R37: 220R, Resistors_SMD:R_0603, F.Cu at (371.6, 108.8)
- added R38: 220R, Resistors_SMD:R_0603, F.Cu at (367.2, 110.3)
- added R39: 220R, Resistors_SMD:R_0603, F.Cu at (360.1, 116.2)
- added R4: 10k, Resistors_SMD:R_0603, F.Cu at (521.9, 36.9)
- added R40: 220R, Resistors_SMD:R_0603, F.Cu at (364.5, 116.2)
- added R41: 220R, Resistors_SMD:R_0603, F.Cu at (376.0, 108.8)
- added R42: 4K7, Resistors_SMD:R_0603, F.Cu at (417.2, 3.48)
- added R43: 680R, Resistors_SMD:R_0603, F.Cu at (413.5, 9.78)
- added R44: 100K, Resistors_SMD:R_0603, F.Cu at (404.0, 25.9)
- added R45: 100K, Resistors_SMD:R_0603, F.Cu at (417.9, 9.38)
- added R5: 820R, Resistors_SMD:R_0603, F.Cu at (509.6, 22.3)
- added R6: 820R, Resistors_SMD:R_0603, F.Cu at (524.7, 27.0)
- added R7: 820R, Resistors_SMD:R_0603, F.Cu at (524.9, 21.1)
- added R8: 820R, Resistors_SMD:R_0603, F.Cu at (524.9, 15.2)
- added R9: 10k, Resistors_SMD:R_0603, F.Cu at (520.9, 22.2)
- added RT1: PTC_FUSE, Resistors_SMD:R_1210, F.Cu at (490.6, 57.8)
- added SW1: SW_PUSH, Buttons_Switches_SMD:SW_SPST_FSMSM, F.Cu at (405.0, 107.9)
- added SW2: SP3T, local-footprints:OS103011MA7QP1, F.Cu at (324.3, 92.1)
- added U1: NCP1117DT50G, SMD_Packages:DPAK-2, F.Cu at (480.6, 45.5)
- added U2: NCP1117DT33G, SMD_Packages:DPAK-2, F.Cu at (480.6, 58.9)
- added U3: ISL83491, Housings_SOIC:SOIC-14_3.9x8.7mm_Pitch1.27mm, F.Cu at (516.8, 6.96)
- added U4: LPC11U24FBD48/401, Housings_QFP:LQFP-48_7x7mm_Pitch0.5mm, F.Cu at (391.7, 95.2)
- added U5: PCA9685, Housings_SSOP:TSSOP-28_4.4x9.7mm_Pitch0.65mm, F.Cu at (325.1, 103.2)
- added Y1: 12MHz, Crystals:Crystal_HC49-SD_SMD, F.Cu at (391.1, 108.3)
Other:
- board size 249.4 x 87.7 mm -> 249.4 x 60 mm

Commit message: pcb: importing netlist after remove channel selector
Parts:
- removed the R25 at (377.9, 97.0)
- removed the R26 at (356.2, 116.2)
- removed the R27 at (377.9, 102.9)
- removed SW2: SP3T, local-footprints:OS103011MA7QP1
- moved DS1 294.4 mm to (40.2, 59.5)
- moved P4 281.2 mm to (69.8, 111.8), turned to 270 degrees
- moved P6 246.3 mm to (77.1, 111.7), turned to 270 degrees
- moved DS2 137.8 mm to (192.6, 59.5)
- moved P7 109.3 mm to (229.5, 111.7), turned to 270 degrees
- moved P5 109.1 mm to (222.2, 111.7), turned to 270 degrees
- renumbered R28 to R25, R29 to R26, R30 to R27, R31 to R28, R32 to R29, R33 to R30, R34 to R31, R35 to R32, R36 to R33, R37 to R34, R38 to R35, R39 to R36, R40 to R37, R41 to R38, R42 to R39, R43 to R40, R44 to R41, R45 to R42
Connections:
- U4 pad 13: CH2 -> Net-(U4-Pad13)
- U4 pad 2: CH1 -> Net-(U4-Pad2)
- U4 pad 26: CH3 -> Net-(U4-Pad26)

Commit message: pcb: initial placement of footprint with mandatory position
Parts:
- added H1: HOLE, local-footprints:M3-screw-hole, F.Cu at (28.2, 64.0)
- added H2: HOLE, local-footprints:M3-screw-hole, F.Cu at (117.2, 93.0)
- added H3: HOLE, local-footprints:M3-screw-hole, F.Cu at (28.2, 111.5)
- added H4: HOLE, local-footprints:M3-screw-hole, F.Cu at (179.6, 93.0)
- added H5: HOLE, local-footprints:M3-screw-hole, F.Cu at (268.6, 64.0)
- added H6: HOLE, local-footprints:M3-screw-hole, F.Cu at (268.6, 111.5)
- added H7: KEYSTONE, local-footprints:Keystone-7790, F.Cu at (173.9, 66.2)
- added H8: KEYSTONE, local-footprints:Keystone-7790, F.Cu at (115.4, 66.2)
- DS1, DS2: footprint Display:WC1602A -> local-footprints:WC1602A
- P4, P5, P6, P7: moved to B.Cu
- moved J1 354.8 mm to (130.6, 67.6)
- moved J2 345.7 mm to (159.1, 67.6)
- moved D5 319.6 mm to (34.1, 100.8)
- moved P2 258.8 mm to (148.4, 64.6), turned to 270 degrees
- moved D6 254.7 mm to (110.2, 100.8)
- moved R4 189.3 mm to (335.6, 70.5)
- moved C6 188.2 mm to (336.5, 76.4)
- moved C7 188.1 mm to (316.3, 69.4)
- moved D2 182.6 mm to (334.6, 64.4)
- moved U1 178.4 mm to (305.5, 79.2)
- moved R1 178.3 mm to (344.1, 70.5)
- moved C8 177.1 mm to (341.7, 76.4)
- moved D1 176.3 mm to (316.7, 59.1)
- moved Q1 176.3 mm to (341.9, 57.5)
- moved C1 176.3 mm to (325.9, 68.3)
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
Commit message: pcb: rear board layout done
Parts:
- removed the C10 at (330.0, 31.6)
- removed the C13 at (334.8, 37.9)
- removed the C9 at (418.9, 25.2)
- removed the D4 at (412.1, 37.8)
- removed the P2 at (148.4, 64.6)
- removed the Q4 at (426.5, 25.6)
- removed the Q5 at (417.6, 31.5)
- removed the Q6 at (407.8, 25.6)
- removed the R10 at (431.4, 31.1)
- removed the R11 at (426.9, 37.8)
- removed the R12 at (423.0, 32.1)
- removed the R14 at (336.1, 31.1)
- removed the R15 at (342.1, 37.0)
- removed the R16 at (345.1, 25.2)
- removed the R17 at (348.5, 25.2)
- removed the R18 at (343.8, 31.1)
- removed the R19 at (347.2, 31.1)
- removed the R20 at (338.7, 37.0)
- removed the R21 at (334.5, 43.8)
- removed the R5 at (411.3, 31.9)
- removed the R6 at (417.6, 37.8)
- removed the R7 at (431.8, 25.2)
- removed the R8 at (422.0, 38.2)
- removed the R9 at (426.8, 31.9)
- added C23: 100nF X7R, Capacitors_SMD:C_0603, F.Cu at (173.9, 72.5)
- added C24: 10nF 500V, Capacitors_SMD:C_1206, F.Cu at (151.4, 66.3)
- added C25: 10nF, Capacitors_SMD:C_0603, F.Cu at (310.1, 75.8)
- added D8: 1N4148, Diodes_SMD:SOD-323, F.Cu at (172.1, 72.6)
- added P7: CONN_01X16, Pin_Headers:Pin_Header_Straight_1x16, F.Cu at (167.5, 74.8)
- added P8: USB_OTG, Connect:USB_Mini-B, F.Cu at (148.4, 60.0)
- added P9: CONN_01X16, Pin_Headers:Pin_Header_Angled_1x16, F.Cu at (362.5, 127.2)
- added Q10: BC857, Housings_SOT-23_SOT-143_TSOT-6:SOT-23, F.Cu at (305.3, 76.1)
- added Q8: 2N7002, Housings_SOT-23_SOT-143_TSOT-6:SOT-23, F.Cu at (152.2, 69.3)
- added Q9: IRFML8244TRPBF, Housings_SOT-23_SOT-143_TSOT-6:SOT-23, F.Cu at (176.5, 69.5)
- added R27: 10k, Resistors_SMD:R_0603, F.Cu at (141.3, 71.8)
- added R28: 820R, Resistors_SMD:R_0603, F.Cu at (138.5, 71.8)
- added R29: 820R, Resistors_SMD:R_0603, F.Cu at (129.6, 71.8)
- added R30: 820R, Resistors_SMD:R_0603, F.Cu at (169.5, 71.9)
- added R31: 820R, Resistors_SMD:R_0603, F.Cu at (158.1, 71.9)
- added R32: 10k, Resistors_SMD:R_0603, F.Cu at (155.3, 71.9)
- added R33: 10k, Resistors_SMD:R_0603, F.Cu at (175.6, 72.5)
- added R34: 100R, Resistors_SMD:R_0805, F.Cu at (179.3, 69.5)
- added R35: 1M, Resistors_SMD:R_0603, F.Cu at (144.0, 66.2)
- added R36: 3k, Resistors_SMD:R_0603, F.Cu at (309.7, 81.7)
- added R37: 24k, Resistors_SMD:R_0603, F.Cu at (314.0, 75.8)
- added R38: 1k5, Resistors_SMD:R_0603, F.Cu at (317.4, 75.8)
- added R39: 33R, Resistors_SMD:R_0603, F.Cu at (320.9, 75.8)
- added R40: 33R, Resistors_SMD:R_0603, F.Cu at (313.2, 81.7)
- added R41: 2K, Resistors_SMD:R_0603, F.Cu at (316.6, 81.7)
- added R42: 3K3, Resistors_SMD:R_0603, F.Cu at (320.1, 81.7)
- Q7: value BC857 -> 2N7002
- moved Q7 188.0 mm to (144.6, 69.3)
- moved R5 73.5 mm to (365.9, 72.2)
- moved U3 60.3 mm to (360.3, 75.7)
- moved Q4 51.6 mm to (369.1, 15.6)
- moved C21 49.3 mm to (374.8, 15.3)
- moved R23 47.6 mm to (379.1, 15.3)
- moved C22 43.9 mm to (361.6, 22.1)
- moved R24 42.7 mm to (370.1, 27.8)
- moved C20 42.7 mm to (354.8, 17.3)
- moved Q5 42.7 mm to (362.7, 15.6)
- moved R26 42.2 mm to (379.7, 21.2)
- moved C19 41.9 mm to (365.8, 22.1)
- moved Q6 41.0 mm to (353.2, 25.5)
- moved R25 38.4 mm to (375.3, 21.2)
- moved C18 37.7 mm to (370.5, 21.9)
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- renumbered C12 to C10, C14 to C11, C15 to C12, C16 to C13, C17 to C14, C18 to C15, C19 to C16, C20 to C17, C21 to C18, C22 to C19, C23 to C20, C24 to C21, C25 to C22, C11 to C9, D5 to D4, D6 to D5, D7 to D6, D8 to D7, P3 to P2, P4 to P3, P5 to P4, P6 to P5, P7 to P6, Q8 to Q4, Q9 to Q5, Q10 to Q6, R26 to R10, R27 to R11, R28 to R12, R29 to R13, R30 to R14, R31 to R15, R32 to R16, R33 to R17, R34 to R18, R35 to R19, R36 to R20, R37 to R21, R38 to R22, R39 to R23, R40 to R24, R41 to R25, R42 to R26, R13 to R5, R22 to R6, R23 to R7, R24 to R8, R25 to R9
Connections:
- net RS485_TX_LED renamed RJ45_TX_LED
- net VCC renamed USB_VCC
- H1 pad 1: Net-(H1-Pad1) -> (no net)
- H2 pad 1: Net-(H2-Pad1) -> (no net)
- H3 pad 1: Net-(H3-Pad1) -> (no net)
- H4 pad 1: Net-(H4-Pad1) -> (no net)
- H5 pad 1: Net-(H5-Pad1) -> (no net)
- H6 pad 1: Net-(H6-Pad1) -> (no net)
- H7 pad 1: Net-(H7-Pad1) -> (no net)
- H7 pad 2: Net-(H7-Pad2) -> (no net)
- H7 pad 3: Net-(H7-Pad3) -> (no net)
- H7 pad 4: Net-(H7-Pad4) -> (no net)
- H8 pad 1: Net-(H8-Pad1) -> (no net)
- H8 pad 2: Net-(H8-Pad2) -> (no net)
- H8 pad 3: Net-(H8-Pad3) -> (no net)
- H8 pad 4: Net-(H8-Pad4) -> (no net)
- J1 pad : (no net) -> GNDD
- J1 pad 1: RS485_RX+ -> RJ45_RX+
- J1 pad 11: RS485_RX_LED -> RJ45_RX_LED
- J1 pad 2: RS485_RX- -> RJ45_RX-
- J1 pad 3: RS485_TX+ -> RJ45_TX+
- J1 pad 5: POWER_INPUT -> RJ45_POWER_INPUT
- J1 pad 6: RS485_TX- -> RJ45_TX-
- J2 pad : (no net) -> GNDD
- J2 pad 1: RS485_TX+ -> RJ45_TX+
- J2 pad 11: RS485_RX_LED -> RJ45_RX_LED
- J2 pad 2: RS485_TX- -> RJ45_TX-
- J2 pad 3: RS485_RX+ -> RJ45_RX+
- J2 pad 6: RS485_RX- -> RJ45_RX-
- P2 pad 1: Net-(P3-Pad1) -> (no net)
- P2 pad 7: Net-(P3-Pad7) -> (no net)
- P2 pad 8: Net-(P3-Pad8) -> (no net)
- Q7 pad 1: Net-(Q7-Pad1) -> RX_LED
- Q7 pad 2: +3V3 -> GNDD
- Q7 pad 3: Net-(Q7-Pad3) -> RJ45_RX_LED
- U4 pad 10: Net-(U4-Pad10) -> (no net)
- U4 pad 12: Net-(U4-Pad12) -> (no net)
- U4 pad 13: Net-(U4-Pad13) -> (no net)
- U4 pad 18: Net-(U4-Pad18) -> (no net)
- U4 pad 19: USB_DM -> USB_DM_CPU
- U4 pad 2: Net-(U4-Pad2) -> (no net)
- U4 pad 20: USB_DP -> USB_DP_CPU
- U4 pad 24: Net-(U4-Pad24) -> (no net)
- U4 pad 25: Net-(U4-Pad25) -> (no net)
- U4 pad 26: Net-(U4-Pad26) -> (no net)
- U4 pad 31: Net-(U4-Pad31) -> (no net)
- U4 pad 38: Net-(U4-Pad38) -> (no net)
- U4 pad 46: RX_LED -> RX_LED_CPU
- U4 pad 47: TX_LED -> TX_LED_CPU
- U4 pad 48: Net-(U4-Pad48) -> (no net)
- U5 pad 13: Net-(U5-Pad13) -> (no net)
- U5 pad 18: Net-(U5-Pad18) -> (no net)
- U5 pad 22: Net-(U5-Pad22) -> (no net)
- U5 pad 9: Net-(U5-Pad9) -> (no net)
Routing:
- net +9V: track 0.00 -> 104.9 mm, vias 0 -> 3
- net GNDD: track 0.00 -> 67.4 mm, vias 0 -> 9
- net RJ45_RX-: track 0.00 -> 61.6 mm, vias 0 -> 1
- net RJ45_RX+: track 0.00 -> 61.4 mm
- net RJ45_TX+: track 0.00 -> 48.9 mm
- net RJ45_RX_LED: track 0.00 -> 42.5 mm
- net RJ45_TX_LED: track 0.00 -> 38.5 mm
- net RJ45_TX-: track 0.00 -> 38.3 mm
- net RJ45_POWER_INPUT: track 0.00 -> 27.4 mm
- net Net-(C24-Pad1): track 0.00 -> 25.0 mm
- net USB_PLUG_VCC: track 0.00 -> 12.6 mm
- net USB_DM: track 0.00 -> 12.6 mm
- net TX_LED: track 0.00 -> 12.2 mm, vias 0 -> 1
- net Net-(D8-Pad1): track 0.00 -> 12.0 mm, vias 0 -> 1
- net USB_DP: track 0.00 -> 11.8 mm
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- added copper zone on B.Cu, net GNDD
- added copper zone on F.Cu, net GNDD
Other:
- outline, holes or cut-outs redrawn
- net class Default: clearance 0.2 -> 0.15; trace_width 0.25 -> 0.3048; via_drill 0.4 -> 0.3
- rule trace_clearance: 0.2 -> 0.15
- rule trace_min: 0.2 -> 0.2032
- rule via_min_size: 0.4 -> 0.6

Commit message: importing netlist
Parts:
- removed the C14 at (368.6, 50.1)
- removed the C15 at (377.4, 44.2)
- removed the C16 at (368.6, 44.2)
- removed the C17 at (360.8, 58.1)
- removed the P1 at (319.2, 18.5)
- removed the P7 at (167.5, 74.8)
- removed the P9 at (362.5, 127.2)
- removed the Q7 at (144.6, 69.3)
- removed the Q8 at (152.2, 69.3)
- removed the R27 at (141.3, 71.8)
- removed the R28 at (138.5, 71.8)
- removed the R29 at (129.6, 71.8)
- removed the R30 at (169.5, 71.9)
- removed the R31 at (158.1, 71.9)
- removed the R32 at (155.3, 71.9)
- removed U5: PCA9685, Housings_SSOP:TSSOP-28_4.4x9.7mm_Pitch0.65mm
- added P3: CHAIN, Pin_Headers:Pin_Header_Straight_1x03, F.Cu at (319.2, 18.5)
- added P6: CONN_01X12, Pin_Headers:Pin_Header_Angled_1x12, F.Cu at (162.4, 75.2)
- added P8: CONN_01X12, Pin_Headers:Pin_Header_Angled_1x12, F.Cu at (162.4, 92.7)
- J1: value CC_INPUT -> CC_MAIN; footprint Connect:RJHSE538X -> local-footprints:54602-908LF
- J2: value CC_OUTPUT -> CC_NEXT; footprint Connect:RJHSE538X -> local-footprints:54602-908LF
- R3: renamed from R1; value 3K6 -> 10K
- R4: renamed from R2; value 5K6 -> 10K
- moved R22 363.6 mm to (29.0, 99.1)
- moved R24 357.9 mm to (29.0, 102.5)
- moved R23 353.3 mm to (29.0, 100.8)
- moved R1 329.1 mm to (60.2, 112.4)
- moved R10 296.3 mm to (85.0, 113.2)
- moved R25 293.0 mm to (105.1, 99.1)
- moved R27 287.0 mm to (105.1, 102.5)
- moved R26 279.2 mm to (105.1, 100.8)
- moved R30 200.7 mm to (181.4, 102.5)
- moved R28 197.2 mm to (181.4, 99.1)
- moved R29 191.3 mm to (181.4, 100.8)
- moved R2 169.1 mm to (209.9, 112.5)
- moved R11 150.7 mm to (237.2, 113.0)
- moved R31 137.8 mm to (257.6, 99.1)
- moved R32 122.7 mm to (257.6, 100.8)
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- renumbered C18 to C1, C4 to C10, C5 to C11, C11 to C12, C12 to C13, C25 to C14, C21 to C15, C22 to C16, C6 to C17, C24 to C18, C7 to C19, C19 to C2, C8 to C20, C13 to C21, C20 to C3, C9 to C4, C1 to C5, C10 to C6, C3 to C7, C2 to C8, C23 to C9, D8 to D2, D2 to D3, D3 to D4, D4 to D5, D5 to D6, D6 to D7, D7 to D8, P3 to P1, P4 to P2, P5 to P4, P6 to P5, P8 to P7, P2 to P9, Q4 to Q1, Q1 to Q2, Q10 to Q3, Q2 to Q4, Q3 to Q5, Q9 to Q6, Q5 to Q7, Q6 to Q8, R7 to R1, R9 to R10, R10 to R11, R4 to R12, R38 to R13, R34 to R14, R5 to R15, R33 to R16, R39 to R17, R40 to R18, R25 to R19, R8 to R2, R41 to R20, R42 to R21, R11 to R22, R12 to R23, R13 to R24, R14 to R25, R15 to R26, R16 to R27, R17 to R28, R18 to R29, R19 to R30, R20 to R31, R21 to R32, R22 to R33, R35 to R34, R26 to R35, R6 to R36, R23 to R5, R36 to R6, R37 to R7, R24 to R8, R3 to R9, U3 to U1, U1 to U2, U4 to U3, U2 to U4
Connections:
- D1 pad 2: POWER_INPUT -> +12V
- H1 pad 1: (no net) -> Net-(H1-Pad1)
- H2 pad 1: (no net) -> Net-(H2-Pad1)
- H3 pad 1: (no net) -> Net-(H3-Pad1)
- H4 pad 1: (no net) -> Net-(H4-Pad1)
- H5 pad 1: (no net) -> Net-(H5-Pad1)
- H6 pad 1: (no net) -> Net-(H6-Pad1)
- H7 pad 1: (no net) -> Net-(H7-Pad1)
- H7 pad 2: (no net) -> Net-(H7-Pad2)
- H7 pad 3: (no net) -> Net-(H7-Pad3)
- H7 pad 4: (no net) -> Net-(H7-Pad4)
- H8 pad 1: (no net) -> Net-(H8-Pad1)
- H8 pad 2: (no net) -> Net-(H8-Pad2)
- H8 pad 3: (no net) -> Net-(H8-Pad3)
- H8 pad 4: (no net) -> Net-(H8-Pad4)
- J1 pad 4: +9V -> +12V
- J1 pad 5: RJ45_POWER_INPUT -> +12V
- J2 pad 1: RJ45_TX+ -> RJ45_RX+
- J2 pad 2: RJ45_TX- -> RJ45_RX-
- J2 pad 3: RJ45_RX+ -> RJ45_TX+
- J2 pad 4: +9V -> +12V
- J2 pad 5: +9V -> +12V
- J2 pad 6: RJ45_RX- -> RJ45_TX-
- P7 pad 4: (no net) -> Net-(P7-Pad4)
- P9 pad 1: (no net) -> Net-(P9-Pad1)
- P9 pad 7: (no net) -> Net-(P9-Pad7)
- P9 pad 8: (no net) -> Net-(P9-Pad8)
- R16 pad 1: +9V -> +12V
- R22 pad 1: Net-(R11-Pad1) -> LED_B1
- R23 pad 1: Net-(R12-Pad1) -> LED_R1
- R24 pad 1: Net-(R13-Pad1) -> LED_G1
- R25 pad 1: Net-(R14-Pad1) -> LED_B2
- R26 pad 1: Net-(R15-Pad1) -> LED_R2
- R27 pad 1: Net-(R16-Pad1) -> LED_G2
- R28 pad 1: Net-(R17-Pad1) -> LED_B3
- R29 pad 1: Net-(R18-Pad1) -> LED_R3
- R3 pad 1: POWER_INPUT -> +12V
- R30 pad 1: Net-(R19-Pad1) -> LED_G3
- R31 pad 1: Net-(R20-Pad1) -> LED_B4
- R32 pad 1: Net-(R21-Pad1) -> LED_R4
- R33 pad 1: Net-(R22-Pad1) -> LED_G4
- U3 pad 1: FS3 -> LED_R3
- U3 pad 10: (no net) -> FS2
- U3 pad 11: FS4 -> LED_G3
- U3 pad 12: (no net) -> LED_B4
- U3 pad 13: (no net) -> LED_G1
- U3 pad 15: LEDS_SCL -> FS3
- U3 pad 16: LEDS_SDA -> FS4
- U3 pad 18: (no net) -> LED_G2
- U3 pad 2: (no net) -> LED_R1
- U3 pad 21: FS2 -> LED_B3
- U3 pad 23: LEDS_OE -> Net-(U3-Pad23)
- U3 pad 24: (no net) -> LED_R4
- U3 pad 25: (no net) -> Net-(U3-Pad25)
- U3 pad 26: (no net) -> LED_B2
- U3 pad 31: (no net) -> LED_G4
- U3 pad 38: (no net) -> LED_R2
- U3 pad 46: RX_LED_CPU -> Net-(U3-Pad46)
- U3 pad 47: TX_LED_CPU -> Net-(U3-Pad47)
- U3 pad 48: (no net) -> LED_B1
Routing:
- net +9V: track 104.9 -> 0.00 mm, vias 3 -> 0
- net GNDD: track 67.4 -> 0.00 mm, vias 9 -> 0
- net RJ45_RX-: track 61.6 -> 0.00 mm, vias 1 -> 0
- net RJ45_RX+: track 61.4 -> 0.00 mm
- net RJ45_TX+: track 48.9 -> 0.00 mm
- net RJ45_RX_LED: track 42.5 -> 0.00 mm
- net RJ45_TX_LED: track 38.5 -> 0.00 mm
- net RJ45_TX-: track 38.3 -> 0.00 mm
- net RJ45_POWER_INPUT: track 27.4 -> 0.00 mm
- net Net-(C18-Pad1): track 25.0 -> 0.00 mm
- net USB_PLUG_VCC: track 12.6 -> 0.00 mm
- net USB_DM: track 12.6 -> 0.00 mm
- net TX_LED: track 12.2 -> 0.00 mm, vias 1 -> 0
- net Net-(D2-Pad1): track 12.0 -> 0.00 mm, vias 1 -> 0
- net USB_DP: track 11.8 -> 0.00 mm
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- removed copper zone on B.Cu, net GNDD
- removed copper zone on F.Cu, net GNDD
Other:
- outline, holes or cut-outs redrawn
