File: hw-design/board/footswitch.kicad_pcb (KiCad board)
At the start: 2 copper layers, 249.4 x 60 mm, 101 parts, among them J1 CC_MAIN, J2 CC_NEXT, P1 FOOT, P2 FOOT, P3 CHAIN, P4 FOOT, P5 FOOT, P6 CONN_01X12, P7 USB_OTG, P8 CONN_01X12, P9 SWD, Q1 2N7002, Q2 2N7002, Q3 BC857, Q4 2N7002, Q5 FDN306P, Q6 IRFML8244TRPBF, Q7 2N7002, Q8 2N7002, SW1 SW_PUSH, U1 ISL83491, U2 NCP1117DT50G, U3 LPC11U24FBD48/401, U4 NCP1117DT33G, Y1 12MHz

Commit message: first placement
Parts:
- P6: footprint Pin_Headers:Pin_Header_Angled_1x12 -> Pin_Headers:Pin_Header_Straight_1x12
- moved C21 226.6 mm to (115.4, 86.7)
- moved R36 221.3 mm to (115.3, 83.1)
- moved U1 213.4 mm to (147.9, 96.3), turned to 270 degrees
- moved C6 210.4 mm to (135.9, 82.8)
- moved R15 204.7 mm to (154.3, 90.3), turned to 180 degrees
- moved SW1 204.3 mm to (124.1, 84.0), turned to 180 degrees
- moved C4 197.1 mm to (144.0, 82.8), turned to 180 degrees
- moved R17 196.1 mm to (125.6, 94.5)
- moved R21 195.6 mm to (125.2, 98.8)
- moved R18 192.4 mm to (121.5, 98.8)
- moved R20 191.9 mm to (125.4, 96.5)
- moved C14 189.5 mm to (121.2, 90.8)
- moved R13 189.5 mm to (128.5, 90.8)
- moved R7 189.5 mm to (125.0, 90.8)
- moved Q3 189.1 mm to (118.1, 102.1)
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Other:
- outline, holes or cut-outs redrawn
