File: hw-design/board/footswitch.kicad_pcb (KiCad board)
At the start: 2 copper layers, 249.4 x 58.5 mm, 101 parts, among them J1 CC_MAIN, J2 CC_NEXT, P1 FOOT, P10 CPU_RESET, P2 FOOT, P3 CHAIN, P4 FOOT, P5 FOOT, P6 CONN_01X12, P7 USB_OTG, P8 CONN_01X12, P9 SWD, Q1 2N7002, Q2 2N7002, Q3 BC857, Q4 2N7002, Q5 FDN306P, Q6 IRFML8244TRPBF, Q7 2N7002, Q8 2N7002, U1 ISL83491, U2 NCP1117DT50G, U3 LPC11U24FBD48/401, U4 NCP1117DT33G, Y1 12MHz

Commit message: footswitches signals connected
Parts:
- moved R1 12.1 mm to (69.5, 105.7), turned to 90 degrees
- moved R2 9.08 mm to (221.9, 105.7), turned to 90 degrees
- moved R11 2.13 mm to (230.8, 105.7), turned to 90 degrees
- moved R10 0.81 mm to (78.4, 105.7), turned to 90 degrees
- moved P1 0.29 mm to (66.8, 104.9)
- moved P4 0.29 mm to (75.8, 104.9)
- moved P2 0.28 mm to (219.2, 104.9)
- moved P5 0.28 mm to (228.2, 104.9)
- moved P8 0.28 mm to (157.3, 104.9)
Connections:
- U3 pad 1: FS3 -> Net-(U3-Pad1)
- U3 pad 21: LCD1_EN -> LCD1_BL
- U3 pad 23: LCD1_BL -> FS1
- U3 pad 24: Net-(U3-Pad24) -> FS2
- U3 pad 38: FS4 -> Net-(U3-Pad38)
- U3 pad 4: FS1 -> Net-(U3-Pad4)
- U3 pad 43: FS2 -> FS4
- U3 pad 45: Net-(U3-Pad45) -> FS3
- U3 pad 48: Net-(U3-Pad48) -> LCD1_EN
Routing:
- net FS4: track 0.00 -> 103.5 mm, vias 0 -> 1
- net FS3: track 0.00 -> 98.8 mm, vias 0 -> 1
- net FS1: track 0.00 -> 73.6 mm, vias 0 -> 2
- net FS2: track 0.00 -> 64.4 mm, vias 0 -> 2
- net USB_VCC: track 6.23 -> 28.2 mm, vias 0 -> 1
- net RS485_TX+: track 0.00 -> 7.73 mm
- net RS485_RX+: track 0.00 -> 7.61 mm
- net RS485_TX-: track 0.00 -> 7.20 mm
- net RS485_RX-: track 0.00 -> 7.09 mm
- net LCD1_EN: track 111.5 -> 118.2 mm
- net LCD2_EN: track 98.4 -> 99.1 mm
Other:
- outline, holes or cut-outs redrawn
