File: hw-design/board/footswitch.kicad_pcb (KiCad board)
At the start: 2 copper layers, 249.4 x 58.5 mm, 101 parts, among them J1 CC_MAIN, J2 CC_NEXT, P1 FOOT, P10 CPU_RESET, P2 FOOT, P3 CHAIN, P4 FOOT, P5 FOOT, P6 CONN_01X12, P7 USB_OTG, P8 CONN_01X12, P9 SWD, Q1 2N7002, Q2 2N7002, Q3 BC857, Q4 2N7002, Q5 FDN306P, Q6 IRFML8244TRPBF, Q7 2N7002, Q8 2N7002, U1 ISL83491, U2 NCP1117DT50G, U3 LPC11U24FBD48/401, U4 NCP1117DT33G, Y1 12MHz

Commit message: update layout according last RJ45 position
Parts:
- moved D2 3.62 mm to (160.9, 75.6)
- moved C9 2.63 mm to (161.2, 77.5)
- moved R16 2.45 mm to (163.6, 74.9)
- moved J1 2.18 mm to (138.3, 68.9)
- moved J2 2.18 mm to (167.4, 69.0)
- moved P6 1.00 mm to (157.3, 76.4)
- moved R14 0.45 mm to (168.9, 75.7)
- moved Q6 0.43 mm to (166.1, 75.7)
Routing:
- net USB_PLUG_VCC: track 31.7 -> 24.0 mm
- net GNDD: track 107.2 -> 111.5 mm, vias 10 -> 12
- net RJ45_RX+: track 47.1 -> 44.0 mm
- net CC_OUTPUT_DET: track 9.00 -> 6.01 mm
- net RJ45_RX-: track 40.2 -> 37.3 mm
- net RJ45_TX+: track 44.1 -> 41.9 mm
- net RJ45_TX-: track 39.6 -> 37.6 mm
- net Net-(P6-Pad11): track 25.5 -> 27.2 mm
- net Net-(D2-Pad1): track 5.23 -> 6.67 mm
- net VIN: track 51.4 -> 52.7 mm, vias 1 -> 3
- net Net-(P6-Pad10): track 26.4 -> 25.7 mm
Other:
- outline, holes or cut-outs redrawn

Commit message: lcd contrast comps connected
Parts:
- removed the Q1 at (193.5, 96.7)
- removed the R5 at (192.6, 99.8)
- removed the R8 at (194.4, 99.8)
- added C17: 1uF, Capacitors_SMD:C_0805, F.Cu at (197.7, 96.4)
- added Q3: 2N7002, Housings_SOT-23_SOT-143_TSOT-6:SOT-23, F.Cu at (123.6, 120.5)
- added R10: 10K, Resistors_SMD:R_0603, F.Cu at (148.7, 120.7)
- added R15: 2K, Resistors_SMD:R_0603, F.Cu at (47.4, 96.1)
- added R22: 2K, Resistors_SMD:R_0603, F.Cu at (199.8, 96.2)
- added R6: 10K, Resistors_SMD:R_0603, F.Cu at (142.4, 123.1)
- added R9: 2K4, Resistors_SMD:R_0603, F.Cu at (49.3, 96.1)
- C11: renamed from C14; value 10nF -> 100nF
- C13: renamed from C12; value 100nF X7R -> 100nF
- C14: renamed from C13; value 100nF X7R -> 100nF
- C21, C9: value 100nF X7R -> 100nF
- C3: value 47uF -> 1uF; footprint Capacitors_SMD:c_elec_6.3x5.3 -> Capacitors_SMD:C_0805
- P6: footprint Pin_Headers:Pin_Header_Straight_1x12 -> Pin_Headers:Pin_Header_Angled_1x12
- R1, R2: value 10k -> 10K
- R11: renamed from R10; value 10k -> 10K
- R12: renamed from R11; value 10k -> 10K
- R13: renamed from R12; value 10k -> 10K
- R14: renamed from R13; value 1k5 -> 1K5
- R17: renamed from R15; value 10k -> 10K
- R18: renamed from R16; value 10k -> 10K
- R20: value 2K -> 100R
- R21: value 3K3 -> 2K4
- R39: renamed from R36; value 10k -> 10K
- R5: renamed from R6; value 3k -> 3K
- R7: value 24k -> 24K
- R8: renamed from R9; value 10k -> 10K
- moved C3 155.2 mm to (45.3, 96.3), turned to 270 degrees
- moved R21 74.2 mm to (201.6, 96.2), turned to 270 degrees
- renumbered C11 to C12, C17 to C18, C18 to C19, C19 to C20, C20 to C22, Q2 to Q1, Q3 to Q2, R14 to R16, R22 to R23, R23 to R24, R24 to R25, R17 to R26, R18 to R27, R25 to R28, R26 to R29, R27 to R30, R28 to R31, R29 to R32, R30 to R33, R31 to R34, R32 to R35, R33 to R36, R34 to R37, R35 to R38
Connections:
- C3 pad 1: LCD_VO -> Net-(C3-Pad1)
- DS1 pad 3: LCD_VO -> Net-(C3-Pad1)
- DS2 pad 3: LCD_VO -> Net-(C17-Pad1)
- H1 pad 1: Net-(H1-Pad1) -> (no net)
- H2 pad 1: Net-(H2-Pad1) -> (no net)
- H3 pad 1: Net-(H3-Pad1) -> (no net)
- H4 pad 1: Net-(H4-Pad1) -> (no net)
- H5 pad 1: Net-(H5-Pad1) -> (no net)
- H6 pad 1: Net-(H6-Pad1) -> (no net)
- H7 pad 1: Net-(H7-Pad1) -> (no net)
- H7 pad 2: Net-(H7-Pad2) -> (no net)
- H7 pad 3: Net-(H7-Pad3) -> (no net)
- H7 pad 4: Net-(H7-Pad4) -> (no net)
- H8 pad 1: Net-(H8-Pad1) -> (no net)
- H8 pad 2: Net-(H8-Pad2) -> (no net)
- H8 pad 3: Net-(H8-Pad3) -> (no net)
- H8 pad 4: Net-(H8-Pad4) -> (no net)
- P7 pad 4: Net-(P7-Pad4) -> (no net)
- P9 pad 1: Net-(P9-Pad1) -> (no net)
- P9 pad 7: Net-(P9-Pad7) -> (no net)
- P9 pad 8: Net-(P9-Pad8) -> (no net)
- R21 pad 1: GNDD -> Net-(C17-Pad1)
- R21 pad 2: USB_VBUS -> +3V3
- U3 pad 1: Net-(U3-Pad1) -> (no net)
- U3 pad 2: Net-(U3-Pad2) -> (no net)
- U3 pad 38: Net-(U3-Pad38) -> (no net)
- U3 pad 4: Net-(U3-Pad4) -> ISP_TRIGGER
- U3 pad 42: LCD_CONTRAST -> (no net)
Routing:
- net LCD_VO: track 228.2 -> 0.00 mm, vias 2 -> 0
- net LCD_CONTRAST: track 56.9 -> 0.00 mm, vias 2 -> 0
- net Net-(C17-Pad1): track 0.00 -> 39.9 mm
- net Net-(C3-Pad1): track 0.00 -> 39.8 mm
- net +3V3: track 632.9 -> 651.1 mm, vias 29 -> 31
- net Net-(Q1-Pad2): track 3.14 -> 0.00 mm
- net GNDD: track 111.5 -> 109.9 mm

Commit message: update layout adding last sch changes
Parts:
- R6: value 10K -> 100K
- moved R10 36.7 mm to (123.4, 94.0), turned to 270 degrees
- moved R6 33.8 mm to (125.2, 94.0), turned to 270 degrees
- moved Q3 27.0 mm to (127.9, 93.8)
- moved R14 5.99 mm to (122.9, 97.2), turned to 270 degrees
- moved R20 0.92 mm to (128.1, 90.6), turned to 90 degrees
- moved C11 0.82 mm to (126.2, 90.6)
Routing:
- net ISP_TRIGGER: track 0.00 -> 19.2 mm, vias 0 -> 3
- net USB_DP_CPU: track 13.3 -> 21.9 mm, vias 0 -> 2
- net FS1: track 75.7 -> 81.2 mm, vias 2 -> 3
- net Net-(Q2-Pad3): track 5.32 -> 1.92 mm, vias 2 -> 0
- net +3V3: track 651.1 -> 654.3 mm
- net USB_VBUS: track 6.85 -> 3.97 mm, vias 2 -> 0
- net USB_VCC: track 65.0 -> 67.0 mm
- net LED_G3: track 48.2 -> 49.2 mm
- net LCD1_EN: track 118.2 -> 117.5 mm
- net GNDD: track 109.9 -> 110.4 mm, vias 12 -> 10
Other:
- board text added: "MOD - Footswitch Extension Rev.: 2016.07.18"

Commit message: pcb: update layout
Parts:
- removed C18, C22: 100nF, Capacitors_SMD:C_0603
- removed C20: 100uF, Capacitors_SMD:c_elec_6.3x5.3
- removed D4: 1N5819, Diodes_SMD:SOD-123
- removed U4: NCP1117DT33G, SMD_Packages:DPAK-2
- added R40: 10K, Resistors_SMD:R_0603, F.Cu at (149.6, 90.2)
- P10: footprint Pin_Headers:Pin_Header_Straight_1x02 -> Resistors_SMD:R_0402
- P6: footprint Pin_Headers:Pin_Header_Angled_1x12 -> Pin_Headers:Pin_Header_Straight_1x12
- U2: value NCP1117DT50G -> NCP1117DT33G
- moved P3 22.5 mm to (167.2, 96.3)
- moved C12 21.1 mm to (210.2, 107.2), turned to 270 degrees
- moved C5 19.0 mm to (181.7, 110.3), turned to 270 degrees
- moved R3 18.5 mm to (171.2, 106.8), turned to 270 degrees
- moved R4 17.7 mm to (171.2, 109.6), turned to 270 degrees
- moved U2 16.1 mm to (187.4, 109.2)
- moved D3 15.8 mm to (167.2, 113.5)
- moved C10 14.4 mm to (205.6, 109.2), turned to 90 degrees
- moved D1 13.3 mm to (174.5, 106.9)
- moved Q4 12.4 mm to (168.4, 110.6), turned to 90 degrees
- moved C7 12.1 mm to (177.4, 109.0), turned to 90 degrees
- moved Q1 11.9 mm to (168.5, 107.0)
- moved RT1 10.5 mm to (176.0, 112.5), turned to 0 degrees
- moved R13 10.5 mm to (160.0, 108.2), turned to 270 degrees
- moved C8 10.4 mm to (165.5, 108.7), turned to 90 degrees
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Connections:
- C10 pad 1: Net-(C10-Pad1) -> +3V3
- C12 pad 1: Net-(C10-Pad1) -> +3V3
- D1 pad 1: Net-(D1-Pad1) -> +5V
- H1 pad 1: (no net) -> Net-(H1-Pad1)
- H2 pad 1: (no net) -> Net-(H2-Pad1)
- H3 pad 1: (no net) -> Net-(H3-Pad1)
- H4 pad 1: (no net) -> Net-(H4-Pad1)
- H5 pad 1: (no net) -> Net-(H5-Pad1)
- H6 pad 1: (no net) -> Net-(H6-Pad1)
- H7 pad 1: (no net) -> Net-(H7-Pad1)
- H7 pad 2: (no net) -> Net-(H7-Pad2)
- H7 pad 3: (no net) -> Net-(H7-Pad3)
- H7 pad 4: (no net) -> Net-(H7-Pad4)
- H8 pad 1: (no net) -> Net-(H8-Pad1)
- H8 pad 2: (no net) -> Net-(H8-Pad2)
- H8 pad 3: (no net) -> Net-(H8-Pad3)
- H8 pad 4: (no net) -> Net-(H8-Pad4)
- P7 pad 4: (no net) -> Net-(P7-Pad4)
- P9 pad 1: (no net) -> Net-(P9-Pad1)
- P9 pad 7: (no net) -> Net-(P9-Pad7)
- P9 pad 8: (no net) -> Net-(P9-Pad8)
- Q7 pad 2: Net-(DS1-Pad16) -> GNDD
- Q7 pad 3: GNDD -> Net-(DS1-Pad16)
- Q8 pad 2: Net-(DS2-Pad16) -> GNDD
- Q8 pad 3: GNDD -> Net-(DS2-Pad16)
- RT1 pad 1: Net-(D1-Pad1) -> +5V
- U1 pad 3: GNDD -> CHAIN_RE
- U2 pad 2: Net-(C10-Pad1) -> +3V3
- U3 pad 1: (no net) -> Net-(U3-Pad1)
- U3 pad 2: (no net) -> Net-(U3-Pad2)
- U3 pad 38: (no net) -> CHAIN_RE
- U3 pad 42: (no net) -> Net-(U3-Pad42)
Routing:
- net +3V3: track 654.3 -> 680.2 mm, vias 31 -> 11
- net Net-(C10-Pad1): track 24.3 -> 0.00 mm
- net CHAIN_TX: track 21.7 -> 38.3 mm
- net CHAIN_RX: track 22.8 -> 38.5 mm, vias 2 -> 0
- net CHAIN_RE: track 0.00 -> 14.0 mm
- net RESET: track 54.1 -> 40.8 mm, vias 5 -> 1
- net Net-(Q1-Pad1): track 16.7 -> 4.23 mm, vias 2 -> 0
- net USB_VCC: track 67.0 -> 57.2 mm, vias 3 -> 1
- net Net-(C8-Pad1): track 12.2 -> 6.70 mm, vias 2 -> 0
- net GNDD: track 110.4 -> 105.1 mm, vias 10 -> 8
- net +12V: track 16.0 -> 20.9 mm, vias 1 -> 0
- net Net-(C8-Pad2): track 14.1 -> 9.92 mm, vias 4 -> 0
- net Net-(D1-Pad1): track 3.80 -> 0.00 mm
- net LCD2_BL: track 95.7 -> 99.3 mm
- net SWDIO: track 40.7 -> 37.4 mm
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- removed copper zone on F.Cu, net Net-(C10-Pad1)
Other:
- board text added: "MOD - Footswitch Extension Rev.: 2017.07.14"
- board text removed: "MOD - Footswitch Extension Rev.: 2016.07.18"

Commit message: sch,pcb: add open hardware symbol
Parts:
- added LOGO1: Logo_Open_Hardware_Small, Symbols:OSHW-Logo2_9.8x8mm_SilkScreen, F.Cu at (247.9, 107.2)
- P1, P2, P4, P5: moved to B.Cu
- moved R2 7.96 mm to (213.9, 105.7)
- moved R11 7.96 mm to (70.5, 105.7)
- moved R1 7.95 mm to (61.5, 105.7)
- moved R12 7.94 mm to (222.9, 105.7)
- moved P4 2.54 mm to (73.2, 104.9)
- moved P1 2.54 mm to (64.3, 104.9)
- moved P2 2.54 mm to (216.7, 104.9)
- moved P5 2.54 mm to (225.6, 104.9)
Routing:
- net LCD_D5: track 215.4 -> 209.3 mm
- net FS1: track 81.2 -> 83.9 mm
- net +3V3: track 680.2 -> 677.6 mm
- net FS2: track 66.3 -> 68.9 mm
- net FS4: track 106.6 -> 104.1 mm
- net FS3: track 99.1 -> 96.7 mm
- net LED_B4: track 125.2 -> 122.9 mm
- net LCD_RW: track 212.9 -> 210.7 mm
Other:
- board text added: "Footswitch Extension Rev.: 2017.07.14"
- board text removed: "MOD - Footswitch Extension Rev.: 2017.07.14"

Commit message: Changed R40 RE from pull-up to pull-down
Parts:
- R15, R22: value 2K -> 1.2K
Connections:
- R40 pad 2: +3V3 -> GNDD
Routing:
- net +3V3: track 677.6 -> 676.3 mm, vias 11 -> 10
Changed lines of the file:
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@@
-(kicad_pcb (version 20170123) (host pcbnew "(2017-04-07 revision 7b4ea2a38)-master")
+(kicad_pcb (version 20171130) (host pcbnew 5.0.2-bee76a0~70~ubuntu18.04.1)
   (general
-    (links 249)
-    (no_connects 4)
-    (area 11.31416 48.06698 273.174461 115.739701)
     (thickness 1.6)
     (drawings 124)
-    (tracks 895)
+    (tracks 893)
     (zones 0)
     (modules 102)
@@
   )
   (setup
-    (last_trace_width 0.254)
+    (last_trace_width 0.3048)
     (user_trace_width 0.2032)
     (user_trace_width 0.254)
@@
     (pad_drill 0.89916)
     (pad_to_mask_clearance 0.1)
+    (solder_mask_min_width 0.25)
     (pad_to_paste_clearance -0.003)
     (aux_axis_origin 28.20416 64.01308)
@@
       (layerselection 0x3d0f0_ffffffff)
       (usegerberextensions false)
+      (usegerberattributes false)
+      (usegerberadvancedattributes false)
+      (creategerberjobfile false)
       (excludeedgelayer true)
       (linewidth 0.100000)
@@
       (hpglpennumber 1)
       (hpglpenspeed 20)
-      (hpglpendiameter 15)
+      (hpglpendiameter 15.000000)
       (psnegative false)
       (psa4output false)
@@
       (drillshape 0)
       (scaleselection 1)
-      (outputdirectory gerber))
+      (outputdirectory "gerber"))
   )
   (net 0 "")
@@
       (net 38 FS3))
     (model Pin_Headers.3dshapes/Pin_Header_Angled_1x02.wrl
-      (at (xyz 0 -0.05 0))
+      (offset (xyz 0 -1.269999980926514 0))
       (scale (xyz 1 1 1))
       (rotate (xyz 0 0 90))
@@
       (net 40 FS4))
     (model Pin_Headers.3dshapes/Pin_Header_Angled_1x02.wrl
-      (at (xyz 0 -0.05 0))
+      (offset (xyz 0 -1.269999980926514 0))
       (scale (xyz 1 1 1))
       (rotate (xyz 0 0 90))
@@
       (net 39 FS2))
     (model Pin_Headers.3dshapes/Pin_Header_Angled_1x02.wrl
-      (at (xyz 0 -0.05 0))
+      (offset (xyz 0 -1.269999980926514 0))
       (scale (xyz 1 1 1))
       (rotate (xyz 0 0 90))
@@
       (net 37 FS1))
     (model Pin_Headers.3dshapes/Pin_Header_Angled_1x02.wrl
-      (at (xyz 0 -0.05 0))
+      (offset (xyz 0 -1.269999980926514 0))
       (scale (xyz 1 1 1))
       (rotate (xyz 0 0 90))
@@
       (net 1 GNDD))
     (model Pin_Headers.3dshapes/Pin_Header_Angled_1x12.wrl
-      (at (xyz 0 -0.55 0))
+      (offset (xyz 0 -13.96999979019165 0))
       (scale (xyz 1 1 1))
       (rotate (xyz 0 0 90))
@@
       (effects (font (size 0.7 0.7) (thickness 0.1)))
     )
-    (fp_text value 2K (at 0 0 270) (layer F.Fab)
+    (fp_text value 1.2K (at 0 0 270) (layer F.Fab)
       (effects (font (size 0.7 0.7) (thickness 0.1)))
     )
@@
       (effects (font (size 0.7 0.7) (thickness 0.1)))
     )
-    (fp_text value 2K (at 0 0 270) (layer F.Fab)
+    (fp_text value 1.2K (at 0 0 270) (layer F.Fab)
       (effects (font (size 0.7 0.7) (thickness 0.1)))
     )
@@
       (net 1 GNDD))
     (model Pin_Headers.3dshapes/Pin_Header_Straight_1x12.wrl
-      (at (xyz 0 -0.55 0))
+      (offset (xyz 0 -13.96999979019165 0))
       (scale (xyz 1 1 1))
       (rotate (xyz 0 0 90))
@@
       (net 105 CHAIN_RE))
     (pad 2 smd rect (at 0.75 0 90) (size 0.5 0.9) (layers F.Cu F.Paste F.Mask)
-      (net 4 +3V3))
+      (net 1 GNDD))
     (model Resistors_SMD.3dshapes/R_0603.wrl
       (at (xyz 0 0 0))
@@
   (segment (start 210.21 106.47) (end 233.31 106.47) (width 0.381) (layer F.Cu) (net 4) (status 10))
   (segment (start 146.67 88.1888) (end 149.5688 88.1888) (width 0.254) (layer B.Cu) (net 4))
-  (segment (start 149.57 88.19) (end 149.57 89.41) (width 0.254) (layer F.Cu) (net 4) (status 20))
-  (via (at 149.57 88.19) (size 0.6) (drill 0.3) (layers F.Cu B.Cu) (net 4))
   (segment (start 149.5688 88.1888) (end 149.57 88.19) (width 0.254) (layer B.Cu) (net 4))
   (segment (start 123.4313 94.7808) (end 120.5292 94.7808) (width 0.381) (layer F.Cu) (net 4) (status 10))

Commit message: updated silk screen
Parts:
- added G***: LOGO, local-footprints:mod-logo, B.Cu at (70.5, 77.2)
Other:
- board text added: "MOD Devices GmbH http:/moddevices.com [FS-ELE-001] Footswitch Extension Rev.: 2019.04.15"
- board text added: "[FS-ELE-002]"
- board text removed: "Footswitch Extension Rev.: 2017.07.14"
