File: hw-design/board/rear-board.sch (KiCad schematic (older format))
At the start: 12 parts, among them J1 CC_MAIN, J2 CC_NEXT, P7 CONN_01X16, P8 USB_OTG, P9 CONN_01X16, Q9 IRFML8244TRPBF

Commit message: update 'boards connector' signals
Parts:
- P7: value CONN_01X16 -> CONN_01X12; footprint Pin_Headers:Pin_Header_Straight_1x16 -> Pin_Headers:Pin_Header_Straight_1x12; symbol CONN_01X16 -> CONN_01X12
- P9: value CONN_01X16 -> CONN_01X12; footprint Pin_Headers:Pin_Header_Angled_1x16 -> Pin_Headers:Pin_Header_Angled_1x12; symbol CONN_01X16 -> CONN_01X12
Connections:
- net RX_LED is gone; now on net GNDD: P7.12 (P12)
- net RX_LED_CPU is gone; now on net GNDD: P9.12 (P12)
- net TX_LED is gone; now on net USB_DP: P7.11 (P11)
- net TX_LED_CPU is gone; now on net USB_DP_CPU: P9.11 (P11)
- net +12V: now also P7.1 (P1), P7.2 (P2), P9.1 (P1), P9.2 (P2)
- net GNDD: now also P7.5 (P5), P7.8 (P8), P9.5 (P5), P9.8 (P8); no longer P7.10 (P10), P7.13 (P13), P7.3 (P3), P7.6 (P6), P9.10 (P10), P9.13 (P13), P9.3 (P3), P9.6 (P6)
- net RJ45_RX+: now also P7.3 (P3); no longer P7.1 (P1)
- net RJ45_RX-: now also P7.4 (P4); no longer P7.2 (P2)
- net RJ45_TX+: now also P7.7 (P7); no longer P7.5 (P5)
- net RJ45_TX-: now also P7.6 (P6); no longer P7.4 (P4)
- net RS485_RX+: now also P9.3 (P3); no longer P9.1 (P1)
- net RS485_RX-: now also P9.4 (P4); no longer P9.2 (P2)
- net RS485_TX+: now also P9.7 (P7); no longer P9.5 (P5)
- net RS485_TX-: now also P9.6 (P6); no longer P9.4 (P4)
- net USB_DM: now also P7.10 (P10); no longer P7.8 (P8)
- net USB_DM_CPU: now also P9.10 (P10); no longer P9.8 (P8)
- net USB_DP: no longer P7.9 (P9)
- net USB_DP_CPU: no longer P9.9 (P9)
- net USB_PLUG_VCC: now also P7.9 (P9); no longer P7.7 (P7)
- net USB_VCC: now also P9.9 (P9); no longer P9.7 (P7)
- removed net POWER_INPUT: P9.14 (P14), P9.15 (P15), P9.16 (P16)
- removed net RJ45_POWER_INPUT: P7.14 (P14), P7.15 (P15), P7.16 (P16)
Changed lines of the file:
@@
 Text GLabel 4500 3500 2    50   Output ~ 0
 CC_OUTPUT_DET
-Text GLabel 8150 1350 0    50   Input ~ 0
+Text GLabel 8150 1650 0    50   Input ~ 0
 RJ45_RX+
-Text GLabel 8150 1450 0    50   Input ~ 0
+Text GLabel 8150 1750 0    50   Input ~ 0
 RJ45_RX-
-Text GLabel 8150 1750 0    50   Output ~ 0
+Text GLabel 8150 2050 0    50   Output ~ 0
 RJ45_TX+
-Text GLabel 8150 1650 0    50   Output ~ 0
+Text GLabel 8150 1950 0    50   Output ~ 0
 RJ45_TX-
-Text GLabel 8150 2650 0    50   Input ~ 0
-RJ45_POWER_INPUT
-Text GLabel 8150 2750 0    50   Input ~ 0
-RJ45_POWER_INPUT
-Text GLabel 8150 1950 0    50   Input ~ 0
+Text GLabel 8150 2250 0    50   Input ~ 0
 USB_PLUG_VCC
 $Comp
@@
 Text Notes 8100 900  0    100  ~ 0
 BOARDS CONNECTORS
-Text GLabel 8150 2450 0    50   Output ~ 0
-RX_LED
-Text GLabel 8150 2350 0    50   Output ~ 0
-TX_LED
-Text GLabel 9650 1350 2    50   Output ~ 0
+Text GLabel 9650 1650 2    50   Output ~ 0
 RS485_RX+
-Text GLabel 9650 1450 2    50   Output ~ 0
+Text GLabel 9650 1750 2    50   Output ~ 0
 RS485_RX-
-Text GLabel 9650 1750 2    50   Input ~ 0
+Text GLabel 9650 2050 2    50   Input ~ 0
 RS485_TX+
-Text GLabel 9650 1650 2    50   Input ~ 0
+Text GLabel 9650 1950 2    50   Input ~ 0
 RS485_TX-
-Text GLabel 9650 2450 2    50   Input ~ 0
-RX_LED_CPU
-Text GLabel 9650 2350 2    50   Input ~ 0
-TX_LED_CPU
-Text GLabel 9650 2650 2    50   Output ~ 0
-POWER_INPUT
-Text GLabel 9650 2750 2    50   Output ~ 0
-POWER_INPUT
 NoConn ~ 8850 5350
 $Comp
-L CONN_01X16 P7
+L CONN_01X12 P7
 U 1 1 55B42C87
-P 8550 2100
-F 0 "P7" H 8550 2950 50  0000 C CNN
-F 1 "CONN_01X16" V 8650 2100 50  0000 C CNN
-F 2 "Pin_Headers:Pin_Header_Straight_1x16" H 8550 2100 60  0001 C CNN
-F 3 "" H 8550 2100 60  0000 C CNN
-	1    8550 2100
-	1    0    0    -1
-$EndComp
-$Comp
-L CONN_01X16 P9
+P 8550 2000
+F 0 "P7" H 8550 2650 50  0000 C CNN
+F 1 "CONN_01X12" V 8650 2000 50  0000 C CNN
+F 2 "Pin_Headers:Pin_Header_Straight_1x12" H 8550 2000 60  0001 C CNN
+F 3 "" H 8550 2000 60  0000 C CNN
+	1    8550 2000
+	1    0    0    -1
+$EndComp
+$Comp
+L CONN_01X12 P9
 U 1 1 55B42DAB
-P 9250 2100
-F 0 "P9" H 9250 2950 50  0000 C CNN
-F 1 "CONN_01X16" V 9350 2100 50  0000 C CNN
-F 2 "Pin_Headers:Pin_Header_Angled_1x16" H 9250 2100 60  0001 C CNN
-F 3 "" H 9250 2100 60  0000 C CNN
-	1    9250 2100
+P 9250 2000
+F 0 "P9" H 9250 2650 50  0000 C CNN
+F 1 "CONN_01X12" V 9350 2000 50  0000 C CNN
+F 2 "Pin_Headers:Pin_Header_Angled_1x12" H 9250 2000 60  0001 C CNN
+F 3 "" H 9250 2000 60  0000 C CNN
+	1    9250 2000
 	-1   0    0    -1
 $EndComp
-Text GLabel 8150 2050 0    50   BiDi ~ 0
+Text GLabel 8150 2350 0    50   BiDi ~ 0
 USB_DM
-Text GLabel 8150 2150 0    50   BiDi ~ 0
+Text GLabel 8150 2450 0    50   BiDi ~ 0
 USB_DP
-Text GLabel 9650 2050 2    50   BiDi ~ 0
+Text GLabel 9650 2350 2    50   BiDi ~ 0
 USB_DM_CPU
-Text GLabel 9650 2150 2    50   BiDi ~ 0
+Text GLabel 9650 2450 2    50   BiDi ~ 0
 USB_DP_CPU
-Text GLabel 9650 1950 2    50   Output ~ 0
+Text GLabel 9650 2250 2    50   Output ~ 0
 USB_VCC
 $Comp
 L GNDD #PWR097
 U 1 1 55B45519
-P 8250 2950
-F 0 "#PWR097" H 8250 2700 50  0001 C CNN
-F 1 "GNDD" H 8250 2800 50  0000 C CNN
-F 2 "" H 8250 2950 60  0000 C CNN
-F 3 "" H 8250 2950 60  0000 C CNN
-	1    8250 2950
+P 8250 2700
+F 0 "#PWR097" H 8250 2450 50  0001 C CNN
+F 1 "GNDD" H 8250 2550 50  0000 C CNN
+F 2 "" H 8250 2700 60  0000 C CNN
+F 3 "" H 8250 2700 60  0000 C CNN
+	1    8250 2700
 	1    0    0    -1
 $EndComp
@@
 L GNDD #PWR098
 U 1 1 55B4640F
-P 9550 2950
-F 0 "#PWR098" H 9550 2700 50  0001 C CNN
-F 1 "GNDD" H 9550 2800 50  0000 C CNN
-F 2 "" H 9550 2950 60  0000 C CNN
-F 3 "" H 9550 2950 60  0000 C CNN
-	1    9550 2950
+P 9550 2700
+F 0 "#PWR098" H 9550 2450 50  0001 C CNN
+F 1 "GNDD" H 9550 2550 50  0000 C CNN
+F 2 "" H 9550 2700 60  0000 C CNN
+F 3 "" H 9550 2700 60  0000 C CNN
+	1    9550 2700
 	1    0    0    -1
 $EndComp
@@
 	-1   0    0    -1
 $EndComp
-Text GLabel 8150 2850 0    50   Input ~ 0
-RJ45_POWER_INPUT
-Text GLabel 9650 2850 2    50   Output ~ 0
-POWER_INPUT
 $Comp
 L +12V #PWR?
@@
 Connection ~ 4150 3500
 Wire Wire Line
-	8150 1350 8350 1350
-Wire Wire Line
-	8350 1450 8150 1450
-Wire Wire Line
-	8150 1750 8350 1750
-Wire Wire Line
-	8350 1650 8150 1650
+	8150 1650 8350 1650
+Wire Wire Line
+	8350 1750 8150 1750
+Wire Wire Line
+	8150 2050 8350 2050
+Wire Wire Line
+	8350 1950 8150 1950
+Wire Wire Line
+	8150 2250 8350 2250
+Wire Wire Line
+	8150 2350 8350 2350
 Wire Wire Line
 	8350 2450 8150 2450
-Wire Wire Line
-	8150 2350 8350 2350
-Wire Wire Line
-	8350 2650 8150 2650
-Wire Wire Line
-	8350 2750 8150 2750
-Wire Wire Line
-	8150 1950 8350 1950
-Wire Wire Line
-	8150 2050 8350 2050
-Wire Wire Line
-	8350 2150 8150 2150
 Wire Wire Line
 	8450 5050 8450 4950
@@
 	7200 3900 10400 3900
 Wire Wire Line
-	9450 1350 9650 1350
-Wire Wire Line
-	9650 1450 9450 1450
-Wire Wire Line
-	9450 1750 9650 1750
-Wire Wire Line
-	9650 1650 9450 1650
-Wire Wire Line
-	9650 2450 9450 2450
-Wire Wire Line
-	9450 2350 9650 2350
-Wire Wire Line
-	9650 2650 9450 2650
-Wire Wire Line
-	9450 2750 9650 2750
-Wire Wire Line
-	9650 2050 9450 2050
-Wire Wire Line
-	9450 2150 9650 2150
+	9450 1650 9650 1650
+Wire Wire Line
+	9650 1750 9450 1750
+Wire Wire Line
+	9450 2050 9650 2050
 Wire Wire Line
 	9650 1950 9450 1950
 Wire Wire Line
-	8350 1550 8250 1550
-Wire Wire Line
-	8250 1550 8250 2950
-Wire Wire Line
-	8350 1850 8250 1850
-Connection ~ 8250 1850
-Wire Wire Line
-	9450 1550 9550 1550
-Wire Wire Line
-	9550 1550 9550 2950
-Wire Wire Line
-	9450 1850 9550 1850
-Connection ~ 9550 1850
-Wire Wire Line
-	8350 2250 8250 2250
-Connection ~ 8250 2250
-Wire Wire Line
-	8350 2550 8250 2550
-Connection ~ 8250 2550
-Wire Wire Line
-	9450 2250 9550 2250
-Connection ~ 9550 2250
-Wire Wire Line
-	9450 2550 9550 2550
-Connection ~ 9550 2550
-Wire Wire Line
-	8350 2850 8150 2850
-Wire Wire Line
-	9450 2850 9650 2850
+	9650 2350 9450 2350
+Wire Wire Line
+	9450 2450 9650 2450
+Wire Wire Line
+	9650 2250 9450 2250
 $Comp
 L RJ45 J1
@@
 Wire Wire Line
 	2900 3500 3600 3500
+$Comp
+L +12V #PWR?
+U 1 1 5760ABA5
+P 8250 1300
+F 0 "#PWR?" H 8250 1150 50  0001 C CNN
+F 1 "+12V" H 8268 1474 50  0000 C CNN
+F 2 "" H 8250 1300 60  0000 C CNN
+F 3 "" H 8250 1300 60  0000 C CNN
+	1    8250 1300
+	1    0    0    -1
+$EndComp
+Wire Wire Line
+	8250 1300 8250 1550
+$Comp
+L +12V #PWR?
+U 1 1 5760AF55
+P 9550 1300
+F 0 "#PWR?" H 9550 1150 50  0001 C CNN
+F 1 "+12V" H 9568 1474 50  0000 C CNN
+F 2 "" H 9550 1300 60  0000 C CNN
+F 3 "" H 9550 1300 60  0000 C CNN
+	1    9550 1300
+	1    0    0    -1
+$EndComp
+Wire Wire Line
+	9550 1300 9550 1550
+Connection ~ 8250 1450
+Connection ~ 9550 1450
+Wire Wire Line
+	8250 2700 8250 1850
+Wire Wire Line
+	8250 1850 8350 1850
+Wire Wire Line
+	8350 2150 8250 2150
+Connection ~ 8250 2150
+Wire Wire Line
+	8350 2550 8250 2550
+Connection ~ 8250 2550
+Wire Wire Line
+	8350 1450 8250 1450
+Wire Wire Line
+	8250 1550 8350 1550
+Wire Wire Line
+	9550 1550 9450 1550
+Wire Wire Line
+	9450 1450 9550 1450
+Wire Wire Line
+	9450 1850 9550 1850
+Wire Wire Line
+	9550 1850 9550 2700
+Wire Wire Line
+	9450 2550 9550 2550
+Connection ~ 9550 2550
+Wire Wire Line
+	9450 2150 9550 2150
+Connection ~ 9550 2150
 $EndSCHEMATC

Commit message: annotation and ERC
Parts:
- renumbered C24 to C18, C23 to C9, D8 to D2, P7 to P6, P8 to P7, P9 to P8, Q9 to Q6, R34 to R14, R33 to R16, R35 to R34
Changed lines of the file:
@@
 $EndDescr
 $Comp
-L GNDD #PWR082
+L GNDD #PWR25
 U 1 1 55B26400
 P 3000 2300
-F 0 "#PWR082" H 3000 2050 60  0001 C CNN
+F 0 "#PWR25" H 3000 2050 60  0001 C CNN
 F 1 "GNDD" H 3000 2150 60  0000 C CNN
 F 2 "" H 3000 2300 60  0000 C CNN
@@
 $EndComp
 $Comp
-L C C23
+L C C9
 U 1 1 55B2640D
 P 4150 3800
-F 0 "C23" V 4000 3800 40  0000 L CNN
+F 0 "C9" V 4000 3800 40  0000 L CNN
 F 1 "100nF X7R" V 4300 3650 40  0000 L CNN
 F 2 "Capacitors_SMD:C_0603" H 4188 3650 30  0001 C CNN
@@
 $EndComp
 $Comp
-L R R33
+L R R16
 U 1 1 55B26415
 P 4150 3200
-F 0 "R33" V 4250 3200 40  0000 C CNN
+F 0 "R16" V 4250 3200 40  0000 C CNN
 F 1 "10k" V 4157 3201 40  0000 C CNN
 F 2 "Resistors_SMD:R_0603" V 4080 3200 30  0001 C CNN
@@
 $EndComp
 $Comp
-L GNDD #PWR084
+L GNDD #PWR39
 U 1 1 55B2641C
 P 4150 4050
-F 0 "#PWR084" H 4150 3800 60  0001 C CNN
+F 0 "#PWR39" H 4150 3800 60  0001 C CNN
 F 1 "GNDD" H 4150 3900 60  0000 C CNN
 F 2 "" H 4150 4050 60  0000 C CNN
@@
 $EndComp
 $Comp
-L D D8
+L D D2
 U 1 1 55B26435
 P 3750 3500
-F 0 "D8" H 3750 3600 50  0000 C CNN
+F 0 "D2" H 3750 3600 50  0000 C CNN
 F 1 "1N4148" H 3750 3400 50  0000 C CNN
 F 2 "Diodes_SMD:SOD-323" H 3750 3500 60  0001 C CNN
@@
 USB_PLUG_VCC
 $Comp
-L R R35
+L R R34
 U 1 1 55B2B900
 P 8450 5200
-F 0 "R35" V 8350 5350 50  0000 C CNN
+F 0 "R34" V 8350 5350 50  0000 C CNN
 F 1 "1M" V 8450 5200 50  0000 C CNN
 F 2 "Resistors_SMD:R_0603" V 8380 5200 30  0001 C CNN
@@
 $EndComp
 $Comp
-L GNDD #PWR092
+L GNDD #PWR65
 U 1 1 55B2B90F
 P 8450 5550
-F 0 "#PWR092" H 8450 5300 50  0001 C CNN
+F 0 "#PWR65" H 8450 5300 50  0001 C CNN
 F 1 "GNDD" H 8450 5400 50  0000 C CNN
 F 2 "" H 8450 5550 60  0000 C CNN
@@
 $EndComp
 $Comp
-L C C24
+L C C18
 U 1 1 55B2B908
 P 8250 5200
-F 0 "C24" V 8300 5000 50  0000 L CNN
+F 0 "C18" V 8300 5000 50  0000 L CNN
 F 1 "10nF 500V" V 8100 5000 50  0000 L CNN
 F 2 "Capacitors_SMD:C_1206" H 8288 5050 30  0001 C CNN
@@
 USB_DP
 $Comp
-L Q_NMOS_GSD Q9
+L Q_NMOS_GSD Q6
 U 1 1 55B320E7
 P 3500 5900
-F 0 "Q9" H 3400 6000 50  0000 R CNN
+F 0 "Q6" H 3400 6000 50  0000 R CNN
 F 1 "IRFML8244TRPBF" V 3750 6150 50  0000 R CNN
 F 2 "Housings_SOT-23_SOT-143_TSOT-6:SOT-23" H 3700 6000 29  0001 C CNN
@@
 $EndComp
 $Comp
-L R R34
+L R R14
 U 1 1 55B320EF
 P 3600 6350
-F 0 "R34" V 3680 6350 50  0000 C CNN
+F 0 "R14" V 3680 6350 50  0000 C CNN
 F 1 "100R" V 3600 6350 50  0000 C CNN
 F 2 "Resistors_SMD:R_0805" V 3530 6350 30  0001 C CNN
@@
 NoConn ~ 8850 5350
 $Comp
-L CONN_01X12 P7
+L CONN_01X12 P6
 U 1 1 55B42C87
 P 8550 2000
-F 0 "P7" H 8550 2650 50  0000 C CNN
+F 0 "P6" H 8550 2650 50  0000 C CNN
 F 1 "CONN_01X12" V 8650 2000 50  0000 C CNN
 F 2 "Pin_Headers:Pin_Header_Straight_1x12" H 8550 2000 60  0001 C CNN
@@
 $EndComp
 $Comp
-L CONN_01X12 P9
+L CONN_01X12 P8
 U 1 1 55B42DAB
 P 9250 2000
-F 0 "P9" H 9250 2650 50  0000 C CNN
+F 0 "P8" H 9250 2650 50  0000 C CNN
 F 1 "CONN_01X12" V 9350 2000 50  0000 C CNN
 F 2 "Pin_Headers:Pin_Header_Angled_1x12" H 9250 2000 60  0001 C CNN
@@
 USB_VCC
 $Comp
-L GNDD #PWR097
+L GNDD #PWR63
 U 1 1 55B45519
 P 8250 2700
-F 0 "#PWR097" H 8250 2450 50  0001 C CNN
+F 0 "#PWR63" H 8250 2450 50  0001 C CNN
 F 1 "GNDD" H 8250 2550 50  0000 C CNN
 F 2 "" H 8250 2700 60  0000 C CNN
@@
 $EndComp
 $Comp
-L GNDD #PWR098
+L GNDD #PWR79
 U 1 1 55B4640F
 P 9550 2700
-F 0 "#PWR098" H 9550 2450 50  0001 C CNN
+F 0 "#PWR79" H 9550 2450 50  0001 C CNN
 F 1 "GNDD" H 9550 2550 50  0000 C CNN
 F 2 "" H 9550 2700 60  0000 C CNN
@@
 $EndComp
 $Comp
-L USB_OTG P8
+L USB_OTG P7
 U 1 1 55B4A7CC
 P 8950 5050
-F 0 "P8" H 9275 4925 50  0000 C CNN
+F 0 "P7" H 9275 4925 50  0000 C CNN
 F 1 "USB_OTG" H 8950 5250 50  0000 C CNN
 F 2 "Connect:USB_Mini-B" V 8900 4950 60  0001 C CNN
@@
 $EndComp
 $Comp
-L +12V #PWR?
+L +12V #PWR31
 U 1 1 575F2249
 P 3550 1800
-F 0 "#PWR?" H 3550 1650 50  0001 C CNN
+F 0 "#PWR31" H 3550 1650 50  0001 C CNN
 F 1 "+12V" H 3568 1974 50  0000 C CNN
 F 2 "" H 3550 1800 60  0000 C CNN
@@
 $EndComp
 $Comp
-L +12V #PWR?
+L +12V #PWR38
 U 1 1 575F23FA
 P 4150 2950
-F 0 "#PWR?" H 4150 2800 50  0001 C CNN
+F 0 "#PWR38" H 4150 2800 50  0001 C CNN
 F 1 "+12V" H 4168 3124 50  0000 C CNN
 F 2 "" H 4150 2950 60  0000 C CNN
@@
 Connection ~ 3000 1900
 $Comp
-L GNDD #PWR?
+L GNDD #PWR26
 U 1 1 57607F8B
 P 3000 3700
-F 0 "#PWR?" H 3000 3450 60  0001 C CNN
+F 0 "#PWR26" H 3000 3450 60  0001 C CNN
 F 1 "GNDD" H 3000 3550 60  0000 C CNN
 F 2 "" H 3000 3700 60  0000 C CNN
@@
 RJ45_RX-
 $Comp
-L +12V #PWR?
+L +12V #PWR32
 U 1 1 57607F95
 P 3550 3200
-F 0 "#PWR?" H 3550 3050 50  0001 C CNN
+F 0 "#PWR32" H 3550 3050 50  0001 C CNN
 F 1 "+12V" H 3568 3374 50  0000 C CNN
 F 2 "" H 3550 3200 60  0000 C CNN
@@
 	2900 3500 3600 3500
 $Comp
-L +12V #PWR?
+L +12V #PWR62
 U 1 1 5760ABA5
 P 8250 1300
-F 0 "#PWR?" H 8250 1150 50  0001 C CNN
+F 0 "#PWR62" H 8250 1150 50  0001 C CNN
 F 1 "+12V" H 8268 1474 50  0000 C CNN
 F 2 "" H 8250 1300 60  0000 C CNN
@@
 	8250 1300 8250 1550
 $Comp
-L +12V #PWR?
+L +12V #PWR77
 U 1 1 5760AF55
 P 9550 1300
-F 0 "#PWR?" H 9550 1150 50  0001 C CNN
+F 0 "#PWR77" H 9550 1150 50  0001 C CNN
 F 1 "+12V" H 9568 1474 50  0000 C CNN
 F 2 "" H 9550 1300 60  0000 C CNN

Commit message: set RJ45 footprint
Parts:
- J1, J2: footprint (none) -> local-footprints:54602-908LF
Changed lines of the file:
@@
 F 0 "J1" V 2900 1850 50  0000 L CNN
 F 1 "CC_MAIN" H 2450 2350 50  0000 C CNN
-F 2 "" H 2450 1850 50  0000 C CNN
+F 2 "local-footprints:54602-908LF" H 2450 1850 50  0001 C CNN
 F 3 "" H 2450 1850 50  0000 C CNN
 	1    2450 1850
@@
 F 0 "J2" V 2900 3250 50  0000 L CNN
 F 1 "CC_NEXT" H 2450 3750 50  0000 C CNN
-F 2 "" H 2450 3250 50  0000 C CNN
+F 2 "local-footprints:54602-908LF" H 2450 3250 50  0001 C CNN
 F 3 "" H 2450 3250 50  0000 C CNN
 	1    2450 3250

Commit message: changing footprint of rear board header
Parts:
- P6: footprint Pin_Headers:Pin_Header_Straight_1x12 -> Pin_Headers:Pin_Header_Angled_1x12
Changed lines of the file:
@@
 F 0 "P6" H 8550 2650 50  0000 C CNN
 F 1 "CONN_01X12" V 8650 2000 50  0000 C CNN
-F 2 "Pin_Headers:Pin_Header_Straight_1x12" H 8550 2000 60  0001 C CNN
+F 2 "Pin_Headers:Pin_Header_Angled_1x12" H 8550 2000 60  0001 C CNN
 F 3 "" H 8550 2000 60  0000 C CNN
 	1    8550 2000
