File: hw-design/board/rear-board.sch (KiCad schematic (older format))
At the start: 14 parts, among them J1 CC_MAIN, J2 CC_NEXT, P6 CONN_01X12, P7 USB_OTG, P8 CONN_01X12, Q6 IRFML8244TRPBF

Commit message: rename 12v line to Vin in the rear board
Connections:
- net labels added: VIN
- wire segments 75 -> 74
Changed lines of the file:
@@
-$EndComp
-$Comp
-L +12V #PWR31
-U 1 1 575F2249
-P 3550 1800
-F 0 "#PWR31" H 3550 1650 50  0001 C CNN
-F 1 "+12V" H 3568 1974 50  0000 C CNN
-F 2 "" H 3550 1800 60  0000 C CNN
-F 3 "" H 3550 1800 60  0000 C CNN
-	1    3550 1800
-	1    0    0    -1
-$EndComp
-$Comp
-L +12V #PWR38
-U 1 1 575F23FA
-P 4150 2950
-F 0 "#PWR38" H 4150 2800 50  0001 C CNN
-F 1 "+12V" H 4168 3124 50  0000 C CNN
-F 2 "" H 4150 2950 60  0000 C CNN
-F 3 "" H 4150 2950 60  0000 C CNN
-	1    4150 2950
-	1    0    0    -1
 $EndComp
 $Comp
@@
 RJ45_RX-
 $Comp
-L +12V #PWR32
-U 1 1 57607F95
-P 3550 3200
-F 0 "#PWR32" H 3550 3050 50  0001 C CNN
-F 1 "+12V" H 3568 3374 50  0000 C CNN
-F 2 "" H 3550 3200 60  0000 C CNN
-F 3 "" H 3550 3200 60  0000 C CNN
-	1    3550 3200
-	1    0    0    -1
-$EndComp
-$Comp
 L RJ45 J2
 U 1 1 57607FA3
@@
 NoConn ~ 2100 2400
 NoConn ~ 2100 3800
-$Comp
-L +12V #PWR62
-U 1 1 5760ABA5
-P 8250 1300
-F 0 "#PWR62" H 8250 1150 50  0001 C CNN
-F 1 "+12V" H 8268 1474 50  0000 C CNN
-F 2 "" H 8250 1300 60  0000 C CNN
-F 3 "" H 8250 1300 60  0000 C CNN
-	1    8250 1300
-	1    0    0    -1
-$EndComp
 $Comp
 L +12V #PWR76
@@
 	9650 2250 9450 2250
 Wire Wire Line
-	2900 1900 3550 1900
-Wire Wire Line
-	3550 1900 3550 1800
-Wire Wire Line
-	2900 1800 3000 1800
-Wire Wire Line
-	3000 1800 3000 1900
-Connection ~ 3000 1900
-Wire Wire Line
 	2900 2900 3000 2900
 Wire Wire Line
@@
 	3000 3400 2900 3400
 Wire Wire Line
-	2900 3300 3550 3300
-Wire Wire Line
-	3550 3300 3550 3200
-Wire Wire Line
-	2900 3200 3000 3200
-Wire Wire Line
-	3000 3200 3000 3300
-Connection ~ 3000 3300
-Wire Wire Line
 	2900 3600 3000 3600
 Wire Wire Line
@@
 	2900 3500 3600 3500
 Wire Wire Line
-	8250 1300 8250 1550
-Wire Wire Line
 	9550 1300 9550 1550
-Connection ~ 8250 1450
 Connection ~ 9550 1450
 Wire Wire Line
@@
 Connection ~ 8250 2550
 Wire Wire Line
-	8350 1450 8250 1450
-Wire Wire Line
-	8250 1550 8350 1550
-Wire Wire Line
 	9550 1550 9450 1550
 Wire Wire Line
@@
 Wire Wire Line
 	7850 2450 7750 2450
+Text GLabel 8150 1450 0    50   Input ~ 0
+VIN
+Wire Wire Line
+	8150 1450 8350 1450
+Wire Wire Line
+	8350 1550 8250 1550
+Wire Wire Line
+	8250 1550 8250 1450
+Connection ~ 8250 1450
+Text GLabel 3000 1800 2    50   Output ~ 0
+VIN
+Wire Wire Line
+	2900 1800 3000 1800
+Wire Wire Line
+	2900 1900 2950 1900
+Wire Wire Line
+	2950 1900 2950 1800
+Connection ~ 2950 1800
+Text GLabel 3000 3200 2    50   Output ~ 0
+VIN
+Wire Wire Line
+	2900 3200 3000 3200
+Wire Wire Line
+	2900 3300 2950 3300
+Wire Wire Line
+	2950 3300 2950 3200
+Connection ~ 2950 3200
+Text GLabel 4000 2950 0    50   Input ~ 0
+VIN
+Wire Wire Line
+	4150 2950 4000 2950
 $EndSCHEMATC

Commit message: update MPN
Parts:
- C9: value 100nF X7R -> 100nF
- J1, J2: MPN (none) -> 54602-908LF
- R16: value 10k -> 10K
Changed lines of the file:
@@
 P 4150 3800
 F 0 "C9" V 4000 3800 40  0000 L CNN
-F 1 "100nF X7R" V 4300 3650 40  0000 L CNN
+F 1 "100nF" V 4300 3650 40  0000 L CNN
 F 2 "Capacitors_SMD:C_0603" H 4188 3650 30  0001 C CNN
 F 3 "~" H 4150 3800 60  0000 C CNN
@@
 P 4150 3200
 F 0 "R16" V 4250 3200 40  0000 C CNN
-F 1 "10k" V 4157 3201 40  0000 C CNN
+F 1 "10K" V 4157 3201 40  0000 C CNN
 F 2 "Resistors_SMD:R_0603" V 4080 3200 30  0001 C CNN
 F 3 "~" H 4150 3200 30  0000 C CNN
@@
 F 2 "local-footprints:54602-908LF" H 2450 1850 50  0001 C CNN
 F 3 "" H 2450 1850 50  0000 C CNN
+F 4 "54602-908LF" V 2450 1850 60  0001 C CNN "MPN"
 	1    2450 1850
 	0    -1   1    0
@@
 F 2 "local-footprints:54602-908LF" H 2450 3250 50  0001 C CNN
 F 3 "" H 2450 3250 50  0000 C CNN
+F 4 "54602-908LF" V 2450 3250 60  0001 C CNN "MPN"
 	1    2450 3250
 	0    -1   1    0

Commit message: adding missing MPN
Parts:
- P6, P8: MPN (none) -> 68016-112HLF
Changed lines of the file:
@@
 F 2 "Pin_Headers:Pin_Header_Angled_1x12" H 8550 2000 60  0001 C CNN
 F 3 "" H 8550 2000 60  0000 C CNN
+F 4 "68016-112HLF" H 8550 2000 60  0001 C CNN "MPN"
 	1    8550 2000
 	1    0    0    -1
@@
 F 2 "Pin_Headers:Pin_Header_Angled_1x12" H 9250 2000 60  0001 C CNN
 F 3 "" H 9250 2000 60  0000 C CNN
+F 4 "68016-112HLF" H 9250 2000 60  0001 C CNN "MPN"
 	1    9250 2000
 	-1   0    0    -1

Commit message: DRC done
Parts:
- renumbered C18 to C19, Q6 to Q5, R17 to R24, R18 to R25, R34 to R35
Changed lines of the file:
@@
 $EndDescr
 $Comp
-L GNDD #PWR25
+L GNDD #PWR23
 U 1 1 55B26400
 P 3000 2300
-F 0 "#PWR25" H 3000 2050 60  0001 C CNN
+F 0 "#PWR23" H 3000 2050 60  0001 C CNN
 F 1 "GNDD" H 3000 2150 60  0000 C CNN
 F 2 "" H 3000 2300 60  0000 C CNN
@@
 $EndComp
 $Comp
-L GNDD #PWR39
+L GNDD #PWR35
 U 1 1 55B2641C
 P 4150 4050
-F 0 "#PWR39" H 4150 3800 60  0001 C CNN
+F 0 "#PWR35" H 4150 3800 60  0001 C CNN
 F 1 "GNDD" H 4150 3900 60  0000 C CNN
 F 2 "" H 4150 4050 60  0000 C CNN
@@
 USB_PLUG_VCC
 $Comp
-L R R34
+L R R35
 U 1 1 55B2B900
 P 8450 5200
-F 0 "R34" V 8350 5350 50  0000 C CNN
+F 0 "R35" V 8350 5350 50  0000 C CNN
 F 1 "1M" V 8450 5200 50  0000 C CNN
 F 2 "Resistors_SMD:R_0603" V 8380 5200 30  0001 C CNN
@@
 $EndComp
 $Comp
-L GNDD #PWR65
+L GNDD #PWR61
 U 1 1 55B2B90F
 P 8450 5550
-F 0 "#PWR65" H 8450 5300 50  0001 C CNN
+F 0 "#PWR61" H 8450 5300 50  0001 C CNN
 F 1 "GNDD" H 8450 5400 50  0000 C CNN
 F 2 "" H 8450 5550 60  0000 C CNN
@@
 $EndComp
 $Comp
-L C C18
+L C C19
 U 1 1 55B2B908
 P 8250 5200
-F 0 "C18" V 8300 5000 50  0000 L CNN
+F 0 "C19" V 8300 5000 50  0000 L CNN
 F 1 "10nF 500V" V 8100 5000 50  0000 L CNN
 F 2 "Capacitors_SMD:C_1206" H 8288 5050 30  0001 C CNN
@@
 USB_DP
 $Comp
-L Q_NMOS_GSD Q6
+L Q_NMOS_GSD Q5
 U 1 1 55B320E7
 P 3500 5900
-F 0 "Q6" H 3400 6000 50  0000 R CNN
+F 0 "Q5" H 3400 6000 50  0000 R CNN
 F 1 "IRFML8244TRPBF" V 3750 6150 50  0000 R CNN
 F 2 "Housings_SOT-23_SOT-143_TSOT-6:SOT-23" H 3700 6000 29  0001 C CNN
@@
 USB_VCC
 $Comp
-L GNDD #PWR63
+L GNDD #PWR59
 U 1 1 55B45519
 P 8250 2700
-F 0 "#PWR63" H 8250 2450 50  0001 C CNN
+F 0 "#PWR59" H 8250 2450 50  0001 C CNN
 F 1 "GNDD" H 8250 2550 50  0000 C CNN
 F 2 "" H 8250 2700 60  0000 C CNN
@@
 $EndComp
 $Comp
-L GNDD #PWR78
+L GNDD #PWR76
 U 1 1 55B4640F
 P 9550 2700
-F 0 "#PWR78" H 9550 2450 50  0001 C CNN
+F 0 "#PWR76" H 9550 2450 50  0001 C CNN
 F 1 "GNDD" H 9550 2550 50  0000 C CNN
 F 2 "" H 9550 2700 60  0000 C CNN
@@
 $EndComp
 $Comp
-L GNDD #PWR26
+L GNDD #PWR24
 U 1 1 57607F8B
 P 3000 3700
-F 0 "#PWR26" H 3000 3450 60  0001 C CNN
+F 0 "#PWR24" H 3000 3450 60  0001 C CNN
 F 1 "GNDD" H 3000 3550 60  0000 C CNN
 F 2 "" H 3000 3700 60  0000 C CNN
@@
 NoConn ~ 2100 3800
 $Comp
-L +12V #PWR76
+L +12V #PWR74
 U 1 1 5760AF55
 P 9550 1300
-F 0 "#PWR76" H 9550 1150 50  0001 C CNN
+F 0 "#PWR74" H 9550 1150 50  0001 C CNN
 F 1 "+12V" H 9568 1474 50  0000 C CNN
 F 2 "" H 9550 1300 60  0000 C CNN
@@
 $EndComp
 $Comp
-L R R17
+L R R24
 U 1 1 576041F9
 P 8000 2350
-F 0 "R17" V 8050 2550 50  0000 C CNN
+F 0 "R24" V 8050 2550 50  0000 C CNN
 F 1 "33R" V 8000 2350 50  0000 C CNN
 F 2 "Resistors_SMD:R_0603" V 7930 2350 30  0001 C CNN
@@
 $EndComp
 $Comp
-L R R18
+L R R25
 U 1 1 57604201
 P 8000 2450
-F 0 "R18" V 8050 2650 50  0000 C CNN
+F 0 "R25" V 8050 2650 50  0000 C CNN
 F 1 "33R" V 8000 2450 50  0000 C CNN
 F 2 "Resistors_SMD:R_0603" V 7930 2450 30  0001 C CNN

Commit message: update netlist
Parts:
- renumbered Q5 to Q6, R14 to R16, R16 to R18, R24 to R26, R25 to R27, R35 to R37
Changed lines of the file:
@@
 $EndDescr
 $Comp
-L GNDD #PWR23
+L GNDD #PWR25
 U 1 1 55B26400
 P 3000 2300
-F 0 "#PWR23" H 3000 2050 60  0001 C CNN
+F 0 "#PWR25" H 3000 2050 60  0001 C CNN
 F 1 "GNDD" H 3000 2150 60  0000 C CNN
 F 2 "" H 3000 2300 60  0000 C CNN
@@
 $EndComp
 $Comp
-L R R16
+L R R18
 U 1 1 55B26415
 P 4150 3200
-F 0 "R16" V 4250 3200 40  0000 C CNN
+F 0 "R18" V 4250 3200 40  0000 C CNN
 F 1 "10K" V 4157 3201 40  0000 C CNN
 F 2 "Resistors_SMD:R_0603" V 4080 3200 30  0001 C CNN
@@
 $EndComp
 $Comp
-L GNDD #PWR35
+L GNDD #PWR37
 U 1 1 55B2641C
 P 4150 4050
-F 0 "#PWR35" H 4150 3800 60  0001 C CNN
+F 0 "#PWR37" H 4150 3800 60  0001 C CNN
 F 1 "GNDD" H 4150 3900 60  0000 C CNN
 F 2 "" H 4150 4050 60  0000 C CNN
@@
 USB_PLUG_VCC
 $Comp
-L R R35
+L R R37
 U 1 1 55B2B900
 P 8450 5200
-F 0 "R35" V 8350 5350 50  0000 C CNN
+F 0 "R37" V 8350 5350 50  0000 C CNN
 F 1 "1M" V 8450 5200 50  0000 C CNN
 F 2 "Resistors_SMD:R_0603" V 8380 5200 30  0001 C CNN
@@
 $EndComp
 $Comp
-L GNDD #PWR61
+L GNDD #PWR63
 U 1 1 55B2B90F
 P 8450 5550
-F 0 "#PWR61" H 8450 5300 50  0001 C CNN
+F 0 "#PWR63" H 8450 5300 50  0001 C CNN
 F 1 "GNDD" H 8450 5400 50  0000 C CNN
 F 2 "" H 8450 5550 60  0000 C CNN
@@
 USB_DP
 $Comp
-L Q_NMOS_GSD Q5
+L Q_NMOS_GSD Q6
 U 1 1 55B320E7
 P 3500 5900
-F 0 "Q5" H 3400 6000 50  0000 R CNN
+F 0 "Q6" H 3400 6000 50  0000 R CNN
 F 1 "IRFML8244TRPBF" V 3750 6150 50  0000 R CNN
 F 2 "Housings_SOT-23_SOT-143_TSOT-6:SOT-23" H 3700 6000 29  0001 C CNN
@@
 $EndComp
 $Comp
-L R R14
+L R R16
 U 1 1 55B320EF
 P 3600 6350
-F 0 "R14" V 3680 6350 50  0000 C CNN
+F 0 "R16" V 3680 6350 50  0000 C CNN
 F 1 "100R" V 3600 6350 50  0000 C CNN
 F 2 "Resistors_SMD:R_0805" V 3530 6350 30  0001 C CNN
@@
 USB_VCC
 $Comp
-L GNDD #PWR59
+L GNDD #PWR61
 U 1 1 55B45519
 P 8250 2700
-F 0 "#PWR59" H 8250 2450 50  0001 C CNN
+F 0 "#PWR61" H 8250 2450 50  0001 C CNN
 F 1 "GNDD" H 8250 2550 50  0000 C CNN
 F 2 "" H 8250 2700 60  0000 C CNN
@@
 $EndComp
 $Comp
-L GNDD #PWR76
+L GNDD #PWR78
 U 1 1 55B4640F
 P 9550 2700
-F 0 "#PWR76" H 9550 2450 50  0001 C CNN
+F 0 "#PWR78" H 9550 2450 50  0001 C CNN
 F 1 "GNDD" H 9550 2550 50  0000 C CNN
 F 2 "" H 9550 2700 60  0000 C CNN
@@
 $EndComp
 $Comp
-L GNDD #PWR24
+L GNDD #PWR26
 U 1 1 57607F8B
 P 3000 3700
-F 0 "#PWR24" H 3000 3450 60  0001 C CNN
+F 0 "#PWR26" H 3000 3450 60  0001 C CNN
 F 1 "GNDD" H 3000 3550 60  0000 C CNN
 F 2 "" H 3000 3700 60  0000 C CNN
@@
 NoConn ~ 2100 3800
 $Comp
-L +12V #PWR74
+L +12V #PWR76
 U 1 1 5760AF55
 P 9550 1300
-F 0 "#PWR74" H 9550 1150 50  0001 C CNN
+F 0 "#PWR76" H 9550 1150 50  0001 C CNN
 F 1 "+12V" H 9568 1474 50  0000 C CNN
 F 2 "" H 9550 1300 60  0000 C CNN
@@
 $EndComp
 $Comp
-L R R24
+L R R26
 U 1 1 576041F9
 P 8000 2350
-F 0 "R24" V 8050 2550 50  0000 C CNN
+F 0 "R26" V 8050 2550 50  0000 C CNN
 F 1 "33R" V 8000 2350 50  0000 C CNN
 F 2 "Resistors_SMD:R_0603" V 7930 2350 30  0001 C CNN
@@
 $EndComp
 $Comp
-L R R25
+L R R27
 U 1 1 57604201
 P 8000 2450
-F 0 "R25" V 8050 2650 50  0000 C CNN
+F 0 "R27" V 8050 2650 50  0000 C CNN
 F 1 "33R" V 8000 2450 50  0000 C CNN
 F 2 "Resistors_SMD:R_0603" V 7930 2450 30  0001 C CNN
