File: hw-design/board/rear-board.sch (KiCad schematic (older format))
At the start: 14 parts, among them J1 CC_MAIN, J2 CC_NEXT, P6 CONN_01X12, P7 USB_OTG, P8 CONN_01X12, Q6 IRFML8244TRPBF

Commit message: sch: change angled pin header to straight one
Parts:
- P6: footprint Pin_Headers:Pin_Header_Angled_1x12 -> Pin_Headers:Pin_Header_Straight_1x12
Changed lines of the file:
@@
 LIBS:nxp_armmcu
 LIBS:philips
+LIBS:graphic_symbols
 LIBS:footswitch-cache
 EELAYER 26 0
@@
 F 0 "P6" H 8550 2650 50  0000 C CNN
 F 1 "CONN_01X12" V 8650 2000 50  0000 C CNN
-F 2 "Pin_Headers:Pin_Header_Angled_1x12" H 8550 2000 60  0001 C CNN
+F 2 "Pin_Headers:Pin_Header_Straight_1x12" H 8550 2000 60  0001 C CNN
 F 3 "" H 8550 2000 60  0000 C CNN
 F 4 "68016-112HLF" H 8550 2000 60  0001 C CNN "MPN"

Commit message: update files to KiCAD 5
Parts:
- C19, C9: symbol C -> footswitch-rescue:C
- D2: symbol D -> footswitch-rescue:D
- J1, J2: symbol RJ45 -> footswitch-rescue:RJ45
- P6, P8: symbol CONN_01X12 -> footswitch-rescue:CONN_01X12
- P7: symbol USB_OTG -> footswitch-rescue:USB_OTG
- Q6: symbol Q_NMOS_GSD -> footswitch-rescue:Q_NMOS_GSD
- R16, R18, R26, R27, R37: symbol R -> footswitch-rescue:R
Changed lines of the file:
@@
-EESchema Schematic File Version 2
-LIBS:conn
-LIBS:device
-LIBS:interface
-LIBS:power
-LIBS:regul
-LIBS:transistors
-LIBS:display
-LIBS:nxp_armmcu
-LIBS:philips
-LIBS:graphic_symbols
+EESchema Schematic File Version 4
 LIBS:footswitch-cache
 EELAYER 26 0
@@
 $EndDescr
 $Comp
-L GNDD #PWR069
+L footswitch-rescue:GNDD #PWR069
 U 1 1 55B26400
 P 3000 2300
@@
 $EndComp
 $Comp
-L C C9
+L footswitch-rescue:C C9
 U 1 1 55B2640D
 P 4150 3800
@@
 $EndComp
 $Comp
-L R R18
+L footswitch-rescue:R R18
 U 1 1 55B26415
 P 4150 3200
@@
 $EndComp
 $Comp
-L GNDD #PWR070
+L footswitch-rescue:GNDD #PWR070
 U 1 1 55B2641C
 P 4150 4050
@@
 $EndComp
 $Comp
-L D D2
+L footswitch-rescue:D D2
 U 1 1 55B26435
 P 3750 3500
@@
 USB_PLUG_VCC
 $Comp
-L R R37
+L footswitch-rescue:R R37
 U 1 1 55B2B900
 P 8450 5200
@@
 $EndComp
 $Comp
-L GNDD #PWR071
+L footswitch-rescue:GNDD #PWR071
 U 1 1 55B2B90F
 P 8450 5550
@@
 $EndComp
 $Comp
-L C C19
+L footswitch-rescue:C C19
 U 1 1 55B2B908
 P 8250 5200
@@
 USB_DP
 $Comp
-L Q_NMOS_GSD Q6
+L footswitch-rescue:Q_NMOS_GSD Q6
 U 1 1 55B320E7
 P 3500 5900
@@
 $EndComp
 $Comp
-L R R16
+L footswitch-rescue:R R16
 U 1 1 55B320EF
 P 3600 6350
@@
 NoConn ~ 8850 5350
 $Comp
-L CONN_01X12 P6
+L footswitch-rescue:CONN_01X12 P6
 U 1 1 55B42C87
 P 8550 2000
@@
 $EndComp
 $Comp
-L CONN_01X12 P8
+L footswitch-rescue:CONN_01X12 P8
 U 1 1 55B42DAB
 P 9250 2000
@@
 USB_VCC
 $Comp
-L GNDD #PWR072
+L footswitch-rescue:GNDD #PWR072
 U 1 1 55B45519
 P 8250 2700
@@
 $EndComp
 $Comp
-L GNDD #PWR073
+L footswitch-rescue:GNDD #PWR073
 U 1 1 55B4640F
 P 9550 2700
@@
 $EndComp
 $Comp
-L USB_OTG P7
+L footswitch-rescue:USB_OTG P7
 U 1 1 55B4A7CC
 P 8950 5050
@@
 $EndComp
 $Comp
-L RJ45 J1
+L footswitch-rescue:RJ45 J1
 U 1 1 57607322
 P 2450 1850
@@
 $EndComp
 $Comp
-L GNDD #PWR074
+L footswitch-rescue:GNDD #PWR074
 U 1 1 57607F8B
 P 3000 3700
@@
 RJ45_RX-
 $Comp
-L RJ45 J2
+L footswitch-rescue:RJ45 J2
 U 1 1 57607FA3
 P 2450 3250
@@
 NoConn ~ 2100 3800
 $Comp
-L +12V #PWR075
+L footswitch-rescue:+12V #PWR075
 U 1 1 5760AF55
 P 9550 1300
+AR Path="/5760AF55" Ref="#PWR075"  Part="1"
+AR Path="/55B25118/5760AF55" Ref="#PWR075"  Part="1"
 F 0 "#PWR075" H 9550 1150 50  0001 C CNN
 F 1 "+12V" H 9568 1474 50  0000 C CNN
@@
 $EndComp
 $Comp
-L R R26
+L footswitch-rescue:R R26
 U 1 1 576041F9
 P 8000 2350
@@
 $EndComp
 $Comp
-L R R27
+L footswitch-rescue:R R27
 U 1 1 57604201
 P 8000 2450

Commit message: Changed R40 RE from pull-up to pull-down
Parts:
- C19, C9: symbol footswitch-rescue:C -> footswitch-rescue:C-footswitch-rescue
- D2: symbol footswitch-rescue:D -> footswitch-rescue:D-footswitch-rescue
- J1, J2: symbol footswitch-rescue:RJ45 -> footswitch-rescue:RJ45-footswitch-rescue
- P6, P8: symbol footswitch-rescue:CONN_01X12 -> footswitch-rescue:CONN_01X12-footswitch-rescue
- P7: symbol footswitch-rescue:USB_OTG -> footswitch-rescue:USB_OTG-footswitch-rescue
- Q6: symbol footswitch-rescue:Q_NMOS_GSD -> footswitch-rescue:Q_NMOS_GSD-footswitch-rescue
- R16, R18, R26, R27, R37: symbol footswitch-rescue:R -> footswitch-rescue:R-footswitch-rescue
Changed lines of the file:
@@
 $EndDescr
 $Comp
-L footswitch-rescue:GNDD #PWR069
+L footswitch-rescue:GNDD-footswitch-rescue #PWR069
 U 1 1 55B26400
 P 3000 2300
@@
 $EndComp
 $Comp
-L footswitch-rescue:C C9
+L footswitch-rescue:C-footswitch-rescue C9
 U 1 1 55B2640D
 P 4150 3800
@@
 $EndComp
 $Comp
-L footswitch-rescue:R R18
+L footswitch-rescue:R-footswitch-rescue R18
 U 1 1 55B26415
 P 4150 3200
@@
 $EndComp
 $Comp
-L footswitch-rescue:GNDD #PWR070
+L footswitch-rescue:GNDD-footswitch-rescue #PWR070
 U 1 1 55B2641C
 P 4150 4050
@@
 $EndComp
 $Comp
-L footswitch-rescue:D D2
+L footswitch-rescue:D-footswitch-rescue D2
 U 1 1 55B26435
 P 3750 3500
@@
 USB_PLUG_VCC
 $Comp
-L footswitch-rescue:R R37
+L footswitch-rescue:R-footswitch-rescue R37
 U 1 1 55B2B900
 P 8450 5200
@@
 $EndComp
 $Comp
-L footswitch-rescue:GNDD #PWR071
+L footswitch-rescue:GNDD-footswitch-rescue #PWR071
 U 1 1 55B2B90F
 P 8450 5550
@@
 $EndComp
 $Comp
-L footswitch-rescue:C C19
+L footswitch-rescue:C-footswitch-rescue C19
 U 1 1 55B2B908
 P 8250 5200
@@
 USB_DP
 $Comp
-L footswitch-rescue:Q_NMOS_GSD Q6
+L footswitch-rescue:Q_NMOS_GSD-footswitch-rescue Q6
 U 1 1 55B320E7
 P 3500 5900
@@
 $EndComp
 $Comp
-L footswitch-rescue:R R16
+L footswitch-rescue:R-footswitch-rescue R16
 U 1 1 55B320EF
 P 3600 6350
@@
 NoConn ~ 8850 5350
 $Comp
-L footswitch-rescue:CONN_01X12 P6
+L footswitch-rescue:CONN_01X12-footswitch-rescue P6
 U 1 1 55B42C87
 P 8550 2000
@@
 $EndComp
 $Comp
-L footswitch-rescue:CONN_01X12 P8
+L footswitch-rescue:CONN_01X12-footswitch-rescue P8
 U 1 1 55B42DAB
 P 9250 2000
@@
 USB_VCC
 $Comp
-L footswitch-rescue:GNDD #PWR072
+L footswitch-rescue:GNDD-footswitch-rescue #PWR072
 U 1 1 55B45519
 P 8250 2700
@@
 $EndComp
 $Comp
-L footswitch-rescue:GNDD #PWR073
+L footswitch-rescue:GNDD-footswitch-rescue #PWR073
 U 1 1 55B4640F
 P 9550 2700
@@
 $EndComp
 $Comp
-L footswitch-rescue:USB_OTG P7
+L footswitch-rescue:USB_OTG-footswitch-rescue P7
 U 1 1 55B4A7CC
 P 8950 5050
@@
 $EndComp
 $Comp
-L footswitch-rescue:RJ45 J1
+L footswitch-rescue:RJ45-footswitch-rescue J1
 U 1 1 57607322
 P 2450 1850
@@
 $EndComp
 $Comp
-L footswitch-rescue:GNDD #PWR074
+L footswitch-rescue:GNDD-footswitch-rescue #PWR074
 U 1 1 57607F8B
 P 3000 3700
@@
 RJ45_RX-
 $Comp
-L footswitch-rescue:RJ45 J2
+L footswitch-rescue:RJ45-footswitch-rescue J2
 U 1 1 57607FA3
 P 2450 3250
@@
 NoConn ~ 2100 3800
 $Comp
-L footswitch-rescue:+12V #PWR075
+L footswitch-rescue:+12V-footswitch-rescue #PWR075
 U 1 1 5760AF55
 P 9550 1300
@@
 $EndComp
 $Comp
-L footswitch-rescue:R R26
+L footswitch-rescue:R-footswitch-rescue R26
 U 1 1 576041F9
 P 8000 2350
@@
 $EndComp
 $Comp
-L footswitch-rescue:R R27
+L footswitch-rescue:R-footswitch-rescue R27
 U 1 1 57604201
 P 8000 2450
