File: hw-design/board/mechanic.sch (KiCad schematic (older format))
At the start: 14 parts

Commit message: added keystones to mechanic
Parts:
- removed H? (x3): DS1_HOLE, symbol CONN_01X01
- removed H? (x4): DS2_HOLE, symbol CONN_01X01
- removed H? (x5): STANDOFF_HOLE, symbol CONN_01X01
- added H10, H11, H12, H13, H14: STANDOFF_HOLE, local-footprints:M3-screw-hole, symbol CONN_01X01
- added H15, H16: KEYSTONE, local-footprints:Keystone-7790, symbol CONN_02X02
- added H2, H4, H6, H8: DS2_HOLE, local-footprints:M3-screw-hole, symbol CONN_01X01
- added H3, H5, H7: DS1_HOLE, local-footprints:M3-screw-hole, symbol CONN_01X01
- H1, H9: renamed from H?; footprint (none) -> local-footprints:M3-screw-hole
Connections:
- no-connect marks 14 -> 22
Other:
- note added: "KEYSTONE"
- moved on the sheet: H9

Commit message: sch: fixing mechanic sheet
Parts:
- removed H10, H11, H12, H13, H14, H9: STANDOFF_HOLE, local-footprints:M3-screw-hole, symbol CONN_01X01
- removed H15, H16: KEYSTONE, local-footprints:Keystone-7790, symbol CONN_02X02
- removed H7: DS1_HOLE, local-footprints:M3-screw-hole, symbol CONN_01X01
- removed H8: DS2_HOLE, local-footprints:M3-screw-hole, symbol CONN_01X01
- added H7, H8: KEYSTONE, local-footprints:Keystone-7790, symbol CONN_02X02
- H1, H3, H5: value DS1_HOLE -> HOLE
- H2, H4, H6: value DS2_HOLE -> HOLE
Connections:
- no-connect marks 22 -> 14
Other:
- note added: "BOARD STANDOFF"
- note added: "KEYSTONE HOLES"
- note removed: "DISPLAY HOLES"
- note removed: "KEYSTONE"
- note removed: "STANDOFF"

Commit message: adding missing MPN
Parts:
- H7, H8: MPN (none) -> Keystone 7790
Changed lines of the file:
@@
 F 2 "local-footprints:Keystone-7790" H 4200 1850 60  0001 C CNN
 F 3 "" H 4200 650 60  0000 C CNN
+F 4 "Keystone 7790" H 4200 1850 60  0001 C CNN "MPN"
 	1    4200 1850
 	1    0    0    -1
@@
 F 2 "local-footprints:Keystone-7790" H 4950 1850 60  0001 C CNN
 F 3 "" H 4950 650 60  0000 C CNN
+F 4 "Keystone 7790" H 4950 1850 60  0001 C CNN "MPN"
 	1    4950 1850
 	1    0    0    -1
