File: hw-design/board/mechanic.sch (KiCad schematic (older format))
At the start: 8 parts

Commit message: update files to KiCAD 5
Parts:
- H1, H2, H3, H4, H5, H6: symbol CONN_01X01 -> footswitch-rescue:CONN_01X01; Note (none) -> not a component
- H7, H8: symbol CONN_02X02 -> footswitch-rescue:CONN_02X02
Changed lines of the file:
@@
-EESchema Schematic File Version 2
-LIBS:conn
-LIBS:device
-LIBS:interface
-LIBS:power
-LIBS:regul
-LIBS:transistors
-LIBS:display
-LIBS:nxp_armmcu
-LIBS:philips
-LIBS:graphic_symbols
+EESchema Schematic File Version 4
 LIBS:footswitch-cache
 EELAYER 26 0
@@
 $EndDescr
 $Comp
-L CONN_01X01 H1
+L footswitch-rescue:CONN_01X01 H1
 U 1 1 55B19E56
 P 1850 1800
@@
 F 2 "local-footprints:M3-screw-hole" H 1850 1800 60  0001 C CNN
 F 3 "" H 1850 1800 60  0000 C CNN
+F 4 "not a component" H 1850 1800 50  0001 C CNN "Note"
 	1    1850 1800
 	0    1    1    0
 $EndComp
 $Comp
-L CONN_01X01 H3
+L footswitch-rescue:CONN_01X01 H3
 U 1 1 55B19FA4
 P 2100 1800
@@
 F 2 "local-footprints:M3-screw-hole" H 2100 1800 60  0001 C CNN
 F 3 "" H 2100 1800 60  0000 C CNN
+F 4 "not a component" H 2100 1800 50  0001 C CNN "Note"
 	1    2100 1800
 	0    1    1    0
 $EndComp
 $Comp
-L CONN_01X01 H5
+L footswitch-rescue:CONN_01X01 H5
 U 1 1 55B1A020
 P 2350 1800
@@
 F 2 "local-footprints:M3-screw-hole" H 2350 1800 60  0001 C CNN
 F 3 "" H 2350 1800 60  0000 C CNN
+F 4 "not a component" H 2350 1800 50  0001 C CNN "Note"
 	1    2350 1800
 	0    1    1    0
 $EndComp
 $Comp
-L CONN_01X01 H2
+L footswitch-rescue:CONN_01X01 H2
 U 1 1 55B1A026
 P 1850 2300
@@
 F 2 "local-footprints:M3-screw-hole" H 1850 2300 60  0001 C CNN
 F 3 "" H 1850 2300 60  0000 C CNN
+F 4 "not a component" H 1850 2300 50  0001 C CNN "Note"
 	1    1850 2300
 	0    1    1    0
 $EndComp
 $Comp
-L CONN_01X01 H4
+L footswitch-rescue:CONN_01X01 H4
 U 1 1 55B1A078
 P 2100 2300
@@
 F 2 "local-footprints:M3-screw-hole" H 2100 2300 60  0001 C CNN
 F 3 "" H 2100 2300 60  0000 C CNN
+F 4 "not a component" H 2100 2300 50  0001 C CNN "Note"
 	1    2100 2300
 	0    1    1    0
 $EndComp
 $Comp
-L CONN_01X01 H6
+L footswitch-rescue:CONN_01X01 H6
 U 1 1 55B1A07E
 P 2350 2300
@@
 F 2 "local-footprints:M3-screw-hole" H 2350 2300 60  0001 C CNN
 F 3 "" H 2350 2300 60  0000 C CNN
+F 4 "not a component" H 2350 2300 50  0001 C CNN "Note"
 	1    2350 2300
 	0    1    1    0
@@
 BOARD STANDOFF
 $Comp
-L CONN_02X02 H7
+L footswitch-rescue:CONN_02X02 H7
 U 1 1 55B1AED0
 P 4200 1850
@@
 $EndComp
 $Comp
-L CONN_02X02 H8
+L footswitch-rescue:CONN_02X02 H8
 U 1 1 55B1B1A5
 P 4950 1850

Commit message: Changed R40 RE from pull-up to pull-down
Parts:
- H1, H2, H3, H4, H5, H6: symbol footswitch-rescue:CONN_01X01 -> footswitch-rescue:CONN_01X01-footswitch-rescue
- H7, H8: symbol footswitch-rescue:CONN_02X02 -> footswitch-rescue:CONN_02X02-footswitch-rescue
Changed lines of the file:
@@
 $EndDescr
 $Comp
-L footswitch-rescue:CONN_01X01 H1
+L footswitch-rescue:CONN_01X01-footswitch-rescue H1
 U 1 1 55B19E56
 P 1850 1800
@@
 $EndComp
 $Comp
-L footswitch-rescue:CONN_01X01 H3
+L footswitch-rescue:CONN_01X01-footswitch-rescue H3
 U 1 1 55B19FA4
 P 2100 1800
@@
 $EndComp
 $Comp
-L footswitch-rescue:CONN_01X01 H5
+L footswitch-rescue:CONN_01X01-footswitch-rescue H5
 U 1 1 55B1A020
 P 2350 1800
@@
 $EndComp
 $Comp
-L footswitch-rescue:CONN_01X01 H2
+L footswitch-rescue:CONN_01X01-footswitch-rescue H2
 U 1 1 55B1A026
 P 1850 2300
@@
 $EndComp
 $Comp
-L footswitch-rescue:CONN_01X01 H4
+L footswitch-rescue:CONN_01X01-footswitch-rescue H4
 U 1 1 55B1A078
 P 2100 2300
@@
 $EndComp
 $Comp
-L footswitch-rescue:CONN_01X01 H6
+L footswitch-rescue:CONN_01X01-footswitch-rescue H6
 U 1 1 55B1A07E
 P 2350 2300
@@
 BOARD STANDOFF
 $Comp
-L footswitch-rescue:CONN_02X02 H7
+L footswitch-rescue:CONN_02X02-footswitch-rescue H7
 U 1 1 55B1AED0
 P 4200 1850
@@
 $EndComp
 $Comp
-L footswitch-rescue:CONN_02X02 H8
+L footswitch-rescue:CONN_02X02-footswitch-rescue H8
 U 1 1 55B1B1A5
 P 4950 1850
