File: hw-design/board/usb.sch (KiCad schematic (older format))
At the start: 9 parts, among them Q10 BC857

Commit message: fix power voltage
Changed lines of the file:
@@
 F 0 "R41" V 6200 2100 50  0000 C CNN
 F 1 "2K" V 6300 2100 50  0000 C CNN
-F 2 "Resistors_SMD:R_0603" V 6230 2100 30  0000 C CNN
+F 2 "Resistors_SMD:R_0603" V 6230 2100 30  0001 C CNN
 F 3 "" H 6300 2100 30  0000 C CNN
 F 4 "RMCF0603JT2K00" H 2250 -4350 50  0001 C CNN "MPN"
@@
 F 0 "C25" H 6025 2450 50  0000 L CNN
 F 1 "10nF" V 5850 2150 50  0000 L CNN
-F 2 "Capacitors_SMD:C_0603" H 6038 2200 30  0000 C CNN
+F 2 "Capacitors_SMD:C_0603" H 6038 2200 30  0001 C CNN
 F 3 "" H 6000 2350 60  0000 C CNN
 F 4 "C1608X7R1E103K080AA" H 2250 -4350 50  0001 C CNN "MPN"
@@
 F 0 "R42" V 6500 2350 50  0000 C CNN
 F 1 "3K3" V 6600 2350 50  0000 C CNN
-F 2 "Resistors_SMD:R_0603" V 6530 2350 30  0000 C CNN
+F 2 "Resistors_SMD:R_0603" V 6530 2350 30  0001 C CNN
 F 3 "" H 6600 2350 30  0000 C CNN
 F 4 "RMCF0603JT3K30" H 2550 -4100 50  0001 C CNN "MPN"

Commit message: annotation and ERC
Parts:
- renumbered C25 to C14, Q10 to Q3, R38 to R13, R39 to R17, R40 to R18, R41 to R20, R42 to R21, R36 to R6, R37 to R7
Changed lines of the file:
@@
 $EndDescr
 $Comp
-L R R39
+L R R17
 U 1 1 55B4E32A
 P 4350 2100
-F 0 "R39" V 4250 2100 50  0000 C CNN
+F 0 "R17" V 4250 2100 50  0000 C CNN
 F 1 "33R" V 4350 2100 50  0000 C CNN
 F 2 "Resistors_SMD:R_0603" V 4280 2100 30  0001 C CNN
@@
 $EndComp
 $Comp
-L R R40
+L R R18
 U 1 1 55B4E332
 P 4350 2700
-F 0 "R40" V 4450 2700 50  0000 C CNN
+F 0 "R18" V 4450 2700 50  0000 C CNN
 F 1 "33R" V 4350 2700 50  0000 C CNN
 F 2 "Resistors_SMD:R_0603" V 4280 2700 30  0001 C CNN
@@
 $EndComp
 $Comp
-L R R41
+L R R20
 U 1 1 55B4E33A
 P 6300 2100
-F 0 "R41" V 6200 2100 50  0000 C CNN
+F 0 "R20" V 6200 2100 50  0000 C CNN
 F 1 "2K" V 6300 2100 50  0000 C CNN
 F 2 "Resistors_SMD:R_0603" V 6230 2100 30  0001 C CNN
@@
 $EndComp
 $Comp
-L VCC #PWR099
+L VCC #PWR50
 U 1 1 55B4E341
 P 6000 1950
-F 0 "#PWR099" H 6000 1800 50  0001 C CNN
+F 0 "#PWR50" H 6000 1800 50  0001 C CNN
 F 1 "VCC" H 6000 2100 50  0000 C CNN
 F 2 "" H 6000 1950 60  0000 C CNN
@@
 $EndComp
 $Comp
-L Q_PNP_BEC Q10
+L Q_PNP_BEC Q3
 U 1 1 55B4E348
 P 2700 2450
-F 0 "Q10" H 3000 2450 50  0000 R CNN
+F 0 "Q3" H 3000 2450 50  0000 R CNN
 F 1 "BC857" H 3100 2350 50  0000 R CNN
 F 2 "Housings_SOT-23_SOT-143_TSOT-6:SOT-23" H 2900 2550 29  0001 C CNN
@@
 $EndComp
 $Comp
-L R R36
+L R R6
 U 1 1 55B4E350
 P 2150 2450
-F 0 "R36" V 2230 2450 50  0000 C CNN
+F 0 "R6" V 2230 2450 50  0000 C CNN
 F 1 "3k" V 2150 2450 50  0000 C CNN
 F 2 "Resistors_SMD:R_0603" V 2080 2450 30  0001 C CNN
@@
 $EndComp
 $Comp
-L R R37
+L R R7
 U 1 1 55B4E358
 P 2400 2200
-F 0 "R37" V 2480 2200 50  0000 C CNN
+F 0 "R7" V 2480 2200 50  0000 C CNN
 F 1 "24k" V 2400 2200 50  0000 C CNN
 F 2 "Resistors_SMD:R_0603" V 2330 2200 30  0001 C CNN
@@
 $EndComp
 $Comp
-L +3.3V #PWR0100
+L +3.3V #PWR12
 U 1 1 55B4E35F
 P 2400 1850
-F 0 "#PWR0100" H 2400 1700 50  0001 C CNN
+F 0 "#PWR12" H 2400 1700 50  0001 C CNN
 F 1 "+3.3V" H 2400 1990 50  0000 C CNN
 F 2 "" H 2400 1850 60  0000 C CNN
@@
 $EndComp
 $Comp
-L R R38
+L R R13
 U 1 1 55B4E366
 P 3100 2700
-F 0 "R38" V 3180 2700 50  0000 C CNN
+F 0 "R13" V 3180 2700 50  0000 C CNN
 F 1 "1k5" V 3100 2700 50  0000 C CNN
 F 2 "Resistors_SMD:R_0603" V 3030 2700 30  0001 C CNN
@@
 $EndComp
 $Comp
-L C C25
+L C C14
 U 1 1 55B4E36E
 P 6000 2350
-F 0 "C25" H 6025 2450 50  0000 L CNN
+F 0 "C14" H 6025 2450 50  0000 L CNN
 F 1 "10nF" V 5850 2150 50  0000 L CNN
 F 2 "Capacitors_SMD:C_0603" H 6038 2200 30  0001 C CNN
@@
 $EndComp
 $Comp
-L GNDD #PWR0101
+L GNDD #PWR51
 U 1 1 55B4E375
 P 6000 2550
-F 0 "#PWR0101" H 6000 2300 50  0001 C CNN
+F 0 "#PWR51" H 6000 2300 50  0001 C CNN
 F 1 "GNDD" H 6000 2400 50  0000 C CNN
 F 2 "" H 6000 2550 60  0000 C CNN
@@
 Connection ~ 2400 1950
 $Comp
-L R R42
+L R R21
 U 1 1 55B4E399
 P 6600 2350
-F 0 "R42" V 6500 2350 50  0000 C CNN
+F 0 "R21" V 6500 2350 50  0000 C CNN
 F 1 "3K3" V 6600 2350 50  0000 C CNN
 F 2 "Resistors_SMD:R_0603" V 6530 2350 30  0001 C CNN
@@
 Connection ~ 6600 2100
 $Comp
-L GNDD #PWR0102
+L GNDD #PWR54
 U 1 1 55B4E3A2
 P 6600 2550
-F 0 "#PWR0102" H 6600 2300 50  0001 C CNN
+F 0 "#PWR54" H 6600 2300 50  0001 C CNN
 F 1 "GNDD" H 6600 2400 50  0000 C CNN
 F 2 "" H 6600 2550 60  0000 C CNN

Commit message: fix usb resistors
Parts:
- removed R17, R18: 33R, Resistors_SMD:R_0603, symbol R
Other:
- moved on the sheet: C14, R20, R21
Changed lines of the file:
@@
 $EndDescr
-$Comp
-L R R17
-U 1 1 55B4E32A
-P 4350 2100
-F 0 "R17" V 4250 2100 50  0000 C CNN
-F 1 "33R" V 4350 2100 50  0000 C CNN
-F 2 "Resistors_SMD:R_0603" V 4280 2100 30  0001 C CNN
-F 3 "" H 4350 2100 30  0000 C CNN
-F 4 "MCR03ERTF33R0" H 350 -5100 50  0001 C CNN "MPN"
-	1    4350 2100
-	0    1    1    0
-$EndComp
-$Comp
-L R R18
-U 1 1 55B4E332
-P 4350 2700
-F 0 "R18" V 4450 2700 50  0000 C CNN
-F 1 "33R" V 4350 2700 50  0000 C CNN
-F 2 "Resistors_SMD:R_0603" V 4280 2700 30  0001 C CNN
-F 3 "" H 4350 2700 30  0000 C CNN
-F 4 "MCR03ERTF33R0" H 350 -4650 50  0001 C CNN "MPN"
-	1    4350 2700
-	0    1    1    0
-$EndComp
 $Comp
 L R R20
 U 1 1 55B4E33A
-P 6300 2100
-F 0 "R20" V 6200 2100 50  0000 C CNN
-F 1 "2K" V 6300 2100 50  0000 C CNN
-F 2 "Resistors_SMD:R_0603" V 6230 2100 30  0001 C CNN
-F 3 "" H 6300 2100 30  0000 C CNN
-F 4 "RMCF0603JT2K00" H 2250 -4350 50  0001 C CNN "MPN"
-	1    6300 2100
+P 5300 2100
+F 0 "R20" V 5200 2100 50  0000 C CNN
+F 1 "2K" V 5300 2100 50  0000 C CNN
+F 2 "Resistors_SMD:R_0603" V 5230 2100 30  0001 C CNN
+F 3 "" H 5300 2100 30  0000 C CNN
+F 4 "RMCF0603JT2K00" H 1250 -4350 50  0001 C CNN "MPN"
+	1    5300 2100
 	0    1    1    0
 $EndComp
@@
 L VCC #PWR50
 U 1 1 55B4E341
-P 6000 1950
-F 0 "#PWR50" H 6000 1800 50  0001 C CNN
-F 1 "VCC" H 6000 2100 50  0000 C CNN
-F 2 "" H 6000 1950 60  0000 C CNN
-F 3 "" H 6000 1950 60  0000 C CNN
-	1    6000 1950
+P 5000 1950
+F 0 "#PWR50" H 5000 1800 50  0001 C CNN
+F 1 "VCC" H 5000 2100 50  0000 C CNN
+F 2 "" H 5000 1950 60  0000 C CNN
+F 3 "" H 5000 1950 60  0000 C CNN
+	1    5000 1950
 	1    0    0    -1
 $EndComp
@@
 L C C14
 U 1 1 55B4E36E
-P 6000 2350
-F 0 "C14" H 6025 2450 50  0000 L CNN
-F 1 "10nF" V 5850 2150 50  0000 L CNN
-F 2 "Capacitors_SMD:C_0603" H 6038 2200 30  0001 C CNN
-F 3 "" H 6000 2350 60  0000 C CNN
-F 4 "C1608X7R1E103K080AA" H 2250 -4350 50  0001 C CNN "MPN"
-	1    6000 2350
+P 5000 2350
+F 0 "C14" H 5025 2450 50  0000 L CNN
+F 1 "10nF" V 4850 2150 50  0000 L CNN
+F 2 "Capacitors_SMD:C_0603" H 5038 2200 30  0001 C CNN
+F 3 "" H 5000 2350 60  0000 C CNN
+F 4 "C1608X7R1E103K080AA" H 1250 -4350 50  0001 C CNN "MPN"
+	1    5000 2350
 	1    0    0    -1
 $EndComp
@@
 L GNDD #PWR51
 U 1 1 55B4E375
-P 6000 2550
-F 0 "#PWR51" H 6000 2300 50  0001 C CNN
-F 1 "GNDD" H 6000 2400 50  0000 C CNN
-F 2 "" H 6000 2550 60  0000 C CNN
-F 3 "" H 6000 2550 60  0000 C CNN
-	1    6000 2550
+P 5000 2550
+F 0 "#PWR51" H 5000 2300 50  0001 C CNN
+F 1 "GNDD" H 5000 2400 50  0000 C CNN
+F 2 "" H 5000 2550 60  0000 C CNN
+F 3 "" H 5000 2550 60  0000 C CNN
+	1    5000 2550
 	1    0    0    -1
 $EndComp
-Text GLabel 6750 2100 2    50   Output ~ 0
+Text GLabel 5750 2100 2    50   Output ~ 0
 USB_VBUS
-Text GLabel 4650 2100 2    50   BiDi ~ 0
-USB_DM
-Text GLabel 4650 2700 2    50   BiDi ~ 0
-USB_DP
-Text Notes 3250 1150 0    100  ~ 0
+Text GLabel 3450 2700 2    50   BiDi ~ 0
+USB_DP_CPU
+Text Notes 3500 1150 0    100  ~ 0
 USB DEVICE
 Text GLabel 1850 2450 0    50   Input ~ 0
 USB_CONNECT
 Wire Wire Line
-	4650 2700 4500 2700
+	5450 2100 5750 2100
 Wire Wire Line
-	4650 2100 4500 2100
+	4800 2100 5150 2100
 Wire Wire Line
-	6450 2100 6750 2100
-Wire Wire Line
-	5800 2100 6150 2100
-Wire Wire Line
-	6000 1950 6000 2200
+	5000 1950 5000 2200
 Wire Wire Line
 	2300 2450 2500 2450
@@
 	2800 2700 2950 2700
 Wire Wire Line
-	3250 2700 4200 2700
-Wire Wire Line
-	6000 2550 6000 2500
-Connection ~ 6000 2100
+	5000 2550 5000 2500
+Connection ~ 5000 2100
 Connection ~ 2400 2450
 Connection ~ 2400 1950
@@
 L R R21
 U 1 1 55B4E399
-P 6600 2350
-F 0 "R21" V 6500 2350 50  0000 C CNN
-F 1 "3K3" V 6600 2350 50  0000 C CNN
-F 2 "Resistors_SMD:R_0603" V 6530 2350 30  0001 C CNN
-F 3 "" H 6600 2350 30  0000 C CNN
-F 4 "RMCF0603JT3K30" H 2550 -4100 50  0001 C CNN "MPN"
-	1    6600 2350
+P 5600 2350
+F 0 "R21" V 5500 2350 50  0000 C CNN
+F 1 "3K3" V 5600 2350 50  0000 C CNN
+F 2 "Resistors_SMD:R_0603" V 5530 2350 30  0001 C CNN
+F 3 "" H 5600 2350 30  0000 C CNN
+F 4 "RMCF0603JT3K30" H 1550 -4100 50  0001 C CNN "MPN"
+	1    5600 2350
 	-1   0    0    1
 $EndComp
 Wire Wire Line
-	6600 2200 6600 2100
-Connection ~ 6600 2100
+	5600 2200 5600 2100
+Connection ~ 5600 2100
 $Comp
 L GNDD #PWR54
 U 1 1 55B4E3A2
-P 6600 2550
-F 0 "#PWR54" H 6600 2300 50  0001 C CNN
-F 1 "GNDD" H 6600 2400 50  0000 C CNN
-F 2 "" H 6600 2550 60  0000 C CNN
-F 3 "" H 6600 2550 60  0000 C CNN
-	1    6600 2550
+P 5600 2550
+F 0 "#PWR54" H 5600 2300 50  0001 C CNN
+F 1 "GNDD" H 5600 2400 50  0000 C CNN
+F 2 "" H 5600 2550 60  0000 C CNN
+F 3 "" H 5600 2550 60  0000 C CNN
+	1    5600 2550
 	1    0    0    -1
 $EndComp
 Wire Wire Line
-	6600 2550 6600 2500
-Text GLabel 3800 2100 0    50   BiDi ~ 0
-USB_DM_CPU
-Text GLabel 3800 2400 0    50   BiDi ~ 0
-USB_DP_CPU
-Text GLabel 5800 2100 0    50   Input ~ 0
+	5600 2550 5600 2500
+Text GLabel 4800 2100 0    50   Input ~ 0
 USB_VCC
 Wire Wire Line
-	4200 2100 3800 2100
-Wire Wire Line
-	3800 2400 3950 2400
-Wire Wire Line
-	3950 2400 3950 2700
-Connection ~ 3950 2700
+	3450 2700 3250 2700
 $EndSCHEMATC

Commit message: update MPN
Parts:
- R13: value 1k5 -> 1K5
- R6: value 3k -> 3K
- R7: value 24k -> 24K
Changed lines of the file:
@@
 P 2150 2450
 F 0 "R6" V 2230 2450 50  0000 C CNN
-F 1 "3k" V 2150 2450 50  0000 C CNN
+F 1 "3K" V 2150 2450 50  0000 C CNN
 F 2 "Resistors_SMD:R_0603" V 2080 2450 30  0001 C CNN
 F 3 "" H 2150 2450 30  0000 C CNN
@@
 P 2400 2200
 F 0 "R7" V 2480 2200 50  0000 C CNN
-F 1 "24k" V 2400 2200 50  0000 C CNN
+F 1 "24K" V 2400 2200 50  0000 C CNN
 F 2 "Resistors_SMD:R_0603" V 2330 2200 30  0001 C CNN
 F 3 "" H 2400 2200 30  0000 C CNN
@@
 P 3100 2700
 F 0 "R13" V 3180 2700 50  0000 C CNN
-F 1 "1k5" V 3100 2700 50  0000 C CNN
+F 1 "1K5" V 3100 2700 50  0000 C CNN
 F 2 "Resistors_SMD:R_0603" V 3030 2700 30  0001 C CNN
 F 3 "" H 3100 2700 30  0000 C CNN

Commit message: changing one cap PN
Parts:
- C14: value 10nF -> 100nF; MPN C1608X7R1E103K080AA -> C1608X7R1E104K080AA
Changed lines of the file:
@@
 P 5000 2350
 F 0 "C14" H 5025 2450 50  0000 L CNN
-F 1 "10nF" V 4850 2150 50  0000 L CNN
+F 1 "100nF" V 4850 2150 50  0000 L CNN
 F 2 "Capacitors_SMD:C_0603" H 5038 2200 30  0001 C CNN
 F 3 "" H 5000 2350 60  0000 C CNN
-F 4 "C1608X7R1E103K080AA" H 1250 -4350 50  0001 C CNN "MPN"
+F 4 "C1608X7R1E104K080AA" H 1250 -4350 50  0001 C CNN "MPN"
 	1    5000 2350
 	1    0    0    -1

Commit message: remove resistors divider of usb vbus
Parts:
- removed R21: 3K3, Resistors_SMD:R_0603, symbol R
- R20: value 2K -> 100R; MPN RMCF0603JT2K00 -> RMCF0603JT100R
Other:
- moved on the sheet: R20
Changed lines of the file:
@@
 L R R20
 U 1 1 55B4E33A
-P 5300 2100
-F 0 "R20" V 5200 2100 50  0000 C CNN
-F 1 "2K" V 5300 2100 50  0000 C CNN
-F 2 "Resistors_SMD:R_0603" V 5230 2100 30  0001 C CNN
-F 3 "" H 5300 2100 30  0000 C CNN
-F 4 "RMCF0603JT2K00" H 1250 -4350 50  0001 C CNN "MPN"
-	1    5300 2100
+P 5350 2100
+F 0 "R20" V 5250 2100 50  0000 C CNN
+F 1 "100R" V 5350 2100 50  0000 C CNN
+F 2 "Resistors_SMD:R_0603" V 5280 2100 30  0001 C CNN
+F 3 "" H 5350 2100 30  0000 C CNN
+F 4 "RMCF0603JT100R" H 1300 -4350 50  0001 C CNN "MPN"
+	1    5350 2100
 	0    1    1    0
 $EndComp
@@
 	1    0    0    -1
 $EndComp
-Text GLabel 5750 2100 2    50   Output ~ 0
+Text GLabel 5650 2100 2    50   Output ~ 0
 USB_VBUS
 Text GLabel 3450 2700 2    50   BiDi ~ 0
@@
 USB_CONNECT
 Wire Wire Line
-	5450 2100 5750 2100
+	5500 2100 5650 2100
 Wire Wire Line
-	4800 2100 5150 2100
+	4800 2100 5000 2100
 Wire Wire Line
-	5000 1950 5000 2200
+	5000 2100 5200 2100
 Wire Wire Line
-	2300 2450 2500 2450
+	5000 1950 5000 2100
+Wire Wire Line
+	5000 2100 5000 2200
+Wire Wire Line
+	2300 2450 2400 2450
+Wire Wire Line
+	2400 2450 2500 2450
 Wire Wire Line
 	2400 2350 2400 2450
@@
 	2000 2450 1850 2450
 Wire Wire Line
-	2400 1850 2400 2050
+	2400 1850 2400 1950
+Wire Wire Line
+	2400 1950 2400 2050
 Wire Wire Line
 	2800 2250 2800 1950
@@
 Connection ~ 2400 2450
 Connection ~ 2400 1950
-$Comp
-L R R21
-U 1 1 55B4E399
-P 5600 2350
-F 0 "R21" V 5500 2350 50  0000 C CNN
-F 1 "3K3" V 5600 2350 50  0000 C CNN
-F 2 "Resistors_SMD:R_0603" V 5530 2350 30  0001 C CNN
-F 3 "" H 5600 2350 30  0000 C CNN
-F 4 "RMCF0603JT3K30" H 1550 -4100 50  0001 C CNN "MPN"
-	1    5600 2350
-	-1   0    0    1
-$EndComp
-Wire Wire Line
-	5600 2200 5600 2100
-Connection ~ 5600 2100
-$Comp
-L GNDD #PWR54
-U 1 1 55B4E3A2
-P 5600 2550
-F 0 "#PWR54" H 5600 2300 50  0001 C CNN
-F 1 "GNDD" H 5600 2400 50  0000 C CNN
-F 2 "" H 5600 2550 60  0000 C CNN
-F 3 "" H 5600 2550 60  0000 C CNN
-	1    5600 2550
-	1    0    0    -1
-$EndComp
-Wire Wire Line
-	5600 2550 5600 2500
 Text GLabel 4800 2100 0    50   Input ~ 0
 USB_VCC

Commit message: DRC done
Parts:
- renumbered C14 to C11, Q3 to Q2, R13 to R12, R20 to R18, R6 to R5, R7 to R6
Changed lines of the file:
@@
 $EndDescr
 $Comp
-L R R20
+L R R18
 U 1 1 55B4E33A
 P 5350 2100
-F 0 "R20" V 5250 2100 50  0000 C CNN
+F 0 "R18" V 5250 2100 50  0000 C CNN
 F 1 "100R" V 5350 2100 50  0000 C CNN
 F 2 "Resistors_SMD:R_0603" V 5280 2100 30  0001 C CNN
@@
 $EndComp
 $Comp
-L VCC #PWR50
+L VCC #PWR41
 U 1 1 55B4E341
 P 5000 1950
-F 0 "#PWR50" H 5000 1800 50  0001 C CNN
+F 0 "#PWR41" H 5000 1800 50  0001 C CNN
 F 1 "VCC" H 5000 2100 50  0000 C CNN
 F 2 "" H 5000 1950 60  0000 C CNN
@@
 $EndComp
 $Comp
-L Q_PNP_BEC Q3
+L Q_PNP_BEC Q2
 U 1 1 55B4E348
 P 2700 2450
-F 0 "Q3" H 3000 2450 50  0000 R CNN
+F 0 "Q2" H 3000 2450 50  0000 R CNN
 F 1 "BC857" H 3100 2350 50  0000 R CNN
 F 2 "Housings_SOT-23_SOT-143_TSOT-6:SOT-23" H 2900 2550 29  0001 C CNN
@@
 $EndComp
 $Comp
-L R R6
+L R R5
 U 1 1 55B4E350
 P 2150 2450
-F 0 "R6" V 2230 2450 50  0000 C CNN
+F 0 "R5" V 2230 2450 50  0000 C CNN
 F 1 "3K" V 2150 2450 50  0000 C CNN
 F 2 "Resistors_SMD:R_0603" V 2080 2450 30  0001 C CNN
@@
 $EndComp
 $Comp
-L R R7
+L R R6
 U 1 1 55B4E358
 P 2400 2200
-F 0 "R7" V 2480 2200 50  0000 C CNN
+F 0 "R6" V 2480 2200 50  0000 C CNN
 F 1 "24K" V 2400 2200 50  0000 C CNN
 F 2 "Resistors_SMD:R_0603" V 2330 2200 30  0001 C CNN
@@
 $EndComp
 $Comp
-L +3.3V #PWR12
+L +3.3V #PWR10
 U 1 1 55B4E35F
 P 2400 1850
-F 0 "#PWR12" H 2400 1700 50  0001 C CNN
+F 0 "#PWR10" H 2400 1700 50  0001 C CNN
 F 1 "+3.3V" H 2400 1990 50  0000 C CNN
 F 2 "" H 2400 1850 60  0000 C CNN
@@
 $EndComp
 $Comp
-L R R13
+L R R12
 U 1 1 55B4E366
 P 3100 2700
-F 0 "R13" V 3180 2700 50  0000 C CNN
+F 0 "R12" V 3180 2700 50  0000 C CNN
 F 1 "1K5" V 3100 2700 50  0000 C CNN
 F 2 "Resistors_SMD:R_0603" V 3030 2700 30  0001 C CNN
@@
 $EndComp
 $Comp
-L C C14
+L C C11
 U 1 1 55B4E36E
 P 5000 2350
-F 0 "C14" H 5025 2450 50  0000 L CNN
+F 0 "C11" H 5025 2450 50  0000 L CNN
 F 1 "100nF" V 4850 2150 50  0000 L CNN
 F 2 "Capacitors_SMD:C_0603" H 5038 2200 30  0001 C CNN
@@
 $EndComp
 $Comp
-L GNDD #PWR51
+L GNDD #PWR42
 U 1 1 55B4E375
 P 5000 2550
-F 0 "#PWR51" H 5000 2300 50  0001 C CNN
+F 0 "#PWR42" H 5000 2300 50  0001 C CNN
 F 1 "GNDD" H 5000 2400 50  0000 C CNN
 F 2 "" H 5000 2550 60  0000 C CNN
@@
 	5500 2100 5650 2100
 Wire Wire Line
-	4800 2100 5000 2100
+	4800 2100 5200 2100
 Wire Wire Line
-	5000 2100 5200 2100
+	5000 1950 5000 2200
 Wire Wire Line
-	5000 1950 5000 2100
-Wire Wire Line
-	5000 2100 5000 2200
-Wire Wire Line
-	2300 2450 2400 2450
-Wire Wire Line
-	2400 2450 2500 2450
+	2300 2450 2500 2450
 Wire Wire Line
 	2400 2350 2400 2450
@@
 	2000 2450 1850 2450
 Wire Wire Line
-	2400 1850 2400 1950
-Wire Wire Line
-	2400 1950 2400 2050
+	2400 1850 2400 2050
 Wire Wire Line
 	2800 2250 2800 1950

Commit message: only trigger isp when usb is connected
Parts:
- added Q?: 2N7002, Housings_SOT-23_SOT-143_TSOT-6:SOT-23, symbol Q_NMOS_GSD
- added R? (x2): 10K, Resistors_SMD:R_0603, symbol R
Connections:
- net +3V3: now also R?.2
- net GNDD: now also R?.1
- net VCC: now also Q?.1 (G), R?.2
- new net FS1: Q?.2 (S)
- new net ISP_TRIGGER: Q?.3 (D), R?.1
Changed lines of the file:
@@
 Text GLabel 1850 2450 0    50   Input ~ 0
 USB_CONNECT
+Text GLabel 4800 2100 0    50   Input ~ 0
+USB_VCC
+Text GLabel 2100 4000 0    50   Input ~ 0
+USB_VCC
+$Comp
+L Q_NMOS_GSD Q?
+U 1 1 578D24B0
+P 2700 4000
+F 0 "Q?" H 2600 4050 50  0000 R CNN
+F 1 "2N7002" H 2650 3900 50  0000 R CNN
+F 2 "Housings_SOT-23_SOT-143_TSOT-6:SOT-23" H 2900 4100 29  0001 C CNN
+F 3 "" H 2700 4000 60  0000 C CNN
+F 4 "2N7002P,215" H -6200 1050 50  0001 C CNN "MPN"
+	1    2700 4000
+	1    0    0    -1
+$EndComp
+$Comp
+L R R?
+U 1 1 578D27BF
+P 2300 4300
+F 0 "R?" V 2380 4300 50  0000 C CNN
+F 1 "10K" V 2300 4300 50  0000 C CNN
+F 2 "Resistors_SMD:R_0603" V 2230 4300 30  0001 C CNN
+F 3 "" H 2300 4300 30  0000 C CNN
+F 4 "RMCF0603JT10K0" H 250 -2550 50  0001 C CNN "MPN"
+	1    2300 4300
+	-1   0    0    1
+$EndComp
+$Comp
+L GNDD #PWR?
+U 1 1 578D2C8E
+P 2300 4550
+F 0 "#PWR?" H 2300 4300 50  0001 C CNN
+F 1 "GNDD" H 2300 4400 50  0000 C CNN
+F 2 "" H 2300 4550 60  0000 C CNN
+F 3 "" H 2300 4550 60  0000 C CNN
+	1    2300 4550
+	1    0    0    -1
+$EndComp
+Text GLabel 2700 4300 0    50   Input ~ 0
+FS1
+Text GLabel 2950 3700 2    50   Output ~ 0
+ISP_TRIGGER
+$Comp
+L +3.3V #PWR?
+U 1 1 578D3853
+P 2800 3200
+F 0 "#PWR?" H 2800 3050 50  0001 C CNN
+F 1 "+3.3V" H 2800 3340 50  0000 C CNN
+F 2 "" H 2800 3200 60  0000 C CNN
+F 3 "" H 2800 3200 60  0000 C CNN
+	1    2800 3200
+	1    0    0    -1
+$EndComp
 Wire Wire Line
 	5500 2100 5650 2100
@@
 Connection ~ 2400 2450
 Connection ~ 2400 1950
-Text GLabel 4800 2100 0    50   Input ~ 0
-USB_VCC
 Wire Wire Line
 	3450 2700 3250 2700
+Wire Wire Line
+	2100 4000 2500 4000
+Wire Wire Line
+	2300 4150 2300 4000
+Connection ~ 2300 4000
+Wire Wire Line
+	2300 4450 2300 4550
+Wire Wire Line
+	2700 4300 2800 4300
+Wire Wire Line
+	2800 4300 2800 4200
+Wire Wire Line
+	2800 3600 2800 3800
+Wire Wire Line
+	2950 3700 2800 3700
+Connection ~ 2800 3700
+$Comp
+L R R?
+U 1 1 578D3A95
+P 2800 3450
+F 0 "R?" V 2880 3450 50  0000 C CNN
+F 1 "10K" V 2800 3450 50  0000 C CNN
+F 2 "Resistors_SMD:R_0603" V 2730 3450 30  0001 C CNN
+F 3 "" H 2800 3450 30  0000 C CNN
+F 4 "RMCF0603JT10K0" H 750 -3400 50  0001 C CNN "MPN"
+	1    2800 3450
+	-1   0    0    1
+$EndComp
+Wire Wire Line
+	2800 3200 2800 3300
 $EndSCHEMATC
