File: hw-design/board/usb.sch (KiCad schematic (older format))
At the start: 9 parts, among them Q2 BC857

Commit message: update netlist
Parts:
- gave numbers to parts that had none: 3
- renumbered R12 to R14, R18 to R20, R6 to R7
Changed lines of the file:
@@
 $EndDescr
 $Comp
-L R R18
+L R R20
 U 1 1 55B4E33A
 P 5350 2100
-F 0 "R18" V 5250 2100 50  0000 C CNN
+F 0 "R20" V 5250 2100 50  0000 C CNN
 F 1 "100R" V 5350 2100 50  0000 C CNN
 F 2 "Resistors_SMD:R_0603" V 5280 2100 30  0001 C CNN
@@
 $EndComp
 $Comp
-L VCC #PWR41
+L VCC #PWR43
 U 1 1 55B4E341
 P 5000 1950
-F 0 "#PWR41" H 5000 1800 50  0001 C CNN
+F 0 "#PWR43" H 5000 1800 50  0001 C CNN
 F 1 "VCC" H 5000 2100 50  0000 C CNN
 F 2 "" H 5000 1950 60  0000 C CNN
@@
 $EndComp
 $Comp
-L R R6
+L R R7
 U 1 1 55B4E358
 P 2400 2200
-F 0 "R6" V 2480 2200 50  0000 C CNN
+F 0 "R7" V 2480 2200 50  0000 C CNN
 F 1 "24K" V 2400 2200 50  0000 C CNN
 F 2 "Resistors_SMD:R_0603" V 2330 2200 30  0001 C CNN
@@
 $EndComp
 $Comp
-L +3.3V #PWR10
+L +3.3V #PWR11
 U 1 1 55B4E35F
 P 2400 1850
-F 0 "#PWR10" H 2400 1700 50  0001 C CNN
+F 0 "#PWR11" H 2400 1700 50  0001 C CNN
 F 1 "+3.3V" H 2400 1990 50  0000 C CNN
 F 2 "" H 2400 1850 60  0000 C CNN
@@
 $EndComp
 $Comp
-L R R12
+L R R14
 U 1 1 55B4E366
 P 3100 2700
-F 0 "R12" V 3180 2700 50  0000 C CNN
+F 0 "R14" V 3180 2700 50  0000 C CNN
 F 1 "1K5" V 3100 2700 50  0000 C CNN
 F 2 "Resistors_SMD:R_0603" V 3030 2700 30  0001 C CNN
@@
 $EndComp
 $Comp
-L GNDD #PWR42
+L GNDD #PWR44
 U 1 1 55B4E375
 P 5000 2550
-F 0 "#PWR42" H 5000 2300 50  0001 C CNN
+F 0 "#PWR44" H 5000 2300 50  0001 C CNN
 F 1 "GNDD" H 5000 2400 50  0000 C CNN
 F 2 "" H 5000 2550 60  0000 C CNN
@@
 USB_VCC
 $Comp
-L Q_NMOS_GSD Q?
+L Q_NMOS_GSD Q3
 U 1 1 578D24B0
 P 2700 4000
-F 0 "Q?" H 2600 4050 50  0000 R CNN
+F 0 "Q3" H 2600 4050 50  0000 R CNN
 F 1 "2N7002" H 2650 3900 50  0000 R CNN
 F 2 "Housings_SOT-23_SOT-143_TSOT-6:SOT-23" H 2900 4100 29  0001 C CNN
@@
 $EndComp
 $Comp
-L R R?
+L R R6
 U 1 1 578D27BF
 P 2300 4300
-F 0 "R?" V 2380 4300 50  0000 C CNN
+F 0 "R6" V 2380 4300 50  0000 C CNN
 F 1 "10K" V 2300 4300 50  0000 C CNN
 F 2 "Resistors_SMD:R_0603" V 2230 4300 30  0001 C CNN
@@
 $EndComp
 $Comp
-L GNDD #PWR?
+L GNDD #PWR10
 U 1 1 578D2C8E
 P 2300 4550
-F 0 "#PWR?" H 2300 4300 50  0001 C CNN
+F 0 "#PWR10" H 2300 4300 50  0001 C CNN
 F 1 "GNDD" H 2300 4400 50  0000 C CNN
 F 2 "" H 2300 4550 60  0000 C CNN
@@
 ISP_TRIGGER
 $Comp
-L +3.3V #PWR?
+L +3.3V #PWR16
 U 1 1 578D3853
 P 2800 3200
-F 0 "#PWR?" H 2800 3050 50  0001 C CNN
+F 0 "#PWR16" H 2800 3050 50  0001 C CNN
 F 1 "+3.3V" H 2800 3340 50  0000 C CNN
 F 2 "" H 2800 3200 60  0000 C CNN
@@
 Connection ~ 2800 3700
 $Comp
-L R R?
+L R R10
 U 1 1 578D3A95
 P 2800 3450
-F 0 "R?" V 2880 3450 50  0000 C CNN
+F 0 "R10" V 2880 3450 50  0000 C CNN
 F 1 "10K" V 2800 3450 50  0000 C CNN
 F 2 "Resistors_SMD:R_0603" V 2730 3450 30  0001 C CNN

Commit message: increase usb vcc pull down resistor
Parts:
- R6: value 10K -> 100K; MPN RMCF0603JT10K0 -> RMCF0603JT100K
Changed lines of the file:
@@
 P 2300 4300
 F 0 "R6" V 2380 4300 50  0000 C CNN
-F 1 "10K" V 2300 4300 50  0000 C CNN
+F 1 "100K" V 2300 4300 50  0000 C CNN
 F 2 "Resistors_SMD:R_0603" V 2230 4300 30  0001 C CNN
 F 3 "" H 2300 4300 30  0000 C CNN
-F 4 "RMCF0603JT10K0" H 250 -2550 50  0001 C CNN "MPN"
+F 4 "RMCF0603JT100K" H 250 -2550 50  0001 C CNN "MPN"
 	1    2300 4300
 	-1   0    0    1
