File: hw-design/board/usb.sch (KiCad schematic (older format))
At the start: 9 parts, among them Q2 BC857, Q3 2N7002

Commit message: update files to KiCAD 5
Parts:
- C11: symbol C -> footswitch-rescue:C
- Q2: symbol Q_PNP_BEC -> footswitch-rescue:Q_PNP_BEC
- Q3: symbol Q_NMOS_GSD -> footswitch-rescue:Q_NMOS_GSD
- R10, R14, R20, R5, R6, R7: symbol R -> footswitch-rescue:R
Changed lines of the file:
@@
-EESchema Schematic File Version 2
-LIBS:conn
-LIBS:device
-LIBS:interface
-LIBS:power
-LIBS:regul
-LIBS:transistors
-LIBS:display
-LIBS:nxp_armmcu
-LIBS:philips
-LIBS:graphic_symbols
+EESchema Schematic File Version 4
 LIBS:footswitch-cache
 EELAYER 26 0
@@
 $EndDescr
 $Comp
-L R R20
+L footswitch-rescue:R R20
 U 1 1 55B4E33A
 P 5350 2100
@@
 $EndComp
 $Comp
-L VCC #PWR076
+L footswitch-rescue:VCC #PWR076
 U 1 1 55B4E341
 P 5000 1950
@@
 $EndComp
 $Comp
-L Q_PNP_BEC Q2
+L footswitch-rescue:Q_PNP_BEC Q2
 U 1 1 55B4E348
 P 2700 2450
@@
 $EndComp
 $Comp
-L R R5
+L footswitch-rescue:R R5
 U 1 1 55B4E350
 P 2150 2450
@@
 $EndComp
 $Comp
-L R R7
+L footswitch-rescue:R R7
 U 1 1 55B4E358
 P 2400 2200
@@
 $EndComp
 $Comp
-L +3.3V #PWR077
+L footswitch-rescue:+3.3V #PWR077
 U 1 1 55B4E35F
 P 2400 1850
@@
 $EndComp
 $Comp
-L R R14
+L footswitch-rescue:R R14
 U 1 1 55B4E366
 P 3100 2700
@@
 $EndComp
 $Comp
-L C C11
+L footswitch-rescue:C C11
 U 1 1 55B4E36E
 P 5000 2350
@@
 $EndComp
 $Comp
-L GNDD #PWR078
+L footswitch-rescue:GNDD #PWR078
 U 1 1 55B4E375
 P 5000 2550
@@
 USB_VCC
 $Comp
-L Q_NMOS_GSD Q3
+L footswitch-rescue:Q_NMOS_GSD Q3
 U 1 1 578D24B0
 P 2700 4000
@@
 $EndComp
 $Comp
-L R R6
+L footswitch-rescue:R R6
 U 1 1 578D27BF
 P 2300 4300
@@
 $EndComp
 $Comp
-L GNDD #PWR079
+L footswitch-rescue:GNDD #PWR079
 U 1 1 578D2C8E
 P 2300 4550
@@
 ISP_TRIGGER
 $Comp
-L +3.3V #PWR080
+L footswitch-rescue:+3.3V #PWR080
 U 1 1 578D3853
 P 2800 3200
@@
 Connection ~ 2800 3700
 $Comp
-L R R10
+L footswitch-rescue:R R10
 U 1 1 578D3A95
 P 2800 3450

Commit message: Changed R40 RE from pull-up to pull-down
Parts:
- C11: symbol footswitch-rescue:C -> footswitch-rescue:C-footswitch-rescue
- Q2: symbol footswitch-rescue:Q_PNP_BEC -> footswitch-rescue:Q_PNP_BEC-footswitch-rescue
- Q3: symbol footswitch-rescue:Q_NMOS_GSD -> footswitch-rescue:Q_NMOS_GSD-footswitch-rescue
- R10, R14, R20, R5, R6, R7: symbol footswitch-rescue:R -> footswitch-rescue:R-footswitch-rescue
Changed lines of the file:
@@
 $EndDescr
 $Comp
-L footswitch-rescue:R R20
+L footswitch-rescue:R-footswitch-rescue R20
 U 1 1 55B4E33A
 P 5350 2100
@@
 $EndComp
 $Comp
-L footswitch-rescue:VCC #PWR076
+L footswitch-rescue:VCC-footswitch-rescue #PWR076
 U 1 1 55B4E341
 P 5000 1950
@@
 $EndComp
 $Comp
-L footswitch-rescue:Q_PNP_BEC Q2
+L footswitch-rescue:Q_PNP_BEC-footswitch-rescue Q2
 U 1 1 55B4E348
 P 2700 2450
@@
 $EndComp
 $Comp
-L footswitch-rescue:R R5
+L footswitch-rescue:R-footswitch-rescue R5
 U 1 1 55B4E350
 P 2150 2450
@@
 $EndComp
 $Comp
-L footswitch-rescue:R R7
+L footswitch-rescue:R-footswitch-rescue R7
 U 1 1 55B4E358
 P 2400 2200
@@
 $EndComp
 $Comp
-L footswitch-rescue:+3.3V #PWR077
+L footswitch-rescue:+3.3V-footswitch-rescue #PWR077
 U 1 1 55B4E35F
 P 2400 1850
@@
 $EndComp
 $Comp
-L footswitch-rescue:R R14
+L footswitch-rescue:R-footswitch-rescue R14
 U 1 1 55B4E366
 P 3100 2700
@@
 $EndComp
 $Comp
-L footswitch-rescue:C C11
+L footswitch-rescue:C-footswitch-rescue C11
 U 1 1 55B4E36E
 P 5000 2350
@@
 $EndComp
 $Comp
-L footswitch-rescue:GNDD #PWR078
+L footswitch-rescue:GNDD-footswitch-rescue #PWR078
 U 1 1 55B4E375
 P 5000 2550
@@
 USB_VCC
 $Comp
-L footswitch-rescue:Q_NMOS_GSD Q3
+L footswitch-rescue:Q_NMOS_GSD-footswitch-rescue Q3
 U 1 1 578D24B0
 P 2700 4000
@@
 $EndComp
 $Comp
-L footswitch-rescue:R R6
+L footswitch-rescue:R-footswitch-rescue R6
 U 1 1 578D27BF
 P 2300 4300
@@
 $EndComp
 $Comp
-L footswitch-rescue:GNDD #PWR079
+L footswitch-rescue:GNDD-footswitch-rescue #PWR079
 U 1 1 578D2C8E
 P 2300 4550
@@
 ISP_TRIGGER
 $Comp
-L footswitch-rescue:+3.3V #PWR080
+L footswitch-rescue:+3.3V-footswitch-rescue #PWR080
 U 1 1 578D3853
 P 2800 3200
@@
 Connection ~ 2800 3700
 $Comp
-L footswitch-rescue:R R10
+L footswitch-rescue:R-footswitch-rescue R10
 U 1 1 578D3A95
 P 2800 3450
